File: cpu030/design-files/cpu030.kicad_pcb (KiCad board)
At the start: 4 copper layers, 200 x 154.9 mm, 110 parts, among them J101 Reset, J102 SYSCTL JTAG, J103 NMI, J201 DRAM0SZ, J202 DRAM0 JTAG, J301 UART0 FTDI, J302 UART1 FTDI, J303 UART1, J304 UART0, SW101 Reset, SW102 NMI, U101 MC68030RC, U102 ATF1508AS, U103 MC74ACT05DG, U104 DS1813, U105 SST39SF040 (E), U106 SST39SF040 (O), U107 MC68882, U108 GAL22V10, U109 MC74ACT05DG, U110 DS1813, U201 ATF1508AS, U202 CY7C1061GE (U16), U203 CY7C1061GE (L16), U204 SIMM72-0A, U205 SIMM72-0B, U206 MC74ACT05DG, U301 TL16C2552, U401 CP82C54-10Z, U402 GAL22V10, Y101 50MHz, Y301 1.8432MHz

Commit message: Eliminate the external D-FF clocking on INTC-1; use the same trick with /DS as we do on TMRGLUE.
Connections:
- U108 pad 1: Net-(U108-I1/CLK) -> ~{DS}
- U108 pad 13: ~{DS} -> RnW
- U108 pad 14: RnW -> unconnected-(U108-IO1-Pad14)
- U108 pad 23: Net-(U108-I1/CLK) -> unconnected-(U108-IO10-Pad23)
- U109 pad 5: GND -> TMR_O0
- U109 pad 6: unconnected-(U109-Pad6) -> ~{INT6}
Changed lines of the file:
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@@
 	(net 251 "Net-(U107-A0)")
 	(net 252 "~{INT5}")
-	(net 253 "Net-(U108-I1{slash}CLK)")
-	(net 254 "~{INT1}")
-	(net 255 "~{INT7}")
-	(net 256 "~{INT6}")
-	(net 257 "~{INT2}")
-	(net 258 "~{INT4}")
-	(net 259 "~{INT3}")
-	(net 260 "unconnected-(U108-IO9-Pad22)")
-	(net 261 "unconnected-(U109-Pad10)")
-	(net 262 "unconnected-(U109-Pad8)")
-	(net 263 "unconnected-(U109-Pad6)")
-	(net 264 "unconnected-(U109-Pad12)")
-	(net 265 "Net-(U401-OUT0)")
-	(net 266 "Net-(U401-G2)")
-	(net 267 "Net-(U401-~{CS})")
-	(net 268 "Net-(U401-OUT2)")
-	(net 269 "Net-(U401-G1)")
-	(net 270 "Net-(U401-OUT1)")
-	(net 271 "Net-(U401-G0)")
-	(net 272 "unconnected-(U402-I8-Pad8)")
-	(net 273 "unconnected-(U402-I11-Pad11)")
-	(net 274 "unconnected-(U402-I9-Pad9)")
-	(net 275 "TMR_O2")
-	(net 276 "unconnected-(U402-I10-Pad10)")
-	(net 277 "TMR_O0")
-	(net 278 "TMR_O1")
+	(net 253 "~{INT1}")
+	(net 254 "~{INT7}")
+	(net 255 "~{INT6}")
+	(net 256 "~{INT2}")
+	(net 257 "~{INT4}")
+	(net 258 "~{INT3}")
+	(net 259 "unconnected-(U108-IO9-Pad22)")
+	(net 260 "unconnected-(U109-Pad10)")
+	(net 261 "unconnected-(U109-Pad8)")
+	(net 262 "unconnected-(U109-Pad12)")
+	(net 263 "Net-(U401-OUT0)")
+	(net 264 "Net-(U401-G2)")
+	(net 265 "Net-(U401-~{CS})")
+	(net 266 "Net-(U401-OUT2)")
+	(net 267 "Net-(U401-G1)")
+	(net 268 "Net-(U401-OUT1)")
+	(net 269 "Net-(U401-G0)")
+	(net 270 "unconnected-(U402-I8-Pad8)")
+	(net 271 "unconnected-(U402-I11-Pad11)")
+	(net 272 "unconnected-(U402-I9-Pad9)")
+	(net 273 "TMR_O2")
+	(net 274 "unconnected-(U402-I10-Pad10)")
+	(net 275 "TMR_O0")
+	(net 276 "TMR_O1")
+	(net 277 "unconnected-(U108-IO1-Pad14)")
+	(net 278 "unconnected-(U108-IO10-Pad23)")
 	(footprint "Package_QFP:TQFP-100_14x14mm_P0.5mm"
 		(layer "F.Cu")
@@
 			(layers "*.Cu" "*.Mask")
 			(remove_unused_layers no)
-			(net 265 "Net-(U401-OUT0)")
+			(net 263 "Net-(U401-OUT0)")
 			(pinfunction "I5")
 			(pintype "input")
@@
 			(layers "*.Cu" "*.Mask")
 			(remove_unused_layers no)
-			(net 270 "Net-(U401-OUT1)")
+			(net 268 "Net-(U401-OUT1)")
 			(pinfunction "I6")
 			(pintype "input")
@@
 			(layers "*.Cu" "*.Mask")
 			(remove_unused_layers no)
-			(net 268 "Net-(U401-OUT2)")
+			(net 266 "Net-(U401-OUT2)")
 			(pinfunction "I7")
 			(pintype "input")
@@
 			(layers "*.Cu" "*.Mask")
 			(remove_unused_layers no)
-			(net 272 "unconnected-(U402-I8-Pad8)")
+			(net 270 "unconnected-(U402-I8-Pad8)")
 			(pinfunction "I8")
 			(pintype "input+no_connect")
@@
 			(layers "*.Cu" "*.Mask")
 			(remove_unused_layers no)
-			(net 274 "unconnected-(U402-I9-Pad9)")
+			(net 272 "unconnected-(U402-I9-Pad9)")
 			(pinfunction "I9")
 			(pintype "input+no_connect")
@@
 			(layers "*.Cu" "*.Mask")
 			(remove_unused_layers no)
-			(net 276 "unconnected-(U402-I10-Pad10)")
+			(net 274 "unconnected-(U402-I10-Pad10)")
 			(pinfunction "I10")
 			(pintype "input+no_connect")
@@
 			(layers "*.Cu" "*.Mask")
 			(remove_unused_layers no)
-			(net 273 "unconnected-(U402-I11-Pad11)")
+			(net 271 "unconnected-(U402-I11-Pad11)")
 			(pinfunction "I11")
 			(pintype "input+no_connect")
@@
 			(layers "*.Cu" "*.Mask")
 			(remove_unused_layers no)
-			(net 277 "TMR_O0")
+			(net 275 "TMR_O0")
 			(pinfunction "IO4")
 			(pintype "tri_state")
@@
 			(layers "*.Cu" "*.Mask")
 			(remove_unused_layers no)
-			(net 278 "TMR_O1")
+			(net 276 "TMR_O1")
 			(pinfunction "IO5")
 			(pintype "tri_state")
@@
 			(layers "*.Cu" "*.Mask")
 			(remove_unused_layers no)
-			(net 275 "TMR_O2")
+			(net 273 "TMR_O2")
 			(pinfunction "IO6")
 			(pintype "tri_state")
@@
 			(layers "*.Cu" "*.Mask")
 			(remove_unused_layers no)
-			(net 271 "Net-(U401-G0)")
+			(net 269 "Net-(U401-G0)")
 			(pinfunction "IO7")
 			(pintype "tri_state")
@@
 			(layers "*.Cu" "*.Mask")
 			(remove_unused_layers no)
-			(net 269 "Net-(U401-G1)")
+			(net 267 "Net-(U401-G1)")
 			(pinfunction "IO8")
 			(pintype "tri_state")
@@
 			(layers "*.Cu" "*.Mask")
 			(remove_unused_layers no)
-			(net 266 "Net-(U401-G2)")
+			(net 264 "Net-(U401-G2)")
 			(pinfunction "IO9")
 			(pintype "tri_state")
@@
 			(layers "*.Cu" "*.Mask")
 			(remove_unused_layers no)
-			(net 267 "Net-(U401-~{CS})")
+			(net 265 "Net-(U401-~{CS})")
 			(pinfunction "IO10")
 			(pintype "tri_state")
@@
 			(layers "*.Cu" "*.Mask")
 			(remove_unused_layers no)
-			(net 265 "Net-(U401-OUT0)")
+			(net 263 "Net-(U401-OUT0)")
 			(pinfunction "OUT0")
 			(pintype "output")
@@
 			(layers "*.Cu" "*.Mask")
 			(remove_unused_layers no)
-			(net 271 "Net-(U401-G0)")
+			(net 269 "Net-(U401-G0)")
 			(pinfunction "G0")
 			(pintype "input")
@@
 			(layers "*.Cu" "*.Mask")
 			(remove_unused_layers no)
-			(net 270 "Net-(U401-OUT1)")
+			(net 268 "Net-(U401-OUT1)")
 			(pinfunction "OUT1")
 			(pintype "output")
@@
 			(layers "*.Cu" "*.Mask")
 			(remove_unused_layers no)
-			(net 269 "Net-(U401-G1)")
+			(net 267 "Net-(U401-G1)")
 			(pinfunction "G1")
 			(pintype "input")
@@
 			(layers "*.Cu" "*.Mask")
 			(remove_unused_layers no)
-			(net 266 "Net-(U401-G2)")
+			(net 264 "Net-(U401-G2)")
 			(pinfunction "G2")
 			(pintype "input")
@@
 			(layers "*.Cu" "*.Mask")
 			(remove_unused_layers no)
-			(net 268 "Net-(U401-OUT2)")
+			(net 266 "Net-(U401-OUT2)")
 			(pinfunction "OUT2")
 			(pintype "output")
@@
 			(layers "*.Cu" "*.Mask")
 			(remove_unused_layers no)
-			(net 267 "Net-(U401-~{CS})")
+			(net 265 "Net-(U401-~{CS})")
 			(pinfunction "~{CS}")
 			(pintype "input")
@@
 			(layers "F.Cu" "F.Mask" "F.Paste")
 			(roundrect_rratio 0.25)
-			(net 11 "GND")
+			(net 275 "TMR_O0")
 			(pintype "input")
 		)
@@
 			(layers "F.Cu" "F.Mask" "F.Paste")
 			(roundrect_rratio 0.25)
-			(net 263 "unconnected-(U109-Pad6)")
-			(pintype "open_collector+no_connect")
+			(net 255 "~{INT6}")
+			(pintype "open_collector")
 		)
 		(pad "7" smd roundrect
@@
 			(layers "F.Cu" "F.Mask" "F.Paste")
 			(roundrect_rratio 0.25)
-			(net 262 "unconnected-(U109-Pad8)")
+			(net 261 "unconnected-(U109-Pad8)")
 			(pintype "open_collector+no_connect")
 		)
@@
 			(layers "F.Cu" "F.Mask" "F.Paste")
 			(roundrect_rratio 0.25)
-			(net 261 "unconnected-(U109-Pad10)")
+			(net 260 "unconnected-(U109-Pad10)")
 			(pintype "open_collector+no_connect")
 		)
@@
 			(layers "F.Cu" "F.Mask" "F.Paste")
 			(roundrect_rratio 0.25)
-			(net 264 "unconnected-(U109-Pad12)")
+			(net 262 "unconnected-(U109-Pad12)")
 			(pintype "open_collector+no_connect")
 		)
@@
 			(layers "*.Cu" "*.Mask")
 			(remove_unused_layers no)
-			(net 255 "~{INT7}")
+			(net 254 "~{INT7}")
 			(pinfunction "1")
 			(pintype "passive")
@@
 			(layers "*.Cu" "*.Mask")
 			(remove_unused_layers no)
-			(net 255 "~{INT7}")
+			(net 254 "~{INT7}")
 			(pinfunction "1")
 			(pintype "passive")
@@
 			(remove_unused_layers no)
 			(roundrect_rratio 0.15625)
-			(net 253 "Net-(U108-I1{slash}CLK)")
+			(net 86 "~{DS}")
 			(pinfunction "I1/CLK")
 			(pintype "input")
@@
 			(layers "*.Cu" "*.Mask")
 			(remove_unused_layers no)
-			(net 254 "~{INT1}")
+			(net 253 "~{INT1}")
 			(pinfunction "I2")
 			(pintype "input")
@@
 			(layers "*.Cu" "*.Mask")
 			(remove_unused_layers no)
-			(net 257 "~{INT2}")
+			(net 256 "~{INT2}")
 			(pinfunction "I3")
 			(pintype "input")
@@
 			(layers "*.Cu" "*.Mask")
 			(remove_unused_layers no)
-			(net 259 "~{INT3}")
+			(net 258 "~{INT3}")
 			(pinfunction "I4")
 			(pintype "input")
@@
 			(layers "*.Cu" "*.Mask")
 			(remove_unused_layers no)
-			(net 258 "~{INT4}")
+			(net 257 "~{INT4}")
 			(pinfunction "I5")
 			(pintype "input")
@@
 			(layers "*.Cu" "*.Mask")
 			(remove_unused_layers no)
-			(net 256 "~{INT6}")
+			(net 255 "~{INT6}")
 			(pinfunction "I7")
 			(pintype "input")
@@
 			(layers "*.Cu" "*.Mask")
 			(remove_unused_layers no)
-			(net 255 "~{INT7}")
+			(net 254 "~{INT7}")
 			(pinfunction "I8")
 			(pintype "input")
@@
 			(layers "*.Cu" "*.Mask")
 			(remove_unused_layers no)
-			(net 86 "~{DS}")
+			(net 28 "RnW")
 			(pinfunction "I12")
 			(pintype "input")
@@
 			(layers "*.Cu" "*.Mask")
 			(remove_unused_layers no)
-			(net 28 "RnW")
+			(net 277 "unconnected-(U108-IO1-Pad14)")
 			(pinfunction "IO1")
-			(pintype "tri_state")
+			(pintype "tri_state+no_connect")
 		)
 		(pad "15" thru_hole circle
@@
 			(layers "*.Cu" "*.Mask")
 			(remove_unused_layers no)
-			(net 260 "unconnected-(U108-IO9-Pad22)")
+			(net 259 "unconnected-(U108-IO9-Pad22)")
 			(pinfunction "IO9")
 			(pintype "tri_state+no_connect")
@@
 			(layers "*.Cu" "*.Mask")
 			(remove_unused_layers no)
-			(net 253 "Net-(U108-I1{slash}CLK)")
+			(net 278 "unconnected-(U108-IO10-Pad23)")
 			(pinfunction "IO10")
-			(pintype "tri_state")
+			(pintype "tri_state+no_connect")
 		)
 		(pad "24" thru_hole circle
@@
 			(layers "*.Cu" "*.Mask")
 			(remove_unused_layers no)
-			(net 255 "~{INT7}")
+			(net 254 "~{INT7}")
 			(pinfunction "Pin_1")
 			(pintype "passive")
@@
 			(layers "F.Cu" "F.Mask" "F.Paste")
 			(roundrect_rratio 0.25)
-			(net 255 "~{INT7}")
+			(net 254 "~{INT7}")
 			(pinfunction "~{RST}")
 			(pintype "open_collector")

Commit message: Add ISACTL ISA bus controller and re-do ATA interface with it.
Parts:
- added C403: 220nF, Capacitor_SMD:C_0805_2012Metric, F.Cu at (216.1, 129.0)
- added C404: 220nF, Capacitor_SMD:C_0805_2012Metric, F.Cu at (218.6, 129.0)
- added C405: 220nF, Capacitor_SMD:C_0805_2012Metric, F.Cu at (228.5, 124.5)
- added C406: 220nF, Capacitor_SMD:C_0805_2012Metric, F.Cu at (228.5, 117.0)
- added C407: 220nF, Capacitor_SMD:C_0805_2012Metric, F.Cu at (221.1, 108.2)
- added C408: 220nF, Capacitor_SMD:C_0805_2012Metric, F.Cu at (215.3, 108.1)
- added C409: 220nF, Capacitor_SMD:C_0805_2012Metric, F.Cu at (207.7, 113.6)
- added C501: 100nF, Capacitor_SMD:C_0805_2012Metric, F.Cu at (124.2, 100.2)
- added C502: 100nF, Capacitor_SMD:C_0805_2012Metric, F.Cu at (135.1, 100.2)
- added C503: 100nF, Capacitor_SMD:C_0805_2012Metric, F.Cu at (123.3, 132.9)
- added D501: ATA Active, LED_THT:LED_D3.0mm, F.Cu at (145.7, 228.4)
- added J401: ISACTL JTAG, Connector_PinHeader_2.54mm:PinHeader_2x05_P2.54mm_Vertical, F.Cu at (223.2, 101.2)
- added J501: ATA connector, Connector_IDC:IDC-Header_2x20_P2.54mm_Vertical, F.Cu at (105.4, 106.8)
- added R401: 10K, Resistor_SMD:R_0805_2012Metric, F.Cu at (223.3, 108.1)
- added R402: 10K, Resistor_SMD:R_0805_2012Metric, F.Cu at (213.2, 108.1)
- added R403: 10K, Resistor_SMD:R_0805_2012Metric, F.Cu at (218.2, 107.3)
- added R501: 47K, Resistor_SMD:R_0805_2012Metric, F.Cu at (125.3, 131.0)
- added R502: 47K, Resistor_SMD:R_0805_2012Metric, F.Cu at (128.5, 131.0)
- added R503: 330, Resistor_SMD:R_0805_2012Metric, F.Cu at (150.6, 228.4)
- added U501: 74ACT245, Package_DIP:DIP-20_W7.62mm_Socket, F.Cu at (115.6, 102.8)
- added U502: 74ACT245, Package_DIP:DIP-20_W7.62mm_Socket, F.Cu at (126.6, 102.8)
- added U503: 74ACT245, Package_DIP:DIP-20_W7.62mm_Socket, F.Cu at (115.6, 136.2)
- C402: value 100nF -> 220nF
- J301: value UART0 FTDI -> UART1 FTDI
- J302: value UART1 FTDI -> UART0 FTDI
- J303: value UART1 -> UART0
- J304: value UART0 -> UART1
- U401: value CP82C54-10Z -> ATF1508AS; footprint Package_DIP:DIP-24_W15.24mm_Socket -> Package_QFP:TQFP-100_14x14mm_P0.5mm
- U402: value GAL22V10 -> MC74ACT05DG; footprint Package_DIP:DIP-24_W7.62mm_Socket -> Package_SO:SOIC-14_3.9x8.7mm_P1.27mm
- moved C401 39.8 mm to (197.5, 120.2), turned to 90 degrees
- moved C402 25.7 mm to (207.7, 121.1), turned to 180 degrees
- moved U401 20.7 mm to (218.1, 118.6)
- moved U402 19.0 mm to (202.2, 117.3)
Connections:
- U102 pad 53: ~{IORD} -> unconnected-(U102-I/O-Pad53)
- U102 pad 54: ~{IOWR} -> unconnected-(U102-I/O-Pad54)
- U102 pad 55: ~{FPUSEL} -> unconnected-(U102-I/O-Pad55)
- U102 pad 56: ~{IACKSEL} -> unconnected-(U102-I/O-Pad56)
- U102 pad 64: ~{ATASEL} -> ~{INTCSEL}
- U102 pad 65: ~{TMRSEL} -> ~{ISASEL}
- U102 pad 67: ~{DUARTSEL} -> ~{IACKSEL}
- U102 pad 68: ~{INTCSEL} -> ~{FPUSEL}
- U109 pad 5: TMR_O0 -> TMRINT
- U109 pad 8: unconnected-(U109-Pad8) -> ~{INT3}
- U109 pad 9: GND -> ATA_INT
- U201 pad 99: unconnected-(U201-I/O-Pad99) -> /FRAM + DRAM0/DRAM0_STERM
- U206 pad 10: unconnected-(U206-Pad10) -> ~{CPU_STERM}
- U206 pad 11: GND -> /FRAM + DRAM0/DRAM0_STERM
- U301 pad 16: A3 -> A8
- U301 pad 20: ~{IOWR} -> ~{ISA_IOWR}
- U301 pad 24: ~{IORD} -> ~{ISA_IORD}
- U401 pad 1: D31 -> /ISA bus interface/ISACTL_DSACK0
- U401 pad 10: Net-(U401-OUT0) -> A2
- U401 pad 11: Net-(U401-G0) -> GND
- U401 pad 12: GND -> A3
- U401 pad 13: Net-(U401-OUT1) -> A4
- U401 pad 14: Net-(U401-G1) -> A5
- U401 pad 15: CLK_6_25 -> /ISA bus interface/ISACTL_TMS
- U401 pad 16: Net-(U401-G2) -> A6
- U401 pad 17: Net-(U401-OUT2) -> A7
- U401 pad 18: CLK_6_25 -> +5V
- U401 pad 19: A0 -> A8
- U401 pad 2: D30 -> /ISA bus interface/ISACTL_DSACK1
- U401 pad 20: A1 -> A9
- U401 pad 21: Net-(U401-~{CS}) -> D24
- U401 pad 22: ~{IORD} -> D25
- U401 pad 23: ~{IOWR} -> D26
- U401 pad 24: +5V -> D27
- U401 pad 3: D29 -> +5V
- U401 pad 4: D28 -> unconnected-(U401-I/O/TDI-Pad4)
- U401 pad 5: D27 -> RnW
- U401 pad 6: D26 -> SIZ0
- U401 pad 7: D25 -> SIZ1
- U401 pad 8: D24 -> A0
- U401 pad 9: CLK_6_25 -> A1
- U402 pad 1: ~{IOWR} -> /ISA bus interface/ISACTL_DSACK0
- U402 pad 11: unconnected-(U402-I11-Pad11) -> GND
- U402 pad 12: GND -> unconnected-(U402-Pad12)
- U402 pad 13: ~{RESET} -> GND
- U402 pad 14: D24 -> GND
- U402 pad 2: ~{IORD} -> ~{CPU_DSACK0}
- U402 pad 3: ~{TMRSEL} -> /ISA bus interface/ISACTL_DSACK1
- U402 pad 4: A2 -> ~{CPU_DSACK1}
- U402 pad 5: Net-(U401-OUT0) -> /ISA bus interface/ISACTL_BERR
- U402 pad 6: Net-(U401-OUT1) -> ~{CPU_BERR}
- U402 pad 7: Net-(U401-OUT2) -> +5V
- U402 pad 9: unconnected-(U402-I9-Pad9) -> GND
Routing:
- net +5V: track 160.1 -> 176.8 mm
- net /ISA bus interface/ISACTL_TDI: track 0.00 -> 4.45 mm
- net /ISA bus interface/ISACTL_TCK: track 0.00 -> 4.21 mm
- net /ISA bus interface/ISACTL_TMS: track 0.00 -> 3.44 mm
Other:
- board size 200 x 154.9 mm -> 259.9 x 154.9 mm
- board text added: "ISACTL"
- board text removed: "TMRGLUE"
