File: cpu030/design-files/cpu030.kicad_pcb (KiCad board)
At the start: 4 copper layers, 259.9 x 154.9 mm, 184 parts, among them J101 Reset, J102 SYSCTL JTAG, J103 NMI, J201 DRAM0SZ, J202 DRAM0 JTAG, J301 UART1 FTDI, J302 UART0 FTDI, J303 UART0, J304 UART1, J401 ISACTL JTAG, J501 ATA connector, J701 RJ45_Amphenol_RJMG1BD3B8K1ANR, J801 DIN41612_03x32_ABC, J901 ATX-24, SW101 Reset, SW102 NMI, U101 MC68030RC, U102 ATF1508AS, U103 MC74ACT05DG, U104 DS1813, U105 SST39SF040 (E), U106 SST39SF040 (O), U107 MC68882, U108 GAL22V10, U109 MC74ACT05DG, U110 DS1813, U201 ATF1508AS, U202 CY7C1061GE (U16), U203 CY7C1061GE (L16), U204 SIMM72-0A, U205 SIMM72-0B, U206 MC74ACT05DG, U301 TL16C2552, U401 ATF1508AS, U402 MC74ACT05DG, U501 74ACT245, U502 74ACT245, U503 74ACT245, U601 PCF8584, U602 DS3231MZ, U701 RTL8019AS, U702 AT93C46D-PU, U801 74ACT245, U802 74ACT245, U803 74ACT245, U804 74ACT245, U805 74ACT245, U806 74ACT245, U807 74ACT245, U808 74ACT245, U809 74ACT245, Y101 50MHz, Y301 1.8432MHz, Y701 20MHz

Commit message: Checkpoint: layout mostly the way I want it now.
Parts:
- removed the R501 at (119.4, 120.3)
- added H105: MountingHole, MountingHole:MountingHole_3.2mm_M3_DIN965_Pad, F.Cu at (216.3, 88.4)
- added H106: MountingHole, MountingHole:MountingHole_3.2mm_M3_DIN965_Pad, F.Cu at (216.3, 235.2)
- added J502: 5V CF Power, Connector_PinHeader_2.54mm:PinHeader_1x04_P2.54mm_Vertical, F.Cu at (117.3, 99.2)
- H101, H102, H103, H104: footprint MountingHole:MountingHole_3.2mm_M3 -> MountingHole:MountingHole_3.2mm_M3_DIN965_Pad
- J801: footprint Connector_DIN:DIN41612_R_3x32_Female_Horizontal_THT -> Connector_DIN:DIN41612_C_3x32_Female_Vertical_THT
- U501, U502, U503, U801, U802, U803, U804, U805, U806, U807, U808, U809: footprint Package_DIP:DIP-20_W7.62mm_Socket -> Package_SO:SOIC-20W_7.5x12.8mm_P1.27mm
- moved J801 88.6 mm to (98.1, 126.5), turned to 0 degrees
- moved C801 65.7 mm to (119.5, 128.9)
- moved U801 60.7 mm to (112.6, 133.7)
- moved U804 46.9 mm to (112.6, 182.2)
- moved J501 45.3 mm to (129.9, 143.6), turned to 180 degrees
- moved C804 41.4 mm to (119.5, 177.5)
- moved C503 35.9 mm to (146.7, 97.3), turned to -90 degrees
- moved SW101 34.2 mm to (180.0, 226.5)
- moved R501 34.0 mm to (149.9, 108.6), turned to -90 degrees
- moved U803 33.2 mm to (112.5, 166.0)
- moved C809 28.2 mm to (119.5, 113.0)
- moved U503 26.9 mm to (139.7, 102.0), turned to 0 degrees
- moved C803 26.7 mm to (119.5, 161.2)
- moved U808 25.6 mm to (126.4, 189.7)
- moved C807 25.1 mm to (133.5, 169.1)
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- renumbered R502 to R501
Connections:
- J801 pad a20: /Expansion interface/EXP_A20 -> /Expansion interface/EXP_A16
- J801 pad a21: /Expansion interface/EXP_A21 -> /Expansion interface/EXP_A18
- J801 pad a22: /Expansion interface/EXP_A22 -> /Expansion interface/EXP_A20
- J801 pad a23: /Expansion interface/EXP_A23 -> /Expansion interface/EXP_A22
- J801 pad a24: /Expansion interface/EXP_A24 -> GND
- J801 pad a26: /Expansion interface/EXP_nMMIOSEL -> /Expansion interface/EXP_nIACKSEL
- J801 pad a27: unconnected-(J801-Pin_a27-Pada27) -> /Expansion interface/EXP_nMMIOSEL
- J801 pad b20: /Expansion interface/EXP_nCI -> ~{CPU_CIIN}
- J801 pad b21: /Expansion interface/EXP_nBR -> ~{CPU_BERR}
- J801 pad b22: /Expansion interface/EXP_nBG -> ~{INT1}
- J801 pad b23: /Expansion interface/EXP_nBGACK -> ~{INT2}
- J801 pad b24: /Expansion interface/EXP_nBERR -> ~{INT3}
- J801 pad b25: /Expansion interface/EXP_nRESET -> ~{INT4}
- J801 pad b26: /Expansion interface/EXP_nDRAMSEL1 -> ~{INT5}
- J801 pad b27: /Expansion interface/EXP_nDRAMSEL2 -> ~{INT6}
- J801 pad b28: /Expansion interface/EXP_nDRAMSEL3 -> /Expansion interface/EXP_nRESET
- J801 pad c20: /Expansion interface/EXP_A25 -> /Expansion interface/EXP_A17
- J801 pad c21: /Expansion interface/EXP_A26 -> /Expansion interface/EXP_A19
- J801 pad c22: /Expansion interface/EXP_A27 -> /Expansion interface/EXP_A21
- J801 pad c23: /Expansion interface/EXP_A28 -> /Expansion interface/EXP_A23
- J801 pad c24: /Expansion interface/EXP_A29 -> GND
- J801 pad c28: /Expansion interface/EXP_nDSACK0 -> ~{CPU_DSACK0}
- J801 pad c29: /Expansion interface/EXP_nDSACK1 -> ~{CPU_DSACK1}
- U502 pad 11: D23 -> D16
- U502 pad 12: D22 -> D17
- U502 pad 13: D21 -> D18
- U502 pad 14: D20 -> D19
- U502 pad 15: D19 -> D20
- U502 pad 16: D18 -> D21
- U502 pad 17: D17 -> D22
- U502 pad 18: D16 -> D23
- U502 pad 2: /IDE interface/ATA_D8 -> /IDE interface/ATA_D15
- U502 pad 3: /IDE interface/ATA_D9 -> /IDE interface/ATA_D14
- U502 pad 4: /IDE interface/ATA_D10 -> /IDE interface/ATA_D13
- U502 pad 5: /IDE interface/ATA_D11 -> /IDE interface/ATA_D12
- U502 pad 6: /IDE interface/ATA_D12 -> /IDE interface/ATA_D11
- U502 pad 7: /IDE interface/ATA_D13 -> /IDE interface/ATA_D10
- U502 pad 8: /IDE interface/ATA_D14 -> /IDE interface/ATA_D9
- U502 pad 9: /IDE interface/ATA_D15 -> /IDE interface/ATA_D8
- U801 pad 11: A0 -> D7
- U801 pad 12: A1 -> D6
- U801 pad 13: A2 -> D5
- U801 pad 14: A3 -> D4
- U801 pad 15: A4 -> D3
- U801 pad 16: A5 -> D2
- U801 pad 17: A6 -> D1
- U801 pad 18: A7 -> D0
- U801 pad 2: /Expansion interface/EXP_A7 -> /Expansion interface/EXP_D0
- U801 pad 3: /Expansion interface/EXP_A6 -> /Expansion interface/EXP_D1
- U801 pad 4: /Expansion interface/EXP_A5 -> /Expansion interface/EXP_D2
- U801 pad 5: /Expansion interface/EXP_A4 -> /Expansion interface/EXP_D3
- U801 pad 6: /Expansion interface/EXP_A3 -> /Expansion interface/EXP_D4
- U801 pad 7: /Expansion interface/EXP_A2 -> /Expansion interface/EXP_D5
- U801 pad 8: /Expansion interface/EXP_A1 -> /Expansion interface/EXP_D6
- U801 pad 9: /Expansion interface/EXP_A0 -> /Expansion interface/EXP_D7
- U802 pad 11: A8 -> D15
- U802 pad 12: A9 -> D14
- U802 pad 13: A10 -> D13
- U802 pad 14: A11 -> D12
- U802 pad 15: A12 -> D11
- U802 pad 16: A13 -> D10
- U802 pad 17: A14 -> D9
- U802 pad 18: A15 -> D8
- U802 pad 2: /Expansion interface/EXP_A15 -> /Expansion interface/EXP_D8
- U802 pad 3: /Expansion interface/EXP_A14 -> /Expansion interface/EXP_D9
- U802 pad 4: /Expansion interface/EXP_A13 -> /Expansion interface/EXP_D10
- U802 pad 5: /Expansion interface/EXP_A12 -> /Expansion interface/EXP_D11
- U802 pad 6: /Expansion interface/EXP_A11 -> /Expansion interface/EXP_D12
- U802 pad 7: /Expansion interface/EXP_A10 -> /Expansion interface/EXP_D13
- U802 pad 8: /Expansion interface/EXP_A9 -> /Expansion interface/EXP_D14
- U802 pad 9: /Expansion interface/EXP_A8 -> /Expansion interface/EXP_D15
- U803 pad 11: A16 -> D31
- U803 pad 12: A17 -> D30
- U803 pad 13: A18 -> D29
- U803 pad 14: A19 -> D28
- U803 pad 15: A20 -> D27
- U803 pad 16: A21 -> D26
- U803 pad 17: A22 -> D25
- U803 pad 18: A23 -> D24
- U803 pad 2: /Expansion interface/EXP_A23 -> /Expansion interface/EXP_D24
- U803 pad 3: /Expansion interface/EXP_A22 -> /Expansion interface/EXP_D25
- U803 pad 4: /Expansion interface/EXP_A21 -> /Expansion interface/EXP_D26
- U803 pad 5: /Expansion interface/EXP_A20 -> /Expansion interface/EXP_D27
- U803 pad 6: /Expansion interface/EXP_A19 -> /Expansion interface/EXP_D28
- U803 pad 7: /Expansion interface/EXP_A18 -> /Expansion interface/EXP_D29
- U803 pad 8: /Expansion interface/EXP_A17 -> /Expansion interface/EXP_D30
- U803 pad 9: /Expansion interface/EXP_A16 -> /Expansion interface/EXP_D31
- U804 pad 11: A24 -> unconnected-(U804-B7-Pad11)
- U804 pad 12: A25 -> unconnected-(U804-B6-Pad12)
- U804 pad 13: A26 -> unconnected-(U804-B5-Pad13)
- U804 pad 14: A27 -> unconnected-(U804-B4-Pad14)
- U804 pad 15: A28 -> unconnected-(U804-B3-Pad15)
- U804 pad 16: A29 -> unconnected-(U804-B2-Pad16)
- U804 pad 17: SIZ0 -> unconnected-(U804-B1-Pad17)
- U804 pad 18: SIZ1 -> unconnected-(U804-B0-Pad18)
- U804 pad 2: /Expansion interface/EXP_SIZ1 -> unconnected-(U804-A0-Pad2)
- U804 pad 3: /Expansion interface/EXP_SIZ0 -> unconnected-(U804-A1-Pad3)
- U804 pad 4: /Expansion interface/EXP_A29 -> unconnected-(U804-A2-Pad4)
- U804 pad 5: /Expansion interface/EXP_A28 -> unconnected-(U804-A3-Pad5)
- U804 pad 6: /Expansion interface/EXP_A27 -> unconnected-(U804-A4-Pad6)
- U804 pad 7: /Expansion interface/EXP_A26 -> unconnected-(U804-A5-Pad7)
- U804 pad 8: /Expansion interface/EXP_A25 -> unconnected-(U804-A6-Pad8)
- U804 pad 9: /Expansion interface/EXP_A24 -> unconnected-(U804-A7-Pad9)
- U805 pad 11: D0 -> CPU_CLK
- U805 pad 12: D1 -> SIZ1
- U805 pad 13: D2 -> SIZ0
- U805 pad 14: D3 -> ~{IACKSEL}
- U805 pad 15: D4 -> ~{MMIOSEL}
- U805 pad 16: D5 -> RnW
- U805 pad 17: D6 -> ~{DS}
- U805 pad 18: D7 -> ~{AS}
- U805 pad 2: /Expansion interface/EXP_D7 -> /Expansion interface/EXP_nAS
- U805 pad 3: /Expansion interface/EXP_D6 -> /Expansion interface/EXP_nDS
- U805 pad 4: /Expansion interface/EXP_D5 -> /Expansion interface/EXP_RnW
- U805 pad 5: /Expansion interface/EXP_D4 -> /Expansion interface/EXP_nMMIOSEL
- U805 pad 6: /Expansion interface/EXP_D3 -> /Expansion interface/EXP_nIACKSEL
- U805 pad 7: /Expansion interface/EXP_D2 -> /Expansion interface/EXP_SIZ0
- U805 pad 8: /Expansion interface/EXP_D1 -> /Expansion interface/EXP_SIZ1
- U805 pad 9: /Expansion interface/EXP_D0 -> /Expansion interface/EXP_CPU_CLK
- U806 pad 11: D8 -> A7
- U806 pad 12: D9 -> A6
- U806 pad 13: D10 -> A5
- U806 pad 14: D11 -> A4
- U806 pad 15: D12 -> A3
- U806 pad 16: D13 -> A2
- U806 pad 17: D14 -> A1
- U806 pad 18: D15 -> A0
- U806 pad 2: /Expansion interface/EXP_D15 -> /Expansion interface/EXP_A0
- U806 pad 3: /Expansion interface/EXP_D14 -> /Expansion interface/EXP_A1
- U806 pad 4: /Expansion interface/EXP_D13 -> /Expansion interface/EXP_A2
- U806 pad 5: /Expansion interface/EXP_D12 -> /Expansion interface/EXP_A3
- U806 pad 6: /Expansion interface/EXP_D11 -> /Expansion interface/EXP_A4
- U806 pad 7: /Expansion interface/EXP_D10 -> /Expansion interface/EXP_A5
- U806 pad 8: /Expansion interface/EXP_D9 -> /Expansion interface/EXP_A6
- U806 pad 9: /Expansion interface/EXP_D8 -> /Expansion interface/EXP_A7
- U807 pad 11: D16 -> A15
- U807 pad 12: D17 -> A14
- U807 pad 13: D18 -> A13
- U807 pad 14: D19 -> A12
- U807 pad 15: D20 -> A11
- U807 pad 16: D21 -> A10
- U807 pad 17: D22 -> A9
- U807 pad 18: D23 -> A8
- U807 pad 2: /Expansion interface/EXP_D23 -> /Expansion interface/EXP_A8
- U807 pad 3: /Expansion interface/EXP_D22 -> /Expansion interface/EXP_A9
- U807 pad 4: /Expansion interface/EXP_D21 -> /Expansion interface/EXP_A10
- U807 pad 5: /Expansion interface/EXP_D20 -> /Expansion interface/EXP_A11
- U807 pad 6: /Expansion interface/EXP_D19 -> /Expansion interface/EXP_A12
- U807 pad 7: /Expansion interface/EXP_D18 -> /Expansion interface/EXP_A13
- U807 pad 8: /Expansion interface/EXP_D17 -> /Expansion interface/EXP_A14
- U807 pad 9: /Expansion interface/EXP_D16 -> /Expansion interface/EXP_A15
- U808 pad 11: D24 -> A23
- U808 pad 12: D25 -> A22
- U808 pad 13: D26 -> A21
- U808 pad 14: D27 -> A20
- U808 pad 15: D28 -> A19
- U808 pad 16: D29 -> A18
- U808 pad 17: D30 -> A17
- U808 pad 18: D31 -> A16
- U808 pad 2: /Expansion interface/EXP_D31 -> /Expansion interface/EXP_A16
- U808 pad 3: /Expansion interface/EXP_D30 -> /Expansion interface/EXP_A17
- U808 pad 4: /Expansion interface/EXP_D29 -> /Expansion interface/EXP_A18
- U808 pad 5: /Expansion interface/EXP_D28 -> /Expansion interface/EXP_A19
- U808 pad 6: /Expansion interface/EXP_D27 -> /Expansion interface/EXP_A20
- U808 pad 7: /Expansion interface/EXP_D26 -> /Expansion interface/EXP_A21
- U808 pad 8: /Expansion interface/EXP_D25 -> /Expansion interface/EXP_A22
- U808 pad 9: /Expansion interface/EXP_D24 -> /Expansion interface/EXP_A23
- U809 pad 11: ~{AS} -> D23
- U809 pad 12: ~{DS} -> D22
- U809 pad 13: RnW -> D21
- U809 pad 14: ~{DRAM1SEL} -> D20
- U809 pad 15: ~{DRAM2SEL} -> D19
- U809 pad 16: ~{DRAM3SEL} -> D18
- U809 pad 17: ~{MMIOSEL} -> D17
- U809 pad 18: unconnected-(U809-B0-Pad18) -> D16
- U809 pad 2: unconnected-(U809-A0-Pad2) -> /Expansion interface/EXP_D16
- U809 pad 3: /Expansion interface/EXP_nMMIOSEL -> /Expansion interface/EXP_D17
- U809 pad 4: /Expansion interface/EXP_nDRAMSEL3 -> /Expansion interface/EXP_D18
- U809 pad 5: /Expansion interface/EXP_nDRAMSEL2 -> /Expansion interface/EXP_D19
- U809 pad 6: /Expansion interface/EXP_nDRAMSEL1 -> /Expansion interface/EXP_D20
- U809 pad 7: /Expansion interface/EXP_RnW -> /Expansion interface/EXP_D21
- U809 pad 8: /Expansion interface/EXP_nDS -> /Expansion interface/EXP_D22
- U809 pad 9: /Expansion interface/EXP_nAS -> /Expansion interface/EXP_D23
Routing:
- added copper zone on In1.Cu, net +5V
- added copper zone on B.Cu, net GND
- added copper zone on F.Cu, net GND
- added copper zone on In2.Cu, net GND
Other:
- board text added: "Expansion Interface"
- board text added: "Red ->"

Commit message: Ethernet analog magic.
Parts:
- added C711: 100nF, Capacitor_SMD:C_0805_2012Metric, F.Cu at (286.3, 108.2)
- added C712: 100nF, Capacitor_SMD:C_0805_2012Metric, F.Cu at (301.5, 111.0)
- added C713: 100nF, Capacitor_SMD:C_0805_2012Metric, F.Cu at (296.3, 111.0)
- added R705: 49.9, Resistor_SMD:R_0805_2012Metric, F.Cu at (288.3, 108.2)
- added R706: 49.9, Resistor_SMD:R_0805_2012Metric, F.Cu at (284.3, 108.2)
- added R707: 10, Resistor_SMD:R_0805_2012Metric, F.Cu at (300.5, 108.3)
- added R708: 10, Resistor_SMD:R_0805_2012Metric, F.Cu at (297.3, 108.3)
- moved J701 20.5 mm to (298.6, 101.5)
- moved C709 20.5 mm to (303.8, 104.9)
- moved C710 20.5 mm to (284.4, 102.5)
- moved R703 20.5 mm to (284.4, 92.7)
- moved R704 20.5 mm to (303.8, 91.1)
Connections:
- U701 pad 45: /Ethernet/ETH_TD+ -> Net-(U701-TPOUT+)
- U701 pad 46: /Ethernet/ETH_TD- -> Net-(U701-TPOUT-)
