File: cpu030/design-files/cpu030.kicad_pcb (KiCad board)
At the start: 4 copper layers, 259.9 x 154.9 mm, 199 parts, among them J101 Reset, J102 SYSCTL JTAG, J103 NMI, J201 DRAM0SZ, J202 DRAM0 JTAG, J301 UART1 FTDI, J302 UART0 FTDI, J303 UART0, J304 UART1, J401 ISACTL JTAG, J501 ATA connector, J502 5V CF Power, J701 RJ45_Amphenol_RJMG1BD3B8K1ANR, J801 DIN41612_03x32_ABC, J901 ATX-24, SW101 Reset, SW102 NMI, U101 MC68030RC, U102 ATF1508AS, U103 MC74ACT05DG, U104 DS1813, U105 SST39SF040 (E), U106 SST39SF040 (O), U107 MC68882, U108 GAL22V10, U109 MC74ACT05DG, U110 DS1813, U201 ATF1508AS, U202 CY7C1061GE (U16), U203 CY7C1061GE (L16), U204 SIMM72-0A, U205 SIMM72-0B, U206 MC74ACT05DG, U301 TL16C2552, U401 ATF1508AS, U402 MC74ACT05DG, U501 74ACT245, U502 74ACT245, U503 74ACT245, U601 PCF8584, U602 DS3231MZ, U701 RTL8019AS, U702 AT93C46D-PU, U801 74ACT245, U802 74ACT245, U803 74ACT245, U804 74ACT245, U805 74ACT245, U806 74ACT245, U807 74ACT245, U808 74ACT245, Y101 50MHz, Y301 1.8432MHz, Y701 20MHz

Commit message: Manually route +12V and -12V.
Routing:
- net -12V: track 0.00 -> 279.0 mm
- net +12V: track 0.00 -> 252.5 mm
Changed lines of the file:
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@@
+	)
+	(segment
+		(start 224.2312 236.4994)
+		(end 219.4348 231.703)
+		(width 1)
+		(layer "B.Cu")
+		(net 429)
+	)
+	(segment
+		(start 139.2936 236.474)
+		(end 127.0762 224.2566)
+		(width 1)
+		(layer "B.Cu")
+		(net 429)
+	)
+	(segment
+		(start 324.172 232.5288)
+		(end 324.3834 232.7402)
+		(width 1)
+		(layer "B.Cu")
+		(net 429)
+	)
+	(segment
+		(start 127.143123 210.473677)
+		(end 127.143123 205.8162)
+		(width 1)
+		(layer "B.Cu")
+		(net 429)
+	)
+	(segment
+		(start 208.407 236.474)
+		(end 139.2936 236.474)
+		(width 1)
+		(layer "B.Cu")
+		(net 429)
+	)
+	(segment
+		(start 324.172 183.7916)
+		(end 324.172 232.5288)
+		(width 1)
+		(layer "B.Cu")
+		(net 429)
+	)
+	(segment
+		(start 127.0762 210.5406)
+		(end 127.143123 210.473677)
+		(width 1)
+		(layer "B.Cu")
+		(net 429)
+	)
+	(segment
+		(start 219.4348 231.703)
+		(end 213.178 231.703)
+		(width 1)
+		(layer "B.Cu")
+		(net 429)
+	)
+	(segment
+		(start 127.0762 224.2566)
+		(end 127.0762 210.5406)
+		(width 1)
+		(layer "B.Cu")
+		(net 429)
+	)
+	(segment
+		(start 213.178 231.703)
+		(end 208.407 236.474)
+		(width 1)
+		(layer "B.Cu")
+		(net 429)
+	)
+	(segment
+		(start 326.723 181.2406)
+		(end 324.172 183.7916)
+		(width 1)
+		(layer "B.Cu")
+		(net 429)
+	)
+	(segment
+		(start 320.6242 236.4994)
+		(end 224.2312 236.4994)
+		(width 1)
+		(layer "B.Cu")
+		(net 429)
+	)
+	(segment
+		(start 324.3834 232.7402)
+		(end 320.6242 236.4994)
+		(width 1)
+		(layer "B.Cu")
+		(net 429)
+	)
+	(segment
+		(start 127.1524 224.0534)
+		(end 122.3302 224.0534)
+		(width 1)
+		(layer "F.Cu")
+		(net 431)
+	)
+	(segment
+		(start 219.5618 231.703)
+		(end 213.2288 231.703)
+		(width 1)
+		(layer "F.Cu")
+		(net 431)
+	)
+	(segment
+		(start 335.7118 223.7994)
+		(end 323.0372 236.474)
+		(width 1)
+		(layer "F.Cu")
+		(net 431)
+	)
+	(segment
+		(start 208.5086 236.4232)
+		(end 139.7508 236.4232)
+		(width 1)
+		(layer "F.Cu")
+		(net 431)
+	)
+	(segment
+		(start 224.3328 236.474)
+		(end 219.5618 231.703)
+		(width 1)
+		(layer "F.Cu")
+		(net 431)
+	)
+	(segment
+		(start 335.788 222.6056)
+		(end 335.788 223.7232)
+		(width 1)
+		(layer "F.Cu")
+		(net 431)
+	)
+	(segment
+		(start 213.2288 231.703)
+		(end 208.5086 236.4232)
+		(width 1)
+		(layer "F.Cu")
+		(net 431)
+	)
+	(segment
+		(start 323.0372 236.474)
+		(end 224.3328 236.474)
+		(width 1)
+		(layer "F.Cu")
+		(net 431)
+	)
+	(segment
+		(start 139.7 236.474)
+		(end 127.2794 224.0534)
+		(width 1)
+		(layer "F.Cu")
+		(net 431)
+	)
+	(segment
+		(start 122.3302 224.0534)
+		(end 112.0178 213.741)
+		(width 1)
+		(layer "F.Cu")
+		(net 431)
+	)
+	(segment
+		(start 332.223 219.0406)
+		(end 335.788 222.6056)
+		(width 1)
+		(layer "F.Cu")
+		(net 431)
+	)
+	(segment
+		(start 332.223 214.8406)
+		(end 332.223 219.0406)
+		(width 1)
+		(layer "B.Cu")
+		(net 431)
 	)
 	(segment

Commit message: Manually route the parallel SIMM connections.
Routing:
- net +5V: track 77.3 -> 98.2 mm
- net D9: track 0.00 -> 17.9 mm
- net D8: track 0.00 -> 17.9 mm
- net D7: track 0.00 -> 17.9 mm
- net D6: track 0.00 -> 17.9 mm
- net D5: track 0.00 -> 17.9 mm
- net D4: track 0.00 -> 17.9 mm
- net D31: track 0.00 -> 17.9 mm
- net D30: track 0.00 -> 17.9 mm
- net D3: track 0.00 -> 17.9 mm
- net D29: track 0.00 -> 17.9 mm
- net D28: track 0.00 -> 17.9 mm
- net D27: track 0.00 -> 17.9 mm
- net D26: track 0.00 -> 17.9 mm
- net D25: track 0.00 -> 17.9 mm
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
Commit message: Manually route the parallel ROM connections.
Routing:
- net ~{ROMSEL}: track 0.00 -> 46.6 mm
- net A1: track 0.00 -> 20.3 mm
- net A6: track 0.00 -> 20.3 mm
- net A5: track 0.00 -> 20.3 mm
- net A3: track 0.00 -> 20.3 mm
- net A17: track 0.00 -> 20.3 mm
- net A16: track 0.00 -> 20.3 mm
- net A8: track 0.00 -> 20.3 mm
- net A4: track 0.00 -> 20.3 mm
- net A2: track 0.00 -> 20.3 mm
- net A19: track 0.00 -> 20.3 mm
- net A13: track 0.00 -> 20.3 mm
- net A9: track 0.00 -> 20.3 mm
- net A15: track 0.00 -> 20.3 mm
- net A14: track 0.00 -> 20.3 mm
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
Commit message: Manually route the buffered IDE signals.
Connections:
- U503 pad 14: ~{ATAAUXSEL} -> A1
- U503 pad 15: ~{ATASEL} -> A2
- U503 pad 16: A2 -> A0
- U503 pad 17: A1 -> ~{ATAAUXSEL}
- U503 pad 18: A0 -> ~{ATASEL}
- U503 pad 2: /IDE interface/ATA_A0 -> /IDE interface/~{ATA_CS1FX}
- U503 pad 3: /IDE interface/ATA_A1 -> /IDE interface/~{ATA_CS3FX}
- U503 pad 4: /IDE interface/ATA_A2 -> /IDE interface/ATA_A0
- U503 pad 5: /IDE interface/~{ATA_CS1FX} -> /IDE interface/ATA_A2
- U503 pad 6: /IDE interface/~{ATA_CS3FX} -> /IDE interface/ATA_A1
Routing:
- net /IDE interface/~{ATA_RESET}: track 0.00 -> 49.2 mm, vias 0 -> 1
- net /IDE interface/ATA_D7: track 0.00 -> 21.8 mm
- net /IDE interface/ATA_D9: track 0.00 -> 21.1 mm, vias 0 -> 2
- net /IDE interface/ATA_D6: track 0.00 -> 19.7 mm
- net /IDE interface/~{ATA_IORD}: track 0.00 -> 19.4 mm, vias 0 -> 1
- net /IDE interface/ATA_D5: track 0.00 -> 18.5 mm
- net /IDE interface/ATA_D10: track 0.00 -> 18.3 mm, vias 0 -> 2
- net /IDE interface/~{ATA_IOWR}: track 0.00 -> 18.2 mm, vias 0 -> 1
- net /IDE interface/ATA_D4: track 0.00 -> 17.2 mm
- net /IDE interface/ATA_D8: track 0.00 -> 17.1 mm, vias 0 -> 2
- net /IDE interface/ATA_D11: track 0.00 -> 17.1 mm, vias 0 -> 2
- net /IDE interface/ATA_D15: track 0.00 -> 17.0 mm, vias 0 -> 2
- net /IDE interface/ATA_D14: track 0.00 -> 16.1 mm, vias 0 -> 2
- net /IDE interface/ATA_D12: track 0.00 -> 16.1 mm, vias 0 -> 2
- net /IDE interface/ATA_D3: track 0.00 -> 15.9 mm
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
Commit message: Hand-route the parallel SRAM signals.
Connections:
- U202 pad 34: A15 -> A16
- U203 pad 34: A15 -> A16
Routing:
- net A19: track 20.3 -> 43.5 mm, vias 0 -> 2
- net A21: track 0.00 -> 22.9 mm, vias 0 -> 2
- net A3: track 20.3 -> 42.9 mm, vias 0 -> 2
- net A7: track 20.3 -> 42.8 mm, vias 0 -> 2
- net A4: track 20.3 -> 42.6 mm, vias 0 -> 2
- net A8: track 20.3 -> 42.0 mm, vias 0 -> 2
- net A6: track 20.3 -> 41.9 mm, vias 0 -> 2
- net A13: track 20.3 -> 41.6 mm, vias 0 -> 2
- net A18: track 20.3 -> 41.5 mm, vias 0 -> 2
- net ~{FRAM_WR}: track 0.00 -> 21.2 mm, vias 0 -> 2
- net A5: track 20.3 -> 41.0 mm, vias 0 -> 2
- net A9: track 20.3 -> 41.0 mm, vias 0 -> 2
- net A12: track 20.3 -> 40.9 mm, vias 0 -> 2
- net A14: track 20.3 -> 40.7 mm, vias 0 -> 2
- net A20: track 0.00 -> 20.2 mm, vias 0 -> 2
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
Commit message: Manually route some I2C and Ethernet signals.
Routing:
- net D27: track 17.9 -> 142.0 mm, vias 0 -> 3
- net D31: track 17.9 -> 129.5 mm, vias 0 -> 2
- net D30: track 17.9 -> 124.6 mm, vias 0 -> 2
- net D26: track 17.9 -> 123.9 mm, vias 0 -> 2
- net D24: track 17.9 -> 123.6 mm, vias 0 -> 3
- net D28: track 17.9 -> 123.0 mm, vias 0 -> 4
- net D29: track 17.9 -> 122.0 mm, vias 0 -> 2
- net D25: track 17.9 -> 120.6 mm, vias 0 -> 3
- net A0: track 0.00 -> 65.8 mm
- net /I2C interface and devices/I2C_SCL: track 0.00 -> 23.1 mm, vias 0 -> 1
- net +5V: track 112.1 -> 132.6 mm
- net /I2C interface and devices/I2C_SDA: track 0.00 -> 19.6 mm, vias 0 -> 1
- net Net-(BT601-+): track 0.00 -> 16.2 mm, vias 0 -> 2
- net /SYSCTL_TCK: track 0.00 -> 11.1 mm, vias 0 -> 1
- net /ISA bus interface/ISACTL_TCK: track 0.00 -> 11.1 mm, vias 0 -> 1
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
Commit message: Route some ROM/SRAM address signals.
Connections:
- U109 pad 10: unconnected-(U109-Pad10) -> ~{INT4}
- U109 pad 11: GND -> ETH_INT
- U601 pad 5: ~{I2CINT} -> ~{INT5}
Routing:
- net ATA_INT: track 0.00 -> 413.1 mm, vias 0 -> 6
- net ~{INT5}: track 0.00 -> 223.2 mm, vias 0 -> 5
- net ETH_INT: track 0.00 -> 171.2 mm, vias 0 -> 4
- net D16: track 17.9 -> 108.3 mm, vias 0 -> 2
- net D18: track 17.9 -> 106.6 mm, vias 0 -> 2
- net D17: track 17.9 -> 103.4 mm, vias 0 -> 2
- net A16: track 39.8 -> 109.8 mm, vias 2 -> 3
- net A13: track 41.6 -> 103.6 mm, vias 2 -> 4
- net D2: track 17.9 -> 77.1 mm, vias 0 -> 2
- net D1: track 17.9 -> 75.2 mm, vias 0 -> 2
- net D0: track 17.9 -> 75.0 mm, vias 0 -> 2
- net D3: track 17.9 -> 72.4 mm, vias 0 -> 2
- net A15: track 39.6 -> 91.4 mm, vias 2 -> 4
- net A14: track 40.7 -> 89.4 mm, vias 2 -> 4
- net A8: track 42.0 -> 81.8 mm
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