File: cpu030/design-files/cpu030.kicad_sch (KiCad schematic)
At the start: 56 parts, among them J101 Reset, J102 SYSCTL JTAG, SW101 Reset, U101 MC68030RC, U102 ATF1508AS, U103 MC74ACT05DG, U104 DS1813, U105 SST39SF040 (E), U106 SST39SF040 (O), U107 MC68882, U108 GAL22V10, U109 MC74ACT05DG, Y101 50MHz

Commit message: Add NMI button.
Parts:
- added J103: NMI, Connector_PinHeader_2.54mm:PinHeader_1x02_P2.54mm_Vertical, symbol Connector:Conn_01x02_Pin
- added SW102: NMI, Button_Switch_THT:SW_PUSH_6mm, symbol Switch:SW_Push
- added U110: DS1813, Package_TO_SOT_SMD:SOT-23-3, symbol jrt-ICs:DS1813
Connections:
- net +5V: now also U110.2 (Vcc)
- net GND: now also J103.2 (Pin_2), SW102.2, U110.3 (GND)
- net ~{INT7}: now also J103.1 (Pin_1), SW102.1, U110.1 (~{RST})

Commit message: System timer.
Connections:
- net GND: no longer U109.5
- net ~{INT6}: now also U109.6
- new net TMR_O0: U109.5
- no-connect marks 23 -> 22
Other:
- added sheet System Timer (cpu030_sys_timer.kicad_sch)
Changed lines of the file:
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@@
 	)
 	(junction
-		(at 242.57 219.71)
-		(diameter 0)
-		(color 0 0 0 0)
-	)
-	(junction
 		(at 361.95 204.47)
 		(diameter 0)
@@
 	)
 	(no_connect
-		(at 257.81 204.47)
-	)
-	(no_connect
 		(at 102.87 143.51)
 	)
@@
 	(wire
 		(pts
-			(xy 242.57 204.47) (xy 242.57 219.71)
-		)
-		(stroke
-			(width 0)
-			(type default)
-		)
-	)
-	(wire
-		(pts
 			(xy 242.57 234.95) (xy 242.57 250.19)
 		)
@@
 		)
 	)
+	(global_label "TMR_O0"
+		(shape input)
+		(at 242.57 204.47 180)
+		(fields_autoplaced yes)
+		(effects
+			(font
+				(size 1.27 1.27)
+			)
+			(justify right)
+		)
+		(property "Intersheetrefs" "${INTERSHEET_REFS}"
+			(at 232.3882 204.47 0)
+			(effects
+				(font
+					(size 1.27 1.27)
+				)
+				(justify right)
+				(hide yes)
+			)
+		)
+	)
 	(global_label "~{RESET}"
 		(shape input)
@@
 		)
 	)
+	(global_label "~{INT6}"
+		(shape output)
+		(at 257.81 204.47 0)
+		(fields_autoplaced yes)
+		(effects
+			(font
+				(size 1.27 1.27)
+			)
+			(justify left)
+		)
+		(property "Intersheetrefs" "${INTERSHEET_REFS}"
+			(at 264.9076 204.47 0)
+			(effects
+				(font
+					(size 1.27 1.27)
+				)
+				(justify left)
+				(hide yes)
+			)
+		)
+	)
 	(global_label "D19"
 		(shape bidirectional)
@@
 				)
 			)
+		)
+	)
+	(sheet
+		(at 84.074 197.612)
+		(size 20.574 9.906)
+		(exclude_from_sim no)
+		(in_bom yes)
+		(on_board yes)
+		(dnp no)
+		(fields_autoplaced yes)
+		(stroke
+			(width 0.1524)
+			(type solid)
+		)
+		(fill
+			(color 0 0 0 0.0000)
+		)
+		(property "Sheetname" "System Timer"
+			(at 84.074 196.9004 0)
+			(effects
+				(font
+					(size 1.27 1.27)
+				)
+				(justify left bottom)
+			)
+		)
+		(property "Sheetfile" "cpu030_sys_timer.kicad_sch"
+			(at 84.074 208.1026 0)
+			(effects
+				(font
+					(size 1.27 1.27)
+				)
+				(justify left top)
+			)
+		)
+		(instances
+			(project "cpu030"
+				(path "/6696b89f-f6cc-4e49-bcfb-68bdb218d2a6"
+					(page "4")
+				)
+			)

Commit message: Eliminate the external D-FF clocking on INTC-1; use the same trick with /DS as we do on TMRGLUE.
Connections:
- net RnW: now also U108.13 (I12); no longer U108.14 (IO1)
- net ~{DS}: now also U108.1 (I1/CLK); no longer U108.13 (I12)
- net at U108.23 (IO10): no longer U108.1 (I1/CLK)
- no-connect marks 22 -> 24
Changed lines of the file:
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@@
 	)
 	(no_connect
+		(at 300.99 204.47)
+	)
+	(no_connect
 		(at 102.87 143.51)
 	)
 	(no_connect
+		(at 300.99 201.93)
+	)
+	(no_connect
 		(at 102.87 119.38)
 	)
 	(no_connect
+		(at 300.99 181.61)
+	)
+	(no_connect
 		(at 257.81 250.19)
 	)
@@
 	)
 	(no_connect
-		(at 300.99 201.93)
-	)
-	(no_connect
 		(at 264.16 116.84)
 	)
@@
 	(wire
 		(pts
-			(xy 320.04 170.18) (xy 275.59 170.18)
-		)
-		(stroke
-			(width 0)
-			(type default)
-		)
-	)
-	(wire
-		(pts
 			(xy 160.02 137.16) (xy 165.1 137.16)
 		)
@@
 	(wire
 		(pts
-			(xy 300.99 204.47) (xy 320.04 204.47)
-		)
-		(stroke
-			(width 0)
-			(type default)
-		)
-	)
-	(wire
-		(pts
 			(xy 374.65 219.71) (xy 384.81 219.71)
 		)
@@
 	(wire
 		(pts
-			(xy 320.04 204.47) (xy 320.04 170.18)
-		)
-		(stroke
-			(width 0)
-			(type default)
-		)
-	)
-	(wire
-		(pts
 			(xy 264.16 49.53) (xy 264.16 48.26)
 		)
@@
 	(wire
 		(pts
-			(xy 275.59 170.18) (xy 275.59 181.61)
-		)
-		(stroke
-			(width 0)
-			(type default)
-		)
-	)
-	(wire
-		(pts
 			(xy 208.28 46.99) (xy 208.28 45.72)
 		)
@@
 	(global_label "~{DS}"
 		(shape input)
-		(at 275.59 209.55 180)
+		(at 275.59 181.61 180)
 		(fields_autoplaced yes)
 		(effects
@@
 		)
 		(property "Intersheetrefs" "${INTERSHEET_REFS}"
-			(at 270.1253 209.55 0)
+			(at 270.1253 181.61 0)
 			(effects
 				(font
@@
 	(global_label "RnW"
 		(shape input)
-		(at 300.99 181.61 0)
+		(at 275.59 209.55 180)
 		(fields_autoplaced yes)
 		(effects
@@
 				(size 1.27 1.27)
 			)
-			(justify left)
+			(justify right)
 		)
 		(property "Intersheetrefs" "${INTERSHEET_REFS}"
-			(at 307.8456 181.61 0)
+			(at 268.7344 209.55 0)
 			(effects
 				(font
 					(size 1.27 1.27)
 				)
-				(justify left)
+				(justify right)
 				(hide yes)
 			)

Commit message: Add ISACTL ISA bus controller and re-do ATA interface with it.
Connections:
- net ~{ATASEL} is gone; now on net ~{INTCSEL}: U102.64 (I/O)
- net ~{DUARTSEL} is gone; now on net ~{IACKSEL}: U102.67 (I/O)
- net GND: no longer U109.9
- net ~{FPUSEL}: now also U102.68 (I/O); no longer U102.55 (I/O)
- net ~{IACKSEL}: no longer U102.56 (I/O)
- net ~{INT3}: now also U109.8
- net ~{INTCSEL}: no longer U102.68 (I/O)
- net TMR_O0 renamed TMRINT
- net ~{IORD}: no longer names the net of U102.53 (I/O)
- net ~{IOWR}: no longer names the net of U102.54 (I/O)
- net ~{TMRSEL} renamed ~{ISASEL}
- new net ATA_INT: U109.9
- no-connect marks 24 -> 27
Other:
- sheet System Timer renamed ISA bus interface
- added sheet IDE interface (cpu030_ide.kicad_sch)
- sheet ISA bus interface: file cpu030_sys_timer.kicad_sch -> cpu030_isa.kicad_sch
Changed lines of the file:
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@@
 	)
 	(junction
-		(at 242.57 234.95)
-		(diameter 0)
-		(color 0 0 0 0)
-	)
-	(junction
 		(at 248.92 162.56)
 		(diameter 0)
@@
 	)
 	(no_connect
+		(at 264.16 121.92)
+	)
+	(no_connect
 		(at 300.99 204.47)
 	)
@@
 	)
 	(no_connect
-		(at 327.66 191.77)
+		(at 264.16 127)
 	)
 	(no_connect
-		(at 257.81 219.71)
+		(at 327.66 191.77)
 	)
 	(no_connect
@@
 	)
 	(no_connect
+		(at 264.16 129.54)
+	)
+	(no_connect
 		(at 102.87 134.62)
 	)
@@
 		(at 102.87 140.97)
 	)
+	(no_connect
+		(at 264.16 124.46)
+	)
 	(wire
 		(pts
@@
 	(wire
 		(pts
-			(xy 242.57 219.71) (xy 242.57 234.95)
-		)
-		(stroke
-			(width 0)
-			(type default)
-		)
-	)
-	(wire
-		(pts
 			(xy 67.31 19.05) (xy 69.85 19.05)
 		)
@@
 		)
 	)
+	(global_label "~{INT3}"
+		(shape output)
+		(at 257.81 219.71 0)
+		(fields_autoplaced yes)
+		(effects
+			(font
+				(size 1.27 1.27)
+			)
+			(justify left)
+		)
+		(property "Intersheetrefs" "${INTERSHEET_REFS}"
+			(at 264.9076 219.71 0)
+			(effects
+				(font
+					(size 1.27 1.27)
+				)
+				(justify left)
+				(hide yes)
+			)
+		)
+	)
 	(global_label "A15"
 		(shape input)
@@
 		)
 	)
-	(global_label "TMR_O0"
+	(global_label "TMRINT"
 		(shape input)
 		(at 242.57 204.47 180)
@@
 		)
 		(property "Intersheetrefs" "${INTERSHEET_REFS}"
-			(at 232.3882 204.47 0)
+			(at 232.9929 204.47 0)
 			(effects
 				(font
@@
 		)
 	)
-	(global_label "~{DUARTSEL}"
+	(global_label "~{ISASEL}"
 		(shape output)
-		(at 264.16 99.06 0)
+		(at 264.16 101.6 0)
 		(fields_autoplaced yes)
 		(effects
@@
 		)
 		(property "Intersheetrefs" "${INTERSHEET_REFS}"
-			(at 276.4585 99.06 0)
+			(at 273.4347 101.6 0)
 			(effects
 				(font
@@
 	(global_label "~{IACKSEL}"
 		(shape output)
-		(at 264.16 121.92 0)
+		(at 264.16 99.06 0)
 		(fields_autoplaced yes)
 		(effects
@@
 		)
 		(property "Intersheetrefs" "${INTERSHEET_REFS}"
-			(at 274.7652 121.92 0)
+			(at 274.7652 99.06 0)
 			(effects
 				(font
@@
 		)
 	)
-	(global_label "~{ATASEL}"
-		(shape output)
-		(at 264.16 104.14 0)
-		(fields_autoplaced yes)
-		(effects
-			(font
-				(size 1.27 1.27)
-			)
-			(justify left)
-		)
-		(property "Intersheetrefs" "${INTERSHEET_REFS}"
-			(at 273.6766 104.14 0)
-			(effects
-				(font
-					(size 1.27 1.27)
-				)
-				(justify left)
-				(hide yes)
-			)
-		)
-	)
 	(global_label "D30"
 		(shape bidirectional)
@@
 		)
 	)
-	(global_label "~{IOWR}"
-		(shape output)
-		(at 264.16 127 0)
-		(fields_autoplaced yes)
-		(effects
-			(font
-				(size 1.27 1.27)
-			)
-			(justify left)
-		)
-		(property "Intersheetrefs" "${INTERSHEET_REFS}"
-			(at 271.8019 127 0)
-			(effects
-				(font
-					(size 1.27 1.27)
-				)
-				(justify left)
-				(hide yes)
-			)
-		)
-	)
 	(global_label "A29"
 		(shape input)
@@
 	(global_label "~{INTCSEL}"
 		(shape output)
-		(at 264.16 96.52 0)
+		(at 264.16 104.14 0)
 		(fields_autoplaced yes)
 		(effects
@@
 		)
 		(property "Intersheetrefs" "${INTERSHEET_REFS}"
-			(at 274.7047 96.52 0)
+			(at 274.7047 104.14 0)
 			(effects
 				(font
@@
 		)
 	)
-	(global_label "~{IORD}"
-		(shape output)
-		(at 264.16 129.54 0)
-		(fields_autoplaced yes)
-		(effects
-			(font
-				(size 1.27 1.27)
-			)
-			(justify left)
-		)
-		(property "Intersheetrefs" "${INTERSHEET_REFS}"
-			(at 271.6205 129.54 0)
-			(effects
-				(font
-					(size 1.27 1.27)
-				)
-				(justify left)
-				(hide yes)
-			)
-		)
-	)
 	(global_label "RnW"
 		(shape input)
@@
 		)
 	)
-	(global_label "~{TMRSEL}"
-		(shape output)
-		(at 264.16 101.6 0)
-		(fields_autoplaced yes)
-		(effects
-			(font
-				(size 1.27 1.27)
-			)
-			(justify left)
-		)
-		(property "Intersheetrefs" "${INTERSHEET_REFS}"
-			(at 274.2208 101.6 0)
-			(effects
-				(font
-					(size 1.27 1.27)
-				)
-				(justify left)
-				(hide yes)
-			)
-		)
-	)
 	(global_label "D9"
 		(shape bidirectional)
@@
 	(global_label "~{FPUSEL}"
 		(shape output)
-		(at 264.16 124.46 0)
+		(at 264.16 96.52 0)
 		(fields_autoplaced yes)
 		(effects
@@
 		)
 		(property "Intersheetrefs" "${INTERSHEET_REFS}"
-			(at 274.2209 124.46 0)
+			(at 274.2209 96.52 0)
 			(effects
 				(font
@@
 		)
 	)
+	(global_label "ATA_INT"
+		(shape input)
+		(at 242.57 219.71 180)
+		(fields_autoplaced yes)
+		(effects
+			(font
+				(size 1.27 1.27)
+			)
+			(justify right)
+		)
+		(property "Intersheetrefs" "${INTERSHEET_REFS}"
+			(at 232.5695 219.71 0)
+			(effects
+				(font
+					(size 1.27 1.27)
+				)
+				(justify right)
+				(hide yes)
+			)
+		)
+	)
 	(global_label "~{DRAM3SEL}"
 		(shape output)
@@
 	)
 	(sheet
+		(at 19.304 214.122)
+		(size 24.892 8.382)
+		(exclude_from_sim no)
+		(in_bom yes)
+		(on_board yes)
+		(dnp no)
+		(fields_autoplaced yes)
+		(stroke
+			(width 0.1524)
+			(type solid)
+		)
+		(fill
+			(color 0 0 0 0.0000)
+		)
+		(property "Sheetname" "IDE interface"
+			(at 19.304 213.4104 0)
+			(effects
+				(font
+					(size 1.27 1.27)
+				)
+				(justify left bottom)
+			)
+		)
+		(property "Sheetfile" "cpu030_ide.kicad_sch"
+			(at 19.304 223.0886 0)
+			(effects
+				(font
+					(size 1.27 1.27)
+				)
+				(justify left top)
+			)
+		)
+		(instances
+			(project "cpu030"
+				(path "/6696b89f-f6cc-4e49-bcfb-68bdb218d2a6"
+					(page "5")
+				)
+			)
+		)
+	)
+	(sheet
 		(at 19.05 197.612)
 		(size 25.146 9.398)
@@
 			(color 0 0 0 0.0000)
 		)
-		(property "Sheetname" "System Timer"
+		(property "Sheetname" "ISA bus interface"
 			(at 84.074 196.9004 0)
 			(effects
@@
 			)
 		)
-		(property "Sheetfile" "cpu030_sys_timer.kicad_sch"
+		(property "Sheetfile" "cpu030_isa.kicad_sch"
 			(at 84.074 208.1026 0)
 			(effects

Commit message: Add I2C controller and RTC.
Other:
- added sheet I2C interface and devices (cpu030_i2c.kicad_sch)
Changed lines of the file:
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@@
+		)
+	)
+	(sheet
+		(at 50.546 214.122)
+		(size 21.336 8.636)
+		(exclude_from_sim no)
+		(in_bom yes)
+		(on_board yes)
+		(dnp no)
+		(fields_autoplaced yes)
+		(stroke
+			(width 0.1524)
+			(type solid)
+		)
+		(fill
+			(color 0 0 0 0.0000)
+		)
+		(property "Sheetname" "I2C interface and devices"
+			(at 50.546 213.4104 0)
+			(effects
+				(font
+					(size 1.27 1.27)
+				)
+				(justify left bottom)
+			)
+		)
+		(property "Sheetfile" "cpu030_i2c.kicad_sch"
+			(at 50.546 223.3426 0)
+			(effects
+				(font
+					(size 1.27 1.27)
+				)
+				(justify left top)
+			)
+		)
+		(instances
+			(project "cpu030"
+				(path "/6696b89f-f6cc-4e49-bcfb-68bdb218d2a6"
+					(page "6")
+				)
+			)
 		)
 	)

Commit message: Add Ethernet.
Other:
- added sheet Ethernet (cpu030_ethernet.kicad_sch)
Changed lines of the file:
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@@
+	)
+	(sheet
+		(at 78.994 214.122)
+		(size 22.606 9.652)
+		(exclude_from_sim no)
+		(in_bom yes)
+		(on_board yes)
+		(dnp no)
+		(fields_autoplaced yes)
+		(stroke
+			(width 0.1524)
+			(type solid)
+		)
+		(fill
+			(color 0 0 0 0.0000)
+		)
+		(property "Sheetname" "Ethernet"
+			(at 78.994 213.4104 0)
+			(effects
+				(font
+					(size 1.27 1.27)
+				)
+				(justify left bottom)
+			)
+		)
+		(property "Sheetfile" "cpu030_ethernet.kicad_sch"
+			(at 78.994 224.3586 0)
+			(effects
+				(font
+					(size 1.27 1.27)
+				)
+				(justify left top)
+			)
+		)
+		(instances
+			(project "cpu030"
+				(path "/6696b89f-f6cc-4e49-bcfb-68bdb218d2a6"
+					(page "7")
+				)
+			)
+		)
 	)
 	(sheet

Commit message: Checkpoint -- expansion interface and PSU placeholders.  More work to do, but I want to get mounting holes placed.
Parts:
- added H101, H102, H103, H104: MountingHole, MountingHole:MountingHole_3.2mm_M3, symbol Mechanical:MountingHole
Connections:
- net +5V: no longer D101.1 (K), R101.1
- new net PWR_OK: D101.1 (K), R101.1
Other:
- added sheet Expansion interface (cpu030_expansion.kicad_sch)
- added sheet Power Supply (cpu030_psu.kicad_sch)

Commit message: Checkpoint: layout mostly the way I want it now.
Parts:
- added H105, H106: MountingHole, MountingHole:MountingHole_3.2mm_M3_DIN965_Pad, symbol Mechanical:MountingHole_Pad
- H101, H102, H103, H104: footprint MountingHole:MountingHole_3.2mm_M3 -> MountingHole:MountingHole_3.2mm_M3_DIN965_Pad; symbol Mechanical:MountingHole -> Mechanical:MountingHole_Pad
Connections:
- net GND: now also H101.1, H102.1, H103.1, H104.1, H105.1, H106.1
