File: cpu030/design-files/cpu030.kicad_sch (KiCad schematic)
At the start: 65 parts, among them J101 Reset, J102 SYSCTL JTAG, J103 NMI, SW101 Reset, SW102 NMI, U101 MC68030RC, U102 ATF1508AS, U103 MC74ACT05DG, U104 DS1813, U105 SST39SF040 (E), U106 SST39SF040 (O), U107 MC68882, U108 GAL22V10, U109 MC74ACT05DG, U110 DS1813, Y101 50MHz

Commit message: MMIOSEL -> EXPSEL
Connections:
- net ~{MMIOSEL} renamed ~{EXPSEL}
Changed lines of the file:
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@@
 		)
 	)
-	(global_label "~{MMIOSEL}"
+	(global_label "~{EXPSEL}"
 		(shape output)
 		(at 264.16 63.5 0)
@@
 		)
 		(property "Intersheetrefs" "${INTERSHEET_REFS}"
-			(at 275.3699 63.5 0)
+			(at 274.1603 63.5 0)
 			(effects
 				(font

Commit message: Checkpoint: some PSU work, lock down Ethernet analog traces.
Parts:
- added C133, C134: 470µF, Capacitor_THT:CP_Radial_D10.0mm_P5.00mm, symbol Device:C_Polarized_Small
Connections:
- net +5V: now also C133.1, C134.1
- net GND: now also C133.2, C134.2

Commit message: Route some ROM/SRAM address signals.
Connections:
- net GND: no longer U109.11
- net ~{INT4}: now also U109.10
- new net ETH_INT: U109.11
- no-connect marks 27 -> 26
Changed lines of the file:
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@@
 	)
 	(junction
-		(at 242.57 250.19)
-		(diameter 0)
-		(color 0 0 0 0)
-	)
-	(junction
 		(at 179.07 21.59)
 		(diameter 0)
@@
 	)
 	(no_connect
-		(at 257.81 234.95)
-	)
-	(no_connect
 		(at 50.8 147.32)
 	)
@@
 	(wire
 		(pts
-			(xy 242.57 234.95) (xy 242.57 250.19)
-		)
-		(stroke
-			(width 0)
-			(type default)
-		)
-	)
-	(wire
-		(pts
 			(xy 80.01 185.42) (xy 90.17 185.42)
 		)
@@
 		)
 	)
+	(global_label "ETH_INT"
+		(shape input)
+		(at 242.57 234.95 180)
+		(fields_autoplaced yes)
+		(effects
+			(font
+				(size 1.27 1.27)
+			)
+			(justify right)
+		)
+		(property "Intersheetrefs" "${INTERSHEET_REFS}"
+			(at 232.2672 234.95 0)
+			(effects
+				(font
+					(size 1.27 1.27)
+				)
+				(justify right)
+				(hide yes)
+			)
+		)
+	)
 	(global_label "D29"
 		(shape output)
@@
 				(hide yes)
 			)
+		)
+	)
+	(global_label "~{INT4}"
+		(shape output)
+		(at 257.81 234.95 0)
+		(fields_autoplaced yes)
+		(effects
+			(font
+				(size 1.27 1.27)
+			)
+			(justify left)
+		)
+		(property "Intersheetrefs" "${INTERSHEET_REFS}"
+			(at 264.9076 234.95 0)
+			(effects
+				(font
+					(size 1.27 1.27)
+				)
+				(justify left)
+				(hide yes)
+			)

Commit message: Fix some schematic mistakes and checkpoint signal routing on the PCB.
Connections:
- net DUART_INTB is gone; now on net TMRINT: U109.3
- net ATA_INT: now also U109.5; no longer U109.9
- net CPU_CLK: now also U107.C2 (CLK)
- net ETH_INT: now also U109.9; no longer U109.11
- net GND: now also U109.11
- net TMRINT: no longer U109.5
- net ~{FPUSEL}: no longer U107.C2 (CLK)
- net ~{INT3}: now also U109.6; no longer U109.8
- net ~{INT4}: now also U109.8; no longer U109.10
- net ~{INT5}: no longer U109.4
- net ~{INT6}: now also U109.4; no longer U109.6
- net DUART_INTA renamed DUART_INT
- no-connect marks 26 -> 27
Changed lines of the file:
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@@
 	)
 	(junction
-		(at 257.81 181.61)
-		(diameter 0)
-		(color 0 0 0 0)
-	)
-	(junction
 		(at 92.71 172.72)
 		(diameter 0)
@@
 	)
 	(junction
+		(at 242.57 250.19)
+		(diameter 0)
+		(color 0 0 0 0)
+	)
+	(junction
 		(at 87.63 172.72)
 		(diameter 0)
@@
 	)
 	(no_connect
+		(at 257.81 234.95)
+	)
+	(no_connect
 		(at 264.16 119.38)
 	)
@@
 	(wire
 		(pts
-			(xy 257.81 175.26) (xy 257.81 181.61)
-		)
-		(stroke
-			(width 0)
-			(type default)
-		)
-	)
-	(wire
-		(pts
 			(xy 80.01 185.42) (xy 90.17 185.42)
 		)
@@
 	(wire
 		(pts
-			(xy 257.81 181.61) (xy 259.08 181.61)
-		)
-		(stroke
-			(width 0)
-			(type default)
-		)
-	)
-	(wire
-		(pts
 			(xy 228.6 162.56) (xy 238.76 162.56)
 		)
@@
 	(wire
 		(pts
-			(xy 208.28 46.99) (xy 208.28 45.72)
+			(xy 242.57 234.95) (xy 242.57 250.19)
 		)
 		(stroke
@@
 	(wire
 		(pts
-			(xy 59.69 180.34) (xy 69.85 180.34)
+			(xy 208.28 46.99) (xy 208.28 45.72)
 		)
 		(stroke
@@
 	(wire
 		(pts
-			(xy 77.47 172.72) (xy 80.01 172.72)
+			(xy 59.69 180.34) (xy 69.85 180.34)
 		)
 		(stroke
@@
 	(wire
 		(pts
-			(xy 238.76 21.59) (xy 241.3 21.59)
+			(xy 77.47 172.72) (xy 80.01 172.72)
 		)
 		(stroke
@@
 	(wire
 		(pts
-			(xy 163.83 271.78) (xy 167.64 271.78)
+			(xy 238.76 21.59) (xy 241.3 21.59)
 		)
 		(stroke
@@
 	(wire
 		(pts
-			(xy 204.47 189.23) (xy 204.47 198.12)
+			(xy 163.83 271.78) (xy 167.64 271.78)
 		)
 		(stroke
@@
 	(wire
 		(pts
-			(xy 257.81 181.61) (xy 257.81 189.23)
+			(xy 204.47 189.23) (xy 204.47 198.12)
 		)
 		(stroke
@@
 	(global_label "~{INT3}"
 		(shape output)
-		(at 257.81 219.71 0)
+		(at 257.81 204.47 0)
 		(fields_autoplaced yes)
 		(effects
@@
 		)
 		(property "Intersheetrefs" "${INTERSHEET_REFS}"
-			(at 264.9076 219.71 0)
+			(at 264.9076 204.47 0)
 			(effects
 				(font
@@
 	(global_label "TMRINT"
 		(shape input)
-		(at 242.57 204.47 180)
+		(at 242.57 189.23 180)
 		(fields_autoplaced yes)
 		(effects
@@
 		)
 		(property "Intersheetrefs" "${INTERSHEET_REFS}"
-			(at 232.9929 204.47 0)
+			(at 232.9929 189.23 0)
 			(effects
 				(font
@@
 		)
 	)
-	(global_label "DUART_INTA"
+	(global_label "DUART_INT"
 		(shape input)
 		(at 242.57 175.26 180)
@@
 		)
 		(property "Intersheetrefs" "${INTERSHEET_REFS}"
-			(at 228.699 175.26 0)
+			(at 229.7876 175.26 0)
 			(effects
 				(font
@@
 	(global_label "ETH_INT"
 		(shape input)
-		(at 242.57 234.95 180)
+		(at 242.57 219.71 180)
 		(fields_autoplaced yes)
 		(effects
@@
 		)
 		(property "Intersheetrefs" "${INTERSHEET_REFS}"
-			(at 232.2672 234.95 0)
+			(at 232.2672 219.71 0)
 			(effects
 				(font
@@
 		)
 	)
-	(global_label "~{FPUSEL}"
+	(global_label "CPU_CLK"
 		(shape input)
 		(at 327.66 154.94 180)
@@
 		)
 		(property "Intersheetrefs" "${INTERSHEET_REFS}"
-			(at 317.5991 154.94 0)
+			(at 316.2686 154.94 0)
 			(effects
 				(font
@@
 		)
 	)
-	(global_label "DUART_INTB"
-		(shape input)
-		(at 242.57 189.23 180)
-		(fields_autoplaced yes)
-		(effects
-			(font
-				(size 1.27 1.27)
-			)
-			(justify right)
-		)
-		(property "Intersheetrefs" "${INTERSHEET_REFS}"
-			(at 228.5176 189.23 0)
-			(effects
-				(font
-					(size 1.27 1.27)
-				)
-				(justify right)
-				(hide yes)
-			)
-		)
-	)
 	(global_label "A16"
 		(shape input)
@@
 	(global_label "~{INT5}"
 		(shape output)
-		(at 259.08 181.61 0)
+		(at 257.81 175.26 0)
 		(fields_autoplaced yes)
 		(effects
@@
 		)
 		(property "Intersheetrefs" "${INTERSHEET_REFS}"
-			(at 266.1776 181.61 0)
+			(at 264.9076 175.26 0)
 			(effects
 				(font
@@
 	(global_label "~{INT4}"
 		(shape output)
-		(at 257.81 234.95 0)
+		(at 257.81 219.71 0)
 		(fields_autoplaced yes)
 		(effects
@@
 		)
 		(property "Intersheetrefs" "${INTERSHEET_REFS}"
-			(at 264.9076 234.95 0)
+			(at 264.9076 219.71 0)
 			(effects
 				(font
@@
 	(global_label "~{INT6}"
 		(shape output)
-		(at 257.81 204.47 0)
+		(at 257.81 189.23 0)
 		(fields_autoplaced yes)
 		(effects
@@
 		)
 		(property "Intersheetrefs" "${INTERSHEET_REFS}"
-			(at 264.9076 204.47 0)
+			(at 264.9076 189.23 0)
 			(effects
 				(font
@@
 	(global_label "ATA_INT"
 		(shape input)
-		(at 242.57 219.71 180)
+		(at 242.57 204.47 180)
 		(fields_autoplaced yes)
 		(effects
@@
 		)
 		(property "Intersheetrefs" "${INTERSHEET_REFS}"
-			(at 232.5695 219.71 0)
+			(at 232.5695 204.47 0)
 			(effects
 				(font

Commit message: Checkpoint -- I'm going to re-arrange the board a bit and make it 6 layers, putting CPU address and data busses on their own internal signal layers.  Hopefully this detangles the mess a bit.
Parts:
- RN101: footprint Resistor_THT:R_Array_SIP7 -> Resistor_THT:R_Array_SIP9; symbol Device:R_Network06 -> Device:R_Network08
Connections:
- net +5V: no longer U101.F13 (/MMUDIS)
- net ~{CPU_CBACK}: now also RN101.9 (R8); no longer RN101.6 (R5)
- net ~{PSUSEL}: now reaches U102.61 (I/O)
- net at U101.H2 (/HALT): now also RN101.8 (R7)
- new net: RN101.6 (R5), U101.F13 (/MMUDIS)
- no-connect marks 27 -> 26

Commit message: Checkpoint -- more FPU signals connected.
Connections:
- net +5V: no longer U101.A1 (/BR), U101.C3 (/BGACK)
- no-connect marks 26 -> 28
Changed lines of the file:
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@@
 	)
 	(no_connect
+		(at 102.87 137.16)
+	)
+	(no_connect
 		(at 264.16 116.84)
 	)
@@
 	)
 	(no_connect
+		(at 102.87 132.08)
+	)
+	(no_connect
 		(at 264.16 129.54)
 	)
@@
 	)
 	(symbol
-		(lib_id "power:+5V")
-		(at 102.87 137.16 270)
-		(unit 1)
-		(exclude_from_sim no)
-		(in_bom yes)
-		(on_board yes)
-		(dnp no)
-		(fields_autoplaced yes)
-		(property "Reference" "#PWR0114"
-			(at 99.06 137.16 0)
-			(effects
-				(font
-					(size 1.27 1.27)
-				)
-				(hide yes)
-			)
-		)
-		(property "Value" "+5V"
-			(at 106.68 137.1599 90)
-			(effects
-				(font
-					(size 1.27 1.27)
-				)
-				(justify left)
-			)
-		)
-		(property "Footprint" ""
-			(at 102.87 137.16 0)
-			(effects
-				(font
-					(size 1.27 1.27)
-				)
-				(hide yes)
-			)
-		)
-		(property "Datasheet" ""
-			(at 102.87 137.16 0)
-			(effects
-				(font
-					(size 1.27 1.27)
-				)
-				(hide yes)
-			)
-		)
-		(property "Description" "Power symbol creates a global label with name \"+5V\""
-			(at 102.87 137.16 0)
-			(effects
-				(font
-					(size 1.27 1.27)
-				)
-				(hide yes)
-			)
-		)
-		(pin "1"
-		)
-		(instances
-			(project "cpu030"
-				(path "/6696b89f-f6cc-4e49-bcfb-68bdb218d2a6"
-					(reference "#PWR0114")
-					(unit 1)
-				)
-			)
-		)
-	)
-	(symbol
 		(lib_id "Device:C_Small")
 		(at 80.01 182.88 0)
@@
 					(unit 1)
 				)
-			)
-		)
-	)
-	(symbol
-		(lib_id "power:+5V")
-		(at 102.87 132.08 270)
-		(unit 1)
-		(exclude_from_sim no)
-		(in_bom yes)
-		(on_board yes)
-		(dnp no)
-		(fields_autoplaced yes)
-		(property "Reference" "#PWR0113"
-			(at 99.06 132.08 0)
-			(effects
-				(font
-					(size 1.27 1.27)
-				)
-				(hide yes)
-			)
-		)
-		(property "Value" "+5V"
-			(at 106.68 132.0799 90)
-			(effects
-				(font
-					(size 1.27 1.27)
-				)
-				(justify left)
-			)
-		)
-		(property "Footprint" ""
-			(at 102.87 132.08 0)
-			(effects
-				(font
-					(size 1.27 1.27)
-				)
-				(hide yes)
-			)
-		)
-		(property "Datasheet" ""
-			(at 102.87 132.08 0)
-			(effects
-				(font
-					(size 1.27 1.27)
-				)
-				(hide yes)
-			)
-		)
-		(property "Description" "Power symbol creates a global label with name \"+5V\""
-			(at 102.87 132.08 0)
-			(effects
-				(font
-					(size 1.27 1.27)
-				)
-				(hide yes)
-			)
-		)
-		(pin "1"
-		)
-		(instances
-			(project ""
-				(path "/6696b89f-f6cc-4e49-bcfb-68bdb218d2a6"
-					(reference "#PWR0113")
-					(unit 1)
-				)

Commit message: Checkpoint: ROM data bus lines.
Connections:
- net +5V: no longer U101.H12 (/CDIS)
- net at RN101.6 (R5), U101.F13 (/MMUDIS): now also U101.H12 (/CDIS)
Changed lines of the file:
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@@
 	)
 	(junction
+		(at 30.48 140.97)
+		(diameter 0)
+		(color 0 0 0 0)
+	)
+	(junction
 		(at 179.07 21.59)
 		(diameter 0)
@@
 	(wire
 		(pts
+			(xy 30.48 165.1) (xy 50.8 165.1)
+		)
+		(stroke
+			(width 0)
+			(type default)
+		)
+	)
+	(wire
+		(pts
 			(xy 20.32 120.65) (xy 50.8 120.65)
 		)
@@
 	(wire
 		(pts
+			(xy 30.48 140.97) (xy 30.48 165.1)
+		)
+		(stroke
+			(width 0)
+			(type default)
+		)
+	)
+	(wire
+		(pts
 			(xy 13.97 123.19) (xy 22.86 123.19)
 		)
@@
 					(unit 1)
 				)
-			)
-		)
-	)
-	(symbol
-		(lib_id "power:+5V")
-		(at 50.8 165.1 90)
-		(unit 1)
-		(exclude_from_sim no)
-		(in_bom yes)
-		(on_board yes)
-		(dnp no)
-		(fields_autoplaced yes)
-		(property "Reference" "#PWR0103"
-			(at 54.61 165.1 0)
-			(effects
-				(font
-					(size 1.27 1.27)
-				)
-				(hide yes)
-			)
-		)
-		(property "Value" "+5V"
-			(at 46.99 165.0999 90)
-			(effects
-				(font
-					(size 1.27 1.27)
-				)
-				(justify left)
-			)
-		)
-		(property "Footprint" ""
-			(at 50.8 165.1 0)
-			(effects
-				(font
-					(size 1.27 1.27)
-				)
-				(hide yes)
-			)
-		)
-		(property "Datasheet" ""
-			(at 50.8 165.1 0)
-			(effects
-				(font
-					(size 1.27 1.27)
-				)
-				(hide yes)
-			)
-		)
-		(property "Description" "Power symbol creates a global label with name \"+5V\""
-			(at 50.8 165.1 0)
-			(effects
-				(font
-					(size 1.27 1.27)
-				)
-				(hide yes)
-			)
-		)
-		(pin "1"
-		)
-		(instances
-			(project "cpu030"
-				(path "/6696b89f-f6cc-4e49-bcfb-68bdb218d2a6"
-					(reference "#PWR0103")
-					(unit 1)
-				)

Commit message: Fix some connection mistakes on the 74ACT05s, re-arrange pullups on CPU to make layout easier.
Parts:
- RN101: footprint Resistor_THT:R_Array_SIP9 -> Resistor_THT:R_Array_SIP7; symbol Device:R_Network08 -> Device:R_Network06
- U103, U109: value MC74ACT05DG -> 74ACT05
Connections:
- net +5V: now also U103.14 (VCC), U109.14 (VCC); no longer U103.7 (GND), U109.7 (GND)
- net GND: now also U103.7 (GND), U109.7 (GND); no longer U103.14 (VCC), U109.14 (VCC)
- net ~{CPU_BERR}: now also RN101.5 (R4); no longer RN101.4 (R3)
- net ~{CPU_CBACK}: now also RN101.6 (R5); no longer RN101.9 (R8)
- net ~{CPU_CIIN}: now also RN101.7 (R6); no longer RN101.5 (R4)
- net ~{CPU_DSACK1}: now also RN101.4 (R3); no longer RN101.3 (R2)
- net ~{CPU_STERM}: now also RN101.3 (R2); no longer RN101.7 (R6)
- net at U101.H2 (/HALT): no longer RN101.8 (R7)
- now unconnected: U101.F13 (/MMUDIS), U101.H12 (/CDIS)
Other:
- moved on the sheet: U103G, U109G
