File: cpu030/design-files/cpu030.kicad_sch (KiCad schematic)
At the start: 67 parts, among them J101 Reset, J102 SYSCTL JTAG, J103 NMI, SW101 Reset, SW102 NMI, U101 MC68030RC, U102 ATF1508AS, U103 74ACT05, U104 DS1813, U105 SST39SF040 (E), U106 SST39SF040 (O), U107 MC68882, U108 GAL22V10, U109 74ACT05, U110 DS1813, Y101 50MHz

Commit message: Pullups on the INTx inputs.
Parts:
- added RN106: 3K3, Resistor_THT:R_Array_SIP7, symbol Device:R_Network06
Connections:
- net +5V: now also RN106.1 (common)
- net ~{INT1}: now also RN106.2 (R1)
- net ~{INT2}: now also RN106.3 (R2)
- net ~{INT3}: now also RN106.4 (R3)
- net ~{INT4}: now also RN106.5 (R4)
- net ~{INT5}: now also RN106.6 (R5)
- net ~{INT6}: now also RN106.7 (R6)

Commit message: Checkpoint: Nearly done with the expansion interface.
Parts:
- added R106: 3K3, Resistor_SMD:R_0805_2012Metric, symbol Device:R_Small
- RN101: footprint Resistor_THT:R_Array_SIP7 -> Resistor_THT:R_Array_SIP9; symbol Device:R_Network06 -> Device:R_Network08
- RN102, RN103, RN104, RN105: value 10K -> 3K3
- U101: value MC68030RC -> MC68030
Connections:
- net +5V: now also R106.1
- net ~{CPU_BERR}: now also RN101.7 (R6); no longer RN101.5 (R4)
- net ~{CPU_CBACK}: now also RN101.8 (R7); no longer RN101.6 (R5)
- net ~{CPU_CIIN}: now also RN101.9 (R8); no longer RN101.7 (R6)
- net ~{CPU_DSACK0}: now also RN101.4 (R3); no longer RN101.2 (R1)
- net ~{CPU_DSACK1}: now also RN101.6 (R5); no longer RN101.4 (R3)
- net ~{CPU_STERM}: now also RN101.5 (R4); no longer RN101.3 (R2)
- net ~{CPU_BR}: now reaches U101.A1 (/BR)
- net ~{CPU_BR}: now also R106.2
- net ~{CPU_BG}: now reaches U101.B2 (/BG)
- net ~{CPU_BG}: now also RN101.2 (R1)
- net ~{CPU_BGACK}: now reaches U101.C3 (/BGACK)
- net ~{CPU_BGACK}: now also RN101.3 (R2)
- no-connect marks 28 -> 25

Commit message: Couple of missing CPU pullups.
Parts:
- added R107, R108: 3K3, Resistor_SMD:R_0805_2012Metric, symbol Device:R_Small
Connections:
- net +5V: now also R107.1, R108.1
- net ~{MMUDIS}: now reaches U101.F13 (/MMUDIS)
- net ~{MMUDIS}: now also R107.2
- net ~{HALT}: now reaches U101.H2 (/HALT)
- net ~{HALT}: now also R108.2
Changed lines of the file:
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@@
 	)
 	(junction
+		(at 165.1 180.34)
+		(diameter 0)
+		(color 0 0 0 0)
+	)
+	(junction
 		(at 228.6 157.48)
 		(diameter 0)
@@
 	)
 	(junction
+		(at 173.99 180.34)
+		(diameter 0)
+		(color 0 0 0 0)
+	)
+	(junction
 		(at 132.08 166.37)
 		(diameter 0)
@@
 	(wire
 		(pts
+			(xy 182.88 182.88) (xy 182.88 180.34)
+		)
+		(stroke
+			(width 0)
+			(type default)
+		)
+	)
+	(wire
+		(pts
 			(xy 69.85 172.72) (xy 72.39 172.72)
 		)
@@
 	(wire
 		(pts
+			(xy 173.99 180.34) (xy 173.99 182.88)
+		)
+		(stroke
+			(width 0)
+			(type default)
+		)
+	)
+	(wire
+		(pts
 			(xy 142.24 118.11) (xy 142.24 119.38)
 		)
@@
 	(wire
 		(pts
+			(xy 182.88 180.34) (xy 173.99 180.34)
+		)
+		(stroke
+			(width 0)
+			(type default)
+		)
+	)
+	(wire
+		(pts
 			(xy 208.28 44.45) (xy 208.28 43.18)
 		)
@@
 	(wire
 		(pts
+			(xy 48.26 140.97) (xy 50.8 140.97)
+		)
+		(stroke
+			(width 0)
+			(type default)
+		)
+	)
+	(wire
+		(pts
 			(xy 339.09 204.47) (xy 341.63 204.47)
 		)
@@
 	(wire
 		(pts
+			(xy 173.99 180.34) (xy 165.1 180.34)
+		)
+		(stroke
+			(width 0)
+			(type default)
+		)
+	)
+	(wire
+		(pts
 			(xy 154.94 137.16) (xy 160.02 137.16)
 		)
@@
 	(wire
 		(pts
+			(xy 40.64 134.62) (xy 50.8 134.62)
+		)
+		(stroke
+			(width 0)
+			(type default)
+		)
+	)
+	(wire
+		(pts
 			(xy 269.24 228.6) (xy 283.21 228.6)
 		)
@@
 		)
 	)
+	(label "~{MMUDIS}"
+		(at 48.26 140.97 180)
+		(effects
+			(font
+				(size 1.27 1.27)
+			)
+			(justify right bottom)
+		)
+	)
 	(label "SYSCTL_DSACK0"
 		(at 207.01 44.45 180)
@@
 		)
 	)
+	(label "~{MMUDIS}"
+		(at 173.99 187.96 270)
+		(effects
+			(font
+				(size 1.27 1.27)
+			)
+			(justify right bottom)
+		)
+	)
 	(label "SYSCTL_STERM"
 		(at 144.78 85.09 0)
@@
 		)
 	)
+	(label "~{HALT}"
+		(at 182.88 187.96 270)
+		(effects
+			(font
+				(size 1.27 1.27)
+			)
+			(justify right bottom)
+		)
+	)
 	(label "SYSCTL_TDI"
 		(at 207.01 49.53 180)
@@
 		)
 	)
+	(label "~{HALT}"
+		(at 40.64 134.62 180)
+		(effects
+			(font
+				(size 1.27 1.27)
+			)
+			(justify right bottom)
+		)
+	)
 	(label "SYSCTL_BERR"
 		(at 264.16 38.1 0)
@@
 	)
 	(symbol
+		(lib_id "Device:R_Small")
+		(at 182.88 185.42 0)
+		(unit 1)
+		(exclude_from_sim no)
+		(in_bom yes)
+		(on_board yes)
+		(dnp no)
+		(fields_autoplaced yes)
+		(property "Reference" "R108"
+			(at 185.42 184.1499 0)
+			(effects
+				(font
+					(size 1.016 1.016)
+				)
+				(justify left)
+			)
+		)
+		(property "Value" "3K3"
+			(at 185.42 186.6899 0)
+			(effects
+				(font
+					(size 1.27 1.27)
+				)
+				(justify left)
+			)
+		)
+		(property "Footprint" "Resistor_SMD:R_0805_2012Metric"
+			(at 182.88 185.42 0)
+			(effects
+				(font
+					(size 1.27 1.27)
+				)
+				(hide yes)
+			)
+		)
+		(property "Datasheet" "~"
+			(at 182.88 185.42 0)
+			(effects
+				(font
+					(size 1.27 1.27)
+				)
+				(hide yes)
+			)
+		)
+		(property "Description" "Resistor, small symbol"
+			(at 182.88 185.42 0)
+			(effects
+				(font
+					(size 1.27 1.27)
+				)
+				(hide yes)
+			)
+		)
+		(pin "2"
+		)
+		(pin "1"
+		)
+		(instances
+			(project "cpu030"
+				(path "/6696b89f-f6cc-4e49-bcfb-68bdb218d2a6"
+					(reference "R108")
+					(unit 1)
+				)
+			)
+		)
+	)
+	(symbol
 		(lib_id "74xx:74LS05")
 		(at 250.19 189.23 0)
@@
 					(unit 1)
 				)
+			)
+		)
+	)
+	(symbol
+		(lib_id "Device:R_Small")
+		(at 173.99 185.42 0)
+		(unit 1)
+		(exclude_from_sim no)
+		(in_bom yes)
+		(on_board yes)
+		(dnp no)
+		(fields_autoplaced yes)
+		(property "Reference" "R107"
+			(at 176.53 184.1499 0)
+			(effects
+				(font
+					(size 1.016 1.016)
+				)
+				(justify left)
+			)
+		)
+		(property "Value" "3K3"
+			(at 176.53 186.6899 0)
+			(effects
+				(font
+					(size 1.27 1.27)
+				)
+				(justify left)
+			)
+		)
+		(property "Footprint" "Resistor_SMD:R_0805_2012Metric"
+			(at 173.99 185.42 0)
+			(effects
+				(font
+					(size 1.27 1.27)
+				)
+				(hide yes)
+			)
+		)
+		(property "Datasheet" "~"
+			(at 173.99 185.42 0)
+			(effects
+				(font
+					(size 1.27 1.27)
+				)
+				(hide yes)
+			)
+		)
+		(property "Description" "Resistor, small symbol"
+			(at 173.99 185.42 0)
+			(effects
+				(font
+					(size 1.27 1.27)
+				)
+				(hide yes)
+			)
+		)
+		(pin "2"
+		)
+		(pin "1"
+		)
+		(instances
+			(project "cpu030"
+				(path "/6696b89f-f6cc-4e49-bcfb-68bdb218d2a6"
+					(reference "R107")
+					(unit 1)
+				)

Commit message: Re-pin SYSCTL to make signal routing a lot easier.
Connections:
- net ~{DEVSEL} is gone; now on net CLK_6_25: U102.84 (I/O)
- net ~{DRAM1SEL} is gone; now on net A28: U102.70 (I/O)
- net ~{DRAM2SEL} is gone; now on net A29: U102.71 (I/O)
- net ~{DRAM3SEL} is gone; now on net A30: U102.72 (I/O)
- net A0: now also U102.35 (I/O); no longer U102.8 (I/O)
- net A1: now also U102.36 (I/O); no longer U102.9 (I/O)
- net A10: now also U102.48 (I/O); no longer U102.21 (I/O)
- net A11: now also U102.49 (I/O); no longer U102.22 (I/O)
- net A12: now also U102.50 (I/O); no longer U102.23 (I/O)
- net A13: now also U102.52 (I/O); no longer U102.24 (I/O)
- net A14: now also U102.53 (I/O); no longer U102.25 (I/O)
- net A15: now also U102.54 (I/O); no longer U102.27 (I/O)
- net A16: now also U102.55 (I/O); no longer U102.28 (I/O)
- net A17: now also U102.56 (I/O); no longer U102.29 (I/O)
- net A18: now also U102.57 (I/O); no longer U102.30 (I/O)
- net A19: now also U102.58 (I/O); no longer U102.31 (I/O)
- net A2: now also U102.37 (I/O); no longer U102.10 (I/O)
- net A20: now also U102.60 (I/O); no longer U102.32 (I/O)
- net A21: now also U102.61 (I/O); no longer U102.33 (I/O)
- net A22: now also U102.63 (I/O); no longer U102.35 (I/O)
- net A23: now also U102.64 (I/O); no longer U102.36 (I/O)
- net A24: now also U102.65 (I/O); no longer U102.37 (I/O)
- net A25: now also U102.67 (I/O); no longer U102.40 (I/O)
- net A26: now also U102.68 (I/O); no longer U102.41 (I/O/PD2)
- net A27: now also U102.69 (I/O); no longer U102.42 (I/O)
- net A28: no longer U102.44 (I/O)
- net A29: no longer U102.45 (I/O)
- net A3: now also U102.40 (I/O); no longer U102.12 (I/O)
- net A30: no longer U102.46 (I/O)
- net A31: now also U102.75 (I/O); no longer U102.47 (I/O)
- net A4: now also U102.41 (I/O/PD2); no longer U102.13 (I/O)
- net A5: now also U102.42 (I/O); no longer U102.14 (I/O)
- net A6: now also U102.44 (I/O); no longer U102.16 (I/O)
- net A7: now also U102.45 (I/O); no longer U102.17 (I/O)
- net A8: now also U102.46 (I/O); no longer U102.19 (I/O)
- net A9: now also U102.47 (I/O); no longer U102.20 (I/O)
- net CLK_6_25: no longer U102.92 (I/O)
- net CPU_CLK: now also U102.83 (I/O); no longer U102.94 (I/O)
- net FC0: now also U102.76 (I/O); no longer U102.48 (I/O)
- net FC1: now also U102.77 (I/O); no longer U102.49 (I/O)
- net FC2: now also U102.78 (I/O); no longer U102.50 (I/O)
- net RESET: now also U102.92 (I/O); no longer U102.52 (I/O)
- net RnW: now also U102.31 (I/O); no longer U102.5 (I/O)
- net SIZ0: now also U102.32 (I/O); no longer U102.6 (I/O)
- net SIZ1: now also U102.33 (I/O); no longer U102.7 (I/O)
- net SYSCTL_BERR: now also U102.5 (I/O); no longer U102.100 (I/O)
- net SYSCTL_CBACK: now also U102.6 (I/O); no longer U102.98 (I/O)
- net SYSCTL_CI: now also U102.8 (I/O); no longer U102.96 (I/O)
- net SYSCTL_STERM: now also U102.7 (I/O); no longer U102.99 (I/O)
- net ~{CBREQ}: now also U102.30 (I/O); no longer U102.97 (I/O)
- net ~{DRAM0SEL}: now also U102.93 (I/O); no longer U102.69 (I/O)
- net ~{EXPSEL}: now also U102.28 (I/O); no longer U102.83 (I/O)
- net ~{FPUSEL}: now also U102.81 (I/O); no longer U102.68 (I/O)
- net ~{FRAMSEL}: now also U102.9 (I/O); no longer U102.81 (I/O)
- net ~{FRAM_BE0}: now also U102.13 (I/O); no longer U102.75 (I/O)
- net ~{FRAM_BE1}: now also U102.14 (I/O); no longer U102.76 (I/O)
- net ~{FRAM_BE2}: now also U102.16 (I/O); no longer U102.77 (I/O)
- net ~{FRAM_BE3}: now also U102.17 (I/O); no longer U102.78 (I/O)
- net ~{FRAM_RD}: now also U102.10 (I/O); no longer U102.80 (I/O)
- net ~{FRAM_WR}: now also U102.12 (I/O); no longer U102.79 (I/O)
- net ~{I2CSEL}: now also U102.98 (I/O); no longer U102.63 (I/O)
- net ~{IACKSEL}: now also U102.79 (I/O); no longer U102.67 (I/O)
- net ~{INTCSEL}: now also U102.80 (I/O); no longer U102.64 (I/O)
- net ~{ISASEL}: now also U102.99 (I/O); no longer U102.65 (I/O)
- net ~{PSUSEL}: now also U102.29 (I/O); no longer U102.61 (I/O)
- net ~{ROMSEL}: now also U102.100 (I/O); no longer U102.85 (I/O/GCLK3)
- no-connect marks 25 -> 29

Commit message: Add the EXPGLUE GAL.
Connections:
- net ~{CPU_DBEN}: now reaches U101.M1 (/DBEN)
- no-connect marks 29 -> 28
Changed lines of the file:
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@@
 	)
 	(no_connect
-		(at 102.87 146.05)
-	)
-	(no_connect
 		(at 208.28 99.06)
 	)
@@
 				(hide yes)
 			)
+		)
+	)
+	(global_label "~{CPU_DBEN}"
+		(shape output)
+		(at 102.87 146.05 0)
+		(fields_autoplaced yes)
+		(effects
+			(font
+				(size 1.27 1.27)
+			)
+			(justify left)
+		)
+		(property "Intersheetrefs" "${INTERSHEET_REFS}"
+			(at 115.7128 146.05 0)
+			(effects
+				(font
+					(size 1.27 1.27)
+				)
+				(justify left)
+				(hide yes)
+			)

Commit message: Some board tweaks before I take another crack at routing.
Parts:
- removed J103: NMI, Connector_PinHeader_2.54mm:PinHeader_1x02_P2.54mm_Vertical, symbol Connector:Conn_01x02_Pin
- J101: value Reset -> Reset / Power / NMI; footprint Connector_PinHeader_2.54mm:PinHeader_1x02_P2.54mm_Vertical -> Connector_PinHeader_2.54mm:PinHeader_2x03_P2.54mm_Vertical; symbol Connector:Conn_01x02_Pin -> Connector_Generic:Conn_02x03_Odd_Even
Connections:
- net GND: now also J101.1 (Pin_1), J101.3 (Pin_3), J101.5 (Pin_5); no longer J101.2 (Pin_2)
- net ~{INT7}: now also J101.6 (Pin_6)
- net ~{RESET}: now also J101.2 (Pin_2); no longer J101.1 (Pin_1)
- new net ~{PWR_BUT}: J101.4 (Pin_4)

Commit message: Rearrange some pins on U109 to make routing easier.
Connections:
- net ATA_INT: now also U109.1; no longer U109.5
- net DUART_INT: now also U109.11; no longer U109.1
- net ETH_INT: now also U109.13; no longer U109.9
- net GND: now also U109.3, U109.5; no longer U109.11, U109.13
- net TMRINT: now also U109.9; no longer U109.3
- net ~{INT3}: now also U109.2; no longer U109.6
- net ~{INT4}: now also U109.12; no longer U109.8
- net ~{INT5}: now also U109.10; no longer U109.2
- net ~{INT6}: now also U109.8; no longer U109.4
Changed lines of the file:
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@@
 	)
 	(junction
+		(at 242.57 204.47)
+		(diameter 0)
+		(color 0 0 0 0)
+	)
+	(junction
 		(at 80.01 19.05)
 		(diameter 0)
@@
 	)
 	(junction
-		(at 242.57 250.19)
-		(diameter 0)
-		(color 0 0 0 0)
-	)
-	(junction
 		(at 87.63 172.72)
 		(diameter 0)
@@
 	)
 	(no_connect
-		(at 257.81 234.95)
-	)
-	(no_connect
 		(at 208.28 88.9)
 	)
@@
 	)
 	(no_connect
-		(at 257.81 250.19)
-	)
-	(no_connect
 		(at 50.8 162.56)
 	)
@@
 	)
 	(no_connect
+		(at 257.81 189.23)
+	)
+	(no_connect
+		(at 257.81 204.47)
+	)
+	(no_connect
 		(at 208.28 93.98)
 	)
@@
 	(wire
 		(pts
+			(xy 242.57 189.23) (xy 242.57 204.47)
+		)
+		(stroke
+			(width 0)
+			(type default)
+		)
+	)
+	(wire
+		(pts
 			(xy 241.3 21.59) (xy 243.84 21.59)
 		)
@@
 	(wire
 		(pts
-			(xy 242.57 234.95) (xy 242.57 250.19)
-		)
-		(stroke
-			(width 0)
-			(type default)
-		)
-	)
-	(wire
-		(pts
 			(xy 208.28 46.99) (xy 208.28 45.72)
 		)
@@
 	(global_label "~{INT3}"
 		(shape output)
-		(at 257.81 204.47 0)
+		(at 257.81 175.26 0)
 		(fields_autoplaced yes)
 		(effects
@@
 		)
 		(property "Intersheetrefs" "${INTERSHEET_REFS}"
-			(at 264.9076 204.47 0)
+			(at 264.9076 175.26 0)
 			(effects
 				(font
@@
 	(global_label "TMRINT"
 		(shape input)
-		(at 242.57 189.23 180)
+		(at 242.57 219.71 180)
 		(fields_autoplaced yes)
 		(effects
@@
 		)
 		(property "Intersheetrefs" "${INTERSHEET_REFS}"
-			(at 232.9929 189.23 0)
+			(at 232.9929 219.71 0)
 			(effects
 				(font
@@
 	(global_label "DUART_INT"
 		(shape input)
-		(at 242.57 175.26 180)
+		(at 242.57 234.95 180)
 		(fields_autoplaced yes)
 		(effects
@@
 		)
 		(property "Intersheetrefs" "${INTERSHEET_REFS}"
-			(at 229.7876 175.26 0)
+			(at 229.7876 234.95 0)
 			(effects
 				(font
@@
 	(global_label "ETH_INT"
 		(shape input)
-		(at 242.57 219.71 180)
+		(at 242.57 250.19 180)
 		(fields_autoplaced yes)
 		(effects
@@
 		)
 		(property "Intersheetrefs" "${INTERSHEET_REFS}"
-			(at 232.2672 219.71 0)
+			(at 232.2672 250.19 0)
 			(effects
 				(font
@@
 	(global_label "~{INT5}"
 		(shape output)
-		(at 257.81 175.26 0)
+		(at 257.81 234.95 0)
 		(fields_autoplaced yes)
 		(effects
@@
 		)
 		(property "Intersheetrefs" "${INTERSHEET_REFS}"
-			(at 264.9076 175.26 0)
+			(at 264.9076 234.95 0)
 			(effects
 				(font
@@
 	(global_label "~{INT4}"
 		(shape output)
-		(at 257.81 219.71 0)
+		(at 257.81 250.19 0)
 		(fields_autoplaced yes)
 		(effects
@@
 		)
 		(property "Intersheetrefs" "${INTERSHEET_REFS}"
-			(at 264.9076 219.71 0)
+			(at 264.9076 250.19 0)
 			(effects
 				(font
@@
 	(global_label "~{INT6}"
 		(shape output)
-		(at 257.81 189.23 0)
+		(at 257.81 219.71 0)
 		(fields_autoplaced yes)
 		(effects
@@
 		)
 		(property "Intersheetrefs" "${INTERSHEET_REFS}"
-			(at 264.9076 189.23 0)
+			(at 264.9076 219.71 0)
 			(effects
 				(font
@@
 	(global_label "ATA_INT"
 		(shape input)
-		(at 242.57 204.47 180)
+		(at 242.57 175.26 180)
 		(fields_autoplaced yes)
 		(effects
@@
 		)
 		(property "Intersheetrefs" "${INTERSHEET_REFS}"
-			(at 232.5695 204.47 0)
+			(at 232.5695 175.26 0)
 			(effects
 				(font
@@
 	)
 	(symbol
+		(lib_id "power:GND")
+		(at 242.57 204.47 0)
+		(unit 1)
+		(exclude_from_sim no)
+		(in_bom yes)
+		(on_board yes)
+		(dnp no)
+		(fields_autoplaced yes)
+		(property "Reference" "#PWR0113"
+			(at 242.57 210.82 0)
+			(effects
+				(font
+					(size 1.27 1.27)
+				)
+				(hide yes)
+			)
+		)
+		(property "Value" "GND"
+			(at 242.57 209.55 0)
+			(effects
+				(font
+					(size 1.27 1.27)
+				)
+			)
+		)
+		(property "Footprint" ""
+			(at 242.57 204.47 0)
+			(effects
+				(font
+					(size 1.27 1.27)
+				)
+				(hide yes)
+			)
+		)
+		(property "Datasheet" ""
+			(at 242.57 204.47 0)
+			(effects
+				(font
+					(size 1.27 1.27)
+				)
+				(hide yes)
+			)
+		)
+		(property "Description" "Power symbol creates a global label with name \"GND\" , ground"
+			(at 242.57 204.47 0)
+			(effects
+				(font
+					(size 1.27 1.27)
+				)
+				(hide yes)
+			)
+		)
+		(pin "1"
+		)
+		(instances
+			(project ""
+				(path "/6696b89f-f6cc-4e49-bcfb-68bdb218d2a6"
+					(reference "#PWR0113")
+					(unit 1)
+				)
+			)
+		)
+	)
+	(symbol
 		(lib_id "Memory_Flash:SST39SF040")
 		(at 317.5 57.15 0)
@@
 					(unit 1)
 				)
-			)
-		)
-	)
-	(symbol
-		(lib_id "power:GND")
-		(at 242.57 250.19 0)
-		(unit 1)
-		(exclude_from_sim no)
-		(in_bom yes)
-		(on_board yes)
-		(dnp no)
-		(fields_autoplaced yes)
-		(property "Reference" "#PWR0143"
-			(at 242.57 256.54 0)
-			(effects
-				(font
-					(size 1.27 1.27)
-				)
-				(hide yes)
-			)
-		)
-		(property "Value" "GND"
-			(at 242.57 255.27 0)
-			(effects
-				(font
-					(size 1.27 1.27)
-				)
-			)
-		)
-		(property "Footprint" ""
-			(at 242.57 250.19 0)
-			(effects
-				(font
-					(size 1.27 1.27)
-				)
-				(hide yes)
-			)
-		)
-		(property "Datasheet" ""
-			(at 242.57 250.19 0)
-			(effects
-				(font
-					(size 1.27 1.27)
-				)
-				(hide yes)
-			)
-		)
-		(property "Description" "Power symbol creates a global label with name \"GND\" , ground"
-			(at 242.57 250.19 0)
-			(effects
-				(font
-					(size 1.27 1.27)
-				)
-				(hide yes)
-			)
-		)
-		(pin "1"
-		)
-		(instances
-			(project ""
-				(path "/6696b89f-f6cc-4e49-bcfb-68bdb218d2a6"
-					(reference "#PWR0143")
-					(unit 1)
-				)
