File: cpu030/design-files/cpu030_expansion.kicad_sch (KiCad schematic)
At the start: 20 parts, among them J801 DIN41612_03x32_ABC, U801 74ACT245, U802 74ACT245, U803 74ACT245, U804 74ACT245, U805 74ACT245, U806 74ACT245, U807 74ACT245, U808 74ACT245

Commit message: Checkpoint: Nearly done with the expansion interface.
Parts:
- added C812: 100nF, Capacitor_SMD:C_0805_2012Metric, symbol Device:C_Small
- added RN801, RN802, RN803, RN804: 3K3, Resistor_THT:R_Array_SIP9, symbol Device:R_Network08
- added U809: 74ACT245, Package_SO:SOIC-20W_7.5x12.8mm_P1.27mm, symbol 74xx:74HC245
Connections:
- net ~{INT1} is gone; now on net ~{INT5}: J801.b22 (Pin_b22)
- net +12V: now also J801.b32 (Pin_b32)
- net +5V: now also J801.b1 (Pin_b1), J801.b2 (Pin_b2), J801.b3 (Pin_b3), J801.b4 (Pin_b4), C812.1, RN801.1 (common), RN802.1 (common), RN803.1 (common), RN804.1 (common), U809.20 (VCC)
- net -12V: now also J801.c32 (Pin_c32)
- net A0: now also U803.18 (B0); no longer U806.18 (B0)
- net A1: now also U803.17 (B1); no longer U806.17 (B1)
- net A10: now also U805.16 (B2); no longer U807.16 (B2)
- net A11: now also U805.15 (B3); no longer U807.15 (B3)
- net A12: now also U805.14 (B4); no longer U807.14 (B4)
- net A13: now also U805.13 (B5); no longer U807.13 (B5)
- net A14: now also U805.12 (B6); no longer U807.12 (B6)
- net A15: now also U805.11 (B7); no longer U807.11 (B7)
- net A16: now also U806.18 (B0); no longer U808.18 (B0)
- net A17: now also U806.17 (B1); no longer U808.17 (B1)
- net A18: now also U806.16 (B2); no longer U808.16 (B2)
- net A19: now also U806.15 (B3); no longer U808.15 (B3)
- net A2: now also U803.16 (B2); no longer U806.16 (B2)
- net A20: now also U806.14 (B4); no longer U808.14 (B4)
- net A21: now also U806.13 (B5); no longer U808.13 (B5)
- net A22: now also U806.12 (B6); no longer U808.12 (B6)
- net A23: now also U806.11 (B7); no longer U808.11 (B7)
- net A3: now also U803.15 (B3); no longer U806.15 (B3)
- net A4: now also U803.14 (B4); no longer U806.14 (B4)
- net A5: now also U803.13 (B5); no longer U806.13 (B5)
- net A6: now also U803.12 (B6); no longer U806.12 (B6)
- net A7: now also U803.11 (B7); no longer U806.11 (B7)
- net A8: now also U805.18 (B0); no longer U807.18 (B0)
- net A9: now also U805.17 (B1); no longer U807.17 (B1)
- net CPU_CLK: now also U804.11 (B7); no longer U805.11 (B7)
- net D0: now also U809.18 (B0); no longer U802.18 (B0)
- net D1: now also U809.17 (B1); no longer U802.17 (B1)
- net D10: now also U808.16 (B2); no longer U803.16 (B2)
- net D11: now also U808.15 (B3); no longer U803.15 (B3)
- net D12: now also U808.14 (B4); no longer U803.14 (B4)
- net D13: now also U808.13 (B5); no longer U803.13 (B5)
- net D14: now also U808.12 (B6); no longer U803.12 (B6)
- net D15: now also U808.11 (B7); no longer U803.11 (B7)
- net D16: now also U802.18 (B0); no longer U801.18 (B0)
- net D17: now also U802.17 (B1); no longer U801.17 (B1)
- net D18: now also U802.16 (B2); no longer U801.16 (B2)
- net D19: now also U802.15 (B3); no longer U801.15 (B3)
- net D2: now also U809.16 (B2); no longer U802.16 (B2)
- net D20: now also U802.14 (B4); no longer U801.14 (B4)
- net D21: now also U802.13 (B5); no longer U801.13 (B5)
- net D22: now also U802.12 (B6); no longer U801.12 (B6)
- net D23: now also U802.11 (B7); no longer U801.11 (B7)
- net D24: now also U801.18 (B0); no longer U804.18 (B0)
- net D25: now also U801.17 (B1); no longer U804.17 (B1)
- net D26: now also U801.16 (B2); no longer U804.16 (B2)
- net D27: now also U801.15 (B3); no longer U804.15 (B3)
- net D28: now also U801.14 (B4); no longer U804.14 (B4)
- net D29: now also U801.13 (B5); no longer U804.13 (B5)
- net D3: now also U809.15 (B3); no longer U802.15 (B3)
- net D30: now also U801.12 (B6); no longer U804.12 (B6)
- net D31: now also U801.11 (B7); no longer U804.11 (B7)
- net D4: now also U809.14 (B4); no longer U802.14 (B4)
- net D5: now also U809.13 (B5); no longer U802.13 (B5)
- net D6: now also U809.12 (B6); no longer U802.12 (B6)
- net D7: now also U809.11 (B7); no longer U802.11 (B7)
- net D8: now also U808.18 (B0); no longer U803.18 (B0)
- net D9: now also U808.17 (B1); no longer U803.17 (B1)
- net EXP_A0: now also U803.2 (A0); no longer U806.2 (A0)
- net EXP_A1: now also U803.3 (A1); no longer U806.3 (A1)
- net EXP_A10: now also U805.4 (A2); no longer U807.4 (A2)
- net EXP_A11: now also U805.5 (A3); no longer U807.5 (A3)
- net EXP_A12: now also U805.6 (A4); no longer U807.6 (A4)
- net EXP_A13: now also U805.7 (A5); no longer U807.7 (A5)
- net EXP_A14: now also U805.8 (A6); no longer U807.8 (A6)
- net EXP_A15: now also U805.9 (A7); no longer U807.9 (A7)
- net EXP_A16: now also U806.2 (A0); no longer U808.2 (A0)
- net EXP_A17: now also U806.3 (A1); no longer U808.3 (A1)
- net EXP_A18: now also U806.4 (A2); no longer U808.4 (A2)
- net EXP_A19: now also U806.5 (A3); no longer U808.5 (A3)
- net EXP_A2: now also U803.4 (A2); no longer U806.4 (A2)
- net EXP_A20: now also U806.6 (A4); no longer U808.6 (A4)
- net EXP_A21: now also U806.7 (A5); no longer U808.7 (A5)
- net EXP_A22: now also U806.8 (A6); no longer U808.8 (A6)
- net EXP_A23: now also U806.9 (A7); no longer U808.9 (A7)
- net EXP_A24: now also U807.2 (A0)
- net EXP_A25: now also U807.3 (A1)
- net EXP_A26: now also U807.4 (A2)
- net EXP_A27: now also U807.5 (A3)
- net EXP_A3: now also U803.5 (A3); no longer U806.5 (A3)
- net EXP_A4: now also U803.6 (A4); no longer U806.6 (A4)
- net EXP_A5: now also U803.7 (A5); no longer U806.7 (A5)
- net EXP_A6: now also U803.8 (A6); no longer U806.8 (A6)
- net EXP_A7: now also U803.9 (A7); no longer U806.9 (A7)
- net EXP_A8: now also U805.2 (A0); no longer U807.2 (A0)
- net EXP_A9: now also U805.3 (A1); no longer U807.3 (A1)
- net EXP_CPU_CLK: now also J801.b14 (Pin_b14), U804.9 (A7); no longer J801.b31 (Pin_b31), U805.9 (A7)
- net EXP_D0: now also J801.a25 (Pin_a25), RN804.2 (R1), U809.2 (A0); no longer J801.a1 (Pin_a1), U802.2 (A0)
- net EXP_D1: now also J801.a26 (Pin_a26), RN804.3 (R2), U809.3 (A1); no longer J801.a2 (Pin_a2), U802.3 (A1)
- net EXP_D10: now also J801.a19 (Pin_a19), U808.4 (A2), RN803.4 (R3); no longer J801.a11 (Pin_a11), U803.4 (A2)
- net EXP_D11: now also J801.a20 (Pin_a20), U808.5 (A3), RN803.5 (R4); no longer J801.a12 (Pin_a12), U803.5 (A3)
- net EXP_D12: now also J801.a21 (Pin_a21), U808.6 (A4), RN803.6 (R5); no longer J801.a13 (Pin_a13), U803.6 (A4)
- net EXP_D13: now also J801.a22 (Pin_a22), U808.7 (A5), RN803.7 (R6); no longer J801.a14 (Pin_a14), U803.7 (A5)
- net EXP_D14: now also J801.a23 (Pin_a23), U808.8 (A6), RN803.8 (R7); no longer J801.a15 (Pin_a15), U803.8 (A6)
- net EXP_D15: now also J801.a24 (Pin_a24), U808.9 (A7), RN803.9 (R8); no longer J801.a16 (Pin_a16), U803.9 (A7)
- net EXP_D16: now also J801.a9 (Pin_a9), U802.2 (A0), RN802.2 (R1); no longer J801.a17 (Pin_a17), U801.2 (A0)
- net EXP_D17: now also J801.a10 (Pin_a10), U802.3 (A1), RN802.3 (R2); no longer J801.a18 (Pin_a18), U801.3 (A1)
- net EXP_D18: now also J801.a11 (Pin_a11), U802.4 (A2), RN802.4 (R3); no longer J801.a19 (Pin_a19), U801.4 (A2)
- net EXP_D19: now also J801.a12 (Pin_a12), U802.5 (A3), RN802.5 (R4); no longer J801.a20 (Pin_a20), U801.5 (A3)
- net EXP_D2: now also J801.a27 (Pin_a27), RN804.4 (R3), U809.4 (A2); no longer J801.a3 (Pin_a3), U802.4 (A2)
- net EXP_D20: now also J801.a13 (Pin_a13), U802.6 (A4), RN802.6 (R5); no longer J801.a21 (Pin_a21), U801.6 (A4)
- net EXP_D21: now also J801.a14 (Pin_a14), U802.7 (A5), RN802.7 (R6); no longer J801.a22 (Pin_a22), U801.7 (A5)
- net EXP_D22: now also J801.a15 (Pin_a15), U802.8 (A6), RN802.8 (R7); no longer J801.a23 (Pin_a23), U801.8 (A6)
- net EXP_D23: now also J801.a16 (Pin_a16), U802.9 (A7), RN802.9 (R8); no longer J801.a24 (Pin_a24), U801.9 (A7)
- net EXP_D24: now also J801.a1 (Pin_a1), U801.2 (A0), RN801.2 (R1); no longer J801.a25 (Pin_a25), U804.2 (A0)
- net EXP_D25: now also J801.a2 (Pin_a2), U801.3 (A1), RN801.3 (R2); no longer J801.a26 (Pin_a26), U804.3 (A1)
- net EXP_D26: now also J801.a3 (Pin_a3), U801.4 (A2), RN801.4 (R3); no longer J801.a27 (Pin_a27), U804.4 (A2)
- net EXP_D27: now also J801.a4 (Pin_a4), U801.5 (A3), RN801.5 (R4); no longer J801.a28 (Pin_a28), U804.5 (A3)
- net EXP_D28: now also J801.a5 (Pin_a5), U801.6 (A4), RN801.6 (R5); no longer J801.a29 (Pin_a29), U804.6 (A4)
- net EXP_D29: now also J801.a6 (Pin_a6), U801.7 (A5), RN801.7 (R6); no longer J801.a30 (Pin_a30), U804.7 (A5)
- net EXP_D3: now also J801.a28 (Pin_a28), RN804.5 (R4), U809.5 (A3); no longer J801.a4 (Pin_a4), U802.5 (A3)
- net EXP_D30: now also J801.a7 (Pin_a7), U801.8 (A6), RN801.8 (R7); no longer J801.a31 (Pin_a31), U804.8 (A6)
- net EXP_D31: now also J801.a8 (Pin_a8), U801.9 (A7), RN801.9 (R8); no longer J801.a32 (Pin_a32), U804.9 (A7)
- net EXP_D4: now also J801.a29 (Pin_a29), RN804.6 (R5), U809.6 (A4); no longer J801.a5 (Pin_a5), U802.6 (A4)
- net EXP_D5: now also J801.a30 (Pin_a30), RN804.7 (R6), U809.7 (A5); no longer J801.a6 (Pin_a6), U802.7 (A5)
- net EXP_D6: now also J801.a31 (Pin_a31), RN804.8 (R7), U809.8 (A6); no longer J801.a7 (Pin_a7), U802.8 (A6)
- net EXP_D7: now also J801.a32 (Pin_a32), RN804.9 (R8), U809.9 (A7); no longer J801.a8 (Pin_a8), U802.9 (A7)
- net EXP_D8: now also J801.a17 (Pin_a17), U808.2 (A0), RN803.2 (R1); no longer J801.a9 (Pin_a9), U803.2 (A0)
- net EXP_D9: now also J801.a18 (Pin_a18), U808.3 (A1), RN803.3 (R2); no longer J801.a10 (Pin_a10), U803.3 (A1)
- net EXP_RnW: now also J801.b11 (Pin_b11), U804.6 (A4); no longer J801.b29 (Pin_b29), U805.4 (A2)
- net EXP_SIZ0: now also J801.b9 (Pin_b9), U804.4 (A2); no longer U805.7 (A5)
- net EXP_SIZ1: now also J801.b10 (Pin_b10), U804.5 (A3); no longer U805.8 (A6)
- net EXP_nAS: now also J801.b7 (Pin_b7), U804.2 (A0); no longer U805.2 (A0)
- net EXP_nDS: now also J801.b8 (Pin_b8), U804.3 (A1); no longer U805.3 (A1)
- net EXP_nEXPSEL: now also J801.b12 (Pin_b12), U804.7 (A5); no longer U805.6 (A4)
- net GND: now also J801.b27 (Pin_b27), J801.b28 (Pin_b28), J801.b29 (Pin_b29), U803.1 (A->B), U803.19 (CE), U804.1 (A->B), U804.19 (CE), C812.2, U809.10 (GND); no longer J801.b1 (Pin_b1), J801.b2 (Pin_b2), J801.b32 (Pin_b32), U805.15 (B3), U808.1 (A->B), U808.19 (CE)
- net RnW: now also U804.14 (B4), U808.1 (A->B), U809.1 (A->B); no longer U803.1 (A->B), U804.1 (A->B), U805.16 (B2)
- net SIZ0: now also U804.16 (B2); no longer U805.13 (B5)
- net SIZ1: now also U804.15 (B3); no longer U805.12 (B6)
- net ~{AS}: now also U804.18 (B0); no longer U805.18 (B0)
- net ~{CPU_BERR}: now also J801.b18 (Pin_b18); no longer J801.b21 (Pin_b21)
- net ~{CPU_CIIN}: now also J801.b17 (Pin_b17); no longer J801.b20 (Pin_b20)
- net ~{CPU_DSACK0}: now also J801.b15 (Pin_b15)
- net ~{CPU_DSACK1}: now also J801.b16 (Pin_b16)
- net ~{DS}: now also U804.17 (B1); no longer U805.17 (B1)
- net ~{EXPSEL}: now also U804.13 (B5), U808.19 (CE), U809.19 (CE); no longer U803.19 (CE), U804.19 (CE), U805.14 (B4)
- net ~{INT2}: now also J801.b19 (Pin_b19); no longer J801.b23 (Pin_b23)
- net ~{INT3}: now also J801.b20 (Pin_b20); no longer J801.b24 (Pin_b24)
- net ~{INT4}: now also J801.b21 (Pin_b21); no longer J801.b25 (Pin_b25)
- net ~{INT5}: no longer J801.b26 (Pin_b26)
- net ~{INT6}: now also J801.b23 (Pin_b23); no longer J801.b27 (Pin_b27)
- net ~{RESET}: now also U804.12 (B6); no longer J801.b28 (Pin_b28)
- net EXP_nRESET: now reaches J801.b13 (Pin_b13)
- net EXP_nRESET: now also U804.8 (A6)
- net I2C_SDA: now reaches J801.b5 (Pin_b5)
- net I2C_SCL: now reaches J801.b6 (Pin_b6)
- net EXP_A28: now reaches J801.c29 (Pin_c29)
- net EXP_A28: now also U807.6 (A4)
- net EXP_A29: now reaches J801.c30 (Pin_c30)
- net EXP_A29: now also U807.7 (A5)
- net EXP_A30: now reaches J801.c31 (Pin_c31)
- net EXP_A30: now also U807.8 (A6)
- new net A24: U807.18 (B0)
- new net A25: U807.17 (B1)
- new net A26: U807.16 (B2)
- new net A27: U807.15 (B3)
- new net A28: U807.14 (B4)
- new net A29: U807.13 (B5)
- new net A30: U807.12 (B6)
- new net A31: U807.11 (B7)
- new net EXP_A31: J801.b31 (Pin_b31), U807.9 (A7)
- new net ~{CPU_BGACK}: J801.b26 (Pin_b26)
- new net ~{CPU_BG}: J801.b25 (Pin_b25)
- new net ~{CPU_BR}: J801.b24 (Pin_b24)
- no-connect marks 1 -> 0
Other:
- moved on the sheet: C809, C810, C811

Commit message: Add the EXPGLUE GAL.
Parts:
- added C813, C814: 100nF, Capacitor_SMD:C_0805_2012Metric, symbol Device:C_Small
- added R801, R802, R803, R804: 3K3, Resistor_SMD:R_0805_2012Metric, symbol Device:R_Small
- added U810: 74ACT245, Package_SO:SOIC-20W_7.5x12.8mm_P1.27mm, symbol 74xx:74HC245
- added U811: GAL22V10, Package_DIP:DIP-24_W7.62mm_Socket, symbol jrt-ICs:GAL22V10
Connections:
- net +5V: now also C813.1, C814.1, R802.2, R804.2, U810.20 (VCC), U811.24 (VCC)
- net CPU_CLK: now also U810.16 (B2); no longer U804.11 (B7)
- net EXP_CPU_CLK: now also U810.4 (A2); no longer U804.9 (A7)
- net EXP_nEXPSEL: now also U810.2 (A0); no longer U804.7 (A5)
- net EXP_nRESET: now also U810.3 (A1); no longer U804.8 (A6)
- net GND: now also C813.2, C814.2, R801.2, R803.2, U810.1 (A->B), U810.10 (GND), U810.19 (CE), U811.12 (GND); no longer U803.1 (A->B), U804.1 (A->B), U805.1 (A->B), U806.1 (A->B), U807.1 (A->B)
- net RnW: now also U811.2 (I2); no longer U801.1 (A->B), U802.1 (A->B), U808.1 (A->B), U809.1 (A->B)
- net ~{AS}: now also U811.1 (I1/CLK)
- net ~{CPU_BGACK}: now also U811.4 (I4)
- net ~{EXPSEL}: now also U810.18 (B0), U811.5 (I5); no longer U801.19 (CE), U802.19 (CE), U804.13 (B5), U808.19 (CE), U809.19 (CE)
- net ~{RESET}: now also U810.17 (B1); no longer U804.12 (B6)
- new net: R804.1, U804.7 (A5)
- new net: R803.1, U804.8 (A6)
- new net: R802.1, U804.9 (A7)
- new net: R801.1, U810.11 (B7), U810.12 (B6), U810.13 (B5), U810.14 (B4), U810.15 (B3), U810.5 (A3), U810.6 (A4), U810.7 (A5), U810.8 (A6), U810.9 (A7)
- new net EXP_ADIR: U803.1 (A->B), U804.1 (A->B), U805.1 (A->B), U806.1 (A->B), U807.1 (A->B), U811.14 (IO1)
- new net EXP_DDIR: U801.1 (A->B), U802.1 (A->B), U808.1 (A->B), U809.1 (A->B), U811.15 (IO2)
- new net FC0: U804.13 (B5)
- new net FC1: U804.12 (B6)
- new net FC2: U804.11 (B7)
- new net ~{CPU_DBEN}: U811.3 (I3)
- new net ~{EXP_DEN}: U801.19 (CE), U802.19 (CE), U808.19 (CE), U809.19 (CE), U811.16 (IO3)
- no-connect marks 0 -> 14
Other:
- note added: "Codes "Supervisor Data""
- note added: "EXPGLUE"
- moved on the sheet: U803, U804, U805, U807
