File: cpu030/design-files/cpu030_expansion.kicad_sch (KiCad schematic)
At the start: 34 parts, among them J801 DIN41612_03x32_ABC, U801 74ACT245, U802 74ACT245, U803 74ACT245, U804 74ACT245, U805 74ACT245, U806 74ACT245, U807 74ACT245, U808 74ACT245, U809 74ACT245, U810 74ACT245, U811 GAL22V10

Commit message: Update revision to A0, update issue date.  Update 68882's symbol attributes to eliminate ERC errors.
Other:
- company: (none) -> (c) 2025 Jason R. Thorpe.  See LICENSE.
- title: (none) -> Playground 68030 Mk I
Changed lines of the file:
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@@
 	(generator_version "9.0")
 	(paper "A4")
+	(title_block
+		(title "Playground 68030 Mk I")
+		(date "2025-08-29")
+		(rev "A0")
+		(company "(c) 2025 Jason R. Thorpe.  See LICENSE.")
+	)
 	(text "Codes \"Supervisor Data\""
 		(exclude_from_sim no)
