File: cpu030/design-files/cpu030_psu.kicad_sch (KiCad schematic)
At the start: 1 part, among them J901 ATX-24

Commit message: Checkpoint: some PSU work, lock down Ethernet analog traces.
Parts:
- added C901: 470µF, Capacitor_THT:CP_Radial_D10.0mm_P5.00mm, symbol Device:C_Polarized_Small
Connections:
- net +5V: now also C901.1
- net GND: now also C901.2

Commit message: Add ATtiny85 as a PSU controller.
Parts:
- added C902: 100nF, Capacitor_SMD:C_0805_2012Metric, symbol Device:C_Small
- added D901: Power, LED_THT:LED_D3.0mm, symbol Device:LED
- added J902: Power, Connector_PinHeader_2.54mm:PinHeader_1x02_P2.54mm_Vertical, symbol Connector:Conn_01x02_Pin
- added R901: 470, Resistor_SMD:R_0805_2012Metric, symbol Device:R_Small
- added SW901: Power, Button_Switch_THT:SW_PUSH_6mm, symbol Switch:SW_Push
- added U901: ATtiny85-20P, Package_DIP:DIP-8_W7.62mm_Socket, symbol MCU_Microchip_ATtiny:ATtiny85-20P
Connections:
- net GND: now also C902.2, D901.1 (K), J902.2 (Pin_2), SW901.2, U901.4 (GND)
- net Vsb: no longer names the net of J901.9 (+5VSB)
- net Vsb: now also C902.1, U901.8 (VCC)
- net ~{PWR_ON}: no longer names the net of J901.16 (PS_ON#)
- net ~{PWR_ON}: now also U901.2 (XTAL1/PB3)
- new net: D901.2 (A), R901.2
- new net D0: U901.5 (AREF/PB0)
- new net PSU_ATN: U901.6 (PB1)
- new net PWR_LED: R901.1, U901.3 (XTAL2/PB4)
- new net ~{PWR_BUT}: J902.1 (Pin_1), SW901.1, U901.7 (PB2)
- new net ~{RESET}: U901.1 (~{RESET}/PB5)
Other:
- note added: "See psu-ctrl.ino"

Commit message: Checkpoint -- I'm going to re-arrange the board a bit and make it 6 layers, putting CPU address and data busses on their own internal signal layers.  Hopefully this detangles the mess a bit.
Parts:
- added C903: 100nF, Capacitor_SMD:C_0805_2012Metric, symbol Device:C_Small
- added U902: 74HCT74, Package_SO:SOIC-14_3.9x8.7mm_P1.27mm, symbol 74xx:74HC74
Connections:
- net D0: now also U902.12 (D); no longer U901.5 (AREF/PB0)
- net GND: now also C903.2, U902.2 (D), U902.7 (GND)
- net ~{RESET}: now also U902.13 (~{R}), U902.4 (~{S})
- net Vsb: now reaches C902.1, J901.9 (+5VSB), U901.8 (VCC)
- net Vsb: now also C903.1, U902.1 (~{R}), U902.10 (~{S}), U902.14 (VCC)
- net ~{PS_ON}: now reaches J901.16 (PS_ON#), U901.2 (XTAL1/PB3)
- net PSU_ATN renamed PSU_HOST_REQ
- net PSU_HOST_REQ: now also U902.5 (Q)
- new net PSU_HOST_REQ_BIT0: U901.5 (AREF/PB0), U902.9 (Q)
- new net ~{PSUSEL}: U902.11 (C), U902.3 (C)
- no-connect marks 0 -> 2
Other:
- moved on the sheet: J902, SW901

Commit message: Shrink down to JLCPCB's minimum trace / via sizes.
Changed lines of the file:
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@@
+	(netclass_flag ""
+		(length 2.54)
+		(shape rectangle)
+		(at 91.44 101.6 0)
+		(fields_autoplaced yes)
+		(effects
+			(font
+				(size 1.27 1.27)
+			)
+			(justify left bottom)
+		)
+		(property "Netclass" "Power"
+			(at 92.6465 99.06 0)
+			(effects
+				(font
+					(size 1.27 1.27)
+				)
+				(justify left)
+			)
+		)
+		(property "Component Class" ""
+			(at -72.39 -3.81 0)
+			(effects
+				(font
+					(size 1.27 1.27)
+					(italic yes)
+				)
+			)
+		)
+	)
 	(netclass_flag ""
 		(length 2.54)
@@
 	(netclass_flag ""
 		(length 2.54)
+		(shape rectangle)
+		(at 91.44 107.95 0)
+		(fields_autoplaced yes)
+		(effects
+			(font
+				(size 1.27 1.27)
+			)
+			(justify left bottom)
+		)
+		(property "Netclass" "Power"
+			(at 92.6465 105.41 0)
+			(effects
+				(font
+					(size 1.27 1.27)
+				)
+				(justify left)
+			)
+		)
+		(property "Component Class" ""
+			(at -72.39 2.54 0)
+			(effects
+				(font
+					(size 1.27 1.27)
+					(italic yes)
+				)
+			)
+		)
+	)
+	(netclass_flag ""
+		(length 2.54)
 		(shape diamond)
 		(at 91.44 88.9 0)
@@
 	)
 	(symbol
+		(lib_id "power:GND")
+		(at 91.44 107.95 90)
+		(unit 1)
+		(exclude_from_sim no)
+		(in_bom yes)
+		(on_board yes)
+		(dnp no)
+		(fields_autoplaced yes)
+		(property "Reference" "#PWR0916"
+			(at 97.79 107.95 0)
+			(effects
+				(font
+					(size 1.27 1.27)
+				)
+				(hide yes)
+			)
+		)
+		(property "Value" "GND"
+			(at 95.25 107.9499 90)
+			(effects
+				(font
+					(size 1.27 1.27)
+				)
+				(justify right)
+			)
+		)
+		(property "Footprint" ""
+			(at 91.44 107.95 0)
+			(effects
+				(font
+					(size 1.27 1.27)
+				)
+				(hide yes)
+			)
+		)
+		(property "Datasheet" ""
+			(at 91.44 107.95 0)
+			(effects
+				(font
+					(size 1.27 1.27)
+				)
+				(hide yes)
+			)
+		)
+		(property "Description" "Power symbol creates a global label with name \"GND\" , ground"
+			(at 91.44 107.95 0)
+			(effects
+				(font
+					(size 1.27 1.27)
+				)
+				(hide yes)
+			)
+		)
+		(pin "1"
+		)
+		(instances
+			(project "cpu030"
+				(path "/6696b89f-f6cc-4e49-bcfb-68bdb218d2a6/ebdde0e0-0896-4c67-99fd-d2163b7a8e6c"
+					(reference "#PWR0916")
+					(unit 1)
+				)
+			)
+		)
+	)
+	(symbol
 		(lib_id "power:+5V")
 		(at 68.58 95.25 0)
@@
 					(unit 1)
 				)
+			)
+		)
+	)
+	(symbol
+		(lib_id "power:+5V")
+		(at 91.44 101.6 270)
+		(unit 1)
+		(exclude_from_sim no)
+		(in_bom yes)
+		(on_board yes)
+		(dnp no)
+		(fields_autoplaced yes)
+		(property "Reference" "#PWR0915"
+			(at 87.63 101.6 0)
+			(effects
+				(font
+					(size 1.27 1.27)
+				)
+				(hide yes)
+			)
+		)
+		(property "Value" "+5V"
+			(at 95.25 101.5999 90)
+			(effects
+				(font
+					(size 1.27 1.27)
+				)
+				(justify left)
+			)
+		)
+		(property "Footprint" ""
+			(at 91.44 101.6 0)
+			(effects
+				(font
+					(size 1.27 1.27)
+				)
+				(hide yes)
+			)
+		)
+		(property "Datasheet" ""
+			(at 91.44 101.6 0)
+			(effects
+				(font
+					(size 1.27 1.27)
+				)
+				(hide yes)
+			)
+		)
+		(property "Description" "Power symbol creates a global label with name \"+5V\""
+			(at 91.44 101.6 0)
+			(effects
+				(font
+					(size 1.27 1.27)
+				)
+				(hide yes)
+			)
+		)
+		(pin "1"
+		)
+		(instances
+			(project "cpu030"
+				(path "/6696b89f-f6cc-4e49-bcfb-68bdb218d2a6/ebdde0e0-0896-4c67-99fd-d2163b7a8e6c"
+					(reference "#PWR0915")
+					(unit 1)
+				)
