File: cpu030/design-files/cpu030_psu.kicad_sch (KiCad schematic)
At the start: 9 parts, among them J901 ATX-24, SW901 Power, U901 ATtiny85-20P, U902 74HCT74

Commit message: Update revision to A0, update issue date.  Update 68882's symbol attributes to eliminate ERC errors.
Other:
- company: (none) -> (c) 2025 Jason R. Thorpe.  See LICENSE.
- title: (none) -> Playground 68030 Mk I
Changed lines of the file:
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@@
 	(generator_version "9.0")
 	(paper "A4")
+	(title_block
+		(title "Playground 68030 Mk I")
+		(date "2025-08-29")
+		(rev "A0")
+		(company "(c) 2025 Jason R. Thorpe.  See LICENSE.")
+	)
 	(text "See psu-ctrl.ino"
 		(exclude_from_sim no)
