File: cpu030/design-files/cpu030_fram_dram0.kicad_sch (KiCad schematic)
At the start: 36 parts, among them J201 DRAM0SZ, J202 DRAM0 JTAG, U201 ATF1508AS-TQFP100, U202 CY7C1061GE, U203 CY7C1061GE, U204 SIMM72-0A, U205 SIMM72-0B, U206 MC74ACT05DG

Commit message: Group components with their caps.
Parts:
- added C225: 220nF, Capacitor_SMD:C_0805_2012Metric, symbol Device:C_Small
- U201: value ATF1508AS-TQFP100 -> ATF1508AS
- U202: value CY7C1061GE -> CY7C1061GE (U16)
- U203: value CY7C1061GE -> CY7C1061GE (L16)
Connections:
- net +5V: now also C225.1
- net GND: now also C225.2
Other:
- note removed: "DRAMCTL"
- moved on the sheet: C223, C224
Changed lines of the file:
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@@
 	(generator_version "9.0")
 	(paper "A4")
-	(text "DRAMCTL"
-		(exclude_from_sim no)
-		(at 261.112 20.828 0)
-		(effects
-			(font
-				(size 1.27 1.27)
-				(italic yes)
-			)
-		)
-	)
 	(junction
 		(at 158.75 135.89)
@@
 	)
 	(junction
+		(at 157.48 179.07)
+		(diameter 0)
+		(color 0 0 0 0)
+	)
+	(junction
 		(at 158.75 160.02)
 		(diameter 0)
@@
 	)
 	(junction
-		(at 156.21 173.99)
+		(at 147.32 179.07)
 		(diameter 0)
 		(color 0 0 0 0)
@@
 	)
 	(junction
-		(at 156.21 179.07)
+		(at 147.32 184.15)
 		(diameter 0)
 		(color 0 0 0 0)
@@
 	)
 	(junction
+		(at 157.48 184.15)
+		(diameter 0)
+		(color 0 0 0 0)
+	)
+	(junction
 		(at 97.79 105.41)
 		(diameter 0)
@@
 	(wire
 		(pts
-			(xy 156.21 179.07) (xy 166.37 179.07)
+			(xy 147.32 184.15) (xy 157.48 184.15)
 		)
 		(stroke
@@
 	(wire
 		(pts
-			(xy 156.21 173.99) (xy 166.37 173.99)
+			(xy 157.48 179.07) (xy 167.64 179.07)
+		)
+		(stroke
+			(width 0)
+			(type default)
+		)
+	)
+	(wire
+		(pts
+			(xy 147.32 179.07) (xy 157.48 179.07)
 		)
 		(stroke
@@
 	(wire
 		(pts
+			(xy 157.48 184.15) (xy 167.64 184.15)
+		)
+		(stroke
+			(width 0)
+			(type default)
+		)
+	)
+	(wire
+		(pts
 			(xy 168.91 102.87) (xy 167.64 102.87)
 		)
@@
 	(symbol
 		(lib_id "Device:C_Small")
-		(at 156.21 176.53 0)
+		(at 147.32 181.61 0)
 		(unit 1)
 		(exclude_from_sim no)
@@
 		(fields_autoplaced yes)
 		(property "Reference" "C223"
-			(at 158.75 175.2662 0)
+			(at 149.86 180.3462 0)
 			(effects
 				(font
@@
 		)
 		(property "Value" "220nF"
-			(at 158.75 177.8062 0)
+			(at 149.86 182.8862 0)
 			(effects
 				(font
@@
 		)
 		(property "Footprint" "Capacitor_SMD:C_0805_2012Metric"
-			(at 156.21 176.53 0)
+			(at 147.32 181.61 0)
 			(effects
 				(font
@@
 		)
 		(property "Datasheet" "~"
-			(at 156.21 176.53 0)
+			(at 147.32 181.61 0)
 			(effects
 				(font
@@
 		)
 		(property "Description" "Unpolarized capacitor, small symbol"
-			(at 156.21 176.53 0)
+			(at 147.32 181.61 0)
 			(effects
 				(font
@@
 	(symbol
 		(lib_id "power:+5V")
-		(at 156.21 173.99 0)
+		(at 147.32 179.07 0)
 		(unit 1)
 		(exclude_from_sim no)
@@
 		(dnp no)
 		(property "Reference" "#PWR0230"
-			(at 156.21 177.8 0)
+			(at 147.32 182.88 0)
 			(effects
 				(font
@@
 		)
 		(property "Value" "+5V"
-			(at 156.21 168.91 0)
+			(at 147.32 173.99 0)
 			(effects
 				(font
@@
 		)
 		(property "Footprint" ""
-			(at 156.21 173.99 0)
+			(at 147.32 179.07 0)
 			(effects
 				(font
@@
 		)
 		(property "Datasheet" ""
-			(at 156.21 173.99 0)
+			(at 147.32 179.07 0)
 			(effects
 				(font
@@
 		)
 		(property "Description" "Power symbol creates a global label with name \"+5V\""
-			(at 156.21 173.99 0)
+			(at 147.32 179.07 0)
 			(effects
 				(font
@@
 	(symbol
 		(lib_id "power:GND")
-		(at 156.21 179.07 0)
+		(at 147.32 184.15 0)
 		(unit 1)
 		(exclude_from_sim no)
@@
 		(fields_autoplaced yes)
 		(property "Reference" "#PWR0231"
-			(at 156.21 185.42 0)
+			(at 147.32 190.5 0)
 			(effects
 				(font
@@
 		)
 		(property "Value" "GND"
-			(at 156.21 184.15 0)
+			(at 147.32 189.23 0)
 			(effects
 				(font
@@
 		)
 		(property "Footprint" ""
-			(at 156.21 179.07 0)
+			(at 147.32 184.15 0)
 			(effects
 				(font
@@
 		)
 		(property "Datasheet" ""
-			(at 156.21 179.07 0)
+			(at 147.32 184.15 0)
 			(effects
 				(font
@@
 		)
 		(property "Description" "Power symbol creates a global label with name \"GND\" , ground"
-			(at 156.21 179.07 0)
+			(at 147.32 184.15 0)
 			(effects
 				(font
@@
 			)
 		)
-		(property "Value" "ATF1508AS-TQFP100"
+		(property "Value" "ATF1508AS"
 			(at 243.4433 17.78 0)
 			(effects
@@
 	)
 	(symbol
+		(lib_id "Device:C_Small")
+		(at 167.64 181.61 0)
+		(unit 1)
+		(exclude_from_sim no)
+		(in_bom yes)
+		(on_board yes)
+		(dnp no)
+		(fields_autoplaced yes)
+		(property "Reference" "C225"
+			(at 170.18 180.3462 0)
+			(effects
+				(font
+					(size 1.27 1.27)
+				)
+				(justify left)
+			)
+		)
+		(property "Value" "220nF"
+			(at 170.18 182.8862 0)
+			(effects
+				(font
+					(size 1.27 1.27)
+				)
+				(justify left)
+			)
+		)
+		(property "Footprint" "Capacitor_SMD:C_0805_2012Metric"
+			(at 167.64 181.61 0)
+			(effects
+				(font
+					(size 1.27 1.27)
+				)
+				(hide yes)
+			)
+		)
+		(property "Datasheet" "~"
+			(at 167.64 181.61 0)
+			(effects
+				(font
+					(size 1.27 1.27)
+				)
+				(hide yes)
+			)
+		)
+		(property "Description" "Unpolarized capacitor, small symbol"
+			(at 167.64 181.61 0)
+			(effects
+				(font
+					(size 1.27 1.27)
+				)
+				(hide yes)
+			)
+		)
+		(pin "1"
+		)
+		(pin "2"
+		)
+		(instances
+			(project "cpu030"
+				(path "/6696b89f-f6cc-4e49-bcfb-68bdb218d2a6/6473b99a-f5fc-46a4-ae73-90633955ad5d"
+					(reference "C225")
+					(unit 1)
+				)
+			)
+		)
+	)
+	(symbol
 		(lib_id "power:GND")
 		(at 190.5 119.38 0)
@@
 	(symbol
 		(lib_id "Device:C_Small")
-		(at 166.37 176.53 0)
+		(at 157.48 181.61 0)
 		(unit 1)
 		(exclude_from_sim no)
@@
 		(fields_autoplaced yes)
 		(property "Reference" "C224"
-			(at 168.91 175.2662 0)
+			(at 160.02 180.3462 0)
 			(effects
 				(font
@@
 		)
 		(property "Value" "220nF"
-			(at 168.91 177.8062 0)
+			(at 160.02 182.8862 0)
 			(effects
 				(font
@@
 		)
 		(property "Footprint" "Capacitor_SMD:C_0805_2012Metric"
-			(at 166.37 176.53 0)
+			(at 157.48 181.61 0)
 			(effects
 				(font
@@
 		)
 		(property "Datasheet" "~"
-			(at 166.37 176.53 0)
+			(at 157.48 181.61 0)
 			(effects
 				(font
@@
 		)
 		(property "Description" "Unpolarized capacitor, small symbol"
-			(at 166.37 176.53 0)
+			(at 157.48 181.61 0)
 			(effects
 				(font
@@
 		(fields_autoplaced yes)
 		(property "Reference" "U203"
-			(at 102.4733 17.78 0)
+			(at 102.4733 16.51 0)
 			(effects
 				(font
@@
 			)
 		)
-		(property "Value" "CY7C1061GE"
-			(at 102.4733 20.32 0)
+		(property "Value" "CY7C1061GE (L16)"
+			(at 102.4733 19.05 0)
 			(effects
 				(font
@@
 		(fields_autoplaced yes)
 		(property "Reference" "U202"
-			(at 45.3233 17.78 0)
+			(at 45.3233 16.51 0)
 			(effects
 				(font
@@
 			)
 		)
-		(property "Value" "CY7C1061GE"
-			(at 45.3233 20.32 0)
+		(property "Value" "CY7C1061GE (U16)"
+			(at 45.3233 19.05 0)
 			(effects
 				(font

Commit message: PCB grouping pass.
Connections:
- net SYSCTL_TCK is gone; now on net DRAM0_TCK: R204.1
- net SYSCTL_TDI is gone; now on net DRAM0_TDI: R203.1
- net SYSCTL_TMS is gone; now on net DRAM0_TMS: R202.1
Changed lines of the file:
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@@
+		)
+	)
+	(label "DRAM0_TMS"
+		(at 173.99 121.92 180)
+		(effects
+			(font
+				(size 1.27 1.27)
+			)
+			(justify right bottom)
 		)
 	)
@@
 		)
 	)
-	(label "SYSCTL_TDI"
-		(at 181.61 118.11 180)
-		(effects
-			(font
-				(size 1.27 1.27)
-			)
-			(justify right bottom)
-		)
-	)
-	(label "SYSCTL_TMS"
-		(at 173.99 121.92 180)
-		(effects
-			(font
-				(size 1.27 1.27)
-			)
-			(justify right bottom)
-		)
-	)
 	(label "DRAM0_A2"
 		(at 50.8 114.3 180)
@@
 		)
 	)
+	(label "DRAM0_TCK"
+		(at 190.5 114.3 180)
+		(effects
+			(font
+				(size 1.27 1.27)
+			)
+			(justify right bottom)
+		)
+	)
 	(label "~{DRAM0A_RAS3}"
 		(at 50.8 148.59 180)
@@
 		)
 	)
+	(label "DRAM0_TDI"
+		(at 181.61 118.11 180)
+		(effects
+			(font
+				(size 1.27 1.27)
+			)
+			(justify right bottom)
+		)
+	)
 	(label "DRAM0_A0"
 		(at 203.2 133.35 180)
@@
 		)
 	)
-	(label "SYSCTL_TCK"
-		(at 190.5 114.3 180)
-		(effects
-			(font
-				(size 1.27 1.27)
-			)
-			(justify right bottom)
-		)
-	)

Commit message: Add INTC-1.
Other:
- note added: "DRAMCTL"
Changed lines of the file:
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@@
 	(generator_version "9.0")
 	(paper "A4")
+	(text "DRAMCTL"
+		(exclude_from_sim no)
+		(at 255.778 18.034 0)
+		(effects
+			(font
+				(size 1.27 1.27)
+				(italic yes)
+			)
+			(justify left)
+		)
+	)
 	(junction
 		(at 158.75 135.89)

Commit message: Connect /STERM to the DRAM controller.
Connections:
- net GND: no longer U206.11
- net DRAM0_STERM: now reaches U201.99 (I/O)
- net DRAM0_STERM: now also U206.11
- net ~{CPU_STERM}: now reaches U206.10
- no-connect marks 10 -> 8
Other:
- moved on the sheet: U206E
Changed lines of the file:
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@@
 	)
 	(no_connect
-		(at 139.7 82.55)
-	)
-	(no_connect
-		(at 259.08 36.83)
-	)
-	(no_connect
 		(at 139.7 67.31)
 	)
@@
 		)
 	)
+	(label "DRAM0_STERM"
+		(at 144.78 82.55 0)
+		(effects
+			(font
+				(size 1.27 1.27)
+			)
+			(justify left bottom)
+		)
+	)
 	(label "DRAM0B_PD3"
 		(at 113.03 172.72 180)
@@
 		)
 	)
+	(label "DRAM0_STERM"
+		(at 259.08 36.83 0)
+		(effects
+			(font
+				(size 1.27 1.27)
+			)
+			(justify left bottom)
+		)
+	)
 	(label "DRAM0_TMS"
 		(at 201.93 71.12 180)
@@
 		)
 	)
+	(global_label "~{CPU_STERM}"
+		(shape output)
+		(at 129.54 82.55 180)
+		(fields_autoplaced yes)
+		(effects
+			(font
+				(size 1.27 1.27)
+			)
+			(justify right)
+		)
+		(property "Intersheetrefs" "${INTERSHEET_REFS}"
+			(at 115.6692 82.55 0)
+			(effects
+				(font
+					(size 1.27 1.27)
+				)
+				(justify right)
+				(hide yes)
+			)
+		)
+	)
 	(global_label "D14"
 		(shape bidirectional)
@@
 	)
 	(symbol
-		(lib_id "power:GND")
-		(at 154.94 82.55 0)
-		(unit 1)
-		(exclude_from_sim no)
-		(in_bom yes)
-		(on_board yes)
-		(dnp no)
-		(fields_autoplaced yes)
-		(property "Reference" "#PWR0216"
-			(at 154.94 88.9 0)
-			(effects
-				(font
-					(size 1.27 1.27)
-				)
-				(hide yes)
-			)
-		)
-		(property "Value" "GND"
-			(at 154.94 87.63 0)
-			(effects
-				(font
-					(size 1.27 1.27)
-				)
-			)
-		)
-		(property "Footprint" ""
-			(at 154.94 82.55 0)
-			(effects
-				(font
-					(size 1.27 1.27)
-				)
-				(hide yes)
-			)
-		)
-		(property "Datasheet" ""
-			(at 154.94 82.55 0)
-			(effects
-				(font
-					(size 1.27 1.27)
-				)
-				(hide yes)
-			)
-		)
-		(property "Description" "Power symbol creates a global label with name \"GND\" , ground"
-			(at 154.94 82.55 0)
-			(effects
-				(font
-					(size 1.27 1.27)
-				)
-				(hide yes)
-			)
-		)
-		(pin "1"
-		)
-		(instances
-			(project ""
-				(path "/6696b89f-f6cc-4e49-bcfb-68bdb218d2a6/6473b99a-f5fc-46a4-ae73-90633955ad5d"
-					(reference "#PWR0216")
-					(unit 1)
-				)
-			)
-		)
-	)
-	(symbol
 		(lib_id "power:+5V")
 		(at 173.99 127 180)
@@
 	(symbol
 		(lib_id "74xx:74LS05")
-		(at 147.32 82.55 180)
+		(at 137.16 82.55 180)
 		(unit 5)
 		(exclude_from_sim no)
@@
 		(on_board yes)
 		(dnp no)
-		(fields_autoplaced yes)
 		(property "Reference" "U206"
-			(at 147.32 73.66 0)
+			(at 137.16 73.66 0)
 			(effects
 				(font
@@
 		)
 		(property "Value" "MC74ACT05DG"
-			(at 147.32 76.2 0)
+			(at 137.16 76.2 0)
 			(effects
 				(font
@@
 		)
 		(property "Footprint" "Package_SO:SOIC-14_3.9x8.7mm_P1.27mm"
-			(at 147.32 82.55 0)
+			(at 137.16 82.55 0)
 			(effects
 				(font
@@
 		)
 		(property "Datasheet" "http://www.ti.com/lit/gpn/sn74LS05"
-			(at 147.32 82.55 0)
+			(at 137.16 82.55 0)
 			(effects
 				(font
@@
 		)
 		(property "Description" "Inverter Open Collect"
-			(at 147.32 82.55 0)
+			(at 137.16 82.55 0)
 			(effects
 				(font
@@
 		)
 		(property "Part" "MC74ACT05DG"
-			(at 147.32 82.55 0)
+			(at 137.16 82.55 0)
 			(effects
 				(font

Commit message: Fix a mistake!  A15 was connected to the SRAM twice, and A16 wasn't connected at all!  I guess hand-routing is the way to go after all!
Connections:
- net A15: no longer U202.34 (A14), U203.34 (A14)
- net A16: now also U202.34 (A14), U203.34 (A14)
Changed lines of the file:
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@@
 		)
 	)
-	(global_label "A15"
+	(global_label "A16"
 		(shape input)
 		(at 25.4 62.23 180)
@@
 		)
 	)
-	(global_label "A15"
+	(global_label "A16"
 		(shape input)
 		(at 82.55 62.23 180)

Commit message: Need pullups on the PD signals.
Parts:
- added R205, R206, R207, R208, R209, R210, R211, R212: 10K, Resistor_SMD:R_0805_2012Metric, symbol Device:R_Small
Connections:
- net +5V: now also U205.11 (NC), R205.1, R206.1, R207.1, R208.1, R209.1, R210.1, R211.1, R212.1
- net DRAM0A_PD1: now also R205.2
- net DRAM0A_PD2: now also R206.2
- net DRAM0A_PD3: now also R207.2
- net DRAM0A_PD4: now also R208.2
- net DRAM0B_PD1: now also R209.2
- net DRAM0B_PD2: now also R210.2
- net DRAM0B_PD3: now also R211.2
- net DRAM0B_PD4: now also U205.36 (NC), R212.2

Commit message: Fix some connection mistakes on the 74ACT05s, re-arrange pullups on CPU to make layout easier.
Parts:
- U206: value MC74ACT05DG -> 74ACT05
Connections:
- net +5V: now also U206.14 (VCC); no longer U206.7 (GND)
- net GND: now also U206.7 (GND); no longer U206.14 (VCC)
Other:
- moved on the sheet: U206G
Changed lines of the file:
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@@
 	)
 	(junction
+		(at 172.72 85.09)
+		(diameter 0)
+		(color 0 0 0 0)
+	)
+	(junction
 		(at 232.41 146.05)
 		(diameter 0)
@@
 	)
 	(junction
+		(at 172.72 59.69)
+		(diameter 0)
+		(color 0 0 0 0)
+	)
+	(junction
 		(at 35.56 19.05)
 		(diameter 0)
@@
 	)
 	(junction
-		(at 172.72 59.69)
-		(diameter 0)
-		(color 0 0 0 0)
-	)
-	(junction
 		(at 92.71 19.05)
 		(diameter 0)
@@
 	)
 	(junction
-		(at 172.72 85.09)
-		(diameter 0)
-		(color 0 0 0 0)
-	)
-	(junction
 		(at 189.23 160.02)
 		(diameter 0)
@@
 			)
 		)
-		(property "Value" "MC74ACT05DG"
+		(property "Value" "74ACT05"
 			(at 147.32 16.51 0)
 			(effects
@@
 			)
 		)
-		(property "Value" "MC74ACT05DG"
+		(property "Value" "74ACT05"
 			(at 147.32 30.48 0)
 			(effects
@@
 			)
 		)
-		(property "Value" "MC74ACT05DG"
+		(property "Value" "74ACT05"
 			(at 147.32 45.72 0)
 			(effects
@@
 			)
 		)
-		(property "Value" "MC74ACT05DG"
+		(property "Value" "74ACT05"
 			(at 137.16 76.2 0)
 			(effects
@@
 			)
 		)
-		(property "Value" "MC74ACT05DG"
+		(property "Value" "74ACT05"
 			(at 147.32 60.96 0)
 			(effects
@@
 	(symbol
 		(lib_id "74xx:74LS05")
-		(at 172.72 72.39 180)
+		(at 172.72 72.39 0)
 		(unit 7)
 		(exclude_from_sim no)
@@
 					(size 1.27 1.27)
 				)
-				(justify right)
+				(justify left)
 			)
 		)
-		(property "Value" "MC74ACT05DG"
+		(property "Value" "74ACT05"
 			(at 179.07 73.6599 0)
 			(effects
@@
 					(size 1.27 1.27)
 				)
-				(justify right)
+				(justify left)
 			)
 		)
@@
 			)
 		)
-		(property "Value" "MC74ACT05DG"
+		(property "Value" "74ACT05"
 			(at 147.32 91.44 0)
 			(effects

Commit message: Fix silliness in the SIMM-72 symbol that tripped the ERC.
Connections:
- net +5V: no longer U205.11 (NC)
- net DRAM0B_PD4: no longer U205.36 (NC)
- net GND: no longer U202.53 (Vss)
Other:
- moved on the sheet: C201, C202, C203, C204, C205, C206, C207, C208, C210, C211, C212, C213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
