File: cpu030/design-files/cpu030_fram_dram0.kicad_sch (KiCad schematic)
At the start: 45 parts, among them J201 DRAM0SZ, J202 DRAM0 JTAG, U201 ATF1508AS, U202 CY7C1061GE (U16), U203 CY7C1061GE (L16), U204 SIMM72-0A, U205 SIMM72-0B, U206 74ACT05

Commit message: Adjust some constraints for DRC.
Connections:
- net GND: now also U202.53 (Vss)
Changed lines of the file:
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@@
+	)
+	(junction
+		(at 40.64 105.41)
+		(diameter 0)
+		(color 0 0 0 0)
 	)
 	(junction
@@
 		)
 		(stroke
+			(width 0)
+			(type default)
+		)
+	)
+	(wire
+		(pts
+			(xy 40.64 105.41) (xy 43.18 105.41)
+		)
+		(stroke

Commit message: Update revision to A0, update issue date.  Update 68882's symbol attributes to eliminate ERC errors.
Other:
- company: (none) -> (c) 2025 Jason R. Thorpe.  See LICENSE.
- title: (none) -> Playground 68030 Mk I
Changed lines of the file:
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@@
 	(generator_version "9.0")
 	(paper "A4")
+	(title_block
+		(title "Playground 68030 Mk I")
+		(date "2025-08-29")
+		(rev "A0")
+		(company "(c) 2025 Jason R. Thorpe.  See LICENSE.")
+	)
 	(text "DRAMCTL"
 		(exclude_from_sim no)
