File: cpu030/design-files/cpu030_duart.kicad_sch (KiCad schematic)
At the start: 10 parts, among them J301 UART0 FTDI, J302 UART1 FTDI, J303 UART1, J304 UART0, U301 TL16C2552, Y301 1.8432MHz

Commit message: Add ISACTL ISA bus controller and re-do ATA interface with it.
Parts:
- J301: value UART0 FTDI -> UART1 FTDI
- J302: value UART1 FTDI -> UART0 FTDI
- J303: value UART1 -> UART0
- J304: value UART0 -> UART1
Connections:
- net A3 renamed A8
- net ~{IORD} renamed ~{ISA_IORD}
- net ~{IOWR} renamed ~{ISA_IOWR}
Other:
- note added: "Note: A8=0 selects channel B."
- note removed: "Note: A3=0 selects channel B."
Changed lines of the file:
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@@
 		)
 	)
-	(text "Note: A3=0 selects channel B."
+	(text "Note: A8=0 selects channel B."
 		(exclude_from_sim no)
 		(at 136.652 34.798 0)
@@
 		)
 	)
-	(global_label "A3"
+	(global_label "A8"
 		(shape input)
 		(at 58.42 69.85 180)
@@
 		)
 	)
-	(global_label "~{IORD}"
+	(global_label "~{ISA_IORD}"
 		(shape input)
 		(at 58.42 77.47 180)
@@
 		)
 		(property "Intersheetrefs" "${INTERSHEET_REFS}"
-			(at 50.9595 77.47 0)
+			(at 47.089 77.47 0)
 			(effects
 				(font
@@
 		)
 	)
-	(global_label "~{IOWR}"
+	(global_label "~{ISA_IOWR}"
 		(shape input)
 		(at 58.42 80.01 180)
@@
 		)
 		(property "Intersheetrefs" "${INTERSHEET_REFS}"
-			(at 50.7781 80.01 0)
+			(at 46.9076 80.01 0)
 			(effects
 				(font
@@
 			)
 		)
-		(property "Value" "UART1"
+		(property "Value" "UART0"
 			(at 163.83 143.51 0)
 			(effects
@@
 			)
 		)
-		(property "Value" "UART0"
+		(property "Value" "UART1"
 			(at 217.17 143.51 0)
 			(effects
@@
 			)
 		)
-		(property "Value" "UART0 FTDI"
+		(property "Value" "UART1 FTDI"
 			(at 222.885 58.42 0)
 			(effects
@@
 			)
 		)
-		(property "Value" "UART1 FTDI"
+		(property "Value" "UART0 FTDI"
 			(at 221.615 19.05 0)
 			(effects

Commit message: Fix some schematic mistakes and checkpoint signal routing on the PCB.
Parts:
- added C304: 100nF, Capacitor_SMD:C_0805_2012Metric, symbol Device:C_Small
- added U302: 74ACHT32, Package_SO:SOIC-14_3.9x8.7mm_P1.27mm, symbol 74xx:74LS32
Connections:
- net +5V: now also C304.1, U302.14 (VCC)
- net GND: now also C304.2, U302.10, U302.12, U302.13, U302.4, U302.5, U302.7 (GND), U302.9
- net DUART_INTA: no longer names the net of U301.34 (INTA)
- net DUART_INTA: now also U302.1
- net DUART_INTB: no longer names the net of U301.17 (INTB)
- net DUART_INTB: now also U302.2
- new net DUART_INT: U302.3
- no-connect marks 8 -> 11

Commit message: Update revision to A0, update issue date.  Update 68882's symbol attributes to eliminate ERC errors.
Other:
- company: (none) -> (c) 2025 Jason R. Thorpe.  See LICENSE.
- title: (none) -> Playground 68030 Mk I
Changed lines of the file:
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@@
 	(generator_version "9.0")
 	(paper "A4")
+	(title_block
+		(title "Playground 68030 Mk I")
+		(date "2025-08-29")
+		(rev "A0")
+		(company "(c) 2025 Jason R. Thorpe.  See LICENSE.")
+	)
 	(text "IDC 10 connectors are pinned the same as RS232 DB9,\nwith +5V being provided on pin 10.  This allows for\na remote board with RS232 line drivers to be added.\n\nNote: Only connect one kind of external interface to\na port at any given time."
 		(exclude_from_sim no)
