File: cpu030/design-files/cpu030_ethernet.kicad_sch (KiCad schematic)
At the start: 18 parts, among them J701 RJ45_Amphenol_RJMG1BD3B8K1ANR, U701 RTL8019AS, U702 AT93C46D-PU, Y701 20MHz

Commit message: Checkpoint -- expansion interface and PSU placeholders.  More work to do, but I want to get mounting holes placed.
Connections:
- net +5V: no longer U701.31 (~{SMEMRB}), U701.32 (~{SMEMWB})
- net at R701.2: now also U701.31 (~{SMEMRB}), U701.32 (~{SMEMWB}); no longer U701.96 (~{IOCS16B/SLOT16})
- new net ~{ISA_IO16}: U701.96 (~{IOCS16B/SLOT16})
Other:
- moved on the sheet: R701
Changed lines of the file:
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@@
 	)
 	(junction
-		(at 21.59 133.35)
-		(diameter 0)
-		(color 0 0 0 0)
-	)
-	(junction
-		(at 13.97 125.73)
+		(at 76.2 24.13)
 		(diameter 0)
 		(color 0 0 0 0)
 	)
 	(junction
-		(at 76.2 24.13)
+		(at 48.26 135.89)
 		(diameter 0)
 		(color 0 0 0 0)
@@
 	(wire
 		(pts
-			(xy 21.59 133.35) (xy 48.26 133.35)
-		)
-		(stroke
-			(width 0)
-			(type default)
-		)
-	)
-	(wire
-		(pts
 			(xy 163.83 142.24) (xy 177.8 142.24)
 		)
@@
 	(wire
 		(pts
-			(xy 13.97 148.59) (xy 13.97 130.81)
-		)
-		(stroke
-			(width 0)
-			(type default)
-		)
-	)
-	(wire
-		(pts
 			(xy 73.66 179.07) (xy 76.2 179.07)
 		)
@@
 	(wire
 		(pts
-			(xy 21.59 125.73) (xy 21.59 133.35)
-		)
-		(stroke
-			(width 0)
-			(type default)
-		)
-	)
-	(wire
-		(pts
 			(xy 209.55 153.67) (xy 220.98 153.67)
 		)
@@
 	(wire
 		(pts
-			(xy 13.97 125.73) (xy 21.59 125.73)
-		)
-		(stroke
-			(width 0)
-			(type default)
-		)
-	)
-	(wire
-		(pts
 			(xy 187.96 95.25) (xy 187.96 100.33)
 		)
@@
 	(wire
 		(pts
-			(xy 48.26 148.59) (xy 13.97 148.59)
+			(xy 48.26 133.35) (xy 48.26 135.89)
 		)
 		(stroke
@@
 		)
 	)
+	(global_label "~{ISA_IO16}"
+		(shape output)
+		(at 48.26 148.59 180)
+		(fields_autoplaced yes)
+		(effects
+			(font
+				(size 1.27 1.27)
+			)
+			(justify right)
+		)
+		(property "Intersheetrefs" "${INTERSHEET_REFS}"
+			(at 37.05 148.59 0)
+			(effects
+				(font
+					(size 1.27 1.27)
+				)
+				(justify right)
+				(hide yes)
+			)
+		)
+	)
 	(global_label "A13"
 		(shape input)
@@
 	(symbol
 		(lib_id "power:+5V")
-		(at 13.97 125.73 0)
+		(at 21.59 128.27 0)
 		(unit 1)
 		(exclude_from_sim no)
@@
 		(fields_autoplaced yes)
 		(property "Reference" "#PWR0712"
-			(at 13.97 129.54 0)
+			(at 21.59 132.08 0)
 			(effects
 				(font
@@
 		)
 		(property "Value" "+5V"
-			(at 13.97 120.65 0)
+			(at 21.59 123.19 0)
 			(effects
 				(font
@@
 		)
 		(property "Footprint" ""
-			(at 13.97 125.73 0)
+			(at 21.59 128.27 0)
 			(effects
 				(font
@@
 		)
 		(property "Datasheet" ""
-			(at 13.97 125.73 0)
+			(at 21.59 128.27 0)
 			(effects
 				(font
@@
 		)
 		(property "Description" "Power symbol creates a global label with name \"+5V\""
-			(at 13.97 125.73 0)
+			(at 21.59 128.27 0)
 			(effects
 				(font
@@
 	(symbol
 		(lib_id "Device:R_Small")
-		(at 13.97 128.27 0)
+		(at 21.59 130.81 0)
 		(unit 1)
 		(exclude_from_sim no)
@@
 		(dnp no)
 		(property "Reference" "R701"
-			(at 15.24 127 0)
+			(at 22.86 129.54 0)
 			(effects
 				(font
@@
 		)
 		(property "Value" "10K"
-			(at 15.24 129.54 0)
+			(at 22.86 132.08 0)
 			(effects
 				(font
@@
 		)
 		(property "Footprint" "Resistor_SMD:R_0805_2012Metric"
-			(at 13.97 128.27 0)
+			(at 21.59 130.81 0)
 			(effects
 				(font
@@
 		)
 		(property "Datasheet" "~"
-			(at 13.97 128.27 0)
+			(at 21.59 130.81 0)
 			(effects
 				(font
@@
 		)
 		(property "Description" "Resistor, small symbol"
-			(at 13.97 128.27 0)
+			(at 21.59 130.81 0)
 			(effects
 				(font

Commit message: Ethernet analog magic.
Parts:
- added C711, C712, C713: 100nF, Capacitor_SMD:C_0805_2012Metric, symbol Device:C_Small
- added R705, R706: 49.9, Resistor_SMD:R_0805_2012Metric, symbol Device:R_Small
- added R707, R708: 10, Resistor_SMD:R_0805_2012Metric, symbol Device:R_Small
Connections:
- net ETH_RD+: now also R706.1
- net ETH_RD-: now also R705.1
- net ETH_TD+: now also R707.2; no longer U701.45 (TPOUT+)
- net ETH_TD-: now also R708.1; no longer U701.46 (TPOUT-)
- net GND: now also C711.2, C712.2, C713.2
- new net: C713.1, R708.2, U701.46 (TPOUT-)
- new net: C712.1, R707.1, U701.45 (TPOUT+)
- new net: C711.1, R705.2, R706.2

Commit message: Checkpoint: some PSU work, lock down Ethernet analog traces.
Parts:
- added R709: 22, Resistor_SMD:R_0805_2012Metric, symbol Device:R_Small
- C709, C710: value 10nF -> 100nF
- C712, C713: value 100nF -> 10nF
Connections:
- net ETH_CLK: now also R709.1; no longer Y701.5 (OUT)
- new net: R709.2, Y701.5 (OUT)
Other:
- moved on the sheet: C701, C710, Y701
Changed lines of the file:
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@@
 	)
 	(junction
-		(at 177.8 142.24)
+		(at 151.13 157.48)
 		(diameter 0)
 		(color 0 0 0 0)
@@
 	)
 	(junction
-		(at 177.8 157.48)
+		(at 151.13 172.72)
 		(diameter 0)
 		(color 0 0 0 0)
@@
 	)
 	(no_connect
-		(at 170.18 149.86)
+		(at 143.51 165.1)
 	)
 	(no_connect
@@
 	(wire
 		(pts
-			(xy 163.83 142.24) (xy 177.8 142.24)
+			(xy 137.16 157.48) (xy 151.13 157.48)
 		)
 		(stroke
@@
 	(wire
 		(pts
-			(xy 187.96 95.25) (xy 187.96 100.33)
+			(xy 189.23 95.25) (xy 189.23 100.33)
 		)
 		(stroke
@@
 	(wire
 		(pts
-			(xy 205.74 95.25) (xy 187.96 95.25)
+			(xy 205.74 95.25) (xy 189.23 95.25)
 		)
 		(stroke
@@
 	(wire
 		(pts
-			(xy 163.83 157.48) (xy 177.8 157.48)
+			(xy 137.16 172.72) (xy 151.13 172.72)
 		)
 		(stroke
@@
 	(wire
 		(pts
-			(xy 163.83 147.32) (xy 163.83 157.48)
+			(xy 137.16 162.56) (xy 137.16 172.72)
 		)
 		(stroke
@@
 	)
 	(label "ETH_CLK"
-		(at 185.42 149.86 0)
+		(at 163.83 165.1 0)
 		(effects
 			(font
@@
 			)
 		)
-		(property "Value" "100nF"
+		(property "Value" "10nF"
 			(at 168.91 129.5462 0)
 			(effects
@@
 	(symbol
 		(lib_id "Device:C_Small")
-		(at 187.96 102.87 0)
+		(at 189.23 102.87 0)
 		(unit 1)
 		(exclude_from_sim no)
@@
 		(fields_autoplaced yes)
 		(property "Reference" "C710"
-			(at 190.5 101.6062 0)
+			(at 191.77 101.6062 0)
 			(effects
 				(font
@@
 			)
 		)
-		(property "Value" "10nF"
-			(at 190.5 104.1462 0)
+		(property "Value" "100nF"
+			(at 191.77 104.1462 0)
 			(effects
 				(font
@@
 		)
 		(property "Footprint" "Capacitor_SMD:C_0805_2012Metric"
-			(at 187.96 102.87 0)
+			(at 189.23 102.87 0)
 			(effects
 				(font
@@
 		)
 		(property "Datasheet" "~"
-			(at 187.96 102.87 0)
+			(at 189.23 102.87 0)
 			(effects
 				(font
@@
 		)
 		(property "Description" "Unpolarized capacitor, small symbol"
-			(at 187.96 102.87 0)
+			(at 189.23 102.87 0)
 			(effects
 				(font
@@
 	(symbol
 		(lib_id "Device:C_Small")
-		(at 163.83 144.78 0)
+		(at 137.16 160.02 0)
 		(unit 1)
 		(exclude_from_sim no)
@@
 		(fields_autoplaced yes)
 		(property "Reference" "C701"
-			(at 166.37 143.5162 0)
+			(at 139.7 158.7562 0)
 			(effects
 				(font
@@
 		)
 		(property "Value" "100nF"
-			(at 166.37 146.0562 0)
+			(at 139.7 161.2962 0)
 			(effects
 				(font
@@
 		)
 		(property "Footprint" "Capacitor_SMD:C_0805_2012Metric"
-			(at 163.83 144.78 0)
+			(at 137.16 160.02 0)
 			(effects
 				(font
@@
 		)
 		(property "Datasheet" "~"
-			(at 163.83 144.78 0)
+			(at 137.16 160.02 0)
 			(effects
 				(font
@@
 		)
 		(property "Description" "Unpolarized capacitor, small symbol"
-			(at 163.83 144.78 0)
+			(at 137.16 160.02 0)
 			(effects
 				(font
@@
 	(symbol
 		(lib_id "power:GND")
-		(at 177.8 157.48 0)
+		(at 151.13 172.72 0)
 		(unit 1)
 		(exclude_from_sim no)
@@
 		(fields_autoplaced yes)
 		(property "Reference" "#PWR0709"
-			(at 177.8 163.83 0)
+			(at 151.13 179.07 0)
 			(effects
 				(font
@@
 		)
 		(property "Value" "GND"
-			(at 177.8 162.56 0)
+			(at 151.13 177.8 0)
 			(effects
 				(font
@@
 		)
 		(property "Footprint" ""
-			(at 177.8 157.48 0)
+			(at 151.13 172.72 0)
 			(effects
 				(font
@@
 		)
 		(property "Datasheet" ""
-			(at 177.8 157.48 0)
+			(at 151.13 172.72 0)
 			(effects
 				(font
@@
 		)
 		(property "Description" "Power symbol creates a global label with name \"GND\" , ground"
-			(at 177.8 157.48 0)
+			(at 151.13 172.72 0)
 			(effects
 				(font
@@
 	(symbol
 		(lib_id "Device:R_Small")
+		(at 161.29 165.1 270)
+		(unit 1)
+		(exclude_from_sim no)
+		(in_bom yes)
+		(on_board yes)
+		(dnp no)
+		(property "Reference" "R709"
+			(at 162.56 166.37 0)
+			(effects
+				(font
+					(size 1.016 1.016)
+				)
+				(justify left)
+			)
+		)
+		(property "Value" "22"
+			(at 160.02 166.37 0)
+			(effects
+				(font
+					(size 1.27 1.27)
+				)
+				(justify left)
+			)
+		)
+		(property "Footprint" "Resistor_SMD:R_0805_2012Metric"
+			(at 161.29 165.1 0)
+			(effects
+				(font
+					(size 1.27 1.27)
+				)
+				(hide yes)
+			)
+		)
+		(property "Datasheet" "~"
+			(at 161.29 165.1 0)
+			(effects
+				(font
+					(size 1.27 1.27)
+				)
+				(hide yes)
+			)
+		)
+		(property "Description" "Resistor, small symbol"
+			(at 161.29 165.1 0)
+			(effects
+				(font
+					(size 1.27 1.27)
+				)
+				(hide yes)
+			)
+		)
+		(pin "2"
+		)
+		(pin "1"
+		)
+		(instances
+			(project "cpu030"
+				(path "/6696b89f-f6cc-4e49-bcfb-68bdb218d2a6/6336b086-612e-4cdf-a612-7ddcb8084a94"
+					(reference "R709")
+					(unit 1)
+				)
+			)
+		)
+	)
+	(symbol
+		(lib_id "Device:R_Small")
 		(at 143.51 135.89 0)
 		(unit 1)
@@
 			)
 		)
-		(property "Value" "100nF"
+		(property "Value" "10nF"
 			(at 158.75 129.5462 0)
 			(effects
@@
 	(symbol
 		(lib_id "power:GND")
-		(at 187.96 105.41 0)
+		(at 189.23 105.41 0)
 		(unit 1)
 		(exclude_from_sim no)
@@
 		(fields_autoplaced yes)
 		(property "Reference" "#PWR0714"
-			(at 187.96 111.76 0)
+			(at 189.23 111.76 0)
 			(effects
 				(font
@@
 		)
 		(property "Value" "GND"
-			(at 187.96 110.49 0)
+			(at 189.23 110.49 0)
 			(effects
 				(font
@@
 		)
 		(property "Footprint" ""
-			(at 187.96 105.41 0)
+			(at 189.23 105.41 0)
 			(effects
 				(font
@@
 		)
 		(property "Datasheet" ""
-			(at 187.96 105.41 0)
+			(at 189.23 105.41 0)
 			(effects
 				(font
@@
 		)
 		(property "Description" "Power symbol creates a global label with name \"GND\" , ground"
-			(at 187.96 105.41 0)
+			(at 189.23 105.41 0)
 			(effects
 				(font
@@
 	(symbol
 		(lib_id "Oscillator:CXO_DIP8")
-		(at 177.8 149.86 0)
+		(at 151.13 165.1 0)
 		(unit 1)
 		(exclude_from_sim no)
@@
 		(fields_autoplaced yes)
 		(property "Reference" "Y701"
-			(at 189.23 143.4398 0)
+			(at 162.56 158.6798 0)
 			(effects
 				(font
@@
 		)
 		(property "Value" "20MHz"
-			(at 189.23 145.9798 0)
+			(at 162.56 161.2198 0)
 			(effects
 				(font
@@
 		)
 		(property "Footprint" "Oscillator:Oscillator_DIP-8"
-			(at 189.23 158.75 0)
+			(at 162.56 173.99 0)
 			(effects
 				(font
@@
 		)
 		(property "Datasheet" "http://cdn-reichelt.de/documents/datenblatt/B400/OSZI.pdf"
-			(at 175.26 149.86 0)
+			(at 148.59 165.1 0)
 			(effects
 				(font
@@
 		)
 		(property "Description" "Crystal Clock Oscillator, DIP8-style metal package"
-			(at 177.8 149.86 0)
+			(at 151.13 165.1 0)
 			(effects
 				(font
@@
 		)
 		(property "Part" "MXO45HS-3C-20M0000"
-			(at 177.8 149.86 0)
+			(at 151.13 165.1 0)
 			(effects
 				(font
@@
 	(symbol
 		(lib_id "power:+5V")
-		(at 177.8 142.24 0)
+		(at 151.13 157.48 0)
 		(unit 1)
 		(exclude_from_sim no)
@@
 		(fields_autoplaced yes)
 		(property "Reference" "#PWR0708"
-			(at 177.8 146.05 0)
+			(at 151.13 161.29 0)
 			(effects
 				(font
@@
 		)
 		(property "Value" "+5V"
-			(at 177.8 137.16 0)
+			(at 151.13 152.4 0)
 			(effects
 				(font
@@
 		)
 		(property "Footprint" ""
-			(at 177.8 142.24 0)
+			(at 151.13 157.48 0)
 			(effects
 				(font
@@
 		)
 		(property "Datasheet" ""
-			(at 177.8 142.24 0)
+			(at 151.13 157.48 0)
 			(effects
 				(font
@@
 		)
 		(property "Description" "Power symbol creates a global label with name \"+5V\""
-			(at 177.8 142.24 0)
+			(at 151.13 157.48 0)
 			(effects
 				(font
@@
 			)
 		)
-		(property "Value" "10nF"
+		(property "Value" "100nF"
 			(at 180.34 104.1462 0)
 			(effects

Commit message: Checkpoint: address lines for Ethernet.
Connections:
- net A10 is gone; now on net GND: U701.18 (SA10)
- net A11 is gone; now on net GND: U701.19 (SA11)
- net A12 is gone; now on net GND: U701.20 (SA12)
- net A13 is gone; now on net GND: U701.21 (SA13)
- net A14 is gone; now on net GND: U701.22 (SA14)
- net A15 is gone; now on net GND: U701.23 (SA15)
- net A16 is gone; now on net GND: U701.24 (SA16)
- net A17 is gone; now on net GND: U701.25 (SA17)
- net A18 is gone; now on net GND: U701.26 (SA18)
- net A19 is gone; now on net GND: U701.27 (SA19)
- net A5 is gone; now on net GND: U701.11 (SA5)
- net A6 is gone; now on net GND: U701.12 (SA6)
- net A7 is gone; now on net GND: U701.13 (SA7)
- net A8 is gone; now on an unnamed net: U701.15 (SA8)
- net A9 is gone; now on an unnamed net: U701.16 (SA9)
- net ISA_AEN renamed ~{ETHSEL}
Other:
- note added: "The chip is wired for "jumper mode", and the IRQSx and IOSx connections select INT0 and I/O address 0x300. ISACTL only asserts ~{ETHSEL} for 0x300, and the address lines are hard-wired for it. Only A[4..0] need be routed on the board."
- note removed: "The chip is wired for "jumper mode", and the IRQSx and IOSx connections select INT0 and I/O address 0x300."

Commit message: Update revision to A0, update issue date.  Update 68882's symbol attributes to eliminate ERC errors.
Other:
- company: (none) -> (c) 2025 Jason R. Thorpe.  See LICENSE.
- title: (none) -> Playground 68030 Mk I
Changed lines of the file:
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@@
 	(generator_version "9.0")
 	(paper "A4")
+	(title_block
+		(title "Playground 68030 Mk I")
+		(date "2025-08-29")
+		(rev "A0")
+		(company "(c) 2025 Jason R. Thorpe.  See LICENSE.")
+	)
 	(text "The chip is wired for \"jumper mode\", and the IRQSx\nand IOSx connections select INT0 and I/O address\n0x300.  ISACTL only asserts ~{ETHSEL} for 0x300,\nand the address lines are hard-wired for it.  Only\nA[4..0] need be routed on the board."
 		(exclude_from_sim no)
