File: cpu030/design-files/cpu030_ide.kicad_sch (KiCad schematic)
At the start: 10 parts, among them J501 ATA connector, U501 74ACT245, U502 74ACT245, U503 74ACT245, U504 74AHCT138, U505 GAL22V10

Commit message: Add ISACTL ISA bus controller and re-do ATA interface with it.
Parts:
- removed R501: 47K, Resistor_SMD:R_0805_2012Metric, symbol Device:R_Small
- removed U504: 74AHCT138, Package_SO:SOIC-16_3.9x9.9mm_P1.27mm, symbol 74xx:74LS138
- removed U505: GAL22V10, symbol jrt-ICs:GAL22V10
- added C501, C502, C503: 100nF, Capacitor_SMD:C_0805_2012Metric, symbol Device:C_Small
- D501: value ATA Acvity -> ATA Active
- J501: footprint (none) -> Connector_IDC:IDC-Header_2x20_P2.54mm_Vertical
- U501, U502, U503: footprint Package_SO:SOIC-20W_7.5x12.8mm_P1.27mm -> Package_DIP:DIP-20_W7.62mm_Socket; Part 74ACT245SCX -> (none)
Connections:
- net +5V: now also C501.1, C502.1, C503.1
- net ATA_INT: no longer U503.11 (B7)
- net GND: now also C501.2, C502.2, C503.2
- net ~{ATASEL}: now also U503.15 (B3); no longer U501.19 (CE), U502.19 (CE)
- net ~{ATA_IORD}: now also U503.8 (A6)
- net ~{ATA_IOWR}: now also U503.9 (A7)
- net ~{ATAAUXSEL}: now reaches U503.14 (B4)
- net ATA_IORDY renamed ISA_IORDY
- net ISA_IORDY: no longer U503.12 (B6)
- net ~{ATA_CS1} renamed ~{ATA_CS1FX}
- net ~{ATA_CS2} renamed ~{ATA_CS3FX}
- new net ~{ATABEN}: U501.19 (CE), U502.19 (CE)
- new net ~{ISA_IORD}: U503.12 (B6)
- new net ~{ISA_IOWR}: U503.11 (B7)
- no-connect marks 23 -> 6
Other:
- note removed: "ISAGLUE"
- moved on the sheet: D501, R502, R503, U501, U502, U503

Commit message: Add Ethernet.
Connections:
- net ISA_IORDY renamed ISA_RDY
Changed lines of the file:
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@@
 		)
 	)
-	(global_label "ISA_IORDY"
+	(global_label "ISA_RDY"
 		(shape output)
 		(at 222.25 95.25 180)
@@
 		)
 		(property "Intersheetrefs" "${INTERSHEET_REFS}"
-			(at 209.8304 95.25 0)
+			(at 211.7657 95.25 0)
 			(effects
 				(font

Commit message: Checkpoint -- expansion interface and PSU placeholders.  More work to do, but I want to get mounting holes placed.
Parts:
- R503: value 330 -> 470
Connections:
- net ~{ISA_IO16}: now reaches J501.32 (Pin_32)
- no-connect marks 6 -> 5
Changed lines of the file:
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@@
-	)
-	(no_connect
-		(at 246.38 100.33)
 	)
 	(no_connect
@@
 	(wire
 		(pts
-			(xy 222.25 95.25) (xy 233.68 95.25)
+			(xy 247.65 92.71) (xy 247.65 97.79)
 		)
 		(stroke
@@
 	(wire
 		(pts
-			(xy 247.65 92.71) (xy 247.65 97.79)
+			(xy 247.65 87.63) (xy 247.65 90.17)
 		)
 		(stroke
@@
 	(wire
 		(pts
-			(xy 247.65 87.63) (xy 247.65 90.17)
+			(xy 74.93 85.09) (xy 74.93 87.63)
 		)
 		(stroke
@@
 	(wire
 		(pts
-			(xy 74.93 85.09) (xy 74.93 87.63)
+			(xy 247.65 90.17) (xy 247.65 92.71)
 		)
 		(stroke
@@
 	(wire
 		(pts
-			(xy 247.65 90.17) (xy 247.65 92.71)
+			(xy 247.65 97.79) (xy 246.38 97.79)
 		)
 		(stroke
@@
 	(wire
 		(pts
-			(xy 247.65 97.79) (xy 246.38 97.79)
+			(xy 246.38 90.17) (xy 247.65 90.17)
 		)
 		(stroke
@@
 	(wire
 		(pts
-			(xy 246.38 90.17) (xy 247.65 90.17)
+			(xy 143.51 144.78) (xy 154.94 144.78)
 		)
 		(stroke
@@
 	(wire
 		(pts
-			(xy 143.51 144.78) (xy 154.94 144.78)
+			(xy 214.63 100.33) (xy 218.44 100.33)
 		)
 		(stroke
@@
 	(wire
 		(pts
-			(xy 214.63 100.33) (xy 218.44 100.33)
+			(xy 252.73 62.23) (xy 246.38 62.23)
 		)
 		(stroke
@@
 	(wire
 		(pts
-			(xy 252.73 62.23) (xy 246.38 62.23)
+			(xy 246.38 87.63) (xy 247.65 87.63)
 		)
 		(stroke
@@
 	(wire
 		(pts
-			(xy 246.38 87.63) (xy 247.65 87.63)
+			(xy 246.38 92.71) (xy 247.65 92.71)
 		)
 		(stroke
@@
 	(wire
 		(pts
-			(xy 246.38 92.71) (xy 247.65 92.71)
+			(xy 143.51 149.86) (xy 154.94 149.86)
 		)
 		(stroke
@@
 	(wire
 		(pts
-			(xy 143.51 149.86) (xy 154.94 149.86)
+			(xy 154.94 144.78) (xy 166.37 144.78)
 		)
 		(stroke
@@
 		)
 	)
-	(wire
-		(pts
-			(xy 154.94 144.78) (xy 166.37 144.78)
-		)
-		(stroke
-			(width 0)
-			(type default)
-		)
-	)
 	(label "ATA_D0"
 		(at 143.51 31.75 180)
@@
 	(global_label "ISA_RDY"
 		(shape output)
-		(at 222.25 95.25 180)
+		(at 233.68 95.25 180)
 		(fields_autoplaced yes)
 		(effects
@@
 		)
 		(property "Intersheetrefs" "${INTERSHEET_REFS}"
-			(at 211.7657 95.25 0)
+			(at 223.1957 95.25 0)
 			(effects
 				(font
@@
 		(property "Intersheetrefs" "${INTERSHEET_REFS}"
 			(at 176.6955 39.37 0)
+			(effects
+				(font
+					(size 1.27 1.27)
+				)
+				(justify left)
+				(hide yes)
+			)
+		)
+	)
+	(global_label "~{ISA_IO16}"
+		(shape output)
+		(at 246.38 100.33 0)
+		(fields_autoplaced yes)
+		(effects
+			(font
+				(size 1.27 1.27)
+			)
+			(justify left)
+		)
+		(property "Intersheetrefs" "${INTERSHEET_REFS}"
+			(at 257.59 100.33 0)
 			(effects
 				(font
@@
 			)
 		)
-		(property "Value" "330"
+		(property "Value" "470"
 			(at 242.57 123.1899 0)
 			(effects

Commit message: Checkpoint: layout mostly the way I want it now.
Parts:
- added J502: 5V CF Power, Connector_PinHeader_2.54mm:PinHeader_1x04_P2.54mm_Vertical, symbol Connector_Generic:Conn_01x04
- U501, U502, U503: footprint Package_DIP:DIP-20_W7.62mm_Socket -> Package_SO:SOIC-20W_7.5x12.8mm_P1.27mm; Part (none) -> 74ACT245SCX
- renumbered R502 to R501
Connections:
- net +5V: now also J502.1 (Pin_1)
- net ATA_D10: now also U502.7 (A5); no longer U502.4 (A2)
- net ATA_D11: now also U502.6 (A4); no longer U502.5 (A3)
- net ATA_D12: now also U502.5 (A3); no longer U502.6 (A4)
- net ATA_D13: now also U502.4 (A2); no longer U502.7 (A5)
- net ATA_D14: now also U502.3 (A1); no longer U502.8 (A6)
- net ATA_D15: now also U502.2 (A0); no longer U502.9 (A7)
- net ATA_D8: now also U502.9 (A7); no longer U502.2 (A0)
- net ATA_D9: now also U502.8 (A6); no longer U502.3 (A1)
- net D16: now also U502.11 (B7); no longer U502.18 (B0)
- net D17: now also U502.12 (B6); no longer U502.17 (B1)
- net D18: now also U502.13 (B5); no longer U502.16 (B2)
- net D19: now also U502.14 (B4); no longer U502.15 (B3)
- net D20: now also U502.15 (B3); no longer U502.14 (B4)
- net D21: now also U502.16 (B2); no longer U502.13 (B5)
- net D22: now also U502.17 (B1); no longer U502.12 (B6)
- net D23: now also U502.18 (B0); no longer U502.11 (B7)
- net GND: now also J502.2 (Pin_2), J502.3 (Pin_3)
- no-connect marks 5 -> 6

Commit message: Checkpoint: some PSU work, lock down Ethernet analog traces.
Parts:
- added C504: 470µF, Capacitor_THT:CP_Radial_D10.0mm_P5.00mm, symbol Device:C_Polarized_Small
Connections:
- net +5V: now also C504.1
- net GND: now also C504.2
Changed lines of the file:
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@@
+	)
+	(symbol
+		(lib_id "power:GND")
+		(at 182.88 149.86 0)
+		(unit 1)
+		(exclude_from_sim no)
+		(in_bom yes)
+		(on_board yes)
+		(dnp no)
+		(fields_autoplaced yes)
+		(property "Reference" "#PWR0516"
+			(at 182.88 156.21 0)
+			(effects
+				(font
+					(size 1.27 1.27)
+				)
+				(hide yes)
+			)
+		)
+		(property "Value" "GND"
+			(at 182.88 154.94 0)
+			(effects
+				(font
+					(size 1.27 1.27)
+				)
+			)
+		)
+		(property "Footprint" ""
+			(at 182.88 149.86 0)
+			(effects
+				(font
+					(size 1.27 1.27)
+				)
+				(hide yes)
+			)
+		)
+		(property "Datasheet" ""
+			(at 182.88 149.86 0)
+			(effects
+				(font
+					(size 1.27 1.27)
+				)
+				(hide yes)
+			)
+		)
+		(property "Description" "Power symbol creates a global label with name \"GND\" , ground"
+			(at 182.88 149.86 0)
+			(effects
+				(font
+					(size 1.27 1.27)
+				)
+				(hide yes)
+			)
+		)
+		(pin "1"
+		)
+		(instances
+			(project "cpu030"
+				(path "/6696b89f-f6cc-4e49-bcfb-68bdb218d2a6/2f986d8b-f53d-4235-93e5-3fe086aff134"
+					(reference "#PWR0516")
+					(unit 1)
+				)
+			)
+		)
 	)
 	(symbol
@@
 	)
 	(symbol
+		(lib_id "Device:C_Polarized_Small")
+		(at 182.88 147.32 0)
+		(unit 1)
+		(exclude_from_sim no)
+		(in_bom yes)
+		(on_board yes)
+		(dnp no)
+		(fields_autoplaced yes)
+		(property "Reference" "C504"
+			(at 185.42 145.5038 0)
+			(effects
+				(font
+					(size 1.27 1.27)
+				)
+				(justify left)
+			)
+		)
+		(property "Value" "470µF"
+			(at 185.42 148.0438 0)
+			(effects
+				(font
+					(size 1.27 1.27)
+				)
+				(justify left)
+			)
+		)
+		(property "Footprint" "Capacitor_THT:CP_Radial_D10.0mm_P5.00mm"
+			(at 182.88 147.32 0)
+			(effects
+				(font
+					(size 1.27 1.27)
+				)
+				(hide yes)
+			)
+		)
+		(property "Datasheet" "~"
+			(at 182.88 147.32 0)
+			(effects
+				(font
+					(size 1.27 1.27)
+				)
+				(hide yes)
+			)
+		)
+		(property "Description" "Polarized capacitor, small symbol"
+			(at 182.88 147.32 0)
+			(effects
+				(font
+					(size 1.27 1.27)
+				)
+				(hide yes)
+			)
+		)
+		(property "Part" "ESL477M025AH9AA"
+			(at 182.88 147.32 0)
+			(effects
+				(font
+					(size 1.27 1.27)
+				)
+				(hide yes)
+			)
+		)
+		(pin "1"
+		)
+		(pin "2"
+		)
+		(instances
+			(project "cpu030"
+				(path "/6696b89f-f6cc-4e49-bcfb-68bdb218d2a6/2f986d8b-f53d-4235-93e5-3fe086aff134"
+					(reference "C504")
+					(unit 1)
+				)
+			)
+		)
+	)
+	(symbol
 		(lib_id "74xx:74HC245")
 		(at 156.21 101.6 0)
@@
 					(unit 1)
 				)
+			)
+		)
+	)
+	(symbol
+		(lib_id "power:+5V")
+		(at 182.88 144.78 0)
+		(unit 1)
+		(exclude_from_sim no)
+		(in_bom yes)
+		(on_board yes)
+		(dnp no)
+		(fields_autoplaced yes)
+		(property "Reference" "#PWR0515"
+			(at 182.88 148.59 0)
+			(effects
+				(font
+					(size 1.27 1.27)
+				)
+				(hide yes)
+			)
+		)
+		(property "Value" "+5V"
+			(at 182.88 139.7 0)
+			(effects
+				(font
+					(size 1.27 1.27)
+				)
+			)
+		)
+		(property "Footprint" ""
+			(at 182.88 144.78 0)
+			(effects
+				(font
+					(size 1.27 1.27)
+				)
+				(hide yes)
+			)
+		)
+		(property "Datasheet" ""
+			(at 182.88 144.78 0)
+			(effects
+				(font
+					(size 1.27 1.27)
+				)
+				(hide yes)
+			)
+		)
+		(property "Description" "Power symbol creates a global label with name \"+5V\""
+			(at 182.88 144.78 0)
+			(effects
+				(font
+					(size 1.27 1.27)
+				)
+				(hide yes)
+			)
+		)
+		(pin "1"
+		)
+		(instances
+			(project "cpu030"
+				(path "/6696b89f-f6cc-4e49-bcfb-68bdb218d2a6/2f986d8b-f53d-4235-93e5-3fe086aff134"
+					(reference "#PWR0515")
+					(unit 1)
+				)

Commit message: Manually route the buffered IDE signals.
Connections:
- net A0: now also U503.16 (B2); no longer U503.18 (B0)
- net A1: now also U503.14 (B4); no longer U503.17 (B1)
- net A2: now also U503.15 (B3); no longer U503.16 (B2)
- net ATA_A0: now also U503.4 (A2); no longer U503.2 (A0)
- net ATA_A1: now also U503.6 (A4); no longer U503.3 (A1)
- net ATA_A2: now also U503.5 (A3); no longer U503.4 (A2)
- net ~{ATAAUXSEL}: now also U503.17 (B1); no longer U503.14 (B4)
- net ~{ATASEL}: now also U503.18 (B0); no longer U503.15 (B3)
- net ~{ATA_CS1FX}: now also U503.2 (A0); no longer U503.5 (A3)
- net ~{ATA_CS3FX}: now also U503.3 (A1); no longer U503.6 (A4)
Changed lines of the file:
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@@
 	)
 	(label "ATA_A1"
-		(at 74.93 64.77 180)
+		(at 74.93 72.39 180)
 		(effects
 			(font
@@
 	)
 	(label "~{ATA_CS1FX}"
-		(at 74.93 69.85 180)
+		(at 74.93 62.23 180)
 		(effects
 			(font
@@
 	)
 	(label "ATA_A0"
-		(at 74.93 62.23 180)
+		(at 74.93 67.31 180)
 		(effects
 			(font
@@
 	)
 	(label "ATA_A2"
-		(at 74.93 67.31 180)
+		(at 74.93 69.85 180)
 		(effects
 			(font
@@
 	)
 	(label "~{ATA_CS3FX}"
-		(at 74.93 72.39 180)
+		(at 74.93 64.77 180)
 		(effects
 			(font
@@
 	(global_label "A1"
 		(shape input)
-		(at 100.33 64.77 0)
-		(fields_autoplaced yes)
-		(effects
-			(font
-				(size 1.27 1.27)
-			)
-			(justify left)
-		)
-		(property "Intersheetrefs" "${INTERSHEET_REFS}"
-			(at 105.6133 64.77 0)
+		(at 100.33 72.39 0)
+		(fields_autoplaced yes)
+		(effects
+			(font
+				(size 1.27 1.27)
+			)
+			(justify left)
+		)
+		(property "Intersheetrefs" "${INTERSHEET_REFS}"
+			(at 105.6133 72.39 0)
 			(effects
 				(font
@@
 	(global_label "A2"
 		(shape input)
-		(at 100.33 67.31 0)
-		(fields_autoplaced yes)
-		(effects
-			(font
-				(size 1.27 1.27)
-			)
-			(justify left)
-		)
-		(property "Intersheetrefs" "${INTERSHEET_REFS}"
-			(at 105.6133 67.31 0)
+		(at 100.33 69.85 0)
+		(fields_autoplaced yes)
+		(effects
+			(font
+				(size 1.27 1.27)
+			)
+			(justify left)
+		)
+		(property "Intersheetrefs" "${INTERSHEET_REFS}"
+			(at 105.6133 69.85 0)
 			(effects
 				(font
@@
 	(global_label "~{ATASEL}"
 		(shape input)
-		(at 100.33 69.85 0)
-		(fields_autoplaced yes)
-		(effects
-			(font
-				(size 1.27 1.27)
-			)
-			(justify left)
-		)
-		(property "Intersheetrefs" "${INTERSHEET_REFS}"
-			(at 109.8466 69.85 0)
+		(at 100.33 62.23 0)
+		(fields_autoplaced yes)
+		(effects
+			(font
+				(size 1.27 1.27)
+			)
+			(justify left)
+		)
+		(property "Intersheetrefs" "${INTERSHEET_REFS}"
+			(at 109.8466 62.23 0)
 			(effects
 				(font
@@
 	(global_label "~{ATAAUXSEL}"
 		(shape input)
-		(at 100.33 72.39 0)
-		(fields_autoplaced yes)
-		(effects
-			(font
-				(size 1.27 1.27)
-			)
-			(justify left)
-		)
-		(property "Intersheetrefs" "${INTERSHEET_REFS}"
-			(at 113.4752 72.39 0)
+		(at 100.33 64.77 0)
+		(fields_autoplaced yes)
+		(effects
+			(font
+				(size 1.27 1.27)
+			)
+			(justify left)
+		)
+		(property "Intersheetrefs" "${INTERSHEET_REFS}"
+			(at 113.4752 64.77 0)
 			(effects
 				(font
@@
 	(global_label "A0"
 		(shape input)
-		(at 100.33 62.23 0)
-		(fields_autoplaced yes)
-		(effects
-			(font
-				(size 1.27 1.27)
-			)
-			(justify left)
-		)
-		(property "Intersheetrefs" "${INTERSHEET_REFS}"
-			(at 105.6133 62.23 0)
-			(effects
-				(font
+		(at 100.33 67.31 0)
+		(fields_autoplaced yes)
+		(effects
+			(font
+				(size 1.27 1.27)
+			)
+			(justify left)
+		)
+		(property "Intersheetrefs" "${INTERSHEET_REFS}"
+			(at 105.6133 67.31 0)
+			(effects
+				(font

Commit message: Update revision to A0, update issue date.  Update 68882's symbol attributes to eliminate ERC errors.
Other:
- company: (none) -> (c) 2025 Jason R. Thorpe.  See LICENSE.
- title: (none) -> Playground 68030 Mk I
Changed lines of the file:
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@@
 	(generator_version "9.0")
 	(paper "A4")
+	(title_block
+		(title "Playground 68030 Mk I")
+		(date "2025-08-29")
+		(rev "A0")
+		(company "(c) 2025 Jason R. Thorpe.  See LICENSE.")
+	)
 	(junction
 		(at 154.94 144.78)
