File: cpu030/design-files/cpu030_isa.kicad_sch (KiCad schematic)
At the start: 15 parts, among them J401 ISACTL JTAG, U401 ATF1508AS, U402 MC74ACT05DG

Commit message: Checkpoint -- expansion interface and PSU placeholders.  More work to do, but I want to get mounting holes placed.
Parts:
- added R404, R405: 3K3, Resistor_SMD:R_0805_2012Metric, symbol Device:R_Small
Connections:
- net +5V: now also R404.1, R405.1
- net ISA_RDY: now also R404.2
- net ~{ISA_IO16}: now reaches U401.83 (I/O)
- net ~{ISA_IO16}: now also R405.2
- no-connect marks 47 -> 46

Commit message: Fix some schematic mistakes and checkpoint signal routing on the PCB.
Connections:
- net ISACTL_TDI: now also U401.4 (I/O/TDI)
Changed lines of the file:
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@@
+	(wire
+		(pts
+			(xy 116.84 54.61) (xy 115.57 54.61)
+		)
+		(stroke
+			(width 0)
+			(type default)
+		)
+	)
 	(wire
 		(pts
@@
 		)
 		(stroke
+			(width 0)
+			(type default)
+		)
+	)
+	(wire
+		(pts
+			(xy 116.84 53.34) (xy 116.84 54.61)
+		)
+		(stroke

Commit message: Checkpoint: address lines for Ethernet.
Connections:
- net ISA_AEN renamed ~{ETHSEL}
Changed lines of the file:
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@@
 		)
 	)
-	(global_label "ISA_AEN"
+	(global_label "~{ETHSEL}"
 		(shape output)
 		(at 172.72 76.2 0)
@@
 		)
 		(property "Intersheetrefs" "${INTERSHEET_REFS}"
-			(at 183.1438 76.2 0)
+			(at 182.5389 76.2 0)
 			(effects
 				(font

Commit message: Fix some connection mistakes on the 74ACT05s, re-arrange pullups on CPU to make layout easier.
Parts:
- U402: value MC74ACT05DG -> 74ACT05
Connections:
- net +5V: now also U402.14 (VCC); no longer U402.7 (GND)
- net GND: now also U402.7 (GND); no longer U402.14 (VCC)
Other:
- moved on the sheet: U402G
Changed lines of the file:
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@@
 	)
 	(junction
-		(at 77.47 97.79)
+		(at 144.78 173.99)
 		(diameter 0)
 		(color 0 0 0 0)
 	)
 	(junction
-		(at 144.78 173.99)
+		(at 137.16 26.67)
 		(diameter 0)
 		(color 0 0 0 0)
 	)
 	(junction
-		(at 137.16 26.67)
+		(at 77.47 97.79)
 		(diameter 0)
 		(color 0 0 0 0)
@@
 	)
 	(junction
+		(at 77.47 72.39)
+		(diameter 0)
+		(color 0 0 0 0)
+	)
+	(junction
 		(at 146.05 154.94)
 		(diameter 0)
@@
 	)
 	(junction
-		(at 77.47 72.39)
-		(diameter 0)
-		(color 0 0 0 0)
-	)
-	(junction
 		(at 93.98 173.99)
 		(diameter 0)
@@
 			)
 		)
-		(property "Value" "MC74ACT05DG"
+		(property "Value" "74ACT05"
 			(at 52.07 88.9 0)
 			(effects
@@
 			)
 		)
-		(property "Value" "MC74ACT05DG"
+		(property "Value" "74ACT05"
 			(at 52.07 73.66 0)
 			(effects
@@
 			)
 		)
-		(property "Value" "MC74ACT05DG"
+		(property "Value" "74ACT05"
 			(at 52.07 43.18 0)
 			(effects
@@
 			)
 		)
-		(property "Value" "MC74ACT05DG"
+		(property "Value" "74ACT05"
 			(at 52.07 104.14 0)
 			(effects
@@
 			)
 		)
-		(property "Value" "MC74ACT05DG"
+		(property "Value" "74ACT05"
 			(at 52.07 58.42 0)
 			(effects
@@
 			)
 		)
-		(property "Value" "MC74ACT05DG"
+		(property "Value" "74ACT05"
 			(at 52.07 29.21 0)
 			(effects
@@
 	(symbol
 		(lib_id "74xx:74LS05")
-		(at 77.47 85.09 180)
+		(at 77.47 85.09 0)
 		(unit 7)
 		(exclude_from_sim no)
@@
 					(size 1.27 1.27)
 				)
-				(justify right)
+				(justify left)
 			)
 		)
-		(property "Value" "MC74ACT05DG"
+		(property "Value" "74ACT05"
 			(at 83.82 86.3599 0)
 			(effects
@@
 					(size 1.27 1.27)
 				)
-				(justify right)
+				(justify left)
 			)
 		)

Commit message: Checkpoint -- a bunch of device signals.
Connections:
- net TMRINT: now also U401.50 (I/O); no longer U401.98 (I/O)
- net ~{ATAAUXSEL}: now also U401.98 (I/O); no longer U401.75 (I/O)
- net ~{ATABEN}: now also U401.99 (I/O); no longer U401.76 (I/O)
- net ~{ATASEL}: now also U401.97 (I/O); no longer U401.72 (I/O)
- net ~{ETHSEL}: now also U401.75 (I/O); no longer U401.79 (I/O)
- net ~{ISA_IORD}: now also U401.80 (I/O); no longer U401.77 (I/O)
- net ~{ISA_IOWR}: now also U401.81 (I/O); no longer U401.78 (I/O)
Changed lines of the file:
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@@
-	)
-	(no_connect
-		(at 172.72 73.66)
 	)
 	(no_connect
@@
 	)
 	(no_connect
+		(at 172.72 76.2)
+	)
+	(no_connect
 		(at 172.72 96.52)
 	)
@@
 	)
 	(no_connect
-		(at 172.72 45.72)
+		(at 172.72 78.74)
 	)
 	(no_connect
@@
 	)
 	(no_connect
+		(at 172.72 83.82)
+	)
+	(no_connect
 		(at 116.84 121.92)
 	)
@@
 	)
 	(no_connect
-		(at 172.72 71.12)
+		(at 172.72 81.28)
 	)
 	(no_connect
@@
 	)
 	(no_connect
-		(at 172.72 139.7)
-	)
-	(no_connect
 		(at 172.72 134.62)
 	)
@@
 	)
 	(no_connect
+		(at 172.72 91.44)
+	)
+	(no_connect
 		(at 172.72 132.08)
 	)
@@
 	)
 	(no_connect
-		(at 172.72 50.8)
-	)
-	(no_connect
 		(at 44.45 80.01)
 	)
@@
 	(wire
 		(pts
-			(xy 172.72 44.45) (xy 172.72 43.18)
-		)
-		(stroke
-			(width 0)
-			(type default)
-		)
-	)
-	(wire
-		(pts
 			(xy 147.32 26.67) (xy 149.86 26.67)
 		)
@@
 		(pts
 			(xy 144.78 173.99) (xy 154.94 173.99)
-		)
-		(stroke
-			(width 0)
-			(type default)
-		)
-	)
-	(wire
-		(pts
-			(xy 173.99 44.45) (xy 172.72 44.45)
 		)
 		(stroke
@@
 	)
 	(label "ISACTL_BERR"
-		(at 173.99 44.45 0)
+		(at 172.72 43.18 0)
 		(effects
 			(font
@@
 	(global_label "TMRINT"
 		(shape output)
-		(at 172.72 48.26 0)
+		(at 172.72 139.7 0)
 		(fields_autoplaced yes)
 		(effects
@@
 		)
 		(property "Intersheetrefs" "${INTERSHEET_REFS}"
-			(at 182.2971 48.26 0)
+			(at 182.2971 139.7 0)
 			(effects
 				(font
@@
 	(global_label "~{ETHSEL}"
 		(shape output)
-		(at 172.72 76.2 0)
+		(at 172.72 86.36 0)
 		(fields_autoplaced yes)
 		(effects
@@
 		)
 		(property "Intersheetrefs" "${INTERSHEET_REFS}"
-			(at 182.5389 76.2 0)
+			(at 182.5389 86.36 0)
 			(effects
 				(font
@@
 	(global_label "~{ATABEN}"
 		(shape output)
-		(at 172.72 83.82 0)
+		(at 172.72 45.72 0)
 		(fields_autoplaced yes)
 		(effects
@@
 		)
 		(property "Intersheetrefs" "${INTERSHEET_REFS}"
-			(at 182.5995 83.82 0)
+			(at 182.5995 45.72 0)
 			(effects
 				(font
@@
 	(global_label "~{ISA_IOWR}"
 		(shape output)
-		(at 172.72 78.74 0)
+		(at 172.72 71.12 0)
 		(fields_autoplaced yes)
 		(effects
@@
 		)
 		(property "Intersheetrefs" "${INTERSHEET_REFS}"
-			(at 184.2324 78.74 0)
+			(at 184.2324 71.12 0)
 			(effects
 				(font
@@
 	(global_label "~{ATASEL}"
 		(shape output)
-		(at 172.72 91.44 0)
+		(at 172.72 50.8 0)
 		(fields_autoplaced yes)
 		(effects
@@
 		)
 		(property "Intersheetrefs" "${INTERSHEET_REFS}"
-			(at 182.2366 91.44 0)
+			(at 182.2366 50.8 0)
 			(effects
 				(font
@@
 	(global_label "~{ISA_IORD}"
 		(shape output)
-		(at 172.72 81.28 0)
+		(at 172.72 73.66 0)
 		(fields_autoplaced yes)
 		(effects
@@
 		)
 		(property "Intersheetrefs" "${INTERSHEET_REFS}"
-			(at 184.051 81.28 0)
+			(at 184.051 73.66 0)
 			(effects
 				(font
@@
 	(global_label "~{ATAAUXSEL}"
 		(shape output)
-		(at 172.72 86.36 0)
+		(at 172.72 48.26 0)
 		(fields_autoplaced yes)
 		(effects
@@
 		)
 		(property "Intersheetrefs" "${INTERSHEET_REFS}"
-			(at 185.8652 86.36 0)
-			(effects
-				(font
+			(at 185.8652 48.26 0)
+			(effects
+				(font

Commit message: Adjust some constraints for DRC.
Changed lines of the file:
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@@
-	)
-	(symbol
-		(lib_id "power:+5V")
-		(at 73.66 113.03 90)
-		(unit 1)
-		(exclude_from_sim no)
-		(in_bom yes)
-		(on_board yes)
-		(dnp no)
-		(fields_autoplaced yes)
-		(property "Reference" "#PWR0402"
-			(at 77.47 113.03 0)
-			(effects
-				(font
-					(size 1.27 1.27)
-				)
-				(hide yes)
-			)
-		)
-		(property "Value" "+5V"
-			(at 69.85 113.0299 90)
-			(effects
-				(font
-					(size 1.27 1.27)
-				)
-				(justify left)
-			)
-		)
-		(property "Footprint" ""
-			(at 73.66 113.03 0)
-			(effects
-				(font
-					(size 1.27 1.27)
-				)
-				(hide yes)
-			)
-		)
-		(property "Datasheet" ""
-			(at 73.66 113.03 0)
-			(effects
-				(font
-					(size 1.27 1.27)
-				)
-				(hide yes)
-			)
-		)
-		(property "Description" "Power symbol creates a global label with name \"+5V\""
-			(at 73.66 113.03 0)
-			(effects
-				(font
-					(size 1.27 1.27)
-				)
-				(hide yes)
-			)
-		)
-		(pin "1"
-		)
-		(instances
-			(project "cpu030"
-				(path "/6696b89f-f6cc-4e49-bcfb-68bdb218d2a6/73c5e65c-632f-4863-98b7-0d11c2a0ac33"
-					(reference "#PWR0402")
-					(unit 1)
-				)
-			)
-		)
 	)
 	(symbol

Commit message: Update revision to A0, update issue date.  Update 68882's symbol attributes to eliminate ERC errors.
Other:
- company: (none) -> (c) 2025 Jason R. Thorpe.  See LICENSE.
- title: (none) -> Playground 68030 Mk I
Changed lines of the file:
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@@
 	(generator_version "9.0")
 	(paper "A4")
+	(title_block
+		(title "Playground 68030 Mk I")
+		(date "2025-08-29")
+		(rev "A0")
+		(company "(c) 2025 Jason R. Thorpe.  See LICENSE.")
+	)
 	(text "ISACTL"
 		(exclude_from_sim no)
