File: cpu010/design-files/cpu010.kicad_pcb (KiCad board)
At the start: 2 copper layers, 365.8 x 223.5 mm, 54 parts, among them SW401 SW_DIP_x08, SW402 SW_DIP_x08, U101 GAL22V10, U201 MC68010P, U202 74ACT163, U203 74ACT05, U301 ATF1508AS-TQFP100, U302 61C3216, U303 74AHCT245, U304 74AHCT245, U305 7C4098, U306 7C4098, U307 74AHCT245, U308 74AHCT245, U309 74AHCT245, U310 74AHCT245, U311 74AHCT373, U312 74AHCT373, U313 74AHCT373, U314 74AHCT157, U315 74AHCT157, U316 74AHCT157, U317 74AHCT157, U318 74AHCT157, U319 74AHCT157, U320 74AHCT157, U321 74AHCT157, U322 74AHCT157, U323 74AHCT245, U324 74AHCT245, U401 DA04-11SURKWA, U402 74HCT273, U403 74HCT273, U404 GAL22V10, U405 74HC245, U406 74HC245, U407 74HCT273, U408 74HC245, U409 ATF1504AS-PLCC44, U501 GAL22V10, U502 CY62158, U503 CY62158, U504 CY62158, U505 CY62158, U506 SST39SF040, U507 SST39SF040, Y201 40MHz

Commit message: Add reset circuit.
Parts:
- added C201: 100µF, Capacitor_THT:CP_Radial_D6.3mm_P2.50mm, F.Cu at (55.9, 203.2)
- added D201: BAT86,113, Diode_THT:D_DO-35_SOD27_P7.62mm_Horizontal, F.Cu at (66.0, 195.6)
- added D202: 1N4148, Diode_THT:D_DO-35_SOD27_P7.62mm_Horizontal, F.Cu at (39.4, 195.6)
- added R204: 3K3, Resistor_THT:R_Axial_DIN0207_L6.3mm_D2.5mm_P7.62mm_Horizontal, F.Cu at (47.0, 203.2)
- added SW201: Reset, Button_Switch_THT:SW_PUSH_6mm, F.Cu at (35.6, 226.1)
- added U204: DS1813, Package_TO_SOT_THT:TO-92_Inline, F.Cu at (61.0, 203.2)
Connections:
- U201 pad 17: unconnected-(U201-~{HALT}-Pad17) -> ~{HALT}
- U502 pad 15: (no net) -> unconnected-(U502-NC-Pad15)
- U502 pad 16: (no net) -> unconnected-(U502-NC-Pad16)
- U502 pad 37: (no net) -> unconnected-(U502-NC-Pad37)
- U502 pad 38: (no net) -> unconnected-(U502-NC-Pad38)
- U503 pad 15: (no net) -> unconnected-(U503-NC-Pad15)
- U503 pad 16: (no net) -> unconnected-(U503-NC-Pad16)
- U503 pad 37: (no net) -> unconnected-(U503-NC-Pad37)
- U503 pad 38: (no net) -> unconnected-(U503-NC-Pad38)
- U504 pad 15: (no net) -> unconnected-(U504-NC-Pad15)
- U504 pad 16: (no net) -> unconnected-(U504-NC-Pad16)
- U504 pad 37: (no net) -> unconnected-(U504-NC-Pad37)
- U504 pad 38: (no net) -> unconnected-(U504-NC-Pad38)
- U505 pad 15: (no net) -> unconnected-(U505-NC-Pad15)
- U505 pad 16: (no net) -> unconnected-(U505-NC-Pad16)
- U505 pad 37: (no net) -> unconnected-(U505-NC-Pad37)
- U505 pad 38: (no net) -> unconnected-(U505-NC-Pad38)
Other:
- board size 365.8 x 223.5 mm -> 370.8 x 223.5 mm
