File: cpu010/design-files/cpu010.kicad_pcb (KiCad board)
At the start: 2 copper layers, 370.8 x 223.5 mm, 122 parts, among them SW201 Reset, SW401 SW_DIP_x08, SW402 SW_DIP_x08, U101 GAL22V10, U201 MC68010P, U202 74ACT163, U203 74ACT05, U204 DS1813, U301 ATF1508AS-TQFP100, U302 61C3216, U303 74AHCT245, U304 74AHCT245, U305 7C4098, U306 7C4098, U307 74AHCT245, U308 74AHCT245, U309 74AHCT245, U310 74AHCT245, U311 74AHCT373, U312 74AHCT373, U313 74AHCT373, U314 74AHCT157, U315 74AHCT157, U316 74AHCT157, U317 74AHCT157, U318 74AHCT157, U319 74AHCT157, U320 74AHCT157, U321 74AHCT157, U322 74AHCT157, U323 74AHCT245, U324 74AHCT245, U401 DA04-11SURKWA, U402 74HCT273, U403 74HCT273, U404 GAL22V10, U405 74HC245, U406 74HC245, U407 74HCT273, U408 74HC245, U409 ATF1504AS-PLCC44, U501 GAL22V10, U502 CY62158, U503 CY62158, U504 CY62158, U505 CY62158, U506 SST39SF040, U507 SST39SF040, Y201 40MHz

Commit message: Getting a start at on-board i/o.
Parts:
- added BT601: CR1220, Battery:BatteryHolder_Keystone_500, F.Cu at (203.2, 50.6)
- added J601: UART0 FTDI, Connector_PinHeader_2.54mm:PinHeader_1x06_P2.54mm_Horizontal, F.Cu at (114.3, 40.6)
- added J602: UART1 FTDI, Connector_PinHeader_2.54mm:PinHeader_1x06_P2.54mm_Horizontal, F.Cu at (139.7, 40.6)
- added J603: UART0, Connector_IDC:IDC-Header_2x05_P2.54mm_Vertical, F.Cu at (116.8, 50.8)
- added J604: UART1, Connector_IDC:IDC-Header_2x05_P2.54mm_Vertical, F.Cu at (142.2, 50.8)
- added R601: 3K3, Resistor_SMD:R_0805_2012Metric_Pad1.20x1.40mm_HandSolder, F.Cu at (203.2, 64.5)
- added R602: 3K3, Resistor_SMD:R_0805_2012Metric_Pad1.20x1.40mm_HandSolder, F.Cu at (208.3, 64.5)
- added RN601: 3K3, Resistor_THT:R_Array_SIP9, F.Cu at (105.7, 36.3)
- added U601: ATF1508AS-TQFP100, Package_QFP:TQFP-100_14x14mm_P0.5mm, F.Cu at (236.9, 49.9)
- added U602: TL16C2552, Package_LCC:PLCC-44_THT-Socket, F.Cu at (91.4, 40.6)
- added U603: PCF8584, Package_DIP:DIP-20_W7.62mm_Socket, F.Cu at (215.6, 38.1)
- added U604: DS3231MZ+, Package_SO:SOIC-8_3.9x4.9mm_P1.27mm, F.Cu at (205.7, 58.4)
- added Y601: 1.8432MHz, Oscillator:Oscillator_DIP-8, F.Cu at (48.3, 48.3)
- R201: value 0R -> 3K3; footprint Resistor_THT:R_Axial_DIN0207_L6.3mm_D2.5mm_P7.62mm_Horizontal -> Resistor_SMD:R_0805_2012Metric_Pad1.20x1.40mm_HandSolder
- R204, R205: footprint Resistor_THT:R_Axial_DIN0207_L6.3mm_D2.5mm_P7.62mm_Horizontal -> Resistor_SMD:R_0805_2012Metric_Pad1.20x1.40mm_HandSolder
- moved R201 102.4 mm to (45.5, 100.6), turned to -90 degrees
- moved C101 33.1 mm to (243.8, 138.2)
- moved C205 33.1 mm to (117.1, 125.5)
- moved C301 33.1 mm to (94.2, 72.1)
- moved C303 33.1 mm to (140.0, 72.1)
- moved C305 33.1 mm to (140.0, 133.1)
- moved C306 33.1 mm to (157.7, 72.1)
- moved C308 33.1 mm to (173.0, 72.1)
- moved C310 33.1 mm to (190.8, 72.1)
- moved C311 33.1 mm to (190.8, 97.5)
- moved C315 33.1 mm to (226.1, 72.1)
- moved C316 33.1 mm to (226.1, 97.5)
- moved C319 33.1 mm to (243.8, 72.1)
- moved C322 33.1 mm to (210.1, 88.4)
- moved C324 33.1 mm to (210.1, 123.2)
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Connections:
- R201 pad 1: GND -> +5V
- R201 pad 2: Net-(R201-Pad2) -> ~{DTACK}
- U203 pad 8: unconnected-(U203-Pad8) -> ~{DTACK}
- U203 pad 9: Net-(R201-Pad2) -> IOCTL_DTACK
Other:
- board size 370.8 x 223.5 mm -> 370.8 x 185.4 mm
- board text added: "GND CTS (NC) TxD RxD RTS <-- FTDI GND RTS (NC) RxD RxD CTS <-- UART"
- board text added: "I/O Control"

Commit message: More layout.
Parts:
- added C412: 100nF, Capacitor_SMD:C_0805_2012Metric_Pad1.18x1.45mm_HandSolder, F.Cu at (255.0, 61.2)
- added C413: 100nF, Capacitor_SMD:C_0805_2012Metric_Pad1.18x1.45mm_HandSolder, F.Cu at (255.0, 68.8)
- added C414: 100nF, Capacitor_SMD:C_0805_2012Metric_Pad1.18x1.45mm_HandSolder, F.Cu at (263.7, 76.7)
- added C415: 100nF, Capacitor_SMD:C_0805_2012Metric_Pad1.18x1.45mm_HandSolder, F.Cu at (266.2, 76.7)
- added C416: 100nF, Capacitor_SMD:C_0805_2012Metric_Pad1.18x1.45mm_HandSolder, F.Cu at (276.4, 72.1)
- added C417: 100nF, Capacitor_SMD:C_0805_2012Metric_Pad1.18x1.45mm_HandSolder, F.Cu at (276.4, 64.8)
- added C418: 100nF, Capacitor_SMD:C_0805_2012Metric_Pad1.18x1.45mm_HandSolder, F.Cu at (268.7, 53.6)
- added C419: 100nF, Capacitor_SMD:C_0805_2012Metric_Pad1.18x1.45mm_HandSolder, F.Cu at (264.2, 53.6)
- added C601: 100nF, Capacitor_SMD:C_0805_2012Metric_Pad1.18x1.45mm_HandSolder, F.Cu at (141.7, 64.5)
- added C602: 100nF, Capacitor_SMD:C_0805_2012Metric_Pad1.18x1.45mm_HandSolder, F.Cu at (131.6, 48.0)
- added C603: 100nF, Capacitor_SMD:C_0805_2012Metric_Pad1.18x1.45mm_HandSolder, F.Cu at (82.0, 64.5)
- added C604: 100nF, Capacitor_SMD:C_0805_2012Metric_Pad1.18x1.45mm_HandSolder, F.Cu at (210.8, 54.4)
- added C605: 100nF, Capacitor_SMD:C_0805_2012Metric_Pad1.18x1.45mm_HandSolder, F.Cu at (223.5, 54.4)
- added C606: 100nF, Capacitor_SMD:C_0805_2012Metric_Pad1.18x1.45mm_HandSolder, F.Cu at (236.2, 54.4)
- added C607: 100nF, Capacitor_SMD:C_0805_2012Metric_Pad1.18x1.45mm_HandSolder, F.Cu at (248.9, 54.4)
- added D601: ATA Active, LED_SMD:LED_0805_2012Metric_Pad1.15x1.40mm_HandSolder, F.Cu at (264.2, 42.2)
- added H101: MountingHole, MountingHole:MountingHole_3.2mm_M3, F.Cu at (71.1, 33.0)
- added H102: MountingHole, MountingHole:MountingHole_3.2mm_M3, F.Cu at (71.1, 226.1)
- added H103: MountingHole, MountingHole:MountingHole_3.2mm_M3, F.Cu at (353.1, 33.0)
- added H104: MountingHole, MountingHole:MountingHole_3.2mm_M3, F.Cu at (353.1, 226.1)
- added J605: ATA Connector, Connector_IDC:IDC-Header_2x20_P2.54mm_Vertical, F.Cu at (208.3, 45.7)
- added J606: 5V CF Power, Connector_PinHeader_2.54mm:PinHeader_1x04_P2.54mm_Vertical, F.Cu at (271.3, 39.9)
- added J607: I2C, Connector_PinHeader_2.54mm:PinHeader_1x04_P2.54mm_Vertical, F.Cu at (317.5, 39.9)
- added R603: 47K, Resistor_SMD:R_0805_2012Metric_Pad1.20x1.40mm_HandSolder, F.Cu at (270.8, 53.6)
- added R604: 470R, Resistor_SMD:R_0805_2012Metric_Pad1.20x1.40mm_HandSolder, F.Cu at (264.2, 46.7)
- added U605: 74ACT245, Package_DIP:DIP-20_W7.62mm_Socket, F.Cu at (200.7, 53.3)
- added U606: 74ACT245, Package_DIP:DIP-20_W7.62mm_Socket, F.Cu at (213.4, 53.3)
- added U607: 74ACT245, Package_DIP:DIP-20_W7.62mm_Socket, F.Cu at (226.1, 53.3)
- moved BT601 101.4 mm to (304.5, 48.3)
- moved R601 89.3 mm to (288.3, 37.3)
- moved R602 89.3 mm to (293.4, 37.3)
- moved U604 87.6 mm to (292.1, 43.7)
- moved RN601 62.3 mm to (161.5, 63.8), turned to 0 degrees
- moved C202 41.3 mm to (83.8, 128.0)
- moved R201 41.3 mm to (83.8, 115.8)
- moved C509 41.0 mm to (304.8, 207.3)
- moved C511 41.0 mm to (324.6, 207.2)
- moved U101 41.0 mm to (271.5, 152.4)
- moved U320 41.0 mm to (253.7, 111.8)
- moved U322 41.0 mm to (253.7, 162.6)
- moved U324 41.0 mm to (271.5, 116.8)
- moved U502 41.0 mm to (295.9, 177.7)
- moved U503 41.0 mm to (315.7, 177.7)
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Connections:
- C330 pad 1: +5V -> GND
- C330 pad 2: GND -> +5V
- C331 pad 1: +5V -> GND
- C331 pad 2: GND -> +5V
- C404 pad 1: +5V -> GND
- C404 pad 2: GND -> +5V
- C405 pad 1: +5V -> GND
- C405 pad 2: GND -> +5V
- R204 pad 1: Net-(D202-A) -> +5V
- R204 pad 2: +5V -> Net-(D202-A)
- R205 pad 1: ~{RESET} -> +5V
- R205 pad 2: +5V -> ~{RESET}
- RN601 pad 2: /On-board IO/~{UARTA_RI} -> /On-board IO/~{UARTB_RI}
- RN601 pad 3: /On-board IO/~{UARTA_CD} -> /On-board IO/~{UARTB_CD}
- RN601 pad 4: /On-board IO/~{UARTA_DSR} -> /On-board IO/~{UARTB_DSR}
- RN601 pad 5: /On-board IO/~{UARTA_CTS} -> /On-board IO/~{UARTB_CTS}
- RN601 pad 6: /On-board IO/~{UARTB_RI} -> /On-board IO/~{UARTA_RI}
- RN601 pad 7: /On-board IO/~{UARTB_CD} -> /On-board IO/~{UARTA_CD}
- RN601 pad 8: /On-board IO/~{UARTB_DSR} -> /On-board IO/~{UARTA_DSR}
- RN601 pad 9: /On-board IO/~{UARTB_CTS} -> /On-board IO/~{UARTA_CTS}
- U601 pad 11: unconnected-(U601-GND-Pad11) -> GND
- U601 pad 18: unconnected-(U601-VCCio-Pad18) -> +5V
- U601 pad 26: unconnected-(U601-GND-Pad26) -> GND
- U601 pad 3: unconnected-(U601-VCCio-Pad3) -> +5V
- U601 pad 34: unconnected-(U601-VCCio-Pad34) -> +5V
- U601 pad 38: unconnected-(U601-GND-Pad38) -> GND
- U601 pad 39: unconnected-(U601-VCC-Pad39) -> +5V
- U601 pad 43: unconnected-(U601-GND-Pad43) -> GND
- U601 pad 51: unconnected-(U601-VCCio-Pad51) -> +5V
- U601 pad 59: unconnected-(U601-GND-Pad59) -> GND
- U601 pad 66: unconnected-(U601-VCCio-Pad66) -> +5V
- U601 pad 74: unconnected-(U601-GND-Pad74) -> GND
- U601 pad 82: unconnected-(U601-VCCio-Pad82) -> +5V
- U601 pad 86: unconnected-(U601-GND-Pad86) -> GND
- U601 pad 91: unconnected-(U601-VCC-Pad91) -> +5V
- U601 pad 95: unconnected-(U601-GND-Pad95) -> GND
Other:
- board size 370.8 x 185.4 mm -> 292.1 x 203.2 mm
- board text added: "<-- +5V"
- board text added: "<-- GND"
- board text added: "<-- RED"
- board text added: "<-- SDA"
- board text added: "GND CTS (NC) TxD RxD RTS <-- FTDI GND RTS (NC) RxD TxD CTS <-- UART"
- board text added: "UART0"
- board text added: "UART1"
- board text added: "phaethon 1"
- board text removed: "GND CTS (NC) TxD RxD RTS <-- FTDI GND RTS (NC) RxD RxD CTS <-- UART"

Commit message: We have 8MB RAM now.
Parts:
- added C512: 100nF, Capacitor_SMD:C_0805_2012Metric_Pad1.18x1.45mm_HandSolder, F.Cu at (291.1, 124.2)
- added C513: 100nF, Capacitor_SMD:C_0805_2012Metric_Pad1.18x1.45mm_HandSolder, F.Cu at (308.9, 125.0)
- added C514: 100nF, Capacitor_SMD:C_0805_2012Metric_Pad1.18x1.45mm_HandSolder, F.Cu at (310.9, 124.2)
- added C515: 100nF, Capacitor_SMD:C_0805_2012Metric_Pad1.18x1.45mm_HandSolder, F.Cu at (328.7, 125.0)
- added C516: 100nF, Capacitor_SMD:C_0805_2012Metric_Pad1.18x1.45mm_HandSolder, F.Cu at (291.1, 152.1)
- added C517: 100nF, Capacitor_SMD:C_0805_2012Metric_Pad1.18x1.45mm_HandSolder, F.Cu at (308.9, 152.9)
- added C518: 100nF, Capacitor_SMD:C_0805_2012Metric_Pad1.18x1.45mm_HandSolder, F.Cu at (310.9, 152.1)
- added C519: 100nF, Capacitor_SMD:C_0805_2012Metric_Pad1.18x1.45mm_HandSolder, F.Cu at (328.7, 152.9)
- added H105: MountingHole, MountingHole:MountingHole_3.2mm_M3, F.Cu at (205.7, 33.0)
- added H106: MountingHole, MountingHole:MountingHole_3.2mm_M3, F.Cu at (205.7, 226.1)
- added U508: CY62158, Package_SO:TSOP-II-44_10.16x18.41mm_P0.8mm, F.Cu at (300.0, 123.5)
- added U509: CY62158, Package_SO:TSOP-II-44_10.16x18.41mm_P0.8mm, F.Cu at (319.8, 123.5)
- added U510: CY62158, Package_SO:TSOP-II-44_10.16x18.41mm_P0.8mm, F.Cu at (300.0, 151.5)
- added U511: CY62158, Package_SO:TSOP-II-44_10.16x18.41mm_P0.8mm, F.Cu at (319.8, 151.5)
- U501: value GAL22V10 -> ATF1504AS-PLCC44; footprint Package_DIP:DIP-24_W7.62mm_Socket -> Package_LCC:PLCC-44_THT-Socket
- moved C502 27.9 mm to (307.1, 59.4)
- moved C503 27.9 mm to (328.7, 59.4)
- moved U506 27.9 mm to (289.3, 58.4)
- moved U507 27.9 mm to (310.9, 58.4)
- moved C501 5.92 mm to (287.0, 196.6)
- moved U501 5.80 mm to (274.3, 198.1)
- moved C504 4.44 mm to (291.1, 180.1)
- moved C506 4.43 mm to (310.9, 180.1)
- moved C510 4.43 mm to (310.9, 208.3)
- moved C505 4.43 mm to (308.9, 180.8)
- moved C507 4.43 mm to (328.7, 180.8)
- moved C509 4.43 mm to (308.9, 209.0)
- moved C511 4.43 mm to (328.7, 209.0)
- moved U502 4.43 mm to (300.0, 179.4)
- moved U503 4.43 mm to (319.8, 179.4)
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Connections:
- U501 pad 1: ~{UDS} -> unconnected-(U501-I/GCLR-Pad1)
- U501 pad 10: A25 -> GND
- U501 pad 12: GND -> unconnected-(U501-I/O-Pad12)
- U501 pad 14: /On-board memory/OBMEM_nA1 -> unconnected-(U501-I/O-Pad14)
- U501 pad 15: /On-board memory/~{RAMUR} -> +5V
- U501 pad 16: /On-board memory/~{RAMLR} -> unconnected-(U501-I/O-Pad16)
- U501 pad 17: /On-board memory/~{RAMUW} -> unconnected-(U501-I/O-Pad17)
- U501 pad 18: /On-board memory/~{RAMLW} -> unconnected-(U501-I/O-Pad18)
- U501 pad 19: /On-board memory/~{ROMUR} -> unconnected-(U501-I/O-Pad19)
- U501 pad 2: ~{LDS} -> unconnected-(U501-I/OE2/GCLK2-Pad2)
- U501 pad 20: /On-board memory/~{ROMLR} -> unconnected-(U501-I/O-Pad20)
- U501 pad 21: /On-board memory/~{ROMUW} -> unconnected-(U501-I/O-Pad21)
- U501 pad 22: /On-board memory/~{ROMLW} -> GND
- U501 pad 23: OBMEM_DTACK -> +5V
- U501 pad 24: +5V -> unconnected-(U501-I/O-Pad24)
- U501 pad 3: R/~{W} -> +5V
- U501 pad 4: ~{RAMSEL} -> unconnected-(U501-I/O-Pad4)
- U501 pad 5: ~{ROMSEL} -> unconnected-(U501-I/O-Pad5)
- U501 pad 6: A1 -> unconnected-(U501-I/O-Pad6)
- U501 pad 7: A22 -> unconnected-(U501-I/O/TDI-Pad7)
- U501 pad 8: A23 -> unconnected-(U501-I/O-Pad8)
- U501 pad 9: A24 -> unconnected-(U501-I/O-Pad9)
- U502 pad 17: /On-board memory/~{RAMUW} -> /On-board memory/~{RAM0UW}
- U502 pad 40: /On-board memory/OBMEM_nA1 -> +5V
- U502 pad 41: /On-board memory/~{RAMUR} -> /On-board memory/~{RAM0UR}
- U503 pad 17: /On-board memory/~{RAMLW} -> /On-board memory/~{RAM0LW}
- U503 pad 40: /On-board memory/OBMEM_nA1 -> +5V
- U503 pad 41: /On-board memory/~{RAMLR} -> /On-board memory/~{RAM0LR}
- U504 pad 17: /On-board memory/~{RAMUW} -> /On-board memory/~{RAM2UW}
- U504 pad 40: A1 -> +5V
- U504 pad 41: /On-board memory/~{RAMUR} -> /On-board memory/~{RAM2UR}
- U505 pad 17: /On-board memory/~{RAMLW} -> /On-board memory/~{RAM2LW}
- U505 pad 40: A1 -> +5V
- U505 pad 41: /On-board memory/~{RAMLR} -> /On-board memory/~{RAM2LR}
Other:
- board text added: "0-2MB"
- board text added: "2-4MB"
- board text added: "4-6MB"
- board text added: "6-8MB"
- board text added: "Memory Interface Logic"
- board text added: "Rev A Made by @thorpej. https://github.com/thorpej/pg68k/"
- board text added: "System RAM"
- board text removed: "(Lower word)"
- board text removed: "(Upper word)"
- board text removed: "4MB RAM"
- board text removed: "On-board Memory Interface Logic"

Commit message: Add board design constraints.
Other:
- copper layers 2 -> 4
Changed lines of the file:
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@@
 	(layers
 		(0 "F.Cu" signal)
+		(4 "In1.Cu" power)
+		(6 "In2.Cu" power)
 		(2 "B.Cu" signal)
 		(9 "F.Adhes" user "F.Adhesive")
@@
 	)
 	(setup
+		(stackup
+			(layer "F.SilkS"
+				(type "Top Silk Screen")
+			)
+			(layer "F.Paste"
+				(type "Top Solder Paste")
+			)
+			(layer "F.Mask"
+				(type "Top Solder Mask")
+				(thickness 0.01)
+			)
+			(layer "F.Cu"
+				(type "copper")
+				(thickness 0.035)
+			)
+			(layer "dielectric 1"
+				(type "prepreg")
+				(thickness 0.1)
+				(material "FR4")
+				(epsilon_r 4.5)
+				(loss_tangent 0.02)
+			)
+			(layer "In1.Cu"
+				(type "copper")
+				(thickness 0.035)
+			)
+			(layer "dielectric 2"
+				(type "core")
+				(thickness 1.24)
+				(material "FR4")
+				(epsilon_r 4.5)
+				(loss_tangent 0.02)
+			)
+			(layer "In2.Cu"
+				(type "copper")
+				(thickness 0.035)
+			)
+			(layer "dielectric 3"
+				(type "prepreg")
+				(thickness 0.1)
+				(material "FR4")
+				(epsilon_r 4.5)
+				(loss_tangent 0.02)
+			)
+			(layer "B.Cu"
+				(type "copper")
+				(thickness 0.035)
+			)
+			(layer "B.Mask"
+				(type "Bottom Solder Mask")
+				(thickness 0.01)
+			)
+			(layer "B.Paste"
+				(type "Bottom Solder Paste")
+			)
+			(layer "B.SilkS"
+				(type "Bottom Silk Screen")
+			)
+			(copper_finish "None")
+			(dielectric_constraints no)
+		)
 		(pad_to_mask_clearance 0)
 		(allow_soldermask_bridges_in_footprints no)
