File: cpu010/design-files/cpu010.kicad_pcb (KiCad board)
At the start: 4 copper layers, 292.1 x 203.2 mm, 177 parts, among them J601 UART0 FTDI, J602 UART1 FTDI, J603 UART0, J604 UART1, J605 ATA Connector, J606 5V CF Power, J607 I2C, SW201 Reset, SW401 SW_DIP_x08, SW402 SW_DIP_x08, U101 GAL22V10, U201 MC68010P, U202 74ACT163, U203 74ACT05, U204 DS1813, U301 ATF1508AS-TQFP100, U302 61C3216, U303 74AHCT245, U304 74AHCT245, U305 7C4098, U306 7C4098, U307 74AHCT245, U308 74AHCT245, U309 74AHCT245, U310 74AHCT245, U311 74AHCT373, U312 74AHCT373, U313 74AHCT373, U314 74AHCT157, U315 74AHCT157, U316 74AHCT157, U317 74AHCT157, U318 74AHCT157, U319 74AHCT157, U320 74AHCT157, U321 74AHCT157, U322 74AHCT157, U323 74AHCT245, U324 74AHCT245, U401 DA04-11SURKWA, U402 74HCT273, U403 74HCT273, U404 GAL22V10, U405 74HC245, U406 74HC245, U407 74HCT273, U408 74HC245, U409 ATF1504AS-PLCC44, U501 ATF1504AS-PLCC44, U502 CY62158, U503 CY62158, U504 CY62158, U505 CY62158, U506 SST39SF040, U507 SST39SF040, U508 CY62158, U509 CY62158, U510 CY62158, U511 CY62158, U601 ATF1508AS-TQFP100, U602 TL16C2552, U603 PCF8584, U604 DS3231MZ+, U605 74ACT245, U606 74ACT245, U607 74ACT245, Y201 40MHz, Y601 1.8432MHz

Commit message: Route some bypass caps and the diagnostic display.
Parts:
- added C608: 100nF, Capacitor_SMD:C_0805_2012Metric_Pad1.18x1.45mm_HandSolder, F.Cu at (287.0, 43.9)
Routing:
- net +5V: track 0.00 -> 106.1 mm, vias 0 -> 4
- net ~{HALT}: track 0.00 -> 61.8 mm, vias 0 -> 2
- net Net-(RN402-R8.2): track 0.00 -> 41.4 mm, vias 0 -> 2
- net Net-(RN401-R8.2): track 0.00 -> 39.3 mm, vias 0 -> 1
- net Net-(RN401-R3.1): track 0.00 -> 38.1 mm, vias 0 -> 1
- net Net-(RN401-R5.2): track 0.00 -> 35.2 mm, vias 0 -> 1
- net Net-(RN402-R4.1): track 0.00 -> 34.9 mm, vias 0 -> 1
- net Net-(RN402-R5.2): track 0.00 -> 33.9 mm, vias 0 -> 1
- net Net-(RN402-R6.1): track 0.00 -> 33.4 mm, vias 0 -> 1
- net Net-(RN401-R7.1): track 0.00 -> 33.1 mm, vias 0 -> 1
- net Net-(D202-A): track 0.00 -> 31.7 mm, vias 0 -> 1
- net /On-board IO/SCL: track 0.00 -> 31.7 mm
- net Net-(RN402-R7.2): track 0.00 -> 31.6 mm, vias 0 -> 2
- net /On-board IO/SDA: track 0.00 -> 31.5 mm
- net Net-(RN402-R3.1): track 0.00 -> 31.1 mm, vias 0 -> 1
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Other:
- board text added: "<-- SCL"

Commit message: More power traces for SMT components.
Routing:
- net GND: track 3.13 -> 125.3 mm, vias 2 -> 41
- net +5V: track 106.1 -> 219.2 mm, vias 4 -> 26

Commit message: Serial port connectors.
Routing:
- net /On-board IO/~{UARTA_CTS}: track 0.00 -> 34.2 mm, vias 0 -> 1
- net /On-board IO/~{UARTB_CTS}: track 0.00 -> 33.8 mm, vias 0 -> 1
- net /On-board IO/~{UARTB_RTS}: track 0.00 -> 24.7 mm, vias 0 -> 2
- net /On-board IO/~{UARTA_RTS}: track 0.00 -> 24.7 mm, vias 0 -> 2
- net /On-board IO/~{UARTA_RI}: track 0.00 -> 22.9 mm, vias 0 -> 1
- net /On-board IO/UARTB_TXD: track 0.00 -> 22.0 mm, vias 0 -> 2
- net /On-board IO/UARTA_TXD: track 0.00 -> 22.0 mm, vias 0 -> 2
- net /On-board IO/UARTB_RXD: track 0.00 -> 20.0 mm, vias 0 -> 2
- net /On-board IO/UARTA_RXD: track 0.00 -> 20.0 mm, vias 0 -> 2
- net /On-board IO/~{UARTB_CD}: track 0.00 -> 18.7 mm, vias 0 -> 1
- net /On-board IO/~{UARTA_DSR}: track 0.00 -> 17.7 mm, vias 0 -> 1
- net /On-board IO/~{UARTB_DSR}: track 0.00 -> 17.6 mm, vias 0 -> 1
- net /On-board IO/~{UARTA_CD}: track 0.00 -> 10.4 mm, vias 0 -> 1
- net /On-board IO/~{UARTB_RI}: track 0.00 -> 8.29 mm

Commit message: Oscillator outputs.
Routing:
- net Net-(U602-XIN): track 0.00 -> 28.7 mm, vias 0 -> 1
- net Net-(U202-CP): track 0.00 -> 8.67 mm
Changed lines of the file:
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@@
+	)
+	(segment
+		(start 99.06 73.66)
+		(end 101.6 71.12)
+		(width 0.1)
+		(layer "F.Cu")
+		(net 244)
+	)
+	(segment
+		(start 93.98 73.66)
+		(end 99.06 73.66)
+		(width 0.1)
+		(layer "F.Cu")
+		(net 244)
 	)
 	(segment
@@
 	)
 	(segment
+		(start 116.332 55.88)
+		(end 117.602 57.15)
+		(width 0.1)
+		(layer "F.Cu")
+		(net 491)
+	)
+	(segment
+		(start 93.98 55.88)
+		(end 116.332 55.88)
+		(width 0.1)
+		(layer "F.Cu")
+		(net 491)
+	)
+	(via
+		(at 117.602 57.15)
+		(size 0.35)
+		(drill 0.2)
+		(layers "F.Cu" "B.Cu")
+		(net 491)
+	)
+	(segment
+		(start 117.602 59.182)
+		(end 119.38 60.96)
+		(width 0.1)
+		(layer "B.Cu")
+		(net 491)
+	)
+	(segment
+		(start 117.602 57.15)
+		(end 117.602 59.182)
+		(width 0.1)
+		(layer "B.Cu")
+		(net 491)
+	)
+	(segment

Commit message: Route configuration register.
Routing:
- net Net-(RN404-R1): track 0.00 -> 56.9 mm
- net Net-(RN404-R2): track 0.00 -> 54.6 mm, vias 0 -> 1
- net Net-(RN404-R8): track 0.00 -> 53.3 mm, vias 0 -> 1
- net Net-(RN404-R5): track 0.00 -> 53.2 mm, vias 0 -> 1
- net Net-(RN404-R7): track 0.00 -> 53.2 mm, vias 0 -> 1
- net Net-(RN404-R4): track 0.00 -> 53.2 mm, vias 0 -> 1
- net Net-(RN404-R3): track 0.00 -> 53.2 mm, vias 0 -> 1
- net Net-(RN404-R6): track 0.00 -> 53.2 mm, vias 0 -> 1
- net Net-(RN403-R1): track 0.00 -> 49.3 mm
- net Net-(RN403-R7): track 0.00 -> 47.5 mm, vias 0 -> 1
- net Net-(RN403-R4): track 0.00 -> 47.5 mm, vias 0 -> 1
- net Net-(RN403-R8): track 0.00 -> 47.4 mm, vias 0 -> 1
- net Net-(RN403-R6): track 0.00 -> 47.4 mm, vias 0 -> 1
- net Net-(RN403-R5): track 0.00 -> 47.2 mm, vias 0 -> 1
- net Net-(RN403-R3): track 0.00 -> 47.2 mm, vias 0 -> 1
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
Commit message: Route some more signals, but might have to roll some of this back because berr010 isn't fitting in the 1504.
Routing:
- net R/~{W}: track 0.00 -> 236.3 mm, vias 0 -> 3
- net ~{CPU_LDS}: track 0.00 -> 113.3 mm, vias 0 -> 2
- net ~{CPU_UDS}: track 0.00 -> 108.8 mm, vias 0 -> 1
- net /Control Space/~{CSLSEL}: track 0.00 -> 99.3 mm, vias 0 -> 1
- net /Control Space/~{ERWR}: track 0.00 -> 94.6 mm, vias 0 -> 1
- net /Control Space/~{CSUSEL}: track 0.00 -> 80.1 mm, vias 0 -> 2
- net /Control Space/~{DDLSEL}: track 0.00 -> 78.9 mm, vias 0 -> 1
- net /Control Space/~{ERRD}: track 0.00 -> 70.0 mm, vias 0 -> 1
- net /Control Space/~{DDUSEL}: track 0.00 -> 64.3 mm, vias 0 -> 2
- net FC0: track 0.00 -> 41.4 mm, vias 0 -> 1
- net FC2: track 0.00 -> 40.2 mm, vias 0 -> 2
- net VA3: track 0.00 -> 36.6 mm
- net FC1: track 0.00 -> 36.6 mm
- net VA4: track 0.00 -> 36.6 mm
- net VA2: track 0.00 -> 36.6 mm
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
Commit message: Routing some I/O stuff.
Parts:
- removed C101: 100nF, Capacitor_SMD:C_0805_2012Metric_Pad1.18x1.45mm_HandSolder
- removed U101: GAL22V10, Package_DIP:DIP-24_W7.62mm_Socket
- added R605: 3K3, Resistor_SMD:R_0805_2012Metric_Pad1.20x1.40mm_HandSolder, F.Cu at (1.88, 0.97)
- added R606: 3K3, Resistor_SMD:R_0805_2012Metric_Pad1.20x1.40mm_HandSolder, F.Cu at (1.88, 3.92)
- added R607: 3K3, Resistor_SMD:R_0805_2012Metric_Pad1.20x1.40mm_HandSolder, F.Cu at (1.88, 6.88)
- added R608: 3K3, Resistor_SMD:R_0805_2012Metric_Pad1.20x1.40mm_HandSolder, F.Cu at (1.88, 9.82)
- added R609: 3K3, Resistor_SMD:R_0805_2012Metric_Pad1.20x1.40mm_HandSolder, F.Cu at (1.88, 12.8)
- added RN602: 3K3, Resistor_THT:R_Array_SIP9, F.Cu at (281.9, 58.4)
Connections:
- J605 pad 32: /On-board IO/~{ATA_IO16} -> unconnected-(J605-Pin_32-Pad32)
- U501 pad 1: unconnected-(U501-I/GCLR-Pad1) -> ~{AS}
- U501 pad 11: unconnected-(U501-I/O/PD1-Pad11) -> FC2
- U501 pad 12: unconnected-(U501-I/O-Pad12) -> A21
- U501 pad 14: unconnected-(U501-I/O-Pad14) -> A22
- U501 pad 16: unconnected-(U501-I/O-Pad16) -> A23
- U501 pad 17: unconnected-(U501-I/O-Pad17) -> A24
- U501 pad 18: unconnected-(U501-I/O-Pad18) -> A25
- U501 pad 19: unconnected-(U501-I/O-Pad19) -> A26
- U501 pad 2: unconnected-(U501-I/OE2/GCLK2-Pad2) -> ~{UDS}
- U501 pad 20: unconnected-(U501-I/O-Pad20) -> A27
- U501 pad 21: unconnected-(U501-I/O-Pad21) -> /On-board memory/~{OBMEM_URD}
- U501 pad 24: unconnected-(U501-I/O-Pad24) -> /On-board memory/~{OBMEM_UWR}
- U501 pad 25: unconnected-(U501-I/O/PD2-Pad25) -> /On-board memory/~{OBMEM_LRD}
- U501 pad 26: unconnected-(U501-I/O-Pad26) -> /On-board memory/~{OBMEM_LWR}
- U501 pad 27: unconnected-(U501-I/O-Pad27) -> /On-board memory/~{OBMEM_ROMSEL}
- U501 pad 28: unconnected-(U501-I/O-Pad28) -> /On-board memory/~{OBMEM_RAM0SEL}
- U501 pad 29: unconnected-(U501-I/O-Pad29) -> /On-board memory/~{OBMEM_RAM1SEL}
- U501 pad 31: unconnected-(U501-I/O-Pad31) -> /On-board memory/~{OBMEM_RAM2SEL}
- U501 pad 33: unconnected-(U501-I/O-Pad33) -> /On-board memory/~{OBMEM_RAM3SEL}
- U501 pad 34: unconnected-(U501-I/O-Pad34) -> ~{EXPRAMSEL}
- U501 pad 4: unconnected-(U501-I/O-Pad4) -> ~{LDS}
- U501 pad 40: unconnected-(U501-I/O-Pad40) -> OBMEM_DTACK
- U501 pad 5: unconnected-(U501-I/O-Pad5) -> R/~{W}
- U501 pad 6: unconnected-(U501-I/O-Pad6) -> MMU_EN
- U501 pad 8: unconnected-(U501-I/O-Pad8) -> FC0
- U501 pad 9: unconnected-(U501-I/O-Pad9) -> FC1
- U601 pad 1: unconnected-(U601-I/O/PD1-Pad1) -> IOCTL_DTACK
- U601 pad 10: unconnected-(U601-I/O-Pad10) -> FC0
- U601 pad 100: unconnected-(U601-I/O-Pad100) -> ~{AVEC}
- U601 pad 12: unconnected-(U601-I/O-Pad12) -> FC1
- U601 pad 13: unconnected-(U601-I/O-Pad13) -> FC2
- U601 pad 14: unconnected-(U601-I/O-Pad14) -> IPL0
- U601 pad 16: unconnected-(U601-I/O-Pad16) -> IPL1
- U601 pad 17: unconnected-(U601-I/O-Pad17) -> IPL2
- U601 pad 19: unconnected-(U601-I/O-Pad19) -> D8
- U601 pad 2: unconnected-(U601-I/O-Pad2) -> /On-board IO/IO_RST
- U601 pad 20: unconnected-(U601-I/O-Pad20) -> D9
- U601 pad 21: unconnected-(U601-I/O-Pad21) -> D10
- U601 pad 22: unconnected-(U601-I/O-Pad22) -> D11
- U601 pad 23: unconnected-(U601-I/O-Pad23) -> D12
- U601 pad 24: unconnected-(U601-I/O-Pad24) -> D13
- U601 pad 25: unconnected-(U601-I/O-Pad25) -> D14
- U601 pad 27: unconnected-(U601-I/O-Pad27) -> D15
- U601 pad 28: unconnected-(U601-I/O-Pad28) -> VA1
- U601 pad 29: unconnected-(U601-I/O-Pad29) -> VA2
- U601 pad 30: unconnected-(U601-I/O-Pad30) -> VA3
- U601 pad 31: unconnected-(U601-I/O-Pad31) -> VA4
- U601 pad 32: unconnected-(U601-I/O-Pad32) -> VA5
- U601 pad 33: unconnected-(U601-I/O-Pad33) -> VA6
- U601 pad 35: unconnected-(U601-I/O-Pad35) -> VA7
- U601 pad 36: unconnected-(U601-I/O-Pad36) -> VA8
- U601 pad 37: unconnected-(U601-I/O-Pad37) -> VA9
- U601 pad 40: unconnected-(U601-I/O-Pad40) -> VA10
- U601 pad 41: unconnected-(U601-I/O/PD2-Pad41) -> VA11
- U601 pad 42: unconnected-(U601-I/O-Pad42) -> A26
- U601 pad 44: unconnected-(U601-I/O-Pad44) -> A27
- U601 pad 45: unconnected-(U601-I/O-Pad45) -> VA16
- U601 pad 46: unconnected-(U601-I/O-Pad46) -> VA17
- U601 pad 47: unconnected-(U601-I/O-Pad47) -> VA18
- U601 pad 48: unconnected-(U601-I/O-Pad48) -> VA19
- U601 pad 5: unconnected-(U601-I/O-Pad5) -> ~{AS}
- U601 pad 6: unconnected-(U601-I/O-Pad6) -> R/~{W}
- U601 pad 7: unconnected-(U601-I/O-Pad7) -> ~{UDS}
- U601 pad 76: unconnected-(U601-I/O-Pad76) -> ~{EXPSEL}
- U601 pad 77: unconnected-(U601-I/O-Pad77) -> /On-board IO/~{I2CSEL}
- U601 pad 78: unconnected-(U601-I/O-Pad78) -> /On-board IO/~{ATABEN}
- U601 pad 79: unconnected-(U601-I/O-Pad79) -> /On-board IO/~{ATASEL}
- U601 pad 8: unconnected-(U601-I/O-Pad8) -> ~{LDS}
- U601 pad 80: unconnected-(U601-I/O-Pad80) -> /On-board IO/~{ATAAUXSEL}
- U601 pad 81: unconnected-(U601-I/O-Pad81) -> /On-board IO/ATA_INT
- U601 pad 83: unconnected-(U601-I/O-Pad83) -> /On-board IO/~{DUARTSEL}
- U601 pad 84: unconnected-(U601-I/O-Pad84) -> /On-board IO/UARTA_INT
- U601 pad 85: unconnected-(U601-I/O/GCLK3-Pad85) -> /On-board IO/UARTB_INT
- U601 pad 87: unconnected-(U601-I/GCLK1-Pad87) -> CLK10
- U601 pad 89: unconnected-(U601-I/GCLR-Pad89) -> ~{RESET}
- U601 pad 92: unconnected-(U601-I/O-Pad92) -> ~{IRQ3}
- U601 pad 93: unconnected-(U601-I/O-Pad93) -> ~{IRQ4}
- U601 pad 94: unconnected-(U601-I/O-Pad94) -> ~{IRQ5}
- U601 pad 96: unconnected-(U601-I/O-Pad96) -> ~{IRQ6}
- U601 pad 97: unconnected-(U601-I/O-Pad97) -> ~{IRQ7}
- U601 pad 98: unconnected-(U601-I/O-Pad98) -> /On-board IO/~{IO_RD}
- U601 pad 99: unconnected-(U601-I/O-Pad99) -> /On-board IO/~{IO_WR}
- U602 pad 10: A1 -> VA1
- U602 pad 14: A2 -> VA2
- U602 pad 15: A3 -> VA3
- U602 pad 16: A8 -> VA8
- U603 pad 6: A1 -> VA1
- U605 pad 11: D15 -> D7
- U605 pad 12: D14 -> D6
- U605 pad 13: D13 -> D5
- U605 pad 14: D12 -> D4
- U605 pad 15: D11 -> D3
- U605 pad 16: D10 -> D2
- U605 pad 17: D9 -> D1
- U605 pad 18: D8 -> D0
- U605 pad 2: /On-board IO/ATA_D0 -> /On-board IO/ATA_D8
- U605 pad 3: /On-board IO/ATA_D1 -> /On-board IO/ATA_D9
- U605 pad 4: /On-board IO/ATA_D2 -> /On-board IO/ATA_D10
- U605 pad 5: /On-board IO/ATA_D3 -> /On-board IO/ATA_D11
- U605 pad 6: /On-board IO/ATA_D4 -> /On-board IO/ATA_D12
- U605 pad 7: /On-board IO/ATA_D5 -> /On-board IO/ATA_D13
- U605 pad 8: /On-board IO/ATA_D6 -> /On-board IO/ATA_D14
- U605 pad 9: /On-board IO/ATA_D7 -> /On-board IO/ATA_D15
- U606 pad 11: D7 -> D15
- U606 pad 12: D6 -> D14
- U606 pad 13: D5 -> D13
- U606 pad 14: D4 -> D12
- U606 pad 15: D3 -> D11
- U606 pad 16: D2 -> D10
- U606 pad 17: D1 -> D9
- U606 pad 18: D0 -> D8
- U606 pad 2: /On-board IO/ATA_D8 -> /On-board IO/ATA_D0
- U606 pad 3: /On-board IO/ATA_D9 -> /On-board IO/ATA_D1
- U606 pad 4: /On-board IO/ATA_D10 -> /On-board IO/ATA_D2
- U606 pad 5: /On-board IO/ATA_D11 -> /On-board IO/ATA_D3
- U606 pad 6: /On-board IO/ATA_D12 -> /On-board IO/ATA_D4
- U606 pad 7: /On-board IO/ATA_D13 -> /On-board IO/ATA_D5
- U606 pad 8: /On-board IO/ATA_D14 -> /On-board IO/ATA_D6
- U606 pad 9: /On-board IO/ATA_D15 -> /On-board IO/ATA_D7
- U607 pad 11: unconnected-(U607-B7-Pad11) -> /On-board IO/~{IO_WR}
- U607 pad 12: unconnected-(U607-B6-Pad12) -> /On-board IO/~{IO_RD}
- U607 pad 13: unconnected-(U607-B5-Pad13) -> ~{RESET}
- U607 pad 14: unconnected-(U607-B4-Pad14) -> VA3
- U607 pad 15: unconnected-(U607-B3-Pad15) -> VA2
- U607 pad 16: unconnected-(U607-B2-Pad16) -> VA1
- U607 pad 17: unconnected-(U607-B1-Pad17) -> /On-board IO/~{ATAAUXSEL}
- U607 pad 18: unconnected-(U607-B0-Pad18) -> /On-board IO/~{ATASEL}
- U607 pad 2: unconnected-(U607-A0-Pad2) -> /On-board IO/~{ATA_CS1FX}
- U607 pad 3: unconnected-(U607-A1-Pad3) -> /On-board IO/~{ATA_CS3FX}
- U607 pad 4: unconnected-(U607-A2-Pad4) -> /On-board IO/ATA_A0
- U607 pad 5: unconnected-(U607-A3-Pad5) -> /On-board IO/ATA_A1
- U607 pad 6: unconnected-(U607-A4-Pad6) -> /On-board IO/ATA_A2
- U607 pad 7: unconnected-(U607-A5-Pad7) -> /On-board IO/~{ATA_RST}
- U607 pad 8: unconnected-(U607-A6-Pad8) -> /On-board IO/~{ATA_IORD}
- U607 pad 9: unconnected-(U607-A7-Pad9) -> /On-board IO/~{ATA_IOWR}
Routing:
- net /On-board IO/SCL: track 31.7 -> 102.4 mm, vias 0 -> 4
- net /On-board IO/SDA: track 31.5 -> 97.1 mm, vias 0 -> 2
- net /On-board IO/~{UARTA_RTS}: track 24.7 -> 81.0 mm, vias 2 -> 3
- net /On-board IO/~{UARTA_CTS}: track 34.2 -> 90.5 mm, vias 1 -> 2
- net /On-board IO/ATA_D15: track 0.00 -> 55.4 mm, vias 0 -> 2
- net /On-board IO/~{UARTA_DSR}: track 17.7 -> 72.0 mm, vias 1 -> 2
- net ~{IRQ3}: track 0.00 -> 53.7 mm, vias 0 -> 5
- net /On-board IO/~{UARTA_DTR}: track 0.00 -> 53.2 mm, vias 0 -> 1
- net /On-board IO/ATA_D14: track 0.00 -> 50.6 mm, vias 0 -> 2
- net /On-board IO/UARTA_RXD: track 20.0 -> 70.4 mm, vias 2 -> 3
- net /On-board IO/~{UARTA_CD}: track 10.4 -> 60.7 mm, vias 1 -> 2
- net /On-board IO/UARTA_TXD: track 22.0 -> 71.3 mm
- net /On-board IO/ATA_A2: track 0.00 -> 49.3 mm, vias 0 -> 1
- net /On-board IO/~{UARTB_RTS}: track 24.7 -> 73.8 mm, vias 2 -> 3
- net /On-board IO/~{UARTA_RI}: track 22.9 -> 70.4 mm, vias 1 -> 2
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Other:
- board text removed: "Top-level Address Decoding"

Commit message: Expansion slots!
Parts:
- removed R605, R606, R607, R608, R609: 3K3, Resistor_SMD:R_0805_2012Metric_Pad1.20x1.40mm_HandSolder
- added H107: MountingHole, MountingHole:MountingHole_3.2mm_M3, F.Cu at (462.3, 190.5)
- added H108: MountingHole, MountingHole:MountingHole_3.2mm_M3, F.Cu at (76.2, 190.5)
- added H109: MountingHole, MountingHole:MountingHole_3.2mm_M3, F.Cu at (353.1, 190.5)
- added H110: MountingHole, MountingHole:MountingHole_3.2mm_M3, F.Cu at (353.1, 94.0)
- added H111: MountingHole, MountingHole:MountingHole_3.2mm_M3, F.Cu at (353.1, 287.0)
- added H112: MountingHole, MountingHole:MountingHole_3.2mm_M3, F.Cu at (205.7, 94.0)
- added J701: Expansion Slot 1, Connector_DIN:DIN41612_C_3x32_Female_Vertical_THT, F.Cu at (373.4, 149.9)
- added J702: Expansion Slot 2, Connector_DIN:DIN41612_C_3x32_Female_Vertical_THT, F.Cu at (403.9, 149.9)
- added J703: Expansion Slot 3, Connector_DIN:DIN41612_C_3x32_Female_Vertical_THT, F.Cu at (434.3, 149.9)
- added U701: 74ACT245, Package_DIP:DIP-20_W7.62mm_Socket, F.Cu at (337.8, 172.7)
- added U702: 74ACT245, Package_DIP:DIP-20_W7.62mm_Socket, F.Cu at (337.8, 142.2)
- added U703: 74HC08, Package_DIP:DIP-14_W7.62mm_Socket, F.Cu at (337.8, 119.4)
- U319, U320, U321, U322: value 74AHCT157 -> 74ACT157
- U323, U324: value 74AHCT245 -> 74ACT245
- moved H103 125.1 mm to (462.3, 94.0)
- moved H104 125.1 mm to (462.3, 287.0)
- moved H105 88.0 mm to (269.2, 94.0)
- moved H106 88.0 mm to (269.2, 287.0)
- moved C319 61.2 mm to (286.8, 148.3)
- moved C320 61.2 mm to (286.8, 178.8)
- moved C414 61.2 mm to (268.7, 137.7)
- moved C416 61.2 mm to (281.4, 133.1)
- moved C417 61.2 mm to (281.4, 125.7)
- moved C517 61.2 mm to (313.9, 213.9)
- moved U509 61.2 mm to (324.9, 184.5)
- moved U510 61.2 mm to (305.1, 212.5)
- moved C608 61.2 mm to (292.1, 104.9)
- moved C201 61.2 mm to (100.1, 246.4)
- moved C202 61.2 mm to (88.9, 189.0)
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Connections:
- net /On-board IO/SCL renamed SCL
- net /On-board IO/SDA renamed SDA
Other:
- board size 292.1 x 203.2 mm -> 396.2 x 203.2 mm
