File: cpu010/design-files/cpu010-cpu.kicad_sch (KiCad schematic)
At the start: 1 part, among them U201 MC68010P

Commit message: Add clock generator.
Parts:
- added U202: 74ACT163, Package_DIP:DIP-16_W7.62mm_Socket, symbol 74xx:74LS163
- added Y201: 40MHz, Oscillator:Oscillator_DIP-8, symbol Oscillator:CXO_DIP8
- U201: footprint Package_DIP:DIP-64_W22.86mm -> Package_DIP:DIP-64_W22.86mm_Socket
Connections:
- net CLK10: now also U202.13 (Q1)
- net +5V: now reaches U201.14 (V_{CC}), U201.49 (V_{CC})
- net +5V: now also U202.1 (~{MR}), U202.10 (CET), U202.16 (VCC), U202.7 (CEP), U202.9 (~{PE}), Y201.1 (EN), Y201.8 (Vcc)
- net GND: now reaches U201.16 (GND), U201.53 (GND)
- net GND: now also U202.3 (D0), U202.4 (D1), U202.5 (D2), U202.6 (D3), U202.8 (GND), Y201.4 (GND)
- new net: U202.2 (CP), Y201.5 (OUT)
- new net CLK20: U202.14 (Q0)
- no-connect marks 0 -> 3
Other:
- moved on the sheet: U201

Commit message: Wire up Bus Error register.
Connections:
- net ~{RESET}: now reaches U201.18 (~{RESET})
- net ~{CPU_BERR}: now reaches U201.22 (~{BERR})
Changed lines of the file:
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@@
+		)
+	)
+	(global_label "~{CPU_BERR}"
+		(shape input)
+		(at 29.21 118.11 180)
+		(fields_autoplaced yes)
+		(effects
+			(font
+				(size 1.27 1.27)
+			)
+			(justify right)
+		)
+		(property "Intersheetrefs" "${INTERSHEET_REFS}"
+			(at 16.4277 118.11 0)
+			(effects
+				(font
+					(size 1.27 1.27)
+				)
+				(justify right)
+				(hide yes)
+			)
 		)
 	)
@@
 				(hide yes)
 			)
+		)
+	)
+	(global_label "~{RESET}"
+		(shape input)
+		(at 29.21 125.73 180)
+		(fields_autoplaced yes)
+		(effects
+			(font
+				(size 1.27 1.27)
+			)
+			(justify right)
+		)
+		(property "Intersheetrefs" "${INTERSHEET_REFS}"
+			(at 20.4797 125.73 0)
+			(effects
+				(font
+					(size 1.27 1.27)
+				)
+				(justify right)
+				(hide yes)
+			)

Commit message: Open-drain inverter for DTACKs.
Parts:
- added R201, R202, R203: 0R, Resistor_THT:R_Axial_DIN0207_L6.3mm_D2.5mm_P7.62mm_Horizontal, symbol Device:R_Small
- added U203: 74ACT05, Package_DIP:DIP-14_W7.62mm_Socket, symbol 74xx:74LS05
Connections:
- net +5V: now also U203.14 (VCC)
- net GND: now also R201.1, R202.1, R203.1, U203.7 (GND)
- net ~{DTACK}: now also U203.2, U203.4, U203.6
- new net: R201.2, U203.9
- new net: R202.2, U203.11
- new net: R203.2, U203.13
- new net CTLSP_DTACK: U203.5
- new net MMU_DTACK: U203.1
- new net OBMEM_DTACK: U203.3
- no-connect marks 3 -> 6
Other:
- moved on the sheet: U201

Commit message: Add reset circuit.
Parts:
- added C201: 100µF, Capacitor_THT:CP_Radial_D6.3mm_P2.50mm, symbol Device:C_Polarized_Small
- added D201: BAT86,113, Diode_THT:D_DO-35_SOD27_P7.62mm_Horizontal, symbol Diode:BAT86
- added D202: 1N4148, Diode_THT:D_DO-35_SOD27_P7.62mm_Horizontal, symbol Diode:1N4148
- added R204: 3K3, Resistor_THT:R_Axial_DIN0207_L6.3mm_D2.5mm_P7.62mm_Horizontal, symbol Device:R_Small
- added SW201: Reset, Button_Switch_THT:SW_PUSH_6mm, symbol Switch:SW_Push
- added U204: DS1813, Package_TO_SOT_THT:TO-92_Inline, symbol jrt-ICs:DS1813
Connections:
- net +5V: now also D202.1 (K), R204.2
- net GND: now also C201.2, SW201.2, U204.3 (GND)
- net ~{RESET}: now also D201.2 (A)
- net ~{HALT}: now reaches U201.17 (~{HALT})
- net ~{HALT}: now also D201.1 (K), SW201.1, U204.1 (~{RST})
- new net: C201.1, D202.2 (A), R204.1, U204.2 (Vcc)
Other:
- note added: "Vf=0.450"

Commit message: Some decoupling caps.
Parts:
- added C202, C203, C204, C205: 0.1µF, Capacitor_THT:C_Disc_D3.8mm_W2.6mm_P2.50mm, symbol Device:C_Small
Connections:
- net +5V: now also C202.1, C203.1, C204.1, C205.1
- net GND: now also C202.2, C203.2, C204.2, C205.2

Commit message: Need a pull-up on /RESET!
Parts:
- added R205: 3K3, Resistor_THT:R_Axial_DIN0207_L6.3mm_D2.5mm_P7.62mm_Horizontal, symbol Device:R_Small
Connections:
- net +5V: now also R205.2
- net ~{RESET}: now also R205.1
Changed lines of the file:
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@@
 	)
 	(junction
+		(at 97.79 173.99)
+		(diameter 0)
+		(color 0 0 0 0)
+	)
+	(junction
 		(at 92.71 182.88)
 		(diameter 0)
@@
 	(wire
 		(pts
+			(xy 97.79 172.72) (xy 97.79 173.99)
+		)
+		(stroke
+			(width 0)
+			(type default)
+		)
+	)
+	(wire
+		(pts
 			(xy 81.28 88.9) (xy 83.82 88.9)
 		)
@@
 	(wire
 		(pts
+			(xy 97.79 173.99) (xy 114.3 173.99)
+		)
+		(stroke
+			(width 0)
+			(type default)
+		)
+	)
+	(wire
+		(pts
 			(xy 114.3 166.37) (xy 127 166.37)
 		)
@@
 	(wire
 		(pts
-			(xy 111.76 173.99) (xy 114.3 173.99)
+			(xy 95.25 173.99) (xy 97.79 173.99)
 		)
 		(stroke
@@
 	(global_label "~{RESET}"
 		(shape output)
-		(at 111.76 173.99 180)
+		(at 95.25 173.99 180)
 		(fields_autoplaced yes)
 		(effects
@@
 		)
 		(property "Intersheetrefs" "${INTERSHEET_REFS}"
-			(at 103.0297 173.99 0)
+			(at 86.5197 173.99 0)
 			(effects
 				(font
@@
 	)
 	(symbol
+		(lib_id "power:+5V")
+		(at 97.79 167.64 0)
+		(unit 1)
+		(exclude_from_sim no)
+		(in_bom yes)
+		(on_board yes)
+		(dnp no)
+		(fields_autoplaced yes)
+		(property "Reference" "#PWR0218"
+			(at 97.79 171.45 0)
+			(effects
+				(font
+					(size 1.27 1.27)
+				)
+				(hide yes)
+			)
+		)
+		(property "Value" "+5V"
+			(at 97.79 162.56 0)
+			(effects
+				(font
+					(size 1.27 1.27)
+				)
+			)
+		)
+		(property "Footprint" ""
+			(at 97.79 167.64 0)
+			(effects
+				(font
+					(size 1.27 1.27)
+				)
+				(hide yes)
+			)
+		)
+		(property "Datasheet" ""
+			(at 97.79 167.64 0)
+			(effects
+				(font
+					(size 1.27 1.27)
+				)
+				(hide yes)
+			)
+		)
+		(property "Description" "Power symbol creates a global label with name \"+5V\""
+			(at 97.79 167.64 0)
+			(effects
+				(font
+					(size 1.27 1.27)
+				)
+				(hide yes)
+			)
+		)
+		(pin "1"
+		)
+		(instances
+			(project "cpu010"
+				(path "/65f80d66-eea1-4882-b29a-ae1b65892b55/40bef1ee-40eb-4732-8f1f-7a2dee1d9fd5"
+					(reference "#PWR0218")
+					(unit 1)
+				)
+			)
+		)
+	)
+	(symbol
 		(lib_id "power:GND")
 		(at 58.42 187.96 0)
@@
 				)
 			)
+		)
+	)
+	(symbol
+		(lib_id "Device:R_Small")
+		(at 97.79 170.18 180)
+		(unit 1)
+		(exclude_from_sim no)
+		(in_bom yes)
+		(on_board yes)
+		(dnp no)
+		(fields_autoplaced yes)
+		(property "Reference" "R205"
+			(at 100.33 168.9099 0)
+			(effects
+				(font
+					(size 1.016 1.016)
+				)
+				(justify right)
+			)
+		)
+		(property "Value" "3K3"
+			(at 100.33 171.4499 0)
+			(effects
+				(font
+					(size 1.27 1.27)
+				)
+				(justify right)
+			)
+		)
+		(property "Footprint" "Resistor_THT:R_Axial_DIN0207_L6.3mm_D2.5mm_P7.62mm_Horizontal"
+			(at 97.79 170.18 0)
+			(effects
+				(font
+					(size 1.27 1.27)
+				)
+				(hide yes)
+			)
+		)
+		(property "Datasheet" "~"
+			(at 97.79 170.18 0)
+			(effects
+				(font
+					(size 1.27 1.27)
+				)
+				(hide yes)
+			)
+		)
+		(property "Description" "Resistor, small symbol"
+			(at 97.79 170.18 0)
+			(effects
+				(font
+					(size 1.27 1.27)
+				)
+				(hide yes)
+			)
+		)
+		(pin "1"
+		)
+		(pin "2"
+		)
+		(instances
+			(project "cpu010"
+				(path "/65f80d66-eea1-4882-b29a-ae1b65892b55/40bef1ee-40eb-4732-8f1f-7a2dee1d9fd5"
+					(reference "R205")
+					(unit 1)
+				)
+			)

Commit message: SMT 0805 bypass caps everywere.
Parts:
- C202, C203, C204, C205: value 0.1µF -> 100nF; footprint Capacitor_THT:C_Disc_D3.8mm_W2.6mm_P2.50mm -> Capacitor_SMD:C_0805_2012Metric_Pad1.18x1.45mm_HandSolder; Part Kyocera SR125E104MARAP2 -> (none)
Changed lines of the file:
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@@
 			)
 		)
-		(property "Value" "0.1µF"
+		(property "Value" "100nF"
 			(at 107.95 186.6962 0)
 			(effects
@@
 			)
 		)
-		(property "Footprint" "Capacitor_THT:C_Disc_D3.8mm_W2.6mm_P2.50mm"
+		(property "Footprint" "Capacitor_SMD:C_0805_2012Metric_Pad1.18x1.45mm_HandSolder"
 			(at 105.41 185.42 0)
 			(effects
@@
 		)
 		(property "Description" "Unpolarized capacitor, small symbol"
-			(at 105.41 185.42 0)
-			(effects
-				(font
-					(size 1.27 1.27)
-				)
-				(hide yes)
-			)
-		)
-		(property "Part" "Kyocera SR125E104MARAP2"
 			(at 105.41 185.42 0)
 			(effects
@@
 			)
 		)
-		(property "Value" "0.1µF"
+		(property "Value" "100nF"
 			(at 120.65 186.6962 0)
 			(effects
@@
 			)
 		)
-		(property "Footprint" "Capacitor_THT:C_Disc_D3.8mm_W2.6mm_P2.50mm"
+		(property "Footprint" "Capacitor_SMD:C_0805_2012Metric_Pad1.18x1.45mm_HandSolder"
 			(at 118.11 185.42 0)
 			(effects
@@
 		)
 		(property "Description" "Unpolarized capacitor, small symbol"
-			(at 118.11 185.42 0)
-			(effects
-				(font
-					(size 1.27 1.27)
-				)
-				(hide yes)
-			)
-		)
-		(property "Part" "Kyocera SR125E104MARAP2"
 			(at 118.11 185.42 0)
 			(effects
@@
 			)
 		)
-		(property "Value" "0.1µF"
+		(property "Value" "100nF"
 			(at 133.35 186.6962 0)
 			(effects
@@
 			)
 		)
-		(property "Footprint" "Capacitor_THT:C_Disc_D3.8mm_W2.6mm_P2.50mm"
+		(property "Footprint" "Capacitor_SMD:C_0805_2012Metric_Pad1.18x1.45mm_HandSolder"
 			(at 130.81 185.42 0)
 			(effects
@@
 		)
 		(property "Description" "Unpolarized capacitor, small symbol"
-			(at 130.81 185.42 0)
-			(effects
-				(font
-					(size 1.27 1.27)
-				)
-				(hide yes)
-			)
-		)
-		(property "Part" "Kyocera SR125E104MARAP2"
 			(at 130.81 185.42 0)
 			(effects
@@
 			)
 		)
-		(property "Value" "0.1µF"
+		(property "Value" "100nF"
 			(at 95.25 186.6962 0)
 			(effects
@@
 			)
 		)
-		(property "Footprint" "Capacitor_THT:C_Disc_D3.8mm_W2.6mm_P2.50mm"
+		(property "Footprint" "Capacitor_SMD:C_0805_2012Metric_Pad1.18x1.45mm_HandSolder"
 			(at 92.71 185.42 0)
 			(effects
@@
 			(at 92.71 185.42 0)
 			(effects
-				(font
-					(size 1.27 1.27)
-				)
-				(hide yes)
-			)
-		)
-		(property "Part" "Kyocera SR125E104MARAP2"
-			(at 92.71 185.42 0)
-			(effects
