File: cpu010/design-files/cpu010-cpu.kicad_sch (KiCad schematic)
At the start: 18 parts, among them SW201 Reset, U201 MC68010P, U202 74ACT163, U203 74ACT05, U204 DS1813, Y201 40MHz

Commit message: Clock generation is now done in the MMU, and we clock the MMU at 40MHz.
Parts:
- removed C203: 100nF, Capacitor_SMD:C_0805_2012Metric_Pad1.18x1.45mm_HandSolder, symbol Device:C_Small
- removed U202: 74ACT163, Package_DIP:DIP-16_W7.62mm_Socket, symbol 74xx:74LS163
- renumbered U203 to U202, U204 to U203
Connections:
- net CLK40: now reaches Y201.5 (OUT)
- net CLK10 renamed CPU_CLK
- no-connect marks 5 -> 2
Other:
- moved on the sheet: C204, C205

Commit message: Route a bunch of I/O controller signals.
Parts:
- added R206, R207, R208: 3K3, Resistor_SMD:R_0805_2012Metric_Pad1.20x1.40mm_HandSolder, symbol Device:R_Small
Connections:
- net +5V: now also R206.2, R207.2, R208.2
- net IPL2: now reaches U201.23 (~{IPL2})
- net IPL2: now also R208.1
- net IPL1: now reaches U201.24 (~{IPL1})
- net IPL1: now also R207.1
- net IPL0: now reaches U201.25 (~{IPL0})
- net IPL0: now also R206.1

Commit message: More routing of I/O signals.  Change the I2C pullups to 1K.
Parts:
- added C203: 100nF, Capacitor_SMD:C_0805_2012Metric_Pad1.18x1.45mm_HandSolder, symbol Device:C_Small
Connections:
- net +5V: now also C203.1
- net GND: now also C203.2
- net ~{VPA}: now reaches U201.21 (~{VPA})
- no-connect marks 2 -> 5
Changed lines of the file:
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@@
 	)
 	(junction
+		(at 120.65 187.96)
+		(diameter 0)
+		(color 0 0 0 0)
+	)
+	(junction
 		(at 60.96 99.06)
 		(diameter 0)
@@
 	)
 	(junction
+		(at 120.65 182.88)
+		(diameter 0)
+		(color 0 0 0 0)
+	)
+	(junction
 		(at 48.26 57.15)
 		(diameter 0)
@@
 	)
 	(no_connect
+		(at 83.82 66.04)
+	)
+	(no_connect
 		(at 48.26 113.03)
 	)
+	(no_connect
+		(at 83.82 63.5)
+	)
+	(no_connect
+		(at 83.82 53.34)
+	)
 	(wire
 		(pts
@@
 	(wire
 		(pts
+			(xy 120.65 187.96) (xy 132.08 187.96)
+		)
+		(stroke
+			(width 0)
+			(type default)
+		)
+	)
+	(wire
+		(pts
 			(xy 107.95 182.88) (xy 120.65 182.88)
 		)
@@
 	(wire
 		(pts
+			(xy 120.65 182.88) (xy 132.08 182.88)
+		)
+		(stroke
+			(width 0)
+			(type default)
+		)
+	)
+	(wire
+		(pts
 			(xy 116.84 76.2) (xy 114.3 76.2)
 		)
@@
 		)
 	)
+	(global_label "~{VPA}"
+		(shape input)
+		(at 83.82 68.58 180)
+		(fields_autoplaced yes)
+		(effects
+			(font
+				(size 1.27 1.27)
+			)
+			(justify right)
+		)
+		(property "Intersheetrefs" "${INTERSHEET_REFS}"
+			(at 77.3876 68.58 0)
+			(effects
+				(font
+					(size 1.27 1.27)
+				)
+				(justify right)
+				(hide yes)
+			)
+		)
+	)
 	(global_label "D13"
 		(shape bidirectional)
@@
 					(unit 1)
 				)
+			)
+		)
+	)
+	(symbol
+		(lib_id "Device:C_Small")
+		(at 132.08 185.42 0)
+		(unit 1)
+		(exclude_from_sim no)
+		(in_bom yes)
+		(on_board yes)
+		(dnp no)
+		(fields_autoplaced yes)
+		(property "Reference" "C203"
+			(at 134.62 184.1562 0)
+			(effects
+				(font
+					(size 1.27 1.27)
+				)
+				(justify left)
+			)
+		)
+		(property "Value" "100nF"
+			(at 134.62 186.6962 0)
+			(effects
+				(font
+					(size 1.27 1.27)
+				)
+				(justify left)
+			)
+		)
+		(property "Footprint" "Capacitor_SMD:C_0805_2012Metric_Pad1.18x1.45mm_HandSolder"
+			(at 132.08 185.42 0)
+			(effects
+				(font
+					(size 1.27 1.27)
+				)
+				(hide yes)
+			)
+		)
+		(property "Datasheet" "~"
+			(at 132.08 185.42 0)
+			(effects
+				(font
+					(size 1.27 1.27)
+				)
+				(hide yes)
+			)
+		)
+		(property "Description" "Unpolarized capacitor, small symbol"
+			(at 132.08 185.42 0)
+			(effects
+				(font
+					(size 1.27 1.27)
+				)
+				(hide yes)
+			)
+		)
+		(pin "1"
+		)
+		(pin "2"
+		)
+		(instances
+			(project "cpu010"
+				(path "/65f80d66-eea1-4882-b29a-ae1b65892b55/40bef1ee-40eb-4732-8f1f-7a2dee1d9fd5"
+					(reference "C203")
+					(unit 1)
+				)

Commit message: Many many bus connections.
Connections:
- net +5V: no longer D202.1 (K), R204.1
- new net PWR_OK: D202.1 (K), R204.1
Changed lines of the file:
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@@
 	)
 	(junction
-		(at 102.87 146.05)
-		(diameter 0)
-		(color 0 0 0 0)
-	)
-	(junction
 		(at 149.86 166.37)
 		(diameter 0)
@@
 	)
 	(junction
+		(at 102.87 146.05)
+		(diameter 0)
+		(color 0 0 0 0)
+	)
+	(junction
 		(at 107.95 182.88)
 		(diameter 0)
@@
 	(wire
 		(pts
+			(xy 102.87 144.78) (xy 102.87 146.05)
+		)
+		(stroke
+			(width 0)
+			(type default)
+		)
+	)
+	(wire
+		(pts
 			(xy 44.45 29.21) (xy 48.26 29.21)
 		)
@@
 		)
 	)
+	(global_label "PWR_OK"
+		(shape input)
+		(at 102.87 144.78 90)
+		(fields_autoplaced yes)
+		(effects
+			(font
+				(size 1.27 1.27)
+			)
+			(justify left)
+		)
+		(property "Intersheetrefs" "${INTERSHEET_REFS}"
+			(at 102.87 134.2353 90)
+			(effects
+				(font
+					(size 1.27 1.27)
+				)
+				(justify left)
+				(hide yes)
+			)
+		)
+	)
 	(global_label "VA13"
 		(shape output)
@@
 					(unit 1)
 				)
-			)
-		)
-	)
-	(symbol
-		(lib_id "power:+5V")
-		(at 102.87 146.05 0)
-		(unit 1)
-		(exclude_from_sim no)
-		(in_bom yes)
-		(on_board yes)
-		(dnp no)
-		(fields_autoplaced yes)
-		(property "Reference" "#PWR0215"
-			(at 102.87 149.86 0)
-			(effects
-				(font
-					(size 1.27 1.27)
-				)
-				(hide yes)
-			)
-		)
-		(property "Value" "+5V"
-			(at 102.87 140.97 0)
-			(effects
-				(font
-					(size 1.27 1.27)
-				)
-			)
-		)
-		(property "Footprint" ""
-			(at 102.87 146.05 0)
-			(effects
-				(font
-					(size 1.27 1.27)
-				)
-				(hide yes)
-			)
-		)
-		(property "Datasheet" ""
-			(at 102.87 146.05 0)
-			(effects
-				(font
-					(size 1.27 1.27)
-				)
-				(hide yes)
-			)
-		)
-		(property "Description" "Power symbol creates a global label with name \"+5V\""
-			(at 102.87 146.05 0)
-			(effects
-				(font
-					(size 1.27 1.27)
-				)
-				(hide yes)
-			)
-		)
-		(pin "1"
-		)
-		(instances
-			(project ""
-				(path "/65f80d66-eea1-4882-b29a-ae1b65892b55/40bef1ee-40eb-4732-8f1f-7a2dee1d9fd5"
-					(reference "#PWR0215")
-					(unit 1)
-				)

Commit message: Add some passives for signal integrity, work on some additional signal routing.
Parts:
- added R209, R211, R212: 10K, Resistor_SMD:R_0805_2012Metric_Pad1.20x1.40mm_HandSolder, symbol Device:R_Small
- added R210: 33R, Resistor_SMD:R_0805_2012Metric_Pad1.20x1.40mm_HandSolder, symbol Device:R_Small
- added RN201, RN202: 47K, Resistor_THT:R_Array_SIP9, symbol Device:R_Network08
- R201: value 3K3 -> 470
- R206, R207, R208: value 3K3 -> 10K
- U201: value MC68010P -> MC68010
Connections:
- net +5V: now also R209.1, R211.2, R212.2, RN201.1 (common), RN202.1 (common)
- net CLK40: now also R210.2; no longer Y201.5 (OUT)
- net D0: now also RN201.6 (R5)
- net D1: now also RN201.5 (R4)
- net D10: now also RN202.7 (R6)
- net D11: now also RN202.8 (R7)
- net D12: now also RN202.9 (R8)
- net D13: now also RN201.7 (R6)
- net D14: now also RN201.8 (R7)
- net D15: now also RN201.9 (R8)
- net D2: now also RN201.4 (R3)
- net D3: now also RN201.3 (R2)
- net D4: now also RN201.2 (R1)
- net D5: now also RN202.2 (R1)
- net D6: now also RN202.3 (R2)
- net D7: now also RN202.4 (R3)
- net D8: now also RN202.5 (R4)
- net D9: now also RN202.6 (R5)
- net ~{CPU_BERR}: now also R211.1
- net ~{VPA}: now also R212.1
- net at U201.12 (~{BGACK}): now also U201.13 (~{BR}), R209.2
- new net: R210.1, Y201.5 (OUT)
Other:
- note added: "N.B. Since the 68010 is the only bus master, there is not a need to pull-up the CPU address lines to Vcc."

Commit message: Beef up the power supply a little.
Parts:
- added C206: 100µF, Capacitor_THT:CP_Radial_D6.3mm_P2.50mm, symbol Device:C_Polarized_Small
Connections:
- net +5V: now also C206.1
- net GND: now also C206.2
Changed lines of the file:
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@@
 	(wire
 		(pts
+			(xy 80.01 187.96) (xy 92.71 187.96)
+		)
+		(stroke
+			(width 0)
+			(type default)
+		)
+	)
+	(wire
+		(pts
 			(xy 74.93 55.88) (xy 83.82 55.88)
 		)
@@
 	(wire
 		(pts
+			(xy 80.01 182.88) (xy 92.71 182.88)
+		)
+		(stroke
+			(width 0)
+			(type default)
+		)
+	)
+	(wire
+		(pts
 			(xy 114.3 99.06) (xy 116.84 99.06)
 		)
@@
 					(unit 1)
 				)
+			)
+		)
+	)
+	(symbol
+		(lib_id "Device:C_Polarized_Small")
+		(at 80.01 185.42 0)
+		(unit 1)
+		(exclude_from_sim no)
+		(in_bom yes)
+		(on_board yes)
+		(dnp no)
+		(fields_autoplaced yes)
+		(property "Reference" "C206"
+			(at 82.55 183.6038 0)
+			(effects
+				(font
+					(size 1.27 1.27)
+				)
+				(justify left)
+			)
+		)
+		(property "Value" "100µF"
+			(at 82.55 186.1438 0)
+			(effects
+				(font
+					(size 1.27 1.27)
+				)
+				(justify left)
+			)
+		)
+		(property "Footprint" "Capacitor_THT:CP_Radial_D6.3mm_P2.50mm"
+			(at 80.01 185.42 0)
+			(effects
+				(font
+					(size 1.27 1.27)
+				)
+				(hide yes)
+			)
+		)
+		(property "Datasheet" "~"
+			(at 80.01 185.42 0)
+			(effects
+				(font
+					(size 1.27 1.27)
+				)
+				(hide yes)
+			)
+		)
+		(property "Description" "Polarized capacitor, small symbol"
+			(at 80.01 185.42 0)
+			(effects
+				(font
+					(size 1.27 1.27)
+				)
+				(hide yes)
+			)
+		)
+		(property "Part" "Wurth 860040373002"
+			(at 80.01 185.42 0)
+			(effects
+				(font
+					(size 1.27 1.27)
+				)
+				(hide yes)
+			)
+		)
+		(pin "2"
+		)
+		(pin "1"
+		)
+		(instances
+			(project "cpu010"
+				(path "/65f80d66-eea1-4882-b29a-ae1b65892b55/40bef1ee-40eb-4732-8f1f-7a2dee1d9fd5"
+					(reference "C206")
+					(unit 1)
+				)

Commit message: More component labeling.
Parts:
- C201, C206: Mouser (none) -> 710-860040373002
- D201: Mouser (none) -> 771-BAT86113
- RN201, RN202: Mouser (none) -> 652-4609X-1LF-47K
- U202: Mouser (none) -> 595-CD74ACT05E
- U203: Mouser (none) -> 700-DS1813-5+
- Y201: Mouser (none) -> 774-MXO45HST-3C-40.0; Part (none) -> CTS MXO45HST-3C-40M0000
Changed lines of the file:
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@@
 			)
 		)
+		(property "Mouser" "595-CD74ACT05E"
+			(at 40.64 57.15 0)
+			(effects
+				(font
+					(size 1.27 1.27)
+				)
+				(hide yes)
+			)
+		)
 		(pin "4"
 		)
@@
 			)
 		)
+		(property "Mouser" "652-4609X-1LF-47K"
+			(at 158.75 96.52 90)
+			(effects
+				(font
+					(size 1.27 1.27)
+				)
+				(hide yes)
+			)
+		)
 		(pin "3"
 		)
@@
 			)
 		)
+		(property "Mouser" "771-BAT86113"
+			(at 114.3 170.18 90)
+			(effects
+				(font
+					(size 1.27 1.27)
+				)
+				(hide yes)
+			)
+		)
 		(pin "1"
 		)
@@
 			)
 		)
+		(property "Mouser" "595-CD74ACT05E"
+			(at 40.64 71.12 0)
+			(effects
+				(font
+					(size 1.27 1.27)
+				)
+				(hide yes)
+			)
+		)
 		(pin "4"
 		)
@@
 			)
 		)
+		(property "Mouser" "595-CD74ACT05E"
+			(at 40.64 43.18 0)
+			(effects
+				(font
+					(size 1.27 1.27)
+				)
+				(hide yes)
+			)
+		)
 		(pin "4"
 		)
@@
 			)
 		)
+		(property "Part" "CTS MXO45HST-3C-40M0000"
+			(at 24.13 175.26 0)
+			(effects
+				(font
+					(size 1.27 1.27)
+				)
+				(hide yes)
+			)
+		)
+		(property "Mouser" "774-MXO45HST-3C-40.0"
+			(at 24.13 175.26 0)
+			(effects
+				(font
+					(size 1.27 1.27)
+				)
+				(hide yes)
+			)
+		)
 		(pin "5"
 		)
@@
 			)
 		)
+		(property "Mouser" "595-CD74ACT05E"
+			(at 40.64 85.09 0)
+			(effects
+				(font
+					(size 1.27 1.27)
+				)
+				(hide yes)
+			)
+		)
 		(pin "4"
 		)
@@
 			)
 		)
+		(property "Mouser" "595-CD74ACT05E"
+			(at 22.86 133.35 0)
+			(effects
+				(font
+					(size 1.27 1.27)
+				)
+				(hide yes)
+			)
+		)
 		(pin "4"
 		)
@@
 			)
 		)
+		(property "Mouser" "595-CD74ACT05E"
+			(at 40.64 113.03 0)
+			(effects
+				(font
+					(size 1.27 1.27)
+				)
+				(hide yes)
+			)
+		)
 		(pin "4"
 		)
@@
 			)
 		)
+		(property "Mouser" "710-860040373002"
+			(at 102.87 157.48 0)
+			(effects
+				(font
+					(size 1.27 1.27)
+				)
+				(hide yes)
+			)
+		)
 		(pin "2"
 		)
@@
 			)
 		)
+		(property "Mouser" "652-4609X-1LF-47K"
+			(at 158.75 127 90)
+			(effects
+				(font
+					(size 1.27 1.27)
+				)
+				(hide yes)
+			)
+		)
 		(pin "3"
 		)
@@
 			)
 		)
+		(property "Mouser" "710-860040373002"
+			(at 80.01 185.42 0)
+			(effects
+				(font
+					(size 1.27 1.27)
+				)
+				(hide yes)
+			)
+		)
 		(pin "2"
 		)
@@
 			)
 		)
+		(property "Mouser" "700-DS1813-5+"
+			(at 127 154.94 0)
+			(effects
+				(font
+					(size 1.27 1.27)
+				)
+				(hide yes)
+			)
+		)
 		(pin "2"
 		)
@@
 			(at 40.64 99.06 0)
 			(effects
+				(font
+					(size 1.27 1.27)
+				)
+				(hide yes)
+			)
+		)
+		(property "Mouser" "595-CD74ACT05E"
+			(at 40.64 99.06 0)
+			(effects

Commit message: DRC checkpoint - no more errors!  Set copper layers of the mechanical NPTH mounting holes to "none".
Parts:
- U203: footprint Package_TO_SOT_THT:TO-92_Inline -> Package_TO_SOT_THT:TO-92_Inline_Wide
Changed lines of the file:
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@@
 			)
 		)
-		(property "Footprint" "Package_TO_SOT_THT:TO-92_Inline"
+		(property "Footprint" "Package_TO_SOT_THT:TO-92_Inline_Wide"
 			(at 127 175.26 0)
 			(effects
