File: cpu010/design-files/cpu010-control.kicad_sch (KiCad schematic)
At the start: 14 parts, among them SW401 SW_DIP_x08, SW402 SW_DIP_x08, U401 DA04-11SURKWA, U402 74HCT273, U403 74HCT273, U404 GAL22V10, U405 74HC245, U406 74HC245, U407 74HCT273, U408 74HC245

Commit message: Descriptive text for some control space stuff.
Other:
- note added: "Configuration Register"
- note added: "Diagnostic Display Register"
- note added: "System Enable Register"
- note removed: "Diagnostic 2-digit display"
Changed lines of the file:
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@@
 		)
 	)
-	(text "Diagnostic 2-digit display"
+	(text "System Enable Register"
+		(exclude_from_sim no)
+		(at 98.806 158.75 0)
+		(effects
+			(font
+				(size 1.27 1.27)
+			)
+			(justify left)
+		)
+	)
+	(text "Diagnostic Display Register"
 		(exclude_from_sim no)
 		(at 157.734 18.542 0)
 		(effects
 			(font
+				(size 1.27 1.27)
+			)
+			(justify left)
+		)
+	)
+	(text "Configuration Register"
+		(exclude_from_sim no)
+		(at 259.08 124.968 0)
+		(effects
+			(font

Commit message: Wire up Bus Error register.
Parts:
- added U409: ATF1504AS-PLCC44, Package_LCC:PLCC-44_THT-Socket, symbol jrt-ICs:ATF1504AS-PLCC44
Connections:
- net +5V: now also U409.15 (VCC), U409.23 (VCC), U409.3 (VCC), U409.35 (VCC)
- net D10: now also U409.11 (I/O/PD1)
- net D11: now also U409.12 (I/O)
- net D12: now also U409.14 (I/O)
- net D13: now also U409.16 (I/O)
- net D14: now also U409.17 (I/O)
- net D15: now also U409.18 (I/O)
- net D8: now also U409.8 (I/O)
- net D9: now also U409.9 (I/O)
- net GND: now also U409.10 (GND), U409.22 (GND), U409.30 (GND), U409.42 (GND)
- net R/~{W}: now also U409.6 (I/O)
- net ~{BERSEL}: now also U409.44 (I/OE1/Vpp)
- net ~{RESET}: now also U409.1 (I/GCLR)
- new net BERR_DTACK: U409.5 (I/O)
- new net CLK10: U409.43 (I/GCLK1)
- new net MMUERR0: U409.19 (I/O)
- new net MMUERR1: U409.20 (I/O)
- new net MMUERR2: U409.21 (I/O)
- new net ~{CPU_AS}: U409.2 (I/OE2/GCLK2)
- new net ~{CPU_BERR}: U409.4 (I/O)
- no-connect marks 10 -> 24
Other:
- note added: "Bus Error Register Bits in the register: BERR_MMUINV 0x01 BERR_MMUPROT 0x02 BERR_MMUPRIV 0x04 BERR_TIMEOUT 0x10"

Commit message: Fix up the Enable register.
Connections:
- net D10: now also U407.7 (D2)
- net D11: now also U407.8 (D3)
- net D12: now also U407.13 (D4)
- net D13: now also U407.14 (D5)
- net D14: now also U407.17 (D6)
- net D15: now also U407.18 (D7)
- net D8: now also U407.3 (D0)
- net D9: now also U407.4 (D1)
- net GND: now also U408.1 (A->B); no longer U408.19 (CE)
- net MMU_EN: now also U408.18 (B0)
- net ~{ERRD}: now also U408.19 (CE); no longer U408.1 (A->B)
- net at U408.11 (B7): now also U407.19 (Q7); no longer U407.18 (D7)
- net at U408.12 (B6): now also U407.16 (Q6); no longer U407.17 (D6)
- net at U408.13 (B5): now also U407.15 (Q5); no longer U407.14 (D5)
- net at U408.14 (B4): now also U407.12 (Q4); no longer U407.13 (D4)
- net at U408.15 (B3): now also U407.9 (Q3); no longer U407.8 (D3)
- net at U408.16 (B2): now also U407.6 (Q2); no longer U407.7 (D2)
- net at U408.17 (B1): now also U407.5 (Q1); no longer U407.4 (D1)
- no-connect marks 24 -> 17
Other:
- note added: "Bus Error Register Bits in the register: BERR_MMUINV 0x01 BERR_MMUPROT 0x02 BERR_MMUPRIV 0x04 BERR_TIMEOUT 0x10 All other bits reserved for future expansion."
- note added: "System Enable Register Bits in the register: SYSEN_MMU 0x01 SYSEN_SW7 0x80 All other bits reserved for future expansion."
- note removed: "Bit 7 reserved for software"
- note removed: "Bus Error Register Bits in the register: BERR_MMUINV 0x01 BERR_MMUPROT 0x02 BERR_MMUPRIV 0x04 BERR_TIMEOUT 0x10"
- note removed: "System Enable Register"
- moved on the sheet: U407, U408

Commit message: Open-drain inverter for DTACKs.
Connections:
- net ~{DTACK} renamed CTLSP_DTACK
Changed lines of the file:
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@@
 		)
 	)
-	(global_label "~{DTACK}"
+	(global_label "CTLSP_DTACK"
 		(shape output)
 		(at 68.58 71.12 0)
@@
 		)
 		(property "Intersheetrefs" "${INTERSHEET_REFS}"
-			(at 77.4314 71.12 0)
+			(at 84.1442 71.12 0)
 			(effects
 				(font

Commit message: Some decoupling caps.
Parts:
- added C401, C402, C403, C404, C405, C406, C407: 0.1µF, Capacitor_THT:C_Disc_D3.8mm_W2.6mm_P2.50mm, symbol Device:C_Small
Connections:
- net +5V: now also C401.1, C402.1, C403.1, C404.1, C405.1, C406.1, C407.1
- net GND: now also C401.2, C402.2, C403.2, C404.2, C405.2, C406.2, C407.2

Commit message: SMT 0805 bypass caps everywere.
Parts:
- added C408, C409, C410, C411: 220nF, Capacitor_SMD:C_0805_2012Metric_Pad1.18x1.45mm_HandSolder, symbol Device:C_Small
- C401, C402, C403, C404, C405, C406, C407: value 0.1µF -> 100nF; footprint Capacitor_THT:C_Disc_D3.8mm_W2.6mm_P2.50mm -> Capacitor_SMD:C_0805_2012Metric_Pad1.18x1.45mm_HandSolder; Part Kyocera SR125E104MARAP2 -> (none)
- U409: Part (none) -> ATF1504AS-10JU44
Connections:
- net +5V: now also C408.1, C409.1, C410.1, C411.1
- net GND: now also C408.2, C409.2, C410.2, C411.2
- net at U402.12 (Q4): now also RN401.12 (R5.2); no longer RN401.5 (R5.1)
- net at U402.15 (Q5): now also RN401.11 (R6.2); no longer RN401.6 (R6.1)
- net at U402.16 (Q6): now also RN401.10 (R7.2); no longer RN401.7 (R7.1)
- net at U402.19 (Q7): now also RN401.9 (R8.2); no longer RN401.8 (R8.1)
- net at U402.2 (Q0): now also RN401.16 (R1.2); no longer RN401.1 (R1.1)
- net at U402.5 (Q1): now also RN401.15 (R2.2); no longer RN401.2 (R2.1)
- net at U402.6 (Q2): now also RN401.14 (R3.2); no longer RN401.3 (R3.1)
- net at U402.9 (Q3): now also RN401.13 (R4.2); no longer RN401.4 (R4.1)
- net at U401.16 (DIG1_G): now also RN401.7 (R7.1); no longer RN401.10 (R7.2)
- net at U401.14 (DIG1_F): now also RN401.6 (R6.1); no longer RN401.11 (R6.2)
- net at U401.2 (DIG1_E): now also RN401.5 (R5.1); no longer RN401.12 (R5.2)
- net at U401.3 (DIG1_D): now also RN401.4 (R4.1); no longer RN401.13 (R4.2)
- net at U401.1 (DIG1_C): now also RN401.3 (R3.1); no longer RN401.14 (R3.2)
- net at U401.13 (DIG1_B): now also RN401.2 (R2.1); no longer RN401.15 (R2.2)
- net at U401.15 (DIG1_A): now also RN401.1 (R1.1); no longer RN401.16 (R1.2)
- net at U401.10 (DIG2_A): now also RN402.1 (R1.1); no longer RN402.16 (R1.2)
- net at U401.11 (DIG2_F): now also RN402.6 (R6.1); no longer RN402.11 (R6.2)
- net at U401.12 (DIG2_B): now also RN402.2 (R2.1); no longer RN402.15 (R2.2)
- net at U401.6 (DIG2_D): now also RN402.4 (R4.1); no longer RN402.13 (R4.2)
- net at U401.7 (DIG2_E): now also RN402.5 (R5.1); no longer RN402.12 (R5.2)
- net at U401.8 (DIG2_C): now also RN402.3 (R3.1); no longer RN402.14 (R3.2)
- net at U401.9 (DIG2_G): now also RN402.7 (R7.1); no longer RN402.10 (R7.2)
- net at U403.2 (Q0): now also RN402.16 (R1.2); no longer RN402.1 (R1.1)
- net at U403.5 (Q1): now also RN402.15 (R2.2); no longer RN402.2 (R2.1)
- net at U403.6 (Q2): now also RN402.14 (R3.2); no longer RN402.3 (R3.1)
- net at U403.9 (Q3): now also RN402.13 (R4.2); no longer RN402.4 (R4.1)
- net at U403.12 (Q4): now also RN402.12 (R5.2); no longer RN402.5 (R5.1)
- net at U403.15 (Q5): now also RN402.11 (R6.2); no longer RN402.6 (R6.1)
- net at U403.16 (Q6): now also RN402.10 (R7.2); no longer RN402.7 (R7.1)
- net at RN402.8 (R8.1): no longer U403.19 (Q7)
- net at RN402.9 (R8.2): now also U403.19 (Q7)
Other:
- moved on the sheet: RN401, RN402

Commit message: Document IOCTL address decode.
Other:
- note added: "Control space (FC==4): [CTLSPDEC] xxxx.xxxx xxxx.xxxx 0000.0000 - Diagnostic display (upper digit) xxxx.xxxx xxxx.xxxx 0000.0001 - Diagnostic display (lower digit) xxxx.xxxx xxxx.xxxx 0001.000x - Configuration switches xxxx.xxxx xxxx.xxxx 0010.0000 - System Enable register xxxx.xxxx xxxx.xxxx 0011.0000 - Bus Error register [IOCTL010] xxxx.xxxx xxxx.xxxx 0100.0000 - Interrupt Enable xxxx.xxxx xxxx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"
- note removed: "Control space (FC==4): xxxx.xxxx xxxx.xxxx 0000.0000 - Diagnostic display (upper digit) xxxx.xxxx xxxx.xxxx 0000.0001 - Diagnostic display (lower digit) xxxx.xxxx xxxx.xxxx 0001.000x - Configuration switches xxxx.xxxx xxxx.xxxx 0002.0000 - System Enable register xxxx.xxxx xxxx.xxxx 0003.0000 - Bus Error register"
- moved on the sheet: U404
Changed lines of the file:
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@@
 	(generator_version "9.0")
 	(paper "A3")
-	(text "Control space (FC==4):\nxxxx.xxxx xxxx.xxxx 0000.0000 - Diagnostic display (upper digit)\nxxxx.xxxx xxxx.xxxx 0000.0001 - Diagnostic display (lower digit)\nxxxx.xxxx xxxx.xxxx 0001.000x - Configuration switches\nxxxx.xxxx xxxx.xxxx 0002.0000 - System Enable register\nxxxx.xxxx xxxx.xxxx 0003.0000 - Bus Error register"
+	(text "Control space (FC==4):\n[CTLSPDEC]\nxxxx.xxxx xxxx.xxxx 0000.0000 - Diagnostic display (upper digit)\nxxxx.xxxx xxxx.xxxx 0000.0001 - Diagnostic display (lower digit)\nxxxx.xxxx xxxx.xxxx 0001.000x - Configuration switches\nxxxx.xxxx xxxx.xxxx 0010.0000 - System Enable register\nxxxx.xxxx xxxx.xxxx 0011.0000 - Bus Error register\n[IOCTL010]\nxxxx.xxxx xxxx.xxxx 0100.0000 - Interrupt Enable\nxxxx.xxxx xxxx.xxxx 0101.0000 - Interrupt Set\nxxxx.xxxx xxxx.xxxx 0110.0000 - Interrupt Clear\nxxxx.xxxx xxxx.xxxx 0111.0000 - Interrupt Controller Revision"
 		(exclude_from_sim no)
-		(at 16.002 20.066 0)
+		(at 21.336 30.226 0)
 		(effects
 			(font
@@
 	)
 	(no_connect
-		(at 67.31 50.8)
+		(at 67.31 60.96)
 	)
 	(no_connect
@@
 	(wire
 		(pts
-			(xy 68.58 60.96) (xy 67.31 60.96)
+			(xy 68.58 71.12) (xy 67.31 71.12)
 		)
 		(stroke
@@
 	(wire
 		(pts
-			(xy 67.31 68.58) (xy 68.58 68.58)
+			(xy 67.31 78.74) (xy 68.58 78.74)
 		)
 		(stroke
@@
 	(wire
 		(pts
-			(xy 68.58 66.04) (xy 67.31 66.04)
+			(xy 68.58 76.2) (xy 67.31 76.2)
 		)
 		(stroke
@@
 	(wire
 		(pts
-			(xy 68.58 58.42) (xy 67.31 58.42)
+			(xy 68.58 68.58) (xy 67.31 68.58)
 		)
 		(stroke
@@
 	(wire
 		(pts
-			(xy 68.58 48.26) (xy 67.31 48.26)
+			(xy 68.58 58.42) (xy 67.31 58.42)
 		)
 		(stroke
@@
 	(wire
 		(pts
-			(xy 30.48 73.66) (xy 41.91 73.66)
+			(xy 30.48 83.82) (xy 41.91 83.82)
 		)
 		(stroke
@@
 	(wire
 		(pts
-			(xy 68.58 55.88) (xy 67.31 55.88)
+			(xy 68.58 66.04) (xy 67.31 66.04)
 		)
 		(stroke
@@
 	(wire
 		(pts
-			(xy 68.58 71.12) (xy 67.31 71.12)
+			(xy 68.58 81.28) (xy 67.31 81.28)
 		)
 		(stroke
@@
 	(wire
 		(pts
-			(xy 68.58 63.5) (xy 67.31 63.5)
+			(xy 68.58 73.66) (xy 67.31 73.66)
 		)
 		(stroke
@@
 	(wire
 		(pts
-			(xy 68.58 53.34) (xy 67.31 53.34)
+			(xy 68.58 63.5) (xy 67.31 63.5)
 		)
 		(stroke
@@
 	)
 	(label "~{CSLSEL}"
-		(at 68.58 60.96 0)
+		(at 68.58 71.12 0)
 		(effects
 			(font
@@
 	)
 	(label "~{CSUSEL}"
-		(at 68.58 58.42 0)
+		(at 68.58 68.58 0)
 		(effects
 			(font
@@
 	)
 	(label "~{BERSEL}"
-		(at 68.58 68.58 0)
+		(at 68.58 78.74 0)
 		(effects
 			(font
@@
 	)
 	(label "~{DDLSEL}"
-		(at 68.58 55.88 0)
+		(at 68.58 66.04 0)
 		(effects
 			(font
@@
 	)
 	(label "~{ERWR}"
-		(at 68.58 66.04 0)
+		(at 68.58 76.2 0)
 		(effects
 			(font
@@
 	)
 	(label "~{DDUSEL}"
-		(at 68.58 53.34 0)
+		(at 68.58 63.5 0)
 		(effects
 			(font
@@
 	)
 	(label "~{ERRD}"
-		(at 68.58 63.5 0)
+		(at 68.58 73.66 0)
 		(effects
 			(font
@@
 	(global_label "R{slash}~{W}"
 		(shape input)
-		(at 68.58 48.26 0)
+		(at 68.58 58.42 0)
 		(fields_autoplaced yes)
 		(effects
@@
 		)
 		(property "Intersheetrefs" "${INTERSHEET_REFS}"
-			(at 75.6171 48.26 0)
+			(at 75.6171 58.42 0)
 			(effects
 				(font
@@
 	(global_label "VA1"
 		(shape input)
-		(at 41.91 55.88 180)
+		(at 41.91 66.04 180)
 		(fields_autoplaced yes)
 		(effects
@@
 		)
 		(property "Intersheetrefs" "${INTERSHEET_REFS}"
-			(at 35.5381 55.88 0)
+			(at 35.5381 66.04 0)
 			(effects
 				(font
@@
 	(global_label "FC0"
 		(shape input)
-		(at 41.91 48.26 180)
+		(at 41.91 58.42 180)
 		(fields_autoplaced yes)
 		(effects
@@
 		)
 		(property "Intersheetrefs" "${INTERSHEET_REFS}"
-			(at 35.3567 48.26 0)
+			(at 35.3567 58.42 0)
 			(effects
 				(font
@@
 	(global_label "~{CPU_UDS}"
 		(shape input)
-		(at 30.48 73.66 180)
+		(at 30.48 83.82 180)
 		(fields_autoplaced yes)
 		(effects
@@
 		)
 		(property "Intersheetrefs" "${INTERSHEET_REFS}"
-			(at 18.8467 73.66 0)
+			(at 18.8467 83.82 0)
 			(effects
 				(font
@@
 	(global_label "VA2"
 		(shape input)
-		(at 41.91 58.42 180)
+		(at 41.91 68.58 180)
 		(fields_autoplaced yes)
 		(effects
@@
 		)
 		(property "Intersheetrefs" "${INTERSHEET_REFS}"
-			(at 35.5381 58.42 0)
+			(at 35.5381 68.58 0)
 			(effects
 				(font
@@
 	(global_label "FC2"
 		(shape input)
-		(at 41.91 53.34 180)
+		(at 41.91 63.5 180)
 		(fields_autoplaced yes)
 		(effects
@@
 		)
 		(property "Intersheetrefs" "${INTERSHEET_REFS}"
-			(at 35.3567 53.34 0)
+			(at 35.3567 63.5 0)
 			(effects
 				(font
@@
 	(global_label "FC1"
 		(shape input)
-		(at 41.91 50.8 180)
+		(at 41.91 60.96 180)
 		(fields_autoplaced yes)
 		(effects
@@
 		)
 		(property "Intersheetrefs" "${INTERSHEET_REFS}"
-			(at 35.3567 50.8 0)
+			(at 35.3567 60.96 0)
 			(effects
 				(font
@@
 	(global_label "VA7"
 		(shape input)
-		(at 41.91 71.12 180)
+		(at 41.91 81.28 180)
 		(fields_autoplaced yes)
 		(effects
@@
 		)
 		(property "Intersheetrefs" "${INTERSHEET_REFS}"
-			(at 35.5381 71.12 0)
+			(at 35.5381 81.28 0)
 			(effects
 				(font
@@
 	(global_label "~{CPU_LDS}"
 		(shape input)
-		(at 41.91 76.2 180)
+		(at 41.91 86.36 180)
 		(fields_autoplaced yes)
 		(effects
@@
 		)
 		(property "Intersheetrefs" "${INTERSHEET_REFS}"
-			(at 30.5791 76.2 0)
+			(at 30.5791 86.36 0)
 			(effects
 				(font
@@
 	(global_label "VA3"
 		(shape input)
-		(at 41.91 60.96 180)
+		(at 41.91 71.12 180)
 		(fields_autoplaced yes)
 		(effects
@@
 		)
 		(property "Intersheetrefs" "${INTERSHEET_REFS}"
-			(at 35.5381 60.96 0)
+			(at 35.5381 71.12 0)
 			(effects
 				(font
@@
 	(global_label "VA6"
 		(shape input)
-		(at 41.91 68.58 180)
+		(at 41.91 78.74 180)
 		(fields_autoplaced yes)
 		(effects
@@
 		)
 		(property "Intersheetrefs" "${INTERSHEET_REFS}"
-			(at 35.5381 68.58 0)
+			(at 35.5381 78.74 0)
 			(effects
 				(font
@@
 	(global_label "CTLSP_DTACK"
 		(shape output)
-		(at 68.58 71.12 0)
+		(at 68.58 81.28 0)
 		(fields_autoplaced yes)
 		(effects
@@
 		)
 		(property "Intersheetrefs" "${INTERSHEET_REFS}"
-			(at 84.1442 71.12 0)
+			(at 84.1442 81.28 0)
 			(effects
 				(font
@@
 	(global_label "VA4"
 		(shape input)
-		(at 41.91 63.5 180)
+		(at 41.91 73.66 180)
 		(fields_autoplaced yes)
 		(effects
@@
 		)
 		(property "Intersheetrefs" "${INTERSHEET_REFS}"
-			(at 35.5381 63.5 0)
+			(at 35.5381 73.66 0)
 			(effects
 				(font
@@
 	(global_label "VA5"
 		(shape input)
-		(at 41.91 66.04 180)
+		(at 41.91 76.2 180)
 		(fields_autoplaced yes)
 		(effects
@@
 		)
 		(property "Intersheetrefs" "${INTERSHEET_REFS}"
-			(at 35.5381 66.04 0)
+			(at 35.5381 76.2 0)
 			(effects
 				(font
@@
 	(symbol
 		(lib_id "jrt-ICs:GAL22V10")
-		(at 54.61 62.23 0)
+		(at 54.61 72.39 0)
 		(unit 1)
 		(exclude_from_sim no)
@@
 		(fields_autoplaced yes)
 		(property "Reference" "U404"
-			(at 56.7533 40.64 0)
+			(at 56.7533 50.8 0)
 			(effects
 				(font
@@
 		)
 		(property "Value" "GAL22V10"
-			(at 56.7533 43.18 0)
+			(at 56.7533 53.34 0)
 			(effects
 				(font
@@
 		)
 		(property "Footprint" "Package_DIP:DIP-24_W7.62mm_Socket"
-			(at 54.61 62.23 0)
+			(at 54.61 72.39 0)
 			(effects
 				(font
@@
 		)
 		(property "Datasheet" ""
-			(at 54.61 62.23 0)
+			(at 54.61 72.39 0)
 			(effects
 				(font
@@
 		)
 		(property "Description" ""
-			(at 54.61 62.23 0)
+			(at 54.61 72.39 0)
 			(effects
 				(font
@@
 	(symbol
 		(lib_id "power:GND")
-		(at 54.61 81.28 0)
+		(at 54.61 91.44 0)
 		(unit 1)
 		(exclude_from_sim no)
@@
 		(fields_autoplaced yes)
 		(property "Reference" "#PWR0407"
-			(at 54.61 87.63 0)
+			(at 54.61 97.79 0)
 			(effects
 				(font
@@
 		)
 		(property "Value" "GND"
-			(at 54.61 86.36 0)
+			(at 54.61 96.52 0)
 			(effects
 				(font
@@
 		)
 		(property "Footprint" ""
-			(at 54.61 81.28 0)
+			(at 54.61 91.44 0)
 			(effects
 				(font
@@
 		)
 		(property "Datasheet" ""
-			(at 54.61 81.28 0)
+			(at 54.61 91.44 0)
 			(effects
 				(font
@@
 		)
 		(property "Description" "Power symbol creates a global label with name \"GND\" , ground"
-			(at 54.61 81.28 0)
+			(at 54.61 91.44 0)
 			(effects
 				(font
@@
 	(symbol
 		(lib_id "power:+5V")
-		(at 54.61 43.18 0)
+		(at 54.61 53.34 0)
 		(unit 1)
 		(exclude_from_sim no)
@@
 		(fields_autoplaced yes)
 		(property "Reference" "#PWR0406"
-			(at 54.61 46.99 0)
+			(at 54.61 57.15 0)
 			(effects
 				(font
@@
 		)
 		(property "Value" "+5V"
-			(at 54.61 38.1 0)
+			(at 54.61 48.26 0)
 			(effects
 				(font
@@
 		)
 		(property "Footprint" ""
-			(at 54.61 43.18 0)
+			(at 54.61 53.34 0)
 			(effects
 				(font
@@
 		)
 		(property "Datasheet" ""
-			(at 54.61 43.18 0)
+			(at 54.61 53.34 0)
 			(effects
 				(font
@@
 		)
 		(property "Description" "Power symbol creates a global label with name \"+5V\""
-			(at 54.61 43.18 0)
+			(at 54.61 53.34 0)
 			(effects
 				(font

Commit message: More layout.
Parts:
- added C412, C413, C414, C415, C416, C417, C418, C419: 100nF, Capacitor_SMD:C_0805_2012Metric_Pad1.18x1.45mm_HandSolder, symbol Device:C_Small
Connections:
- net +5V: now also C404.2, C405.2, C412.1, C413.1, C414.1, C415.1, C416.1, C417.1, C418.2, C419.2; no longer C404.1, C405.1
- net GND: now also C404.1, C405.1, C412.2, C413.2, C414.2, C415.2, C416.2, C417.2, C418.1, C419.1; no longer C404.2, C405.2
