File: cpu010/design-files/cpu010-control.kicad_sch (KiCad schematic)
At the start: 29 parts, among them SW401 SW_DIP_x08, SW402 SW_DIP_x08, U401 DA04-11SURKWA, U402 74HCT273, U403 74HCT273, U404 GAL22V10, U405 74HCT245, U406 74HCT245, U407 74HCT273, U408 74HCT245

Commit message: Fix Errata A.2 -- Buffer the PWR_OK output to the LED and the DS1813 with a new N-FET / P-FET high-side switch controlled by PWR_OK from the PSU.
Other:
- note added: "Control space (FC==4): [CTLSPDEC] xxxx.xxxx xxxx.xxxx 0000.0000 - Diagnostic display (upper digit) xxxx.xxxx xxxx.xxxx 0000.0001 - Diagnostic display (lower digit) xxxx.xxxx xxxx.xxxx 0001.000x - Configuration switches xxxx.xxxx xxxx.xxxx 0010.0000 - System Enable register [IOCTL010] xxxx.xxxx xxxx.xxxx 0100.0000 - Interrupt Set xxxx.xxxx xxxx.xxxx 0101.0000 - Interrupt Clear xxxx.xxxx xxxx.xxxx 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"
- note removed: "Control space (FC==4): [CTLSPDEC] xxxx.xxxx xxxx.xxxx 0000.0000 - Diagnostic display (upper digit) xxxx.xxxx xxxx.xxxx 0000.0001 - Diagnostic display (lower digit) xxxx.xxxx xxxx.xxxx 0001.000x - Configuration switches xxxx.xxxx xxxx.xxxx 0010.0000 - System Enable register [IOCTL010] xxxx.xxxx xxxx.xxxx 0100.0000 - Interrupt Set xxxx.xxxx xxxx.xxxx 0101.0000 - Interrupt Clear"
Changed lines of the file:
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@@
 	(title_block
 		(title "68k Playground CPU010")
-		(date "2026-06-12")
+		(date "2026-06-20")
 		(rev "B")
 		(company "(c) 2025, 2026 Jason R. Thorpe.  All rights reserved.")
 	)
-	(text "Control space (FC==4):\n[CTLSPDEC]\nxxxx.xxxx xxxx.xxxx 0000.0000 - Diagnostic display (upper digit)\nxxxx.xxxx xxxx.xxxx 0000.0001 - Diagnostic display (lower digit)\nxxxx.xxxx xxxx.xxxx 0001.000x - Configuration switches\nxxxx.xxxx xxxx.xxxx 0010.0000 - System Enable register\n[IOCTL010]\nxxxx.xxxx xxxx.xxxx 0100.0000 - Interrupt Set\nxxxx.xxxx xxxx.xxxx 0101.0000 - Interrupt Clear\n"
+	(text "Control space (FC==4):\n[CTLSPDEC]\nxxxx.xxxx xxxx.xxxx 0000.0000 - Diagnostic display (upper digit)\nxxxx.xxxx xxxx.xxxx 0000.0001 - Diagnostic display (lower digit)\nxxxx.xxxx xxxx.xxxx 0001.000x - Configuration switches\nxxxx.xxxx xxxx.xxxx 0010.0000 - System Enable register\n[IOCTL010]\nxxxx.xxxx xxxx.xxxx 0100.0000 - Interrupt Set\nxxxx.xxxx xxxx.xxxx 0101.0000 - Interrupt Clear\nxxxx.xxxx xxxx.xxxx 1110.0000 - Board revision (< 'A' == simulator)\nxxxx.xxxx xxxx.xxxx 1111.0000 - CPLD revision (entire set)"
 		(exclude_from_sim no)
 		(at 21.336 30.226 0)
