File: cpu010/design-files/cpu010.kicad_sch (KiCad schematic)
At the start: 8 parts, among them U101 GAL22V10

Commit message: Route some bypass caps and the diagnostic display.
Changed lines of the file:
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@@
+		(length 2.54)
+		(shape diamond)
+		(at 160.02 34.29 0)
+		(fields_autoplaced yes)
+		(effects
+			(font
+				(size 1.27 1.27)
+			)
+			(justify left bottom)
+		)
+		(property "Netclass" "Power"
+			(at 161.2265 31.75 0)
+			(effects
+				(font
+					(size 1.27 1.27)
+				)
+				(justify left)
+			)
+		)
+		(property "Component Class" ""
+			(at -31.75 13.97 0)
+			(effects
+				(font
+					(size 1.27 1.27)
+					(italic yes)
+				)
+			)
+		)
+	)
+	(netclass_flag ""
 		(length 2.54)
 		(shape diamond)
@@
 					(unit 1)
 				)
+			)
+		)
+	)
+	(symbol
+		(lib_id "power:GND")
+		(at 160.02 34.29 0)
+		(unit 1)
+		(exclude_from_sim no)
+		(in_bom yes)
+		(on_board yes)
+		(dnp no)
+		(fields_autoplaced yes)
+		(property "Reference" "#PWR0106"
+			(at 160.02 40.64 0)
+			(effects
+				(font
+					(size 1.27 1.27)
+				)
+				(hide yes)
+			)
+		)
+		(property "Value" "GND"
+			(at 160.02 39.37 0)
+			(effects
+				(font
+					(size 1.27 1.27)
+				)
+			)
+		)
+		(property "Footprint" ""
+			(at 160.02 34.29 0)
+			(effects
+				(font
+					(size 1.27 1.27)
+				)
+				(hide yes)
+			)
+		)
+		(property "Datasheet" ""
+			(at 160.02 34.29 0)
+			(effects
+				(font
+					(size 1.27 1.27)
+				)
+				(hide yes)
+			)
+		)
+		(property "Description" "Power symbol creates a global label with name \"GND\" , ground"
+			(at 160.02 34.29 0)
+			(effects
+				(font
+					(size 1.27 1.27)
+				)
+				(hide yes)
+			)
+		)
+		(pin "1"
+		)
+		(instances
+			(project "cpu010"
+				(path "/65f80d66-eea1-4882-b29a-ae1b65892b55"
+					(reference "#PWR0106")
+					(unit 1)
+				)

Commit message: Routing some I/O stuff.
Parts:
- removed C101: 100nF, Capacitor_SMD:C_0805_2012Metric_Pad1.18x1.45mm_HandSolder, symbol Device:C_Small
- removed U101: GAL22V10, Package_DIP:DIP-24_W7.62mm_Socket, symbol jrt-ICs:GAL22V10
Connections:
- no-connect marks 11 -> 0

Commit message: Expansion slots!
Parts:
- added H107, H108, H109, H110, H111, H112: MountingHole, MountingHole:MountingHole_3.2mm_M3, symbol Mechanical:MountingHole
Other:
- added sheet Expansion (cpu010-expansion.kicad_sch)

Commit message: Expansion port + PSU.  Route signals for the expansion slots.
Other:
- added sheet Power Supply (cpu010-psu.kicad_sch)
Changed lines of the file:
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@@
+	)
+	(sheet
+		(at 127 114.554)
+		(size 48.514 27.686)
+		(exclude_from_sim no)
+		(in_bom yes)
+		(on_board yes)
+		(dnp no)
+		(fields_autoplaced yes)
+		(stroke
+			(width 0.1524)
+			(type solid)
+		)
+		(fill
+			(color 0 0 0 0.0000)
+		)
+		(property "Sheetname" "Power Supply"
+			(at 127 113.8424 0)
+			(effects
+				(font
+					(size 1.27 1.27)
+				)
+				(justify left bottom)
+			)
+		)
+		(property "Sheetfile" "cpu010-psu.kicad_sch"
+			(at 127 142.8246 0)
+			(effects
+				(font
+					(size 1.27 1.27)
+				)
+				(justify left top)
+			)
+		)
+		(instances
+			(project "cpu010"
+				(path "/65f80d66-eea1-4882-b29a-ae1b65892b55"
+					(page "8")
+				)
+			)
+		)
 	)
 	(sheet

Commit message: More (NQ)VME tweaks.  Add JTAG chain.
Parts:
- added J101: JTAG, Connector_PinHeader_2.54mm:PinHeader_2x05_P2.54mm_Vertical, symbol Connector_Generic:Conn_02x05_Odd_Even
- added R101, R102, R103: 10K, Resistor_SMD:R_0805_2012Metric_Pad1.20x1.40mm_HandSolder, symbol Device:R_Small
Connections:
- net +5V: now also J101.4 (Pin_4), R101.2, R102.2, R103.2
- net GND: now also J101.10 (Pin_10), J101.2 (Pin_2)
- new net MMU_TDI: J101.9 (Pin_9), R103.1
- new net TCK: J101.1 (Pin_1), R101.1
- new net TDO: J101.3 (Pin_3)
- new net TMS: J101.5 (Pin_5), R102.1
- no-connect marks 0 -> 3
Other:
- note added: "JTAG Chain: MMU (1508) -> IOCTL (1508) -> MEMCTL (1504) -> BERR (1504)"
- note added: "Top-level physical address map: 00xx xxxx.xxxx xxxx.xxxx xxxx.xxxx - RAM 01xx xxxx.xxxx xxxx.xxxx xxxx.xxxx - ROM 10xx xxxx.xxxx xxxx.xxxx xxxx.xxxx - On-board I/O 11xx xxxx.xxxx xxxx.xxxx xxxx.xxxx - (NQ)VME I/O Control space (FC==4): xxxx.xxxx xxxx.xxxx xxxx.000x - see Control Space sheet xxxx.xxxx xxxx.xxxx xxxx.xx1x - reserved for MMU xxxx.xxxx xxxx.xxxx xxxx.x1xx - reserved for MMU xxxx.xxxx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"
- note removed: "Top-level physical address map: 00xx xxxx.xxxx xxxx.xxxx xxxx.xxxx - RAM 01xx xxxx.xxxx xxxx.xxxx xxxx.xxxx - ROM 10xx xxxx.xxxx xxxx.xxxx xxxx.xxxx - I/O 11xx xxxx.xxxx xxxx.xxxx xxxx.xxxx - expansion Control space (FC==4): xxxx.xxxx xxxx.xxxx xxxx.000x - see Control Space sheet xxxx.xxxx xxxx.xxxx xxxx.xx1x - reserved for MMU xxxx.xxxx xxxx.xxxx xxxx.x1xx - reserved for MMU xxxx.xxxx xxxx.xxxx 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"

Commit message: Expansion bus changes: - VME bus arb signals are now total no-ops, no daisy-chain. - Ditto for VMS IACK signals. - Neuter some other VME control signals.
Other:
- note added: "JTAG Chain: MMU (1508) -> IOCTL (1508) -> MEMCTL (1504)"
- note removed: "JTAG Chain: MMU (1508) -> IOCTL (1508) -> MEMCTL (1504) -> BERR (1504)"
Changed lines of the file:
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@@
 		)
 	)
-	(text "JTAG Chain: MMU (1508) -> IOCTL (1508) -> MEMCTL (1504) -> BERR (1504)"
+	(text "JTAG Chain: MMU (1508) -> IOCTL (1508) -> MEMCTL (1504)"
 		(exclude_from_sim no)
 		(at 113.792 55.372 0)

Commit message: Many many bus connections.
Other:
- added sheet VME termination (cpu010-vme-term.kicad_sch)
Changed lines of the file:
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@@
-		)
-	)
-	(netclass_flag ""
-		(length 2.54)
-		(shape diamond)
-		(at 160.02 34.29 0)
-		(fields_autoplaced yes)
-		(effects
-			(font
-				(size 1.27 1.27)
-			)
-			(justify left bottom)
-		)
-		(property "Netclass" "Power"
-			(at 161.2265 31.75 0)
-			(effects
-				(font
-					(size 1.27 1.27)
-				)
-				(justify left)
-			)
-		)
-		(property "Component Class" ""
-			(at -31.75 13.97 0)
-			(effects
-				(font
-					(size 1.27 1.27)
-					(italic yes)
-				)
-			)
-		)
-	)
-	(netclass_flag ""
-		(length 2.54)
-		(shape diamond)
-		(at 160.02 22.86 180)
-		(fields_autoplaced yes)
-		(effects
-			(font
-				(size 1.27 1.27)
-			)
-			(justify right bottom)
-		)
-		(property "Netclass" "Power"
-			(at 161.2265 25.4 0)
-			(effects
-				(font
-					(size 1.27 1.27)
-				)
-				(justify left)
-			)
-		)
-		(property "Component Class" ""
-			(at -31.75 2.54 0)
-			(effects
-				(font
-					(size 1.27 1.27)
-					(italic yes)
-				)
-			)
 		)
 	)
@@
 	)
 	(symbol
-		(lib_id "power:+5V")
-		(at 160.02 22.86 0)
-		(unit 1)
-		(exclude_from_sim no)
-		(in_bom yes)
-		(on_board yes)
-		(dnp no)
-		(fields_autoplaced yes)
-		(property "Reference" "#PWR0105"
-			(at 160.02 26.67 0)
-			(effects
-				(font
-					(size 1.27 1.27)
-				)
-				(hide yes)
-			)
-		)
-		(property "Value" "+5V"
-			(at 160.02 17.78 0)
-			(effects
-				(font
-					(size 1.27 1.27)
-				)
-			)
-		)
-		(property "Footprint" ""
-			(at 160.02 22.86 0)
-			(effects
-				(font
-					(size 1.27 1.27)
-				)
-				(hide yes)
-			)
-		)
-		(property "Datasheet" ""
-			(at 160.02 22.86 0)
-			(effects
-				(font
-					(size 1.27 1.27)
-				)
-				(hide yes)
-			)
-		)
-		(property "Description" "Power symbol creates a global label with name \"+5V\""
-			(at 160.02 22.86 0)
-			(effects
-				(font
-					(size 1.27 1.27)
-				)
-				(hide yes)
-			)
-		)
-		(pin "1"
-		)
-		(instances
-			(project "cpu010"
-				(path "/65f80d66-eea1-4882-b29a-ae1b65892b55"
-					(reference "#PWR0105")
-					(unit 1)
-				)
-			)
-		)
-	)
-	(symbol
 		(lib_id "Mechanical:MountingHole")
 		(at 185.42 62.23 0)
@@
 				(path "/65f80d66-eea1-4882-b29a-ae1b65892b55"
 					(reference "R103")
-					(unit 1)
-				)
-			)
-		)
-	)
-	(symbol
-		(lib_id "power:GND")
-		(at 160.02 34.29 0)
-		(unit 1)
-		(exclude_from_sim no)
-		(in_bom yes)
-		(on_board yes)
-		(dnp no)
-		(fields_autoplaced yes)
-		(property "Reference" "#PWR0106"
-			(at 160.02 40.64 0)
-			(effects
-				(font
-					(size 1.27 1.27)
-				)
-				(hide yes)
-			)
-		)
-		(property "Value" "GND"
-			(at 160.02 39.37 0)
-			(effects
-				(font
-					(size 1.27 1.27)
-				)
-			)
-		)
-		(property "Footprint" ""
-			(at 160.02 34.29 0)
-			(effects
-				(font
-					(size 1.27 1.27)
-				)
-				(hide yes)
-			)
-		)
-		(property "Datasheet" ""
-			(at 160.02 34.29 0)
-			(effects
-				(font
-					(size 1.27 1.27)
-				)
-				(hide yes)
-			)
-		)
-		(property "Description" "Power symbol creates a global label with name \"GND\" , ground"
-			(at 160.02 34.29 0)
-			(effects
-				(font
-					(size 1.27 1.27)
-				)
-				(hide yes)
-			)
-		)
-		(pin "1"
-		)
-		(instances
-			(project "cpu010"
-				(path "/65f80d66-eea1-4882-b29a-ae1b65892b55"
-					(reference "#PWR0106")
 					(unit 1)
 				)
@@
 				)
 			)
+		)
+	)
+	(sheet
+		(at 180.848 114.554)
+		(size 48.006 27.686)
+		(exclude_from_sim no)
+		(in_bom yes)
+		(on_board yes)
+		(dnp no)
+		(fields_autoplaced yes)
+		(stroke
+			(width 0.1524)
+			(type solid)
+		)
+		(fill
+			(color 0 0 0 0.0000)
+		)
+		(property "Sheetname" "VME termination"
+			(at 180.848 113.8424 0)
+			(effects
+				(font
+					(size 1.27 1.27)
+				)
+				(justify left bottom)
+			)
+		)
+		(property "Sheetfile" "cpu010-vme-term.kicad_sch"
+			(at 180.848 142.8246 0)
+			(effects
+				(font
+					(size 1.27 1.27)
+				)
+				(justify left top)
+			)
+		)
+		(instances
+			(project "cpu010"
+				(path "/65f80d66-eea1-4882-b29a-ae1b65892b55"
+					(page "9")
+				)
+			)

Commit message: There is not a separate VME termination sheet.
Other:
- removed sheet VME termination
Changed lines of the file:
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@@
-	)
-	(sheet
-		(at 180.848 114.554)
-		(size 48.006 27.686)
-		(exclude_from_sim no)
-		(in_bom yes)
-		(on_board yes)
-		(dnp no)
-		(fields_autoplaced yes)
-		(stroke
-			(width 0.1524)
-			(type solid)
-		)
-		(fill
-			(color 0 0 0 0.0000)
-		)
-		(property "Sheetname" "VME termination"
-			(at 180.848 113.8424 0)
-			(effects
-				(font
-					(size 1.27 1.27)
-				)
-				(justify left bottom)
-			)
-		)
-		(property "Sheetfile" "cpu010-vme-term.kicad_sch"
-			(at 180.848 142.8246 0)
-			(effects
-				(font
-					(size 1.27 1.27)
-				)
-				(justify left top)
-			)
-		)
-		(instances
-			(project "cpu010"
-				(path "/65f80d66-eea1-4882-b29a-ae1b65892b55"
-					(page "9")
-				)
-			)
-		)
 	)
 	(sheet
