File: cpu010/design-files/cpu010-mmu.kicad_sch (KiCad schematic)
At the start: 24 parts, among them U301 ATF1508AS-TQFP100, U302 61C3216, U303 74AHCT245, U304 74AHCT245, U305 7C4098, U306 7C4098, U307 74AHCT245, U308 74AHCT245, U309 74AHCT245, U310 74AHCT245, U311 74AHCT373, U312 74AHCT373, U313 74AHCT373, U314 74AHCT157, U315 74AHCT157, U316 74AHCT157, U317 74AHCT157, U318 74AHCT157, U319 74AHCT157, U320 74AHCT157, U321 74AHCT157, U322 74AHCT157, U323 74AHCT245, U324 74AHCT245

Commit message: Wire up Bus Error register.
Connections:
- net MMUERR0: now reaches U301.28 (I/O)
- net MMUERR1: now reaches U301.29 (I/O)
- net MMUERR2: now reaches U301.30 (I/O)
- net MMU_FAULT: no longer names the net of U301.2 (I/O)
- no-connect marks 36 -> 34
Changed lines of the file:
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@@
 	)
 	(no_connect
-		(at 43.18 105.41)
-	)
-	(no_connect
 		(at 163.83 151.13)
 	)
 	(no_connect
-		(at 43.18 107.95)
+		(at 43.18 49.53)
 	)
 	(no_connect
@@
 	)
 	(no_connect
-		(at 43.18 110.49)
-	)
-	(no_connect
 		(at 99.06 52.07)
 	)
@@
 	(wire
 		(pts
+			(xy 39.37 110.49) (xy 43.18 110.49)
+		)
+		(stroke
+			(width 0)
+			(type default)
+		)
+	)
+	(wire
+		(pts
 			(xy 288.29 105.41) (xy 289.56 105.41)
 		)
@@
 	(wire
 		(pts
+			(xy 39.37 105.41) (xy 43.18 105.41)
+		)
+		(stroke
+			(width 0)
+			(type default)
+		)
+	)
+	(wire
+		(pts
 			(xy 224.79 207.01) (xy 231.14 207.01)
 		)
@@
 	(wire
 		(pts
+			(xy 39.37 107.95) (xy 43.18 107.95)
+		)
+		(stroke
+			(width 0)
+			(type default)
+		)
+	)
+	(wire
+		(pts
 			(xy 289.56 105.41) (xy 289.56 104.14)
 		)
@@
 	(wire
 		(pts
-			(xy 39.37 49.53) (xy 43.18 49.53)
-		)
-		(stroke
-			(width 0)
-			(type default)
-		)
-	)
-	(wire
-		(pts
 			(xy 67.31 153.67) (xy 69.85 153.67)
 		)
@@
 		)
 	)
-	(global_label "MMU_FAULT"
-		(shape output)
-		(at 39.37 49.53 180)
-		(fields_autoplaced yes)
-		(effects
-			(font
-				(size 1.27 1.27)
-			)
-			(justify right)
-		)
-		(property "Intersheetrefs" "${INTERSHEET_REFS}"
-			(at 25.6805 49.53 0)
-			(effects
-				(font
-					(size 1.27 1.27)
-				)
-				(justify right)
-				(hide yes)
-			)
-		)
-	)
 	(global_label "VA8"
 		(shape input)
@@
 		)
 	)
+	(global_label "MMUERR2"
+		(shape output)
+		(at 39.37 110.49 180)
+		(fields_autoplaced yes)
+		(effects
+			(font
+				(size 1.27 1.27)
+			)
+			(justify right)
+		)
+		(property "Intersheetrefs" "${INTERSHEET_REFS}"
+			(at 27.253 110.49 0)
+			(effects
+				(font
+					(size 1.27 1.27)
+				)
+				(justify right)
+				(hide yes)
+			)
+		)
+	)
 	(global_label "D10"
 		(shape bidirectional)
@@
 		)
 	)
+	(global_label "MMUERR0"
+		(shape output)
+		(at 39.37 105.41 180)
+		(fields_autoplaced yes)
+		(effects
+			(font
+				(size 1.27 1.27)
+			)
+			(justify right)
+		)
+		(property "Intersheetrefs" "${INTERSHEET_REFS}"
+			(at 27.253 105.41 0)
+			(effects
+				(font
+					(size 1.27 1.27)
+				)
+				(justify right)
+				(hide yes)
+			)
+		)
+	)
 	(global_label "D1"
 		(shape bidirectional)
@@
 			(effects
 				(font
+					(size 1.27 1.27)
+				)
+				(justify right)
+				(hide yes)
+			)
+		)
+	)
+	(global_label "MMUERR1"
+		(shape output)
+		(at 39.37 107.95 180)
+		(fields_autoplaced yes)
+		(effects
+			(font
+				(size 1.27 1.27)
+			)
+			(justify right)
+		)
+		(property "Intersheetrefs" "${INTERSHEET_REFS}"
+			(at 27.253 107.95 0)
+			(effects
+				(font

Commit message: Add top-level address decoding.
Changed lines of the file:
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@@
 	(wire
 		(pts
-			(xy 99.06 82.55) (xy 101.6 82.55)
+			(xy 99.06 82.55) (xy 113.03 82.55)
 		)
 		(stroke
@@
 	(wire
 		(pts
-			(xy 99.06 80.01) (xy 101.6 80.01)
+			(xy 99.06 80.01) (xy 106.68 80.01)
 		)
 		(stroke
@@
 	(wire
 		(pts
-			(xy 99.06 77.47) (xy 101.6 77.47)
+			(xy 99.06 77.47) (xy 113.03 77.47)
 		)
 		(stroke
@@
 		)
 	)
-	(label "~{UDS}"
-		(at 101.6 80.01 0)
-		(effects
-			(font
-				(size 1.27 1.27)
-			)
-			(justify left bottom)
-		)
-	)
 	(label "PMIDX3"
 		(at 224.79 186.69 180)
@@
 		)
 	)
-	(label "~{LDS}"
-		(at 101.6 77.47 0)
-		(effects
-			(font
-				(size 1.27 1.27)
-			)
-			(justify left bottom)
-		)
-	)
 	(label "PME_REF"
 		(at 132.08 189.23 180)
@@
 		)
 	)
-	(label "~{AS}"
-		(at 101.6 82.55 0)
-		(effects
-			(font
-				(size 1.27 1.27)
-			)
-			(justify left bottom)
-		)
-	)
 	(label "PMEG3"
 		(at 86.36 248.92 180)
@@
 		)
 	)
+	(global_label "~{LDS}"
+		(shape output)
+		(at 113.03 77.47 0)
+		(fields_autoplaced yes)
+		(effects
+			(font
+				(size 1.27 1.27)
+			)
+			(justify left)
+		)
+		(property "Intersheetrefs" "${INTERSHEET_REFS}"
+			(at 119.5228 77.47 0)
+			(effects
+				(font
+					(size 1.27 1.27)
+				)
+				(justify left)
+				(hide yes)
+			)
+		)
+	)
 	(global_label "A4"
 		(shape output)
@@
 		)
 	)
+	(global_label "~{UDS}"
+		(shape output)
+		(at 106.68 80.01 0)
+		(fields_autoplaced yes)
+		(effects
+			(font
+				(size 1.27 1.27)
+			)
+			(justify left)
+		)
+		(property "Intersheetrefs" "${INTERSHEET_REFS}"
+			(at 113.4752 80.01 0)
+			(effects
+				(font
+					(size 1.27 1.27)
+				)
+				(justify left)
+				(hide yes)
+			)
+		)
+	)
 	(global_label "VA7"
 		(shape input)
@@
 				(hide yes)
 			)
+		)
+	)
+	(global_label "~{AS}"
+		(shape output)
+		(at 113.03 82.55 0)
+		(fields_autoplaced yes)
+		(effects
+			(font
+				(size 1.27 1.27)
+			)
+			(justify left)
+		)
+		(property "Intersheetrefs" "${INTERSHEET_REFS}"
+			(at 118.3133 82.55 0)
+			(effects
+				(font
+					(size 1.27 1.27)
+				)
+				(justify left)
+				(hide yes)
+			)

Commit message: Some decoupling caps.
Parts:
- added C301, C302, C303, C304, C305: 0.1µF, Capacitor_THT:C_Disc_D3.8mm_W2.6mm_P2.50mm, symbol Device:C_Small
Connections:
- net +5V: now also C301.1, C302.1, C303.1, C304.1, C305.1
- net GND: now also C301.2, C302.2, C303.2, C304.2, C305.2

Commit message: SMT 0805 bypass caps everywere.
Parts:
- added C306, C307, C308, C309, C310, C311, C312, C313, C314, C315, C316, C317, C318, C319, C320, C321, C322, C323, C324, C333, C334: 100nF, Capacitor_SMD:C_0805_2012Metric_Pad1.18x1.45mm_HandSolder, symbol Device:C_Small
- added C325, C326, C327, C328, C329, C330, C331, C332: 220nF, Capacitor_SMD:C_0805_2012Metric_Pad1.18x1.45mm_HandSolder, symbol Device:C_Small
- C301, C302, C303, C304, C305: value 0.1µF -> 100nF; footprint Capacitor_THT:C_Disc_D3.8mm_W2.6mm_P2.50mm -> Capacitor_SMD:C_0805_2012Metric_Pad1.18x1.45mm_HandSolder; Part Kyocera SR125E104MARAP2 -> (none)
- U301: JLCPCB (none) -> C1521282; Part (none) -> ATF1508AS-7AX100
- U302: JLCPCB (none) -> C2063204; Part (none) -> ISSI IS61C3216AL-12KLI
- U305, U306: JLCPCB (none) -> C2064107; Part (none) -> Alliance AS7C4098A-12JIN
Connections:
- net +5V: now also C306.1, C307.1, C308.1, C309.1, C310.1, C311.1, C312.1, C313.1, C314.1, C315.1, C316.1, C317.1, C318.1, C319.1, C320.1, C321.1, C322.1, C323.1, C324.1, C325.1, C326.1, C327.1, C328.1, C329.1, C330.1, C331.1, C332.1, C333.1, C334.1
- net GND: now also C306.2, C307.2, C308.2, C309.2, C310.2, C311.2, C312.2, C313.2, C314.2, C315.2, C316.2, C317.2, C318.2, C319.2, C320.2, C321.2, C322.2, C323.2, C324.2, C325.2, C326.2, C327.2, C328.2, C329.2, C330.2, C331.2, C332.2, C333.2, C334.2
Other:
- moved on the sheet: C301, C302, C303, C304, C305

Commit message: More layout.
Connections:
- net +5V: now also C330.2, C331.2; no longer C330.1, C331.1
- net GND: now also C330.1, C331.1; no longer C330.2, C331.2
Changed lines of the file:
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@@
 		(lib_id "Device:C_Small")
 		(at 354.33 242.57 0)
+		(mirror x)
 		(unit 1)
 		(exclude_from_sim no)
@@
 		(on_board yes)
 		(dnp no)
-		(fields_autoplaced yes)
 		(property "Reference" "C331"
-			(at 356.87 241.3062 0)
+			(at 356.87 243.8338 0)
 			(effects
 				(font
@@
 		)
 		(property "Value" "220nF"
-			(at 356.87 243.8462 0)
+			(at 356.87 241.2938 0)
 			(effects
 				(font
@@
 		(lib_id "Device:C_Small")
 		(at 341.63 242.57 0)
+		(mirror x)
 		(unit 1)
 		(exclude_from_sim no)
@@
 		(on_board yes)
 		(dnp no)
-		(fields_autoplaced yes)
 		(property "Reference" "C330"
-			(at 344.17 241.3062 0)
+			(at 344.17 243.8338 0)
 			(effects
 				(font
@@
 		)
 		(property "Value" "220nF"
-			(at 344.17 243.8462 0)
+			(at 344.17 241.2938 0)
 			(effects
 				(font

Commit message: Expansion slots!
Parts:
- U319, U320, U321, U322: value 74AHCT157 -> 74ACT157
- U323, U324: value 74AHCT245 -> 74ACT245
Changed lines of the file:
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@@
 			)
 		)
-		(property "Value" "74AHCT157"
+		(property "Value" "74ACT157"
 			(at 210.4233 73.66 0)
 			(effects
@@
 			)
 		)
-		(property "Value" "74AHCT157"
+		(property "Value" "74ACT157"
 			(at 304.4033 73.66 0)
 			(effects
@@
 			)
 		)
-		(property "Value" "74AHCT245"
+		(property "Value" "74ACT245"
 			(at 277.7333 125.73 0)
 			(effects
@@
 			)
 		)
-		(property "Value" "74AHCT157"
+		(property "Value" "74ACT157"
 			(at 256.1433 73.66 0)
 			(effects
@@
 			)
 		)
-		(property "Value" "74AHCT157"
+		(property "Value" "74ACT157"
 			(at 352.6633 73.66 0)
 			(effects
@@
 			)
 		)
-		(property "Value" "74AHCT245"
+		(property "Value" "74ACT245"
 			(at 229.4733 125.73 0)
 			(effects

Commit message: More (NQ)VME tweaks.  Add JTAG chain.
Connections:
- net TMS: now reaches U301.15 (I/O/TMS)
- net MMU_TDI: now reaches U301.4 (I/O/TDI)
- net TCK: now reaches U301.62 (I/O/TCK)
- net IOCTL_TDI: now reaches U301.73 (I/O/TDO)
Changed lines of the file:
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@@
 	(wire
 		(pts
+			(xy 111.76 87.63) (xy 99.06 87.63)
+		)
+		(stroke
+			(width 0)
+			(type default)
+		)
+	)
+	(wire
+		(pts
 			(xy 101.6 130.81) (xy 99.06 130.81)
 		)
@@
 	(wire
 		(pts
+			(xy 31.75 77.47) (xy 43.18 77.47)
+		)
+		(stroke
+			(width 0)
+			(type default)
+		)
+	)
+	(wire
+		(pts
 			(xy 132.08 80.01) (xy 138.43 80.01)
 		)
@@
 	(wire
 		(pts
+			(xy 99.06 113.03) (xy 111.76 113.03)
+		)
+		(stroke
+			(width 0)
+			(type default)
+		)
+	)
+	(wire
+		(pts
 			(xy 27.94 54.61) (xy 43.18 54.61)
 		)
@@
 		)
 	)
+	(global_label "MMU_TDI"
+		(shape input)
+		(at 43.18 52.07 180)
+		(fields_autoplaced yes)
+		(effects
+			(font
+				(size 1.27 1.27)
+			)
+			(justify right)
+		)
+		(property "Intersheetrefs" "${INTERSHEET_REFS}"
+			(at 32.1515 52.07 0)
+			(effects
+				(font
+					(size 1.27 1.27)
+				)
+				(justify right)
+				(hide yes)
+			)
+		)
+	)
 	(global_label "D8"
 		(shape bidirectional)
@@
 		)
 	)
+	(global_label "TCK"
+		(shape input)
+		(at 111.76 113.03 0)
+		(fields_autoplaced yes)
+		(effects
+			(font
+				(size 1.27 1.27)
+			)
+			(justify left)
+		)
+		(property "Intersheetrefs" "${INTERSHEET_REFS}"
+			(at 118.2528 113.03 0)
+			(effects
+				(font
+					(size 1.27 1.27)
+				)
+				(justify left)
+				(hide yes)
+			)
+		)
+	)
 	(global_label "VA10"
 		(shape input)
@@
 		)
 	)
+	(global_label "IOCTL_TDI"
+		(shape output)
+		(at 111.76 87.63 0)
+		(fields_autoplaced yes)
+		(effects
+			(font
+				(size 1.27 1.27)
+			)
+			(justify left)
+		)
+		(property "Intersheetrefs" "${INTERSHEET_REFS}"
+			(at 123.7562 87.63 0)
+			(effects
+				(font
+					(size 1.27 1.27)
+				)
+				(justify left)
+				(hide yes)
+			)
+		)
+	)
 	(global_label "~{LDS}"
 		(shape output)
@@
 			(effects
 				(font
+					(size 1.27 1.27)
+				)
+				(justify right)
+				(hide yes)
+			)
+		)
+	)
+	(global_label "TMS"
+		(shape input)
+		(at 31.75 77.47 180)
+		(fields_autoplaced yes)
+		(effects
+			(font
+				(size 1.27 1.27)
+			)
+			(justify right)
+		)
+		(property "Intersheetrefs" "${INTERSHEET_REFS}"
+			(at 25.1363 77.47 0)
+			(effects
+				(font

Commit message: Clock generation is now done in the MMU, and we clock the MMU at 40MHz.
Connections:
- net CPU_CLK: now reaches U301.100 (I/O)
- net I2C_CLK: now reaches U301.99 (I/O)
- net CLK20 renamed CLK40
- no-connect marks 34 -> 32
Changed lines of the file:
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@@
 	)
 	(no_connect
-		(at 99.06 41.91)
-	)
-	(no_connect
 		(at 99.06 46.99)
 	)
@@
 	)
 	(no_connect
-		(at 99.06 44.45)
-	)
-	(no_connect
 		(at 99.06 57.15)
 	)
@@
 	(wire
 		(pts
+			(xy 99.06 41.91) (xy 101.6 41.91)
+		)
+		(stroke
+			(width 0)
+			(type default)
+		)
+	)
+	(wire
+		(pts
 			(xy 224.79 212.09) (xy 231.14 212.09)
 		)
@@
 	(wire
 		(pts
+			(xy 99.06 44.45) (xy 101.6 44.45)
+		)
+		(stroke
+			(width 0)
+			(type default)
+		)
+	)
+	(wire
+		(pts
 			(xy 259.08 209.55) (xy 254 209.55)
 		)
@@
 		)
 	)
-	(global_label "CLK20"
+	(global_label "CLK40"
 		(shape input)
 		(at 39.37 41.91 180)
@@
 		)
 	)
+	(global_label "I2C_CLK"
+		(shape output)
+		(at 101.6 44.45 0)
+		(fields_autoplaced yes)
+		(effects
+			(font
+				(size 1.27 1.27)
+			)
+			(justify left)
+		)
+		(property "Intersheetrefs" "${INTERSHEET_REFS}"
+			(at 112.2052 44.45 0)
+			(effects
+				(font
+					(size 1.27 1.27)
+				)
+				(justify left)
+				(hide yes)
+			)
+		)
+	)
 	(global_label "D13"
 		(shape bidirectional)
@@
 			(effects
 				(font
+					(size 1.27 1.27)
+				)
+				(justify left)
+				(hide yes)
+			)
+		)
+	)
+	(global_label "CPU_CLK"
+		(shape output)
+		(at 101.6 41.91 0)
+		(fields_autoplaced yes)
+		(effects
+			(font
+				(size 1.27 1.27)
+			)
+			(justify left)
+		)
+		(property "Intersheetrefs" "${INTERSHEET_REFS}"
+			(at 112.9914 41.91 0)
+			(effects
+				(font
