File: cpu010/design-files/cpu010-mmu.kicad_sch (KiCad schematic)
At the start: 60 parts, among them U301 ATF1508AS-7AX100, U302 61C3216, U303 74AHCT245, U304 74AHCT245, U305 7C4098, U306 7C4098, U307 74AHCT245, U308 74AHCT245, U309 74AHCT245, U310 74AHCT245, U311 74AHCT373, U312 74AHCT373, U313 74AHCT373, U314 74AHCT157, U315 74AHCT157, U316 74AHCT157, U317 74AHCT157, U318 74AHCT157, U319 74AHCT157, U320 74AHCT157, U321 74AHCT157, U322 74AHCT157, U323 74AHCT245, U324 74AHCT245

Commit message: Note some TSOP-II-44 parts for the MMU SRAMs.  Consider these for board rev B.
Other:
- note added: "Consider replacing with IS61C3216AL-12TLI (TSOP-II-44)."
- note added: "Consider replcaing with AS7C4098A-12TIN (TSOP-II-44)."
Changed lines of the file:
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@@
 		(company "(c) 2025, 2026 Jason R. Thorpe.  All rights reserved.")
+	)
+	(text "Consider replacing with\nIS61C3216AL-12TLI (TSOP-II-44)."
+		(exclude_from_sim no)
+		(at 50.8 248.412 0)
+		(effects
+			(font
+				(size 1.27 1.27)
+			)
+		)
+	)
+	(text "Consider replcaing with\nAS7C4098A-12TIN (TSOP-II-44)."
+		(exclude_from_sim no)
+		(at 271.526 251.206 0)
+		(effects
+			(font
+				(size 1.27 1.27)
+			)
+		)
 	)
 	(junction

Commit message: The SOJ-44 package for the 61C3216 has been EOL'd; replace it with the TSOP-II-44 package of the same part.
Parts:
- U302: footprint Package_SO:SOJ-44_10.16x28.575mm_P1.27mm -> Package_SO:TSOP-II-44_10.16x18.41mm_P0.8mm; LCSC C1351200 -> XXX; Mouser 870IS61C3216AL12KLI -> 870IS61C3216AL12TLI; Part ISSI IS61C3216AL-12KLI -> ISSI IS61C3216AL-12TLI
Other:
- note removed: "Consider replacing with IS61C3216AL-12TLI (TSOP-II-44)."
Changed lines of the file:
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@@
 		(company "(c) 2025, 2026 Jason R. Thorpe.  All rights reserved.")
 	)
-	(text "Consider replacing with\nIS61C3216AL-12TLI (TSOP-II-44)."
-		(exclude_from_sim no)
-		(at 50.8 248.412 0)
-		(effects
-			(font
-				(size 1.27 1.27)
-			)
-		)
-	)
 	(text "Consider replcaing with\nAS7C4098A-12TIN (TSOP-II-44)."
 		(exclude_from_sim no)
@@
 		(on_board yes)
 		(dnp no)
-		(fields_autoplaced yes)
 		(property "Reference" "U303"
 			(at 101.2033 179.07 0)
@@
 			)
 		)
-		(property "Footprint" "Package_SO:SOJ-44_10.16x28.575mm_P1.27mm"
+		(property "Footprint" "Package_SO:TSOP-II-44_10.16x18.41mm_P0.8mm"
 			(at 50.8 172.72 0)
 			(effects
@@
 			)
 		)
-		(property "Part" "ISSI IS61C3216AL-12KLI"
+		(property "Part" "ISSI IS61C3216AL-12TLI"
 			(at 50.8 172.72 0)
 			(effects
@@
 			)
 		)
-		(property "LCSC" "C1351200"
+		(property "LCSC" "XXX"
 			(at 50.8 172.72 0)
 			(effects
@@
 			)
 		)
-		(property "Mouser" "870IS61C3216AL12KLI"
+		(property "Mouser" "870IS61C3216AL12TLI"
 			(at 50.8 172.72 0)
 			(effects

Commit message: Note the AS7C513B-12TCN is an alternative to the ISSI part.
Parts:
- U302: Alt (none) -> AS7C513B-12TCN; LCSC XXX -> C443415
Other:
- note added: "Alternative: AS7C513B-12TCN"
Changed lines of the file:
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@@
 		(company "(c) 2025, 2026 Jason R. Thorpe.  All rights reserved.")
 	)
+	(text "Alternative: AS7C513B-12TCN"
+		(exclude_from_sim no)
+		(at 51.308 248.92 0)
+		(effects
+			(font
+				(size 1.27 1.27)
+			)
+		)
+	)
 	(text "Consider replcaing with\nAS7C4098A-12TIN (TSOP-II-44)."
 		(exclude_from_sim no)
@@
 			)
 		)
-		(property "LCSC" "XXX"
+		(property "LCSC" "C443415"
 			(at 50.8 172.72 0)
 			(effects
@@
 			(at 50.8 172.72 0)
 			(effects
+				(font
+					(size 1.27 1.27)
+				)
+				(hide yes)
+			)
+		)
+		(property "Alt" "AS7C513B-12TCN"
+			(at 50.8 172.72 0)
+			(effects
