File: cpu010/design-files/cpu010-obio.kicad_sch (KiCad schematic)
At the start: 29 parts, among them J601 UART0 FTDI, J602 UART1 FTDI, J603 UART0, J604 UART1, J605 ATA Connector, J606 5V CF Power, J607 I2C, U601 ATF1508AS-TQFP100, U602 TL16C2552, U603 PCF8584, U604 DS3231MZ+, U605 74ACT245, U606 74ACT245, U607 74ACT245, Y601 1.8432MHz

Commit message: Route some bypass caps and the diagnostic display.
Parts:
- added C608: 100nF, Capacitor_SMD:C_0805_2012Metric_Pad1.18x1.45mm_HandSolder, symbol Device:C_Small
Connections:
- net +5V: now also C608.1
- net GND: now also C608.2
Changed lines of the file:
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@@
+	)
+	(junction
+		(at 110.49 274.32)
+		(diameter 0)
+		(color 0 0 0 0)
 	)
 	(junction
@@
 	)
 	(junction
+		(at 110.49 269.24)
+		(diameter 0)
+		(color 0 0 0 0)
+	)
+	(junction
 		(at 34.29 274.32)
 		(diameter 0)
@@
 	(wire
 		(pts
+			(xy 110.49 269.24) (xy 123.19 269.24)
+		)
+		(stroke
+			(width 0)
+			(type default)
+		)
+	)
+	(wire
+		(pts
 			(xy 294.64 241.3) (xy 294.64 233.68)
 		)
@@
 		(pts
 			(xy 190.5 31.75) (xy 195.58 31.75)
+		)
+		(stroke
+			(width 0)
+			(type default)
+		)
+	)
+	(wire
+		(pts
+			(xy 110.49 274.32) (xy 123.19 274.32)
 		)
 		(stroke
@@
 					(unit 1)
 				)
+			)
+		)
+	)
+	(symbol
+		(lib_id "Device:C_Small")
+		(at 123.19 271.78 0)
+		(unit 1)
+		(exclude_from_sim no)
+		(in_bom yes)
+		(on_board yes)
+		(dnp no)
+		(fields_autoplaced yes)
+		(property "Reference" "C608"
+			(at 125.73 270.5162 0)
+			(effects
+				(font
+					(size 1.27 1.27)
+				)
+				(justify left)
+			)
+		)
+		(property "Value" "100nF"
+			(at 125.73 273.0562 0)
+			(effects
+				(font
+					(size 1.27 1.27)
+				)
+				(justify left)
+			)
+		)
+		(property "Footprint" "Capacitor_SMD:C_0805_2012Metric_Pad1.18x1.45mm_HandSolder"
+			(at 123.19 271.78 0)
+			(effects
+				(font
+					(size 1.27 1.27)
+				)
+				(hide yes)
+			)
+		)
+		(property "Datasheet" "~"
+			(at 123.19 271.78 0)
+			(effects
+				(font
+					(size 1.27 1.27)
+				)
+				(hide yes)
+			)
+		)
+		(property "Description" "Unpolarized capacitor, small symbol"
+			(at 123.19 271.78 0)
+			(effects
+				(font
+					(size 1.27 1.27)
+				)
+				(hide yes)
+			)
+		)
+		(pin "1"
+		)
+		(pin "2"
+		)
+		(instances
+			(project "cpu010"
+				(path "/65f80d66-eea1-4882-b29a-ae1b65892b55/fbe8e7dc-2cbe-4b65-807d-71ce3f1eb657"
+					(reference "C608")
+					(unit 1)
+				)

Commit message: Routing some I/O stuff.
Parts:
- added RN602: 3K3, Resistor_THT:R_Array_SIP9, symbol Device:R_Network08
Connections:
- net A1 is gone; now on net VA1: U602.10 (A0), U603.6 (A0)
- net A2 is gone; now on net VA2: U602.14 (A1)
- net A3 is gone; now on net VA3: U602.15 (A2)
- net A8 is gone; now on net VA8: U602.16 (CHSEL)
- net +5V: now also RN602.1 (common)
- net ATA_A0: now also U607.4 (A2)
- net ATA_A1: now also U607.5 (A3)
- net ATA_A2: now also U607.6 (A4)
- net ATA_D0: now also U606.2 (A0); no longer U605.2 (A0)
- net ATA_D1: now also U606.3 (A1); no longer U605.3 (A1)
- net ATA_D10: now also U605.4 (A2); no longer U606.4 (A2)
- net ATA_D11: now also U605.5 (A3); no longer U606.5 (A3)
- net ATA_D12: now also U605.6 (A4); no longer U606.6 (A4)
- net ATA_D13: now also U605.7 (A5); no longer U606.7 (A5)
- net ATA_D14: now also U605.8 (A6); no longer U606.8 (A6)
- net ATA_D15: now also U605.9 (A7); no longer U606.9 (A7)
- net ATA_D2: now also U606.4 (A2); no longer U605.4 (A2)
- net ATA_D3: now also U606.5 (A3); no longer U605.5 (A3)
- net ATA_D4: now also U606.6 (A4); no longer U605.6 (A4)
- net ATA_D5: now also U606.7 (A5); no longer U605.7 (A5)
- net ATA_D6: now also U606.8 (A6); no longer U605.8 (A6)
- net ATA_D7: now also U606.9 (A7); no longer U605.9 (A7)
- net ATA_D8: now also U605.2 (A0); no longer U606.2 (A0)
- net ATA_D9: now also U605.3 (A1); no longer U606.3 (A1)
- net ATA_INT: now also U601.81 (I/O)
- net CLK10: now also U601.87 (I/GCLK1)
- net D0: now also U605.18 (B0); no longer U606.18 (B0)
- net D1: now also U605.17 (B1); no longer U606.17 (B1)
- net D10: now also U601.21 (I/O), U606.16 (B2); no longer U605.16 (B2)
- net D11: now also U601.22 (I/O), U606.15 (B3); no longer U605.15 (B3)
- net D12: now also U601.23 (I/O), U606.14 (B4); no longer U605.14 (B4)
- net D13: now also U601.24 (I/O), U606.13 (B5); no longer U605.13 (B5)
- net D14: now also U601.25 (I/O), U606.12 (B6); no longer U605.12 (B6)
- net D15: now also U601.27 (I/O), U606.11 (B7); no longer U605.11 (B7)
- net D2: now also U605.16 (B2); no longer U606.16 (B2)
- net D3: now also U605.15 (B3); no longer U606.15 (B3)
- net D4: now also U605.14 (B4); no longer U606.14 (B4)
- net D5: now also U605.13 (B5); no longer U606.13 (B5)
- net D6: now also U605.12 (B6); no longer U606.12 (B6)
- net D7: now also U605.11 (B7); no longer U606.11 (B7)
- net D8: now also U601.19 (I/O), U606.18 (B0); no longer U605.18 (B0)
- net D9: now also U601.20 (I/O), U606.17 (B1); no longer U605.17 (B1)
- net IO_RST: now also U601.2 (I/O)
- net R/~{W}: now also U601.6 (I/O)
- net UARTA_INT: now also U601.84 (I/O)
- net UARTB_INT: now also U601.85 (I/O/GCLK3)
- net ~{ATABEN}: now also U601.78 (I/O)
- net ~{ATA_CS1FX}: now also U607.2 (A0)
- net ~{ATA_CS3FX}: now also U607.3 (A1)
- net ~{ATA_IORD}: now also U607.8 (A6)
- net ~{ATA_IOWR}: now also U607.9 (A7)
- net ~{ATA_RST}: now also U607.7 (A5)
- net ~{DUARTSEL}: now also U601.83 (I/O)
- net ~{I2CSEL}: now also U601.77 (I/O)
- net ~{IO_RD}: now also U601.98 (I/O), U607.12 (B6)
- net ~{IO_WR}: now also U601.99 (I/O), U607.11 (B7)
- net ~{IRQ3}: now also U601.92 (I/O), RN602.2 (R1)
- net ~{RESET}: now also U601.89 (I/GCLR), U607.13 (B5)
- net VA3: now reaches U607.14 (B4)
- net VA3: now also U601.30 (I/O)
- net VA2: now reaches U607.15 (B3)
- net VA2: now also U601.29 (I/O)
- net VA1: now reaches U607.16 (B2)
- net VA1: now also U601.28 (I/O)
- net ~{ATAAUXSEL}: now reaches U607.17 (B1)
- net ~{ATAAUXSEL}: now also U601.80 (I/O)
- net ~{ATASEL}: now reaches U607.18 (B0)
- net ~{ATASEL}: now also U601.79 (I/O)
- net IOCTL_DTACK: now reaches U601.1 (I/O/PD1)
- net FC0: now reaches U601.10 (I/O)
- net ~{AVEC}: now reaches U601.100 (I/O)
- net FC1: now reaches U601.12 (I/O)
- net FC2: now reaches U601.13 (I/O)
- net IPL0: now reaches U601.14 (I/O)
- net IPL1: now reaches U601.16 (I/O)
- net IPL2: now reaches U601.17 (I/O)
- net VA4: now reaches U601.31 (I/O)
- net VA5: now reaches U601.32 (I/O)
- net VA6: now reaches U601.33 (I/O)
- net VA7: now reaches U601.35 (I/O)
- net VA8: now reaches U601.36 (I/O)
- net VA9: now reaches U601.37 (I/O)
- net VA10: now reaches U601.40 (I/O)
- net VA11: now reaches U601.41 (I/O/PD2)
- net A26: now reaches U601.42 (I/O)
- net A27: now reaches U601.44 (I/O)
- net VA16: now reaches U601.45 (I/O)
- net VA17: now reaches U601.46 (I/O)
- net VA18: now reaches U601.47 (I/O)
- net VA19: now reaches U601.48 (I/O)
- net ~{AS}: now reaches U601.5 (I/O)
- net ~{UDS}: now reaches U601.7 (I/O)
- net ~{EXPSEL}: now reaches U601.76 (I/O)
- net ~{LDS}: now reaches U601.8 (I/O)
- net ~{IRQ4}: now reaches U601.93 (I/O)
- net ~{IRQ4}: now also RN602.3 (R2)
- net ~{IRQ5}: now reaches U601.94 (I/O)
- net ~{IRQ5}: now also RN602.4 (R3)
- net ~{IRQ6}: now reaches U601.96 (I/O)
- net ~{IRQ6}: now also RN602.5 (R4)
- net ~{IRQ7}: now reaches U601.97 (I/O)
- net ~{IRQ7}: now also RN602.6 (R5)
- net ~{ATA_IO16}: no longer names the net of J605.32 (Pin_32)
- no-connect marks 17 -> 45
Other:
- moved on the sheet: D601, J605, J606, R603, R604, U605, U606, U607

Commit message: Expansion slots!
Changed lines of the file:
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@@
 	(wire
 		(pts
-			(xy 152.4 254) (xy 152.4 252.73)
-		)
-		(stroke
-			(width 0)
-			(type default)
-		)
-	)
-	(wire
-		(pts
 			(xy 132.08 179.07) (xy 132.08 177.8)
 		)
@@
 	(wire
 		(pts
-			(xy 152.4 251.46) (xy 152.4 250.19)
-		)
-		(stroke
-			(width 0)
-			(type default)
-		)
-	)
-	(wire
-		(pts
 			(xy 69.85 161.29) (xy 72.39 161.29)
 		)
@@
 	(wire
 		(pts
-			(xy 153.67 254) (xy 152.4 254)
-		)
-		(stroke
-			(width 0)
-			(type default)
-		)
-	)
-	(wire
-		(pts
 			(xy 260.35 157.48) (xy 260.35 170.18)
 		)
@@
 	(wire
 		(pts
-			(xy 153.67 251.46) (xy 152.4 251.46)
-		)
-		(stroke
-			(width 0)
-			(type default)
-		)
-	)
-	(wire
-		(pts
 			(xy 81.28 33.02) (xy 83.82 33.02)
 		)
@@
 		)
 	)
-	(label "SDA"
-		(at 140.97 212.09 180)
-		(effects
-			(font
-				(size 1.27 1.27)
-			)
-			(justify right bottom)
-		)
-	)
 	(label "~{UARTA_DTR}"
 		(at 218.44 58.42 0)
@@
 		)
 	)
-	(label "SDA"
-		(at 95.25 210.82 0)
-		(effects
-			(font
-				(size 1.27 1.27)
-			)
-			(justify left bottom)
-		)
-	)
-	(label "SCL"
-		(at 140.97 209.55 180)
-		(effects
-			(font
-				(size 1.27 1.27)
-			)
-			(justify right bottom)
-		)
-	)
 	(label "~{IO_RD}"
 		(at 105.41 55.88 0)
@@
 		)
 	)
-	(label "SCL"
-		(at 153.67 254 0)
-		(effects
-			(font
-				(size 1.27 1.27)
-			)
-			(justify left bottom)
-		)
-	)
 	(label "~{ATAAUXSEL}"
 		(at 242.57 154.94 0)
@@
 		)
 	)
-	(label "SCL"
-		(at 109.22 215.9 0)
-		(effects
-			(font
-				(size 1.27 1.27)
-			)
-			(justify left bottom)
-		)
-	)
 	(label "~{UARTA_CTS}"
 		(at 303.53 85.09 0)
@@
 		)
 	)
-	(label "SDA"
-		(at 153.67 251.46 0)
-		(effects
-			(font
-				(size 1.27 1.27)
-			)
-			(justify left bottom)
-		)
-	)
 	(label "ATA_D0"
 		(at 175.26 152.4 180)
@@
 		)
 	)
+	(global_label "SCL"
+		(shape output)
+		(at 109.22 215.9 0)
+		(fields_autoplaced yes)
+		(effects
+			(font
+				(size 1.27 1.27)
+			)
+			(justify left)
+		)
+		(property "Intersheetrefs" "${INTERSHEET_REFS}"
+			(at 115.7128 215.9 0)
+			(effects
+				(font
+					(size 1.27 1.27)
+				)
+				(justify left)
+				(hide yes)
+			)
+		)
+	)
 	(global_label "D9"
 		(shape bidirectional)
@@
 		)
 	)
+	(global_label "SCL"
+		(shape input)
+		(at 140.97 209.55 180)
+		(fields_autoplaced yes)
+		(effects
+			(font
+				(size 1.27 1.27)
+			)
+			(justify right)
+		)
+		(property "Intersheetrefs" "${INTERSHEET_REFS}"
+			(at 134.4772 209.55 0)
+			(effects
+				(font
+					(size 1.27 1.27)
+				)
+				(justify right)
+				(hide yes)
+			)
+		)
+	)
 	(global_label "D14"
 		(shape bidirectional)
@@
 		)
 	)
+	(global_label "SDA"
+		(shape bidirectional)
+		(at 95.25 210.82 0)
+		(fields_autoplaced yes)
+		(effects
+			(font
+				(size 1.27 1.27)
+			)
+			(justify left)
+		)
+		(property "Intersheetrefs" "${INTERSHEET_REFS}"
+			(at 102.9146 210.82 0)
+			(effects
+				(font
+					(size 1.27 1.27)
+				)
+				(justify left)
+				(hide yes)
+			)
+		)
+	)
 	(global_label "D12"
 		(shape bidirectional)
@@
 		)
 	)
+	(global_label "SDA"
+		(shape bidirectional)
+		(at 152.4 250.19 0)
+		(fields_autoplaced yes)
+		(effects
+			(font
+				(size 1.27 1.27)
+			)
+			(justify left)
+		)
+		(property "Intersheetrefs" "${INTERSHEET_REFS}"
+			(at 160.0646 250.19 0)
+			(effects
+				(font
+					(size 1.27 1.27)
+				)
+				(justify left)
+				(hide yes)
+			)
+		)
+	)
 	(global_label "VA2"
 		(shape input)
@@
 		)
 	)
+	(global_label "SDA"
+		(shape bidirectional)
+		(at 140.97 212.09 180)
+		(fields_autoplaced yes)
+		(effects
+			(font
+				(size 1.27 1.27)
+			)
+			(justify right)
+		)
+		(property "Intersheetrefs" "${INTERSHEET_REFS}"
+			(at 133.3054 212.09 0)
+			(effects
+				(font
+					(size 1.27 1.27)
+				)
+				(justify right)
+				(hide yes)
+			)
+		)
+	)
 	(global_label "D12"
 		(shape bidirectional)
@@
 			(effects
 				(font
+					(size 1.27 1.27)
+				)
+				(justify left)
+				(hide yes)
+			)
+		)
+	)
+	(global_label "SCL"
+		(shape input)
+		(at 152.4 252.73 0)
+		(fields_autoplaced yes)
+		(effects
+			(font
+				(size 1.27 1.27)
+			)
+			(justify left)
+		)
+		(property "Intersheetrefs" "${INTERSHEET_REFS}"
+			(at 158.8928 252.73 0)
+			(effects
+				(font

Commit message: More (NQ)VME tweaks.  Add JTAG chain.
Connections:
- net TMS: now reaches U601.15 (I/O/TMS)
- net TMS: now also U601.62 (I/O/TCK)
- net IOCTL_TDI: now reaches U601.4 (I/O/TDI)
- net MEMCTL_TDI: now reaches U601.73 (I/O/TDO)
Changed lines of the file:
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@@
+	(wire
+		(pts
+			(xy 107.95 120.65) (xy 104.14 120.65)
+		)
+		(stroke
+			(width 0)
+			(type default)
+		)
+	)
 	(wire
 		(pts
@@
 	(wire
 		(pts
+			(xy 35.56 85.09) (xy 48.26 85.09)
+		)
+		(stroke
+			(width 0)
+			(type default)
+		)
+	)
+	(wire
+		(pts
 			(xy 104.14 67.31) (xy 116.84 67.31)
 		)
@@
 	(wire
 		(pts
+			(xy 104.14 95.25) (xy 111.76 95.25)
+		)
+		(stroke
+			(width 0)
+			(type default)
+		)
+	)
+	(wire
+		(pts
 			(xy 81.28 33.02) (xy 83.82 33.02)
 		)
@@
 		(pts
 			(xy 90.17 215.9) (xy 106.68 215.9)
+		)
+		(stroke
+			(width 0)
+			(type default)
+		)
+	)
+	(wire
+		(pts
+			(xy 35.56 59.69) (xy 48.26 59.69)
 		)
 		(stroke
@@
 		)
 	)
+	(global_label "IOCTL_TDI"
+		(shape input)
+		(at 35.56 59.69 180)
+		(fields_autoplaced yes)
+		(effects
+			(font
+				(size 1.27 1.27)
+			)
+			(justify right)
+		)
+		(property "Intersheetrefs" "${INTERSHEET_REFS}"
+			(at 23.5638 59.69 0)
+			(effects
+				(font
+					(size 1.27 1.27)
+				)
+				(justify right)
+				(hide yes)
+			)
+		)
+	)
 	(global_label "R{slash}~{W}"
 		(shape input)
@@
 		)
 	)
+	(global_label "TMS"
+		(shape input)
+		(at 107.95 120.65 0)
+		(fields_autoplaced yes)
+		(effects
+			(font
+				(size 1.27 1.27)
+			)
+			(justify left)
+		)
+		(property "Intersheetrefs" "${INTERSHEET_REFS}"
+			(at 114.5637 120.65 0)
+			(effects
+				(font
+					(size 1.27 1.27)
+				)
+				(justify left)
+				(hide yes)
+			)
+		)
+	)
 	(global_label "D6"
 		(shape bidirectional)
@@
 		)
 	)
+	(global_label "TMS"
+		(shape input)
+		(at 35.56 85.09 180)
+		(fields_autoplaced yes)
+		(effects
+			(font
+				(size 1.27 1.27)
+			)
+			(justify right)
+		)
+		(property "Intersheetrefs" "${INTERSHEET_REFS}"
+			(at 28.9463 85.09 0)
+			(effects
+				(font
+					(size 1.27 1.27)
+				)
+				(justify right)
+				(hide yes)
+			)
+		)
+	)
 	(global_label "VA11"
 		(shape input)
@@
 			(effects
 				(font
+					(size 1.27 1.27)
+				)
+				(justify left)
+				(hide yes)
+			)
+		)
+	)
+	(global_label "MEMCTL_TDI"
+		(shape output)
+		(at 111.76 95.25 0)
+		(fields_autoplaced yes)
+		(effects
+			(font
+				(size 1.27 1.27)
+			)
+			(justify left)
+		)
+		(property "Intersheetrefs" "${INTERSHEET_REFS}"
+			(at 125.8727 95.25 0)
+			(effects
+				(font

Commit message: Clock generation is now done in the MMU, and we clock the MMU at 40MHz.
Connections:
- net CLK10 renamed CPU_CLK
- net CPU_CLK: no longer U603.1 (CLK)
- new net I2C_CLK: U603.1 (CLK)
Changed lines of the file:
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@@
 		)
 	)
-	(global_label "CLK10"
+	(global_label "I2C_CLK"
 		(shape input)
 		(at 52.07 241.3 180)
@@
 		)
 		(property "Intersheetrefs" "${INTERSHEET_REFS}"
-			(at 43.0977 241.3 0)
+			(at 41.4648 241.3 0)
 			(effects
 				(font
@@
 		)
 	)
-	(global_label "CLK10"
+	(global_label "CPU_CLK"
 		(shape input)
 		(at 48.26 49.53 180)
@@
 		)
 		(property "Intersheetrefs" "${INTERSHEET_REFS}"
-			(at 39.2877 49.53 0)
-			(effects
-				(font
+			(at 36.8686 49.53 0)
+			(effects
+				(font

Commit message: MMU now has Bus Error Register integrated.
Connections:
- net I2C_CLK is gone; now on net CPU_CLK: U603.1 (CLK)
- net INT_EN: now reaches U601.49 (I/O)
- no-connect marks 45 -> 44
Changed lines of the file:
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@@
 	)
 	(no_connect
-		(at 104.14 148.59)
-	)
-	(no_connect
 		(at 135.89 125.73)
 	)
@@
 		)
 	)
+	(wire
+		(pts
+			(xy 107.95 148.59) (xy 104.14 148.59)
+		)
+		(stroke
+			(width 0)
+			(type default)
+		)
+	)
 	(label "~{UARTA_CTS}"
 		(at 254 58.42 180)
@@
 		)
 	)
-	(global_label "I2C_CLK"
+	(global_label "CPU_CLK"
 		(shape input)
 		(at 52.07 241.3 180)
@@
 		)
 		(property "Intersheetrefs" "${INTERSHEET_REFS}"
-			(at 41.4648 241.3 0)
+			(at 40.6786 241.3 0)
 			(effects
 				(font
@@
 				(hide yes)
 			)
+		)
+	)
+	(global_label "INT_EN"
+		(shape input)
+		(at 107.95 148.59 0)
+		(fields_autoplaced yes)
+		(effects
+			(font
+				(size 1.27 1.27)
+			)
+			(justify left)
+		)
+		(property "Intersheetrefs" "${INTERSHEET_REFS}"
+			(at 117.2852 148.59 0)
+			(effects
+				(font
+					(size 1.27 1.27)
+				)
+				(justify left)
+				(hide yes)
+			)

Commit message: Hook up JTAG.
Connections:
- net TMS: no longer U601.62 (I/O/TCK)
- new net TCK: U601.62 (I/O/TCK)
Changed lines of the file:
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@@
 		)
 	)
-	(global_label "TMS"
+	(global_label "TCK"
 		(shape input)
 		(at 107.95 120.65 0)
@@
 		)
 		(property "Intersheetrefs" "${INTERSHEET_REFS}"
-			(at 114.5637 120.65 0)
+			(at 114.4428 120.65 0)
 			(effects
 				(font

Commit message: More routing of I/O signals.  Change the I2C pullups to 1K.
Parts:
- R601, R602: value 3K3 -> 1K
Changed lines of the file:
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@@
 			)
 		)
-		(property "Value" "3K3"
+		(property "Value" "1K"
 			(at 95.25 207.0099 0)
 			(effects
@@
 			)
 		)
-		(property "Value" "3K3"
+		(property "Value" "1K"
 			(at 109.22 207.0099 0)
 			(effects
