File: cpu010/design-files/cpu010-obio.kicad_sch (KiCad schematic)
At the start: 31 parts, among them J601 UART0 FTDI, J602 UART1 FTDI, J603 UART0, J604 UART1, J605 ATA Connector, J606 5V CF Power, J607 I2C, U601 ATF1508AS-TQFP100, U602 TL16C2552, U603 PCF8584, U604 DS3231MZ+, U605 74ACT245, U606 74ACT245, U607 74ACT245, Y601 1.8432MHz

Commit message: I2C controller now has dedicated interrupt input to IOCTL.
Parts:
- added R605: 1K, Resistor_SMD:R_0805_2012Metric_Pad1.20x1.40mm_HandSolder, symbol Device:R_Small
Connections:
- net +5V: now also R605.1
- net ~{EXPSEL}: now also U601.75 (I/O); no longer U601.76 (I/O)
- net ~{IRQ3}: no longer U603.5 (~{INT})
- new net ~{I2C_INT}: R605.2, U601.76 (I/O), U603.5 (~{INT})
- no-connect marks 44 -> 43
Changed lines of the file:
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@@
 	)
 	(junction
+		(at 106.68 236.22)
+		(diameter 0)
+		(color 0 0 0 0)
+	)
+	(junction
 		(at 78.74 33.02)
 		(diameter 0)
@@
 	)
 	(no_connect
-		(at 104.14 92.71)
-	)
-	(no_connect
 		(at 135.89 128.27)
 	)
@@
 	(wire
 		(pts
+			(xy 106.68 236.22) (xy 109.22 236.22)
+		)
+		(stroke
+			(width 0)
+			(type default)
+		)
+	)
+	(wire
+		(pts
 			(xy 67.31 161.29) (xy 69.85 161.29)
 		)
@@
 	(wire
 		(pts
+			(xy 104.14 92.71) (xy 105.41 92.71)
+		)
+		(stroke
+			(width 0)
+			(type default)
+		)
+	)
+	(wire
+		(pts
 			(xy 92.71 210.82) (xy 92.71 208.28)
 		)
@@
 	(wire
 		(pts
+			(xy 106.68 233.68) (xy 106.68 236.22)
+		)
+		(stroke
+			(width 0)
+			(type default)
+		)
+	)
+	(wire
+		(pts
 			(xy 260.35 157.48) (xy 260.35 170.18)
 		)
@@
 	(wire
 		(pts
-			(xy 90.17 236.22) (xy 92.71 236.22)
+			(xy 90.17 236.22) (xy 106.68 236.22)
 		)
 		(stroke
@@
 		)
 	)
+	(label "~{I2C_INT}"
+		(at 105.41 90.17 0)
+		(effects
+			(font
+				(size 1.27 1.27)
+			)
+			(justify left bottom)
+		)
+	)
 	(label "~{UARTA_CTS}"
 		(at 254 58.42 180)
@@
 		)
 	)
+	(label "~{I2C_INT}"
+		(at 109.22 236.22 0)
+		(effects
+			(font
+				(size 1.27 1.27)
+			)
+			(justify left bottom)
+		)
+	)
 	(label "ATA_D9"
 		(at 285.75 124.46 0)
@@
 	(global_label "~{EXPSEL}"
 		(shape output)
-		(at 105.41 90.17 0)
+		(at 105.41 92.71 0)
 		(fields_autoplaced yes)
 		(effects
@@
 		)
 		(property "Intersheetrefs" "${INTERSHEET_REFS}"
-			(at 115.4103 90.17 0)
+			(at 115.4103 92.71 0)
 			(effects
 				(font
@@
 		)
 	)
-	(global_label "~{IRQ3}"
-		(shape output)
-		(at 92.71 236.22 0)
-		(fields_autoplaced yes)
-		(effects
-			(font
-				(size 1.27 1.27)
-			)
-			(justify left)
-		)
-		(property "Intersheetrefs" "${INTERSHEET_REFS}"
-			(at 100.11 236.22 0)
-			(effects
-				(font
-					(size 1.27 1.27)
-				)
-				(justify left)
-				(hide yes)
-			)
-		)
-	)
 	(global_label "D8"
 		(shape bidirectional)
@@
 	(symbol
 		(lib_id "power:+5V")
+		(at 106.68 228.6 0)
+		(unit 1)
+		(exclude_from_sim no)
+		(in_bom yes)
+		(on_board yes)
+		(dnp no)
+		(fields_autoplaced yes)
+		(property "Reference" "#PWR0639"
+			(at 106.68 232.41 0)
+			(effects
+				(font
+					(size 1.27 1.27)
+				)
+				(hide yes)
+			)
+		)
+		(property "Value" "+5V"
+			(at 106.68 223.52 0)
+			(effects
+				(font
+					(size 1.27 1.27)
+				)
+			)
+		)
+		(property "Footprint" ""
+			(at 106.68 228.6 0)
+			(effects
+				(font
+					(size 1.27 1.27)
+				)
+				(hide yes)
+			)
+		)
+		(property "Datasheet" ""
+			(at 106.68 228.6 0)
+			(effects
+				(font
+					(size 1.27 1.27)
+				)
+				(hide yes)
+			)
+		)
+		(property "Description" "Power symbol creates a global label with name \"+5V\""
+			(at 106.68 228.6 0)
+			(effects
+				(font
+					(size 1.27 1.27)
+				)
+				(hide yes)
+			)
+		)
+		(pin "1"
+		)
+		(instances
+			(project "cpu010"
+				(path "/65f80d66-eea1-4882-b29a-ae1b65892b55/fbe8e7dc-2cbe-4b65-807d-71ce3f1eb657"
+					(reference "#PWR0639")
+					(unit 1)
+				)
+			)
+		)
+	)
+	(symbol
+		(lib_id "power:+5V")
 		(at 153.67 204.47 0)
 		(unit 1)
@@
 					(unit 1)
 				)
+			)
+		)
+	)
+	(symbol
+		(lib_id "Device:R_Small")
+		(at 106.68 231.14 0)
+		(unit 1)
+		(exclude_from_sim no)
+		(in_bom yes)
+		(on_board yes)
+		(dnp no)
+		(property "Reference" "R605"
+			(at 109.22 229.8699 0)
+			(effects
+				(font
+					(size 1.016 1.016)
+				)
+				(justify left)
+			)
+		)
+		(property "Value" "1K"
+			(at 109.22 232.4099 0)
+			(effects
+				(font
+					(size 1.27 1.27)
+				)
+				(justify left)
+			)
+		)
+		(property "Footprint" "Resistor_SMD:R_0805_2012Metric_Pad1.20x1.40mm_HandSolder"
+			(at 106.68 231.14 0)
+			(effects
+				(font
+					(size 1.27 1.27)
+				)
+				(hide yes)
+			)
+		)
+		(property "Datasheet" "~"
+			(at 106.68 231.14 0)
+			(effects
+				(font
+					(size 1.27 1.27)
+				)
+				(hide yes)
+			)
+		)
+		(property "Description" "Resistor, small symbol"
+			(at 106.68 231.14 0)
+			(effects
+				(font
+					(size 1.27 1.27)
+				)
+				(hide yes)
+			)
+		)
+		(pin "1"
+		)
+		(pin "2"
+		)
+		(instances
+			(project "cpu010"
+				(path "/65f80d66-eea1-4882-b29a-ae1b65892b55/fbe8e7dc-2cbe-4b65-807d-71ce3f1eb657"
+					(reference "R605")
+					(unit 1)
+				)

Commit message: Auto-vector interrupts are signalled via /VPA on the 68010.
Connections:
- net ~{AVEC} renamed ~{VPA}
Changed lines of the file:
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@@
 	(wire
 		(pts
+			(xy 105.41 49.53) (xy 104.14 49.53)
+		)
+		(stroke
+			(width 0)
+			(type default)
+		)
+	)
+	(wire
+		(pts
 			(xy 77.47 161.29) (xy 80.01 161.29)
 		)
@@
 	(wire
 		(pts
-			(xy 104.14 52.07) (xy 111.76 52.07)
+			(xy 104.14 52.07) (xy 116.84 52.07)
 		)
 		(stroke
@@
 	)
 	(label "~{IO_WR}"
-		(at 111.76 52.07 0)
+		(at 116.84 52.07 0)
 		(effects
 			(font
@@
 		)
 	)
-	(global_label "~{AVEC}"
+	(global_label "~{VPA}"
 		(shape output)
-		(at 104.14 49.53 0)
+		(at 105.41 49.53 0)
 		(fields_autoplaced yes)
 		(effects
@@
 		)
 		(property "Intersheetrefs" "${INTERSHEET_REFS}"
-			(at 111.7214 49.53 0)
+			(at 111.8424 49.53 0)
 			(effects
 				(font

Commit message: Wire up UART interrupts.
Parts:
- added R606, R607: 47K, Resistor_SMD:R_0805_2012Metric_Pad1.20x1.40mm_HandSolder, symbol Device:R_Small
Connections:
- net GND: now also R606.1, R607.1
- net UARTA_INT: now also R607.2
- net UARTB_INT: now also R606.2

Commit message: Add pull-ups to the ATA data bus.
Parts:
- added RN603, RN604: 3K3, Resistor_THT:R_Array_SIP9, symbol Device:R_Network08
Connections:
- net +5V: now also RN603.1 (common), RN604.1 (common)
- net ATA_D0: now also RN603.9 (R8)
- net ATA_D1: now also RN603.8 (R7)
- net ATA_D10: now also RN604.4 (R3)
- net ATA_D11: now also RN604.5 (R4)
- net ATA_D12: now also RN604.6 (R5)
- net ATA_D13: now also RN604.7 (R6)
- net ATA_D14: now also RN604.8 (R7)
- net ATA_D15: now also RN604.9 (R8)
- net ATA_D2: now also RN603.7 (R6)
- net ATA_D3: now also RN603.6 (R5)
- net ATA_D4: now also RN603.5 (R4)
- net ATA_D5: now also RN603.4 (R3)
- net ATA_D6: now also RN603.3 (R2)
- net ATA_D7: now also RN603.2 (R1)
- net ATA_D8: now also RN604.2 (R1)
- net ATA_D9: now also RN604.3 (R2)

Commit message: Add some passives for signal integrity, work on some additional signal routing.
Parts:
- added R608, R609, R610, R611: 33R, Resistor_SMD:R_0805_2012Metric_Pad1.20x1.40mm_HandSolder, symbol Device:R_Small
- added R612: 1K, Resistor_SMD:R_0805_2012Metric_Pad1.20x1.40mm_HandSolder, symbol Device:R_Small
- added R613: 10K, Resistor_SMD:R_0805_2012Metric_Pad1.20x1.40mm_HandSolder, symbol Device:R_Small
- added RN605: 10K, Resistor_THT:R_Array_SIP9, symbol Device:R_Network08
- R603, R606, R607: value 47K -> 10K
- RN601, RN603, RN604: value 3K3 -> 10K
Connections:
- net +5V: now also R612.1, R613.1, RN605.1 (common)
- net ATA_A0: now also RN605.7 (R6)
- net ATA_A1: now also RN605.5 (R4)
- net ATA_A2: now also RN605.6 (R5)
- net ATA_RDY: now also U601.72 (I/O), R612.2
- net ~{ATA_CS1FX}: now also R608.2, RN605.9 (R8); no longer U607.2 (A0)
- net ~{ATA_CS3FX}: now also R609.2, RN605.8 (R7); no longer U607.3 (A1)
- net ~{ATA_IORD}: now also R610.2, RN605.3 (R2); no longer U607.8 (A6)
- net ~{ATA_IOWR}: now also R611.2, RN605.2 (R1); no longer U607.9 (A7)
- net ~{ATA_RST}: now also RN605.4 (R3)
- net at D601.1 (K), J605.39 (Pin_39): now also R613.2
- new net: R608.1, U607.2 (A0)
- new net: R609.1, U607.3 (A1)
- new net: R610.1, U607.8 (A6)
- new net: R611.1, U607.9 (A7)
- no-connect marks 43 -> 42
Other:
- moved on the sheet: U607

Commit message: Beef up the power supply a little.
Parts:
- added C609, C610: 100µF, Capacitor_THT:CP_Radial_D6.3mm_P2.50mm, symbol Device:C_Polarized_Small
Connections:
- net +5V: now also C609.1, C610.1
- net GND: now also C609.2, C610.2
Changed lines of the file:
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@@
 	)
 	(junction
+		(at 134.62 269.24)
+		(diameter 0)
+		(color 0 0 0 0)
+	)
+	(junction
 		(at 190.5 31.75)
 		(diameter 0)
@@
 	)
 	(junction
+		(at 123.19 269.24)
+		(diameter 0)
+		(color 0 0 0 0)
+	)
+	(junction
 		(at 190.5 118.11)
 		(diameter 0)
@@
 	)
 	(junction
+		(at 123.19 274.32)
+		(diameter 0)
+		(color 0 0 0 0)
+	)
+	(junction
 		(at 67.31 161.29)
 		(diameter 0)
@@
 	)
 	(junction
+		(at 134.62 274.32)
+		(diameter 0)
+		(color 0 0 0 0)
+	)
+	(junction
 		(at 59.69 269.24)
 		(diameter 0)
@@
 	(wire
 		(pts
+			(xy 134.62 274.32) (xy 146.05 274.32)
+		)
+		(stroke
+			(width 0)
+			(type default)
+		)
+	)
+	(wire
+		(pts
 			(xy 130.81 179.07) (xy 132.08 179.07)
 		)
@@
 	(wire
 		(pts
+			(xy 123.19 269.24) (xy 134.62 269.24)
+		)
+		(stroke
+			(width 0)
+			(type default)
+		)
+	)
+	(wire
+		(pts
 			(xy 323.85 146.05) (xy 327.66 146.05)
 		)
@@
 	(wire
 		(pts
+			(xy 134.62 269.24) (xy 146.05 269.24)
+		)
+		(stroke
+			(width 0)
+			(type default)
+		)
+	)
+	(wire
+		(pts
 			(xy 46.99 58.42) (xy 48.26 58.42)
 		)
@@
 	(wire
 		(pts
+			(xy 123.19 274.32) (xy 134.62 274.32)
+		)
+		(stroke
+			(width 0)
+			(type default)
+		)
+	)
+	(wire
+		(pts
 			(xy 210.82 186.69) (xy 215.9 186.69)
 		)
@@
 	)
 	(symbol
+		(lib_id "Device:C_Polarized_Small")
+		(at 146.05 271.78 0)
+		(unit 1)
+		(exclude_from_sim no)
+		(in_bom yes)
+		(on_board yes)
+		(dnp no)
+		(fields_autoplaced yes)
+		(property "Reference" "C610"
+			(at 148.59 269.9638 0)
+			(effects
+				(font
+					(size 1.27 1.27)
+				)
+				(justify left)
+			)
+		)
+		(property "Value" "100µF"
+			(at 148.59 272.5038 0)
+			(effects
+				(font
+					(size 1.27 1.27)
+				)
+				(justify left)
+			)
+		)
+		(property "Footprint" "Capacitor_THT:CP_Radial_D6.3mm_P2.50mm"
+			(at 146.05 271.78 0)
+			(effects
+				(font
+					(size 1.27 1.27)
+				)
+				(hide yes)
+			)
+		)
+		(property "Datasheet" "~"
+			(at 146.05 271.78 0)
+			(effects
+				(font
+					(size 1.27 1.27)
+				)
+				(hide yes)
+			)
+		)
+		(property "Description" "Polarized capacitor, small symbol"
+			(at 146.05 271.78 0)
+			(effects
+				(font
+					(size 1.27 1.27)
+				)
+				(hide yes)
+			)
+		)
+		(property "Part" "Wurth 860040373002"
+			(at 146.05 271.78 0)
+			(effects
+				(font
+					(size 1.27 1.27)
+				)
+				(hide yes)
+			)
+		)
+		(pin "2"
+		)
+		(pin "1"
+		)
+		(instances
+			(project "cpu010"
+				(path "/65f80d66-eea1-4882-b29a-ae1b65892b55/fbe8e7dc-2cbe-4b65-807d-71ce3f1eb657"
+					(reference "C610")
+					(unit 1)
+				)
+			)
+		)
+	)
+	(symbol
 		(lib_id "power:+5V")
 		(at 92.71 203.2 0)
@@
 					(unit 1)
 				)
+			)
+		)
+	)
+	(symbol
+		(lib_id "Device:C_Polarized_Small")
+		(at 134.62 271.78 0)
+		(unit 1)
+		(exclude_from_sim no)
+		(in_bom yes)
+		(on_board yes)
+		(dnp no)
+		(fields_autoplaced yes)
+		(property "Reference" "C609"
+			(at 137.16 269.9638 0)
+			(effects
+				(font
+					(size 1.27 1.27)
+				)
+				(justify left)
+			)
+		)
+		(property "Value" "100µF"
+			(at 137.16 272.5038 0)
+			(effects
+				(font
+					(size 1.27 1.27)
+				)
+				(justify left)
+			)
+		)
+		(property "Footprint" "Capacitor_THT:CP_Radial_D6.3mm_P2.50mm"
+			(at 134.62 271.78 0)
+			(effects
+				(font
+					(size 1.27 1.27)
+				)
+				(hide yes)
+			)
+		)
+		(property "Datasheet" "~"
+			(at 134.62 271.78 0)
+			(effects
+				(font
+					(size 1.27 1.27)
+				)
+				(hide yes)
+			)
+		)
+		(property "Description" "Polarized capacitor, small symbol"
+			(at 134.62 271.78 0)
+			(effects
+				(font
+					(size 1.27 1.27)
+				)
+				(hide yes)
+			)
+		)
+		(property "Part" "Wurth 860040373002"
+			(at 134.62 271.78 0)
+			(effects
+				(font
+					(size 1.27 1.27)
+				)
+				(hide yes)
+			)
+		)
+		(pin "2"
+		)
+		(pin "1"
+		)
+		(instances
+			(project "cpu010"
+				(path "/65f80d66-eea1-4882-b29a-ae1b65892b55/fbe8e7dc-2cbe-4b65-807d-71ce3f1eb657"
+					(reference "C609")
+					(unit 1)
+				)

Commit message: More component labeling.
Parts:
- RN601, RN603, RN604, RN605: Mouser (none) -> 652-4609X-1LF-10K
- RN602: Mouser (none) -> 652-4609X-1LF-3.3K
- U601: JLCPCB (none) -> C1521282; Mouser (none) -> 556-AF1508AS7AX100; Part (none) -> ATF1508AS-7AX100
- U602: Mouser (none) -> 595-TL16C2552FN
- U604: Mouser (none) -> 700-DS3231MZ+
- U605, U606, U607: Mouser (none) -> 595-SN74ACT245N
- Y601: Mouser (none) -> 774-MXO45HST-3C-1.8; Part (none) -> MXO45HST-3C-1M8432
Changed lines of the file:
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@@
 			)
 		)
+		(property "Part" "MXO45HST-3C-1M8432"
+			(at 140.97 85.09 0)
+			(effects
+				(font
+					(size 1.27 1.27)
+				)
+				(hide yes)
+			)
+		)
+		(property "Mouser" "774-MXO45HST-3C-1.8"
+			(at 140.97 85.09 0)
+			(effects
+				(font
+					(size 1.27 1.27)
+				)
+				(hide yes)
+			)
+		)
 		(pin "5"
 		)
@@
 			)
 		)
+		(property "Mouser" "595-TL16C2552FN"
+			(at 193.04 74.93 0)
+			(effects
+				(font
+					(size 1.27 1.27)
+				)
+				(hide yes)
+			)
+		)
 		(pin "18"
 		)
@@
 			)
 		)
+		(property "Mouser" "595-SN74ACT245N"
+			(at 242.57 199.39 0)
+			(effects
+				(font
+					(size 1.27 1.27)
+				)
+				(hide yes)
+			)
+		)
 		(pin "6"
 		)
@@
 			)
 		)
+		(property "Mouser" "652-4609X-1LF-10K"
+			(at 318.77 186.69 90)
+			(effects
+				(font
+					(size 1.27 1.27)
+				)
+				(hide yes)
+			)
+		)
 		(pin "3"
 		)
@@
 			)
 		)
+		(property "Mouser" "595-SN74ACT245N"
+			(at 187.96 165.1 0)
+			(effects
+				(font
+					(size 1.27 1.27)
+				)
+				(hide yes)
+			)
+		)
 		(pin "6"
 		)
@@
 			)
 		)
+		(property "Mouser" "652-4609X-1LF-3.3K"
+			(at 140.97 120.65 90)
+			(effects
+				(font
+					(size 1.27 1.27)
+				)
+				(hide yes)
+			)
+		)
 		(pin "3"
 		)
@@
 			)
 		)
+		(property "Mouser" "700-DS3231MZ+"
+			(at 153.67 214.63 0)
+			(effects
+				(font
+					(size 1.27 1.27)
+				)
+				(hide yes)
+			)
+		)
 		(pin "8"
 		)
@@
 			)
 		)
+		(property "Mouser" "595-SN74ACT245N"
+			(at 144.78 165.1 0)
+			(effects
+				(font
+					(size 1.27 1.27)
+				)
+				(hide yes)
+			)
+		)
 		(pin "6"
 		)
@@
 			)
 		)
+		(property "Mouser" "652-4609X-1LF-10K"
+			(at 318.77 156.21 90)
+			(effects
+				(font
+					(size 1.27 1.27)
+				)
+				(hide yes)
+			)
+		)
 		(pin "3"
 		)
@@
 			)
 		)
+		(property "Mouser" "652-4609X-1LF-10K"
+			(at 259.08 50.8 90)
+			(effects
+				(font
+					(size 1.27 1.27)
+				)
+				(hide yes)
+			)
+		)
 		(pin "3"
 		)
@@
 			)
 		)
+		(property "Part" "ATF1508AS-7AX100"
+			(at 76.2 90.17 0)
+			(effects
+				(font
+					(size 1.27 1.27)
+				)
+				(hide yes)
+			)
+		)
+		(property "JLCPCB" "C1521282"
+			(at 76.2 90.17 0)
+			(effects
+				(font
+					(size 1.27 1.27)
+				)
+				(hide yes)
+			)
+		)
+		(property "Mouser" "556-AF1508AS7AX100"
+			(at 76.2 90.17 0)
+			(effects
+				(font
+					(size 1.27 1.27)
+				)
+				(hide yes)
+			)
+		)
 		(pin "33"
 		)
@@
 			(effects
 				(font
+					(size 1.27 1.27)
+				)
+				(hide yes)
+			)
+		)
+		(property "Mouser" "652-4609X-1LF-10K"
+			(at 318.77 125.73 90)
+			(effects
+				(font

Commit message: Connect missing GND pin on ATA connector.
Connections:
- net GND: now also J605.2 (Pin_2)
Changed lines of the file:
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@@
 	(wire
 		(pts
+			(xy 285.75 119.38) (xy 294.64 119.38)
+		)
+		(stroke
+			(width 0)
+			(type default)
+		)
+	)
+	(wire
+		(pts
 			(xy 104.14 95.25) (xy 111.76 95.25)
 		)
@@
 					(unit 1)
 				)
+			)
+		)
+	)
+	(symbol
+		(lib_id "power:GND")
+		(at 294.64 119.38 90)
+		(unit 1)
+		(exclude_from_sim no)
+		(in_bom yes)
+		(on_board yes)
+		(dnp no)
+		(fields_autoplaced yes)
+		(property "Reference" "#PWR0646"
+			(at 300.99 119.38 0)
+			(effects
+				(font
+					(size 1.27 1.27)
+				)
+				(hide yes)
+			)
+		)
+		(property "Value" "GND"
+			(at 298.45 119.3799 90)
+			(effects
+				(font
+					(size 1.27 1.27)
+				)
+				(justify right)
+			)
+		)
+		(property "Footprint" ""
+			(at 294.64 119.38 0)
+			(effects
+				(font
+					(size 1.27 1.27)
+				)
+				(hide yes)
+			)
+		)
+		(property "Datasheet" ""
+			(at 294.64 119.38 0)
+			(effects
+				(font
+					(size 1.27 1.27)
+				)
+				(hide yes)
+			)
+		)
+		(property "Description" "Power symbol creates a global label with name \"GND\" , ground"
+			(at 294.64 119.38 0)
+			(effects
+				(font
+					(size 1.27 1.27)
+				)
+				(hide yes)
+			)
+		)
+		(pin "1"
+		)
+		(instances
+			(project "cpu010"
+				(path "/65f80d66-eea1-4882-b29a-ae1b65892b55/fbe8e7dc-2cbe-4b65-807d-71ce3f1eb657"
+					(reference "#PWR0646")
+					(unit 1)
+				)
