File: cpu010/design-files/cpu010-expansion.kicad_sch (KiCad schematic)
At the start: 6 parts, among them J701 Expansion Slot 1, J702 Expansion Slot 2, J703 Expansion Slot 3, U701 74ACT245, U702 74ACT245, U703 74HC08

Commit message: More (NQ)VME tweaks.  Add JTAG chain.
Parts:
- removed U703: 74HC08, Package_DIP:DIP-14_W7.62mm_Socket, symbol 74xx:74LS08
- added C701, C702, C703, C704, C705: 100nF, Capacitor_SMD:C_0805_2012Metric_Pad1.18x1.45mm_HandSolder, symbol Device:C_Small
- added R701, R702: 470R, Resistor_SMD:R_0805_2012Metric_Pad1.20x1.40mm_HandSolder, symbol Device:R_Small
- added RN701, RN702: 3K3, Resistor_THT:R_Array_SIP9, symbol Device:R_Network08
- added U703: GAL22V10, Package_DIP:DIP-24_W7.62mm_Socket, symbol jrt-ICs:GAL22V10
- added U704: 74ACT32, Package_DIP:DIP-14_W7.62mm_Socket, symbol 74xx:74LS32
- added U705: 74ACT245, Package_DIP:DIP-20_W7.62mm_Socket, symbol 74xx:74HC245
- J701: value Expansion Slot 1 -> NQVME Slot 1
- J702: value Expansion Slot 2 -> NQVME Slot 2
- J703: value Expansion Slot 3 -> NQVME Slot 3
Connections:
- net +5V: now also C701.1, C702.1, C703.1, C704.1, C705.1, R701.1, R702.1, RN701.1 (common), RN702.1 (common), U703.24 (VCC), U704.14 (VCC), U705.1 (A->B), U705.20 (VCC)
- net A23: now also U703.5 (I5)
- net A24: now also U703.6 (I6); no longer J701.b16 (Pin_b16), J702.b16 (Pin_b16), J703.b16 (Pin_b16)
- net A25: now also U703.7 (I7); no longer J701.b17 (Pin_b17), J702.b17 (Pin_b17), J703.b17 (Pin_b17)
- net D0: no longer J701.a1 (Pin_a1), J702.a1 (Pin_a1), J703.a1 (Pin_a1)
- net D1: no longer J701.a2 (Pin_a2), J702.a2 (Pin_a2), J703.a2 (Pin_a2)
- net D10: no longer J701.c3 (Pin_c3), J702.c3 (Pin_c3), J703.c3 (Pin_c3)
- net D11: no longer J701.c4 (Pin_c4), J702.c4 (Pin_c4), J703.c4 (Pin_c4)
- net D12: no longer J701.c5 (Pin_c5), J702.c5 (Pin_c5), J703.c5 (Pin_c5)
- net D13: no longer J701.c6 (Pin_c6), J702.c6 (Pin_c6), J703.c6 (Pin_c6)
- net D14: no longer J701.c7 (Pin_c7), J702.c7 (Pin_c7), J703.c7 (Pin_c7)
- net D15: no longer J701.c8 (Pin_c8), J702.c8 (Pin_c8), J703.c8 (Pin_c8)
- net D2: no longer J701.a3 (Pin_a3), J702.a3 (Pin_a3), J703.a3 (Pin_a3)
- net D3: no longer J701.a4 (Pin_a4), J702.a4 (Pin_a4), J703.a4 (Pin_a4)
- net D4: no longer J701.a5 (Pin_a5), J702.a5 (Pin_a5), J703.a5 (Pin_a5)
- net D5: no longer J701.a6 (Pin_a6), J702.a6 (Pin_a6), J703.a6 (Pin_a6)
- net D6: no longer J701.a7 (Pin_a7), J702.a7 (Pin_a7), J703.a7 (Pin_a7)
- net D7: no longer J701.a8 (Pin_a8), J702.a8 (Pin_a8), J703.a8 (Pin_a8)
- net D8: no longer J701.c1 (Pin_c1), J702.c1 (Pin_c1), J703.c1 (Pin_c1)
- net D9: no longer J701.c2 (Pin_c2), J702.c2 (Pin_c2), J703.c2 (Pin_c2)
- net EXP_D0: now also J701.a1 (Pin_a1), J702.a1 (Pin_a1), J703.a1 (Pin_a1), RN702.2 (R1)
- net EXP_D1: now also J701.a2 (Pin_a2), J702.a2 (Pin_a2), J703.a2 (Pin_a2), RN702.3 (R2)
- net EXP_D10: now also J701.c3 (Pin_c3), J702.c3 (Pin_c3), J703.c3 (Pin_c3), RN701.4 (R3)
- net EXP_D11: now also J701.c4 (Pin_c4), J702.c4 (Pin_c4), J703.c4 (Pin_c4), RN701.5 (R4)
- net EXP_D12: now also J701.c5 (Pin_c5), J702.c5 (Pin_c5), J703.c5 (Pin_c5), RN701.6 (R5)
- net EXP_D13: now also J701.c6 (Pin_c6), J702.c6 (Pin_c6), J703.c6 (Pin_c6), RN701.7 (R6)
- net EXP_D14: now also J701.c7 (Pin_c7), J702.c7 (Pin_c7), J703.c7 (Pin_c7), RN701.8 (R7)
- net EXP_D15: now also J701.c8 (Pin_c8), J702.c8 (Pin_c8), J703.c8 (Pin_c8), RN701.9 (R8)
- net EXP_D2: now also J701.a3 (Pin_a3), J702.a3 (Pin_a3), J703.a3 (Pin_a3), RN702.4 (R3)
- net EXP_D3: now also J701.a4 (Pin_a4), J702.a4 (Pin_a4), J703.a4 (Pin_a4), RN702.5 (R4)
- net EXP_D4: now also J701.a5 (Pin_a5), J702.a5 (Pin_a5), J703.a5 (Pin_a5), RN702.6 (R5)
- net EXP_D5: now also J701.a6 (Pin_a6), J702.a6 (Pin_a6), J703.a6 (Pin_a6), RN702.7 (R6)
- net EXP_D6: now also J701.a8 (Pin_a8), J702.a8 (Pin_a8), J703.a8 (Pin_a8), RN702.9 (R8)
- net EXP_D7: now also J701.a7 (Pin_a7), J702.a7 (Pin_a7), J703.a7 (Pin_a7), RN702.8 (R7)
- net EXP_D8: now also J701.c1 (Pin_c1), J702.c1 (Pin_c1), J703.c1 (Pin_c1), RN701.2 (R1)
- net EXP_D9: now also J701.c2 (Pin_c2), J702.c2 (Pin_c2), J703.c2 (Pin_c2), RN701.3 (R2)
- net GND: now also C701.2, C702.2, C703.2, C704.2, C705.2, U703.12 (GND), U704.12, U704.13, U704.7 (GND), U705.10 (GND), U705.19 (CE), U705.2 (A0)
- net R/~{W}: now also U705.3 (A1); no longer J701.a14 (Pin_a14), J702.a14 (Pin_a14), J703.a14 (Pin_a14)
- net ~{AS}: now also U704.1; no longer J701.a18 (Pin_a18), J702.a18 (Pin_a18), J703.a18 (Pin_a18)
- net ~{EXPRAMSEL}: now also U703.11 (I11); no longer J701.b18 (Pin_b18), J702.b18 (Pin_b18), J703.b18 (Pin_b18)
- net ~{EXPSEL}: now also U703.1 (I1/CLK); no longer J701.b19 (Pin_b19), J702.b19 (Pin_b19), J703.b19 (Pin_b19)
- net ~{LDS}: now also U704.9; no longer J701.a13 (Pin_a13), J702.a13 (Pin_a13), J703.a13 (Pin_a13)
- net ~{UDS}: now also U704.4; no longer J701.a12 (Pin_a12), J702.a12 (Pin_a12), J703.a12 (Pin_a12)
- net ~{EXP_IACK}: now reaches J703.a20 (Pin_a20)
- net ~{EXP_IACK}: now also J701.a20 (Pin_a20), J702.a20 (Pin_a20), R702.2
- net ~{EXP3_IACKIN}: now reaches J703.a21 (Pin_a21)
- net ~{EXP3_IACKIN}: now also J702.a22 (Pin_a22)
- net EXP_AM4: now reaches J703.a23 (Pin_a23)
- net EXP_AM4: now also J701.a23 (Pin_a23), J702.a23 (Pin_a23), U705.15 (B3)
- net ~{EXP3_BG3IN}: now reaches J703.b10 (Pin_b10)
- net ~{EXP3_BG3IN}: now also J702.b11 (Pin_b11)
- net ~{EXP3_BG0IN}: now reaches J703.b4 (Pin_b4)
- net ~{EXP3_BG0IN}: now also J702.b5 (Pin_b5)
- net ~{EXP3_BG1IN}: now reaches J703.b6 (Pin_b6)
- net ~{EXP3_BG1IN}: now also J702.b7 (Pin_b7)
- net ~{EXP3_BG2IN}: now reaches J703.b8 (Pin_b8)
- net ~{EXP3_BG2IN}: now also J702.b9 (Pin_b9)
- net EXP_AM5: now reaches J703.c14 (Pin_c14)
- net EXP_AM5: now also J701.c14 (Pin_c14), J702.c14 (Pin_c14), U705.16 (B2)
- net ~{VMESEL}: now reaches U701.19 (CE), U702.19 (CE)
- net ~{VMESEL}: now also U703.23 (IO10), U704.10, U704.2, U704.5
- net ~{EXP1_BG0IN}: now reaches J701.a21 (Pin_a21)
- net ~{EXP1_BG0IN}: now also J701.b10 (Pin_b10), J701.b4 (Pin_b4), J701.b6 (Pin_b6), J701.b8 (Pin_b8), R701.2
- net ~{EXP2_IACKIN}: now reaches J701.a22 (Pin_a22)
- net ~{EXP2_IACKIN}: now also J702.a21 (Pin_a21)
- net ~{EXP2_BG3IN}: now reaches J701.b11 (Pin_b11)
- net ~{EXP2_BG3IN}: now also J702.b10 (Pin_b10)
- net ~{EXP2_BG0IN}: now reaches J701.b5 (Pin_b5)
- net ~{EXP2_BG0IN}: now also J702.b4 (Pin_b4)
- net ~{EXP2_BG1IN}: now reaches J701.b7 (Pin_b7)
- net ~{EXP2_BG1IN}: now also J702.b6 (Pin_b6)
- net ~{EXP2_BG2IN}: now reaches J701.b9 (Pin_b9)
- net ~{EXP2_BG2IN}: now also J702.b8 (Pin_b8)
- new net: U703.17 (IO4), U705.4 (A2)
- new net: U703.18 (IO5), U705.5 (A3)
- new net: U703.19 (IO6), U705.6 (A4)
- new net: U703.20 (IO7), U705.7 (A5)
- new net: U703.21 (IO8), U705.8 (A6)
- new net: U703.22 (IO9), U705.9 (A7)
- new net EXP_AM0: J701.b16 (Pin_b16), J702.b16 (Pin_b16), J703.b16 (Pin_b16), U705.11 (B7)
- new net EXP_AM1: J701.b17 (Pin_b17), J702.b17 (Pin_b17), J703.b17 (Pin_b17), U705.12 (B6)
- new net EXP_AM2: J701.b18 (Pin_b18), J702.b18 (Pin_b18), J703.b18 (Pin_b18), U705.13 (B5)
- new net EXP_AM3: J701.b19 (Pin_b19), J702.b19 (Pin_b19), J703.b19 (Pin_b19), U705.14 (B4)
- new net EXP_RnW: J701.a14 (Pin_a14), J702.a14 (Pin_a14), J703.a14 (Pin_a14), U705.17 (B1)
- new net FC0: U703.8 (I8)
- new net FC1: U703.9 (I9)
- new net FC2: U703.10 (I10)
- new net ~{EXP_AS}: J701.a18 (Pin_a18), J702.a18 (Pin_a18), J703.a18 (Pin_a18), U704.3
- new net ~{EXP_LDS}: J701.a13 (Pin_a13), J702.a13 (Pin_a13), J703.a13 (Pin_a13), U704.8
- new net ~{EXP_UDS}: J701.a12 (Pin_a12), J702.a12 (Pin_a12), J703.a12 (Pin_a12), U704.6
- no-connect marks 72 -> 43
Other:
- note added: "N.B. DS1 = UDS, DS0 = LDS (It's absoultely VITAl to use clear terminology!)"
- note added: "N.B. The system board is "VME slot 0", The Arbitor, and will never grant to any other slot. Similarly, no slot will ever see an IACK cycle. Interrupts will simply be autovectored by the interrupt controller and handled as such by the operating system."
- moved on the sheet: U701, U702

Commit message: Clock generation is now done in the MMU, and we clock the MMU at 40MHz.
Connections:
- net CLK10 renamed CPU_CLK
Changed lines of the file:
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@@
 		)
 	)
-	(global_label "CLK10"
+	(global_label "CPU_CLK"
 		(shape input)
 		(at 66.04 55.88 180)
@@
 		)
 		(property "Intersheetrefs" "${INTERSHEET_REFS}"
-			(at 57.0677 55.88 0)
+			(at 54.6486 55.88 0)
 			(effects
 				(font
@@
 		)
 	)
-	(global_label "CLK10"
+	(global_label "CPU_CLK"
 		(shape input)
 		(at 146.05 55.88 180)
@@
 		)
 		(property "Intersheetrefs" "${INTERSHEET_REFS}"
-			(at 137.0777 55.88 0)
+			(at 134.6586 55.88 0)
 			(effects
 				(font
@@
 		)
 	)
-	(global_label "CLK10"
+	(global_label "CPU_CLK"
 		(shape input)
 		(at 222.25 55.88 180)
@@
 		)
 		(property "Intersheetrefs" "${INTERSHEET_REFS}"
-			(at 213.2777 55.88 0)
-			(effects
-				(font
+			(at 210.8586 55.88 0)
+			(effects
+				(font

Commit message: Expansion bus changes: - VME bus arb signals are now total no-ops, no daisy-chain. - Ditto for VMS IACK signals. - Neuter some other VME control signals.
Parts:
- added R703, R704, R705, R706, R707: 470R, Resistor_SMD:R_0805_2012Metric_Pad1.20x1.40mm_HandSolder, symbol Device:R_Small
Connections:
- net +5V: now also R703.1, R704.1, R706.1, R707.1
- net GND: now also R705.1
- net ~{EXP_BBSY}: now reaches J703.b1 (Pin_b1)
- net ~{EXP_BBSY}: now also J701.b1 (Pin_b1), J702.b1 (Pin_b1), R705.2
- net ~{EXP_BCLR}: now reaches J703.b2 (Pin_b2)
- net ~{EXP_BCLR}: now also J701.b2 (Pin_b2), J702.b2 (Pin_b2), R706.2
- net ~{EXP_SYSFAIL}: now reaches J703.c10 (Pin_c10)
- net ~{EXP_SYSFAIL}: now also J701.c10 (Pin_c10), J702.c10 (Pin_c10), R707.2
- net ~{EXP_BERR}: now reaches J703.c11 (Pin_c11)
- net ~{EXP_BERR}: now also J701.c11 (Pin_c11), J702.c11 (Pin_c11)
- net ~{EXP_LWORD}: now reaches J703.c13 (Pin_c13)
- net ~{EXP_LWORD}: now also J701.c13 (Pin_c13), J702.c13 (Pin_c13), R704.2
- net ~{EXP1_BG0IN} renamed ~{EXP_BGxIN}
- net ~{EXP_BGxIN}: now also J702.b10 (Pin_b10), J702.b4 (Pin_b4), J702.b6 (Pin_b6), J702.b8 (Pin_b8), J703.b10 (Pin_b10), J703.b4 (Pin_b4), J703.b6 (Pin_b6), J703.b8 (Pin_b8); no longer J701.a21 (Pin_a21)
- net ~{EXP2_BG0IN}: no longer names the net of J701.b5 (Pin_b5)
- net ~{EXP2_BG0IN}: no longer J702.b4 (Pin_b4)
- net ~{EXP2_BG1IN}: no longer names the net of J701.b7 (Pin_b7)
- net ~{EXP2_BG1IN}: no longer J702.b6 (Pin_b6)
- net ~{EXP2_BG2IN}: no longer names the net of J701.b9 (Pin_b9)
- net ~{EXP2_BG2IN}: no longer J702.b8 (Pin_b8)
- net ~{EXP2_BG3IN}: no longer names the net of J701.b11 (Pin_b11)
- net ~{EXP2_BG3IN}: no longer J702.b10 (Pin_b10)
- net ~{EXP2_IACKIN}: no longer names the net of J701.a22 (Pin_a22)
- net ~{EXP2_IACKIN}: no longer J702.a21 (Pin_a21)
- net ~{EXP3_BG0IN}: no longer names the net of J702.b5 (Pin_b5)
- net ~{EXP3_BG0IN}: no longer J703.b4 (Pin_b4)
- net ~{EXP3_BG1IN}: no longer names the net of J702.b7 (Pin_b7)
- net ~{EXP3_BG1IN}: no longer J703.b6 (Pin_b6)
- net ~{EXP3_BG2IN}: no longer names the net of J702.b9 (Pin_b9)
- net ~{EXP3_BG2IN}: no longer J703.b8 (Pin_b8)
- net ~{EXP3_BG3IN}: no longer names the net of J702.b11 (Pin_b11)
- net ~{EXP3_BG3IN}: no longer J703.b10 (Pin_b10)
- net ~{EXP3_IACKIN}: no longer names the net of J702.a22 (Pin_a22)
- net ~{EXP3_IACKIN}: no longer J703.a21 (Pin_a21)
- new net ~{EXP_IACKIN}: J701.a21 (Pin_a21), J702.a21 (Pin_a21), J703.a21 (Pin_a21), R703.2
- no-connect marks 43 -> 39

Commit message: Directly connect R/W to the NQVME slots.
Connections:
- net GND: now also U705.3 (A1)
- net R/~{W}: now also J701.a14 (Pin_a14), J702.a14 (Pin_a14), J703.a14 (Pin_a14); no longer U705.3 (A1)
- removed net EXP_RnW: J701.a14 (Pin_a14), J702.a14 (Pin_a14), J703.a14 (Pin_a14), U705.17 (B1)
- no-connect marks 39 -> 40
Other:
- moved on the sheet: C701, C702, C703, C704, C705

Commit message: Eliminate the '245 between the VME glue GAL and the AM signals.
Parts:
- removed C705: 100nF, Capacitor_SMD:C_0805_2012Metric_Pad1.18x1.45mm_HandSolder, symbol Device:C_Small
- removed U705: 74ACT245, Package_DIP:DIP-20_W7.62mm_Socket, symbol 74xx:74HC245
Connections:
- net EXP_AM0: now also U703.22 (IO9)
- net EXP_AM1: now also U703.21 (IO8)
- net EXP_AM2: now also U703.20 (IO7)
- net EXP_AM3: now also U703.19 (IO6)
- net EXP_AM4: now also U703.18 (IO5)
- net EXP_AM5: now also U703.17 (IO4)
- no-connect marks 40 -> 38

Commit message: Get rid of RN701 and RN702 in preparation for correct active termination.
Parts:
- removed RN701, RN702: 3K3, Resistor_THT:R_Array_SIP9, symbol Device:R_Network08
Other:
- moved on the sheet: R701, R702, R703, R704, R705, R706, R707, U701, U702, U703, U704A, U704B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

Commit message: Many many bus connections.
Parts:
- added C705, C706, C707, C709, C710, C712: 100nF, Capacitor_SMD:C_0805_2012Metric_Pad1.18x1.45mm_HandSolder, symbol Device:C_Small
- added C708, C711, C713: 100µF, Capacitor_THT:CP_Radial_D6.3mm_P2.50mm, symbol Device:C_Polarized_Small
- added R708: 4K7, Resistor_SMD:R_0805_2012Metric_Pad1.20x1.40mm_HandSolder, symbol Device:R_Small
- added R709: 3K3, Resistor_SMD:R_0805_2012Metric_Pad1.20x1.40mm_HandSolder, symbol Device:R_Small
- added RN701, RN702, RN703, RN704, RN705, RN706, RN707: 330R/470R, Resistor_THT:R_Array_SIP10, symbol Device:R_Network_Dividers_x08_SIP
- added U705, U706, U707: 74ACT245, Package_DIP:DIP-20_W7.62mm_Socket, symbol 74xx:74HC245
- added U708: L272D, Package_SO:SOIC-16_3.9x9.9mm_P1.27mm, symbol Amplifier_Operational:L272D
Connections:
- net +5V: now also C705.1, C706.1, C707.1, C708.1, C709.1, R709.1, U705.1 (A->B), U705.20 (VCC), U706.1 (A->B), U706.20 (VCC), U707.1 (A->B), U707.20 (VCC), U708.4 (V+)
- net A1: now also U705.8 (A6); no longer J701.a30 (Pin_a30), J702.a30 (Pin_a30), J703.a30 (Pin_a30)
- net A10: now also U706.8 (A6); no longer J701.c28 (Pin_c28), J702.c28 (Pin_c28), J703.c28 (Pin_c28)
- net A11: now also U706.7 (A5); no longer J701.c27 (Pin_c27), J702.c27 (Pin_c27), J703.c27 (Pin_c27)
- net A12: now also U706.6 (A4); no longer J701.c26 (Pin_c26), J702.c26 (Pin_c26), J703.c26 (Pin_c26)
- net A13: now also U706.5 (A3); no longer J701.c25 (Pin_c25), J702.c25 (Pin_c25), J703.c25 (Pin_c25)
- net A14: now also U706.4 (A2); no longer J701.c24 (Pin_c24), J702.c24 (Pin_c24), J703.c24 (Pin_c24)
- net A15: now also U706.3 (A1); no longer J701.c23 (Pin_c23), J702.c23 (Pin_c23), J703.c23 (Pin_c23)
- net A16: now also U706.2 (A0); no longer J701.c22 (Pin_c22), J702.c22 (Pin_c22), J703.c22 (Pin_c22)
- net A17: now also U707.9 (A7); no longer J701.c21 (Pin_c21), J702.c21 (Pin_c21), J703.c21 (Pin_c21)
- net A18: now also U707.8 (A6); no longer J701.c20 (Pin_c20), J702.c20 (Pin_c20), J703.c20 (Pin_c20)
- net A19: now also U707.7 (A5); no longer J701.c19 (Pin_c19), J702.c19 (Pin_c19), J703.c19 (Pin_c19)
- net A2: now also U705.7 (A5); no longer J701.a29 (Pin_a29), J702.a29 (Pin_a29), J703.a29 (Pin_a29)
- net A20: now also U707.6 (A4); no longer J701.c18 (Pin_c18), J702.c18 (Pin_c18), J703.c18 (Pin_c18)
- net A21: now also U707.5 (A3); no longer J701.c17 (Pin_c17), J702.c17 (Pin_c17), J703.c17 (Pin_c17)
- net A22: now also U707.4 (A2); no longer J701.c16 (Pin_c16), J702.c16 (Pin_c16), J703.c16 (Pin_c16)
- net A23: now also U707.3 (A1); no longer J701.c15 (Pin_c15), J702.c15 (Pin_c15), J703.c15 (Pin_c15)
- net A3: now also U705.6 (A4); no longer J701.a28 (Pin_a28), J702.a28 (Pin_a28), J703.a28 (Pin_a28)
- net A4: now also U705.5 (A3); no longer J701.a27 (Pin_a27), J702.a27 (Pin_a27), J703.a27 (Pin_a27)
- net A5: now also U705.4 (A2); no longer J701.a26 (Pin_a26), J702.a26 (Pin_a26), J703.a26 (Pin_a26)
- net A6: now also U705.3 (A1); no longer J701.a25 (Pin_a25), J702.a25 (Pin_a25), J703.a25 (Pin_a25)
- net A7: now also U705.2 (A0); no longer J701.a24 (Pin_a24), J702.a24 (Pin_a24), J703.a24 (Pin_a24)
- net A8: now also U705.9 (A7); no longer J701.c30 (Pin_c30), J702.c30 (Pin_c30), J703.c30 (Pin_c30)
- net A9: now also U706.9 (A7); no longer J701.c29 (Pin_c29), J702.c29 (Pin_c29), J703.c29 (Pin_c29)
- net CPU_CLK: now also U704.12, U704.13; no longer J701.a10 (Pin_a10), J702.a10 (Pin_a10), J703.a10 (Pin_a10)
- net EXP_AM0: now also RN703.2 (R1)
- net EXP_AM1: now also RN703.3 (R2)
- net EXP_AM2: now also RN703.4 (R3)
- net EXP_AM3: now also RN703.5 (R4)
- net EXP_AM4: now also RN703.6 (R5)
- net EXP_AM5: now also RN703.7 (R6)
- net EXP_D0: now also RN701.2 (R1)
- net EXP_D1: now also RN701.3 (R2)
- net EXP_D10: now also RN702.4 (R3)
- net EXP_D11: now also RN702.5 (R4)
- net EXP_D12: now also RN702.6 (R5)
- net EXP_D13: now also RN702.7 (R6)
- net EXP_D14: now also RN702.8 (R7)
- net EXP_D15: now also RN702.9 (R8)
- net EXP_D2: now also RN701.4 (R3)
- net EXP_D3: now also RN701.5 (R4)
- net EXP_D4: now also RN701.6 (R5)
- net EXP_D5: now also RN701.7 (R6)
- net EXP_D6: now also U702.8 (A6), RN701.8 (R7); no longer U702.9 (A7)
- net EXP_D7: now also U702.9 (A7), RN701.9 (R8); no longer U702.8 (A6)
- net EXP_D8: now also RN702.2 (R1)
- net EXP_D9: now also RN702.3 (R2)
- net GND: now also C705.2, C706.2, C707.2, C708.2, C709.2, C710.2, C711.2, C712.2, C713.2, R708.2, U705.10 (GND), U706.10 (GND), U707.10 (GND), U708.6 (V-); no longer U704.12, U704.13
- net R/~{W}: now also U707.2 (A0); no longer J701.a14 (Pin_a14), J702.a14 (Pin_a14), J703.a14 (Pin_a14)
- net ~{EXP_AS}: now also RN707.5 (R4)
- net ~{EXP_LDS}: now also RN707.4 (R3)
- net ~{EXP_UDS}: now also RN707.3 (R2)
- net ~{IRQ3}: now also RN707.9 (R8)
- net ~{IRQ4}: now also RN707.8 (R7)
- net ~{IRQ5}: now also RN707.7 (R6)
- net ~{IRQ6}: now also RN707.6 (R5)
- net ~{VMESEL}: now also U705.19 (CE), U706.19 (CE), U707.19 (CE)
- net ~{EXP_CLK}: now reaches U704.11
- net ~{EXP_CLK}: now also J701.a10 (Pin_a10), J702.a10 (Pin_a10), J703.a10 (Pin_a10), RN707.2 (R1)
- removed net ~{IRQ1}: J701.b30 (Pin_b30), J702.b30 (Pin_b30), J703.b30 (Pin_b30)
- removed net ~{IRQ2}: J701.b29 (Pin_b29), J702.b29 (Pin_b29), J703.b29 (Pin_b29)
- removed net ~{IRQ7}: J701.b24 (Pin_b24), J702.b24 (Pin_b24), J703.b24 (Pin_b24)
- new net: R708.1, R709.2, U708.12 (+), U708.13 (+)
- new net EXP_A1: J701.a30 (Pin_a30), J702.a30 (Pin_a30), J703.a30 (Pin_a30), RN704.8 (R7), U705.12 (B6)
- new net EXP_A10: J701.c28 (Pin_c28), J702.c28 (Pin_c28), J703.c28 (Pin_c28), RN705.8 (R7), U706.12 (B6)
- new net EXP_A11: J701.c27 (Pin_c27), J702.c27 (Pin_c27), J703.c27 (Pin_c27), RN705.7 (R6), U706.13 (B5)
- new net EXP_A12: J701.c26 (Pin_c26), J702.c26 (Pin_c26), J703.c26 (Pin_c26), RN705.6 (R5), U706.14 (B4)
- new net EXP_A13: J701.c25 (Pin_c25), J702.c25 (Pin_c25), J703.c25 (Pin_c25), RN705.5 (R4), U706.15 (B3)
- new net EXP_A14: J701.c24 (Pin_c24), J702.c24 (Pin_c24), J703.c24 (Pin_c24), RN705.4 (R3), U706.16 (B2)
- new net EXP_A15: J701.c23 (Pin_c23), J702.c23 (Pin_c23), J703.c23 (Pin_c23), RN705.3 (R2), U706.17 (B1)
- new net EXP_A16: J701.c22 (Pin_c22), J702.c22 (Pin_c22), J703.c22 (Pin_c22), RN705.2 (R1), U706.18 (B0)
- new net EXP_A17: J701.c21 (Pin_c21), J702.c21 (Pin_c21), J703.c21 (Pin_c21), RN706.9 (R8), U707.11 (B7)
- new net EXP_A18: J701.c20 (Pin_c20), J702.c20 (Pin_c20), J703.c20 (Pin_c20), RN706.8 (R7), U707.12 (B6)
- new net EXP_A19: J701.c19 (Pin_c19), J702.c19 (Pin_c19), J703.c19 (Pin_c19), RN706.7 (R6), U707.13 (B5)
- new net EXP_A2: J701.a29 (Pin_a29), J702.a29 (Pin_a29), J703.a29 (Pin_a29), RN704.7 (R6), U705.13 (B5)
- new net EXP_A20: J701.c18 (Pin_c18), J702.c18 (Pin_c18), J703.c18 (Pin_c18), RN706.6 (R5), U707.14 (B4)
- new net EXP_A21: J701.c17 (Pin_c17), J702.c17 (Pin_c17), J703.c17 (Pin_c17), RN706.5 (R4), U707.15 (B3)
- new net EXP_A22: J701.c16 (Pin_c16), J702.c16 (Pin_c16), J703.c16 (Pin_c16), RN706.4 (R3), U707.16 (B2)
- new net EXP_A23: J701.c15 (Pin_c15), J702.c15 (Pin_c15), J703.c15 (Pin_c15), RN706.3 (R2), U707.17 (B1)
- new net EXP_A3: J701.a28 (Pin_a28), J702.a28 (Pin_a28), J703.a28 (Pin_a28), RN704.6 (R5), U705.14 (B4)
- new net EXP_A4: J701.a27 (Pin_a27), J702.a27 (Pin_a27), J703.a27 (Pin_a27), RN704.5 (R4), U705.15 (B3)
- new net EXP_A5: J701.a26 (Pin_a26), J702.a26 (Pin_a26), J703.a26 (Pin_a26), RN704.4 (R3), U705.16 (B2)
- new net EXP_A6: J701.a25 (Pin_a25), J702.a25 (Pin_a25), J703.a25 (Pin_a25), RN704.3 (R2), U705.17 (B1)
- new net EXP_A7: J701.a24 (Pin_a24), J702.a24 (Pin_a24), J703.a24 (Pin_a24), RN704.2 (R1), U705.18 (B0)
- new net EXP_A8: J701.c30 (Pin_c30), J702.c30 (Pin_c30), J703.c30 (Pin_c30), RN704.9 (R8), U705.11 (B7)
- new net EXP_A9: J701.c29 (Pin_c29), J702.c29 (Pin_c29), J703.c29 (Pin_c29), RN705.9 (R8), U706.11 (B7)
- new net EXP_RnW: J701.a14 (Pin_a14), J702.a14 (Pin_a14), J703.a14 (Pin_a14), RN706.2 (R1), U707.18 (B0)
- new net EXP_VTERM1: C710.1, C711.1, RN701.1 (COM1), RN701.10 (COM2), RN702.1 (COM1), RN702.10 (COM2), RN703.1 (COM1), RN703.10 (COM2), RN707.1 (COM1), RN707.10 (COM2), U708.14 (-), U708.3
- new net EXP_VTERM2: C712.1, C713.1, RN704.1 (COM1), RN704.10 (COM2), RN705.1 (COM1), RN705.10 (COM2), RN706.1 (COM1), RN706.10 (COM2), U708.11 (-), U708.5
- no-connect marks 38 -> 48
Other:
- moved on the sheet: R701, R702, R703, R704, R705, R706, R707, U701, U702, U703, U704A, U704B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
