File: cpu010/design-files/cpu010-obmem.kicad_sch (KiCad schematic)
At the start: 7 parts, among them U501 GAL22V10, U502 CY62158, U503 CY62158, U504 CY62158, U505 CY62158, U506 SST39SF040, U507 SST39SF040

Commit message: Add reset circuit.
Parts:
- U502, U503, U504, U505: Part (none) -> CY62158H-45ZSXI
Changed lines of the file:
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@@
 	(text "Lower byte"
 		(exclude_from_sim no)
-		(at 60.96 149.86 0)
+		(at 60.96 147.32 0)
 		(effects
 			(font
@@
 	(text "Upper byte"
 		(exclude_from_sim no)
-		(at 60.452 62.484 0)
+		(at 60.452 59.69 0)
 		(effects
 			(font
@@
 			)
 		)
+		(property "Part" "CY62158H-45ZSXI"
+			(at 44.45 114.3 0)
+			(effects
+				(font
+					(size 1.27 1.27)
+				)
+				(hide yes)
+			)
+		)
 		(pin "20"
 		)
@@
 		(pin "35"
 		)
+		(pin "15"
+		)
+		(pin "16"
+		)
+		(pin "37"
+		)
+		(pin "38"
+		)
 		(instances
 			(project "cpu010"
@@
 			)
 		)
+		(property "Part" "CY62158H-45ZSXI"
+			(at 44.45 26.67 0)
+			(effects
+				(font
+					(size 1.27 1.27)
+				)
+				(hide yes)
+			)
+		)
 		(pin "20"
 		)
@@
 		(pin "35"
 		)
+		(pin "15"
+		)
+		(pin "16"
+		)
+		(pin "37"
+		)
+		(pin "38"
+		)
 		(instances
 			(project ""
@@
 			)
 		)
+		(property "Part" "CY62158H-45ZSXI"
+			(at 91.44 26.67 0)
+			(effects
+				(font
+					(size 1.27 1.27)
+				)
+				(hide yes)
+			)
+		)
 		(pin "20"
 		)
@@
 		(pin "35"
 		)
+		(pin "37"
+		)
+		(pin "15"
+		)
+		(pin "38"
+		)
+		(pin "16"
+		)
 		(instances
 			(project "cpu010"
@@
 			)
 		)
+		(property "Part" "CY62158H-45ZSXI"
+			(at 91.44 114.3 0)
+			(effects
+				(font
+					(size 1.27 1.27)
+				)
+				(hide yes)
+			)
+		)
 		(pin "20"
 		)
@@
 		(pin "35"
 		)
+		(pin "15"
+		)
+		(pin "16"
+		)
+		(pin "37"
+		)
+		(pin "38"
+		)
 		(instances

Commit message: SMT 0805 bypass caps everywere.
Parts:
- added C501, C502, C503, C504, C505, C506, C507, C508, C509, C510, C511: 100nF, Capacitor_SMD:C_0805_2012Metric_Pad1.18x1.45mm_HandSolder, symbol Device:C_Small
- U502, U503, U504, U505: JLCPCB (none) -> C2950517
Connections:
- net +5V: now also C501.1, C502.1, C503.1, C504.1, C505.1, C506.1, C507.1, C508.1, C509.1, C510.1, C511.1
- net GND: now also C501.2, C502.2, C503.2, C504.2, C505.2, C506.2, C507.2, C508.2, C509.2, C510.2, C511.2

Commit message: We have 8MB RAM now.
Parts:
- removed U501: GAL22V10, Package_DIP:DIP-24_W7.62mm_Socket, symbol jrt-ICs:GAL22V10
- added C512, C513, C514, C515, C516, C517, C518, C519: 100nF, Capacitor_SMD:C_0805_2012Metric_Pad1.18x1.45mm_HandSolder, symbol Device:C_Small
- added U501: ATF1504AS-PLCC44, Package_LCC:PLCC-44_THT-Socket, symbol jrt-ICs:ATF1504AS-PLCC44
- added U508, U509, U510, U511: CY62158, Package_SO:TSOP-II-44_10.16x18.41mm_P0.8mm, symbol jrt-Memory:CY62158
Connections:
- net A1 is gone; now on net +5V: U504.40 (CE2), U505.40 (CE2)
- net OBMEM_nA1 is gone; now on net +5V: U502.40 (CE2), U503.40 (CE2)
- net +5V: now also C512.1, C513.1, C514.1, C515.1, C516.1, C517.1, C518.1, C519.1, U501.15 (VCC), U501.23 (VCC), U501.3 (VCC), U501.35 (VCC), U508.11 (VDD), U508.33 (VDD), U508.40 (CE2), U509.11 (VDD), U509.33 (VDD), U509.40 (CE2), U510.11 (VDD), U510.33 (VDD), U510.40 (CE2), U511.11 (VDD), U511.33 (VDD), U511.40 (CE2)
- net A10: now also U508.39 (A8), U509.39 (A8), U510.39 (A8), U511.39 (A8)
- net A11: now also U508.28 (A9), U509.28 (A9), U510.28 (A9), U511.28 (A9)
- net A12: now also U508.27 (A10), U509.27 (A10), U510.27 (A10), U511.27 (A10)
- net A13: now also U508.26 (A11), U509.26 (A11), U510.26 (A11), U511.26 (A11)
- net A14: now also U508.25 (A12), U509.25 (A12), U510.25 (A12), U511.25 (A12)
- net A15: now also U508.24 (A13), U509.24 (A13), U510.24 (A13), U511.24 (A13)
- net A16: now also U508.23 (A14), U509.23 (A14), U510.23 (A14), U511.23 (A14)
- net A17: now also U508.22 (A15), U509.22 (A15), U510.22 (A15), U511.22 (A15)
- net A18: now also U508.21 (A16), U509.21 (A16), U510.21 (A16), U511.21 (A16)
- net A19: now also U508.20 (A17), U509.20 (A17), U510.20 (A17), U511.20 (A17)
- net A2: now also U508.5 (A0), U509.5 (A0), U510.5 (A0), U511.5 (A0)
- net A20: now also U508.19 (A18), U509.19 (A18), U510.19 (A18), U511.19 (A18)
- net A21: now also U508.18 (A19), U509.18 (A19), U510.18 (A19), U511.18 (A19)
- net A3: now also U508.4 (A1), U509.4 (A1), U510.4 (A1), U511.4 (A1)
- net A4: now also U508.3 (A2), U509.3 (A2), U510.3 (A2), U511.3 (A2)
- net A5: now also U508.2 (A3), U509.2 (A3), U510.2 (A3), U511.2 (A3)
- net A6: now also U508.1 (A4), U509.1 (A4), U510.1 (A4), U511.1 (A4)
- net A7: now also U508.44 (A5), U509.44 (A5), U510.44 (A5), U511.44 (A5)
- net A8: now also U508.43 (A6), U509.43 (A6), U510.43 (A6), U511.43 (A6)
- net A9: now also U508.42 (A7), U509.42 (A7), U510.42 (A7), U511.42 (A7)
- net D0: now also U509.9 (IO0), U511.9 (IO0)
- net D1: now also U509.10 (IO1), U511.10 (IO1)
- net D10: now also U508.13 (IO2), U510.13 (IO2)
- net D11: now also U508.14 (IO3), U510.14 (IO3)
- net D12: now also U508.31 (IO4), U510.31 (IO4)
- net D13: now also U508.32 (IO5), U510.32 (IO5)
- net D14: now also U508.35 (IO6), U510.35 (IO6)
- net D15: now also U508.36 (IO7), U510.36 (IO7)
- net D2: now also U509.13 (IO2), U511.13 (IO2)
- net D3: now also U509.14 (IO3), U511.14 (IO3)
- net D4: now also U509.31 (IO4), U511.31 (IO4)
- net D5: now also U509.32 (IO5), U511.32 (IO5)
- net D6: now also U509.35 (IO6), U511.35 (IO6)
- net D7: now also U509.36 (IO7), U511.36 (IO7)
- net D8: now also U508.9 (IO0), U510.9 (IO0)
- net D9: now also U508.10 (IO1), U510.10 (IO1)
- net GND: now also C512.2, C513.2, C514.2, C515.2, C516.2, C517.2, C518.2, C519.2, U501.10 (GND), U501.22 (GND), U501.30 (GND), U501.42 (GND), U508.12 (GND), U508.34 (GND), U508.6 (~{CE1}), U509.12 (GND), U509.34 (GND), U509.6 (~{CE1}), U510.12 (GND), U510.34 (GND), U510.6 (~{CE1}), U511.12 (GND), U511.34 (GND), U511.6 (~{CE1})
- net ~{RAMLR} renamed ~{RAM0LR}
- net ~{RAM0LR}: no longer U505.41 (~{OE})
- net ~{RAMLW} renamed ~{RAM0LW}
- net ~{RAM0LW}: no longer U505.17 (~{WE})
- net ~{RAMUR} renamed ~{RAM0UR}
- net ~{RAM0UR}: no longer U504.41 (~{OE})
- net ~{RAMUW} renamed ~{RAM0UW}
- net ~{RAM0UW}: no longer U504.17 (~{WE})
- new net ~{RAM2LR}: U505.41 (~{OE})
- new net ~{RAM2LW}: U505.17 (~{WE})
- new net ~{RAM2UR}: U504.41 (~{OE})
- new net ~{RAM2UW}: U504.17 (~{WE})
- new net ~{RAM4LR}: U509.41 (~{OE})
- new net ~{RAM4LW}: U509.17 (~{WE})
- new net ~{RAM4UR}: U508.41 (~{OE})
- new net ~{RAM4UW}: U508.17 (~{WE})
- new net ~{RAM6LR}: U511.41 (~{OE})
- new net ~{RAM6LW}: U511.17 (~{WE})
- new net ~{RAM6UR}: U510.41 (~{OE})
- new net ~{RAM6UW}: U510.17 (~{WE})
- no-connect marks 2 -> 0
Other:
- note added: "0-2MB"
- note added: "2-4MB"
- note added: "4-6MB"
- note added: "6-8MB"
- note removed: "Lower Word"
- note removed: "Upper word"
- moved on the sheet: C501, C502, C503, C504, C505, C506, C507, C508, C509, C510, C511, U506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

Commit message: Routing some I/O stuff.
Connections:
- net A21: now also U501.12 (I/O)
- net ~{AS}: now reaches U501.1 (I/GCLR)
- net FC2: now reaches U501.11 (I/O/PD1)
- net A22: now reaches U501.14 (I/O)
- net A23: now reaches U501.16 (I/O)
- net A24: now reaches U501.17 (I/O)
- net A25: now reaches U501.18 (I/O)
- net A26: now reaches U501.19 (I/O)
- net ~{UDS}: now reaches U501.2 (I/OE2/GCLK2)
- net A27: now reaches U501.20 (I/O)
- net ~{OBMEM_URD}: now reaches U501.21 (I/O)
- net ~{OBMEM_UWR}: now reaches U501.24 (I/O)
- net ~{OBMEM_LRD}: now reaches U501.25 (I/O/PD2)
- net ~{OBMEM_LWR}: now reaches U501.26 (I/O)
- net ~{OBMEM_ROMSEL}: now reaches U501.27 (I/O)
- net ~{OBMEM_RAM0SEL}: now reaches U501.28 (I/O)
- net ~{OBMEM_RAM1SEL}: now reaches U501.29 (I/O)
- net ~{OBMEM_RAM2SEL}: now reaches U501.31 (I/O)
- net ~{OBMEM_RAM3SEL}: now reaches U501.33 (I/O)
- net ~{EXPRAMSEL}: now reaches U501.34 (I/O)
- net ~{LDS}: now reaches U501.4 (I/O)
- net OBMEM_DTACK: now reaches U501.40 (I/O)
- net R/~{W}: now reaches U501.5 (I/O)
- net MMU_EN: now reaches U501.6 (I/O)
- net FC0: now reaches U501.8 (I/O)
- net FC1: now reaches U501.9 (I/O)
- no-connect marks 0 -> 6

Commit message: More (NQ)VME tweaks.  Add JTAG chain.
Parts:
- added C520, C521, C522: 100nF, Capacitor_SMD:C_0805_2012Metric_Pad1.18x1.45mm_HandSolder, symbol Device:C_Small
Connections:
- net ~{RAM0LR} is gone; now on net ~{OBMEM_LRD}: U503.41 (~{OE})
- net ~{RAM0LW} is gone; now on net ~{OBMEM_LWR}: U503.17 (~{WE})
- net ~{RAM0UR} is gone; now on net ~{OBMEM_URD}: U502.41 (~{OE})
- net ~{RAM0UW} is gone; now on net ~{OBMEM_UWR}: U502.17 (~{WE})
- net ~{RAM2LR} is gone; now on net ~{OBMEM_LRD}: U505.41 (~{OE})
- net ~{RAM2LW} is gone; now on net ~{OBMEM_LWR}: U505.17 (~{WE})
- net ~{RAM2UR} is gone; now on net ~{OBMEM_URD}: U504.41 (~{OE})
- net ~{RAM2UW} is gone; now on net ~{OBMEM_UWR}: U504.17 (~{WE})
- net ~{RAM4LR} is gone; now on net ~{OBMEM_LRD}: U509.41 (~{OE})
- net ~{RAM4LW} is gone; now on net ~{OBMEM_LWR}: U509.17 (~{WE})
- net ~{RAM4UR} is gone; now on net ~{OBMEM_URD}: U508.41 (~{OE})
- net ~{RAM4UW} is gone; now on net ~{OBMEM_UWR}: U508.17 (~{WE})
- net ~{RAM6LR} is gone; now on net ~{OBMEM_LRD}: U511.41 (~{OE})
- net ~{RAM6LW} is gone; now on net ~{OBMEM_LWR}: U511.17 (~{WE})
- net ~{RAM6UR} is gone; now on net ~{OBMEM_URD}: U510.41 (~{OE})
- net ~{RAM6UW} is gone; now on net ~{OBMEM_UWR}: U510.17 (~{WE})
- net ~{ROMLR} is gone; now on net ~{OBMEM_LRD}: U507.24 (OE)
- net ~{ROMLW} is gone; now on net ~{OBMEM_LWR}: U507.31 (PGM)
- net ~{ROMUR} is gone; now on net ~{OBMEM_URD}: U506.24 (OE)
- net ~{ROMUW} is gone; now on net ~{OBMEM_UWR}: U506.31 (PGM)
- net +5V: now also C520.1, C521.1, C522.1
- net A10: now also U502.28 (A9), U503.28 (A9), U504.28 (A9), U505.28 (A9), U506.26 (A9), U507.26 (A9), U508.28 (A9), U509.28 (A9), U510.28 (A9), U511.28 (A9); no longer U502.39 (A8), U503.39 (A8), U504.39 (A8), U505.39 (A8), U506.27 (A8), U507.27 (A8), U508.39 (A8), U509.39 (A8), U510.39 (A8), U511.39 (A8)
- net A11: now also U502.27 (A10), U503.27 (A10), U504.27 (A10), U505.27 (A10), U506.23 (A10), U507.23 (A10), U508.27 (A10), U509.27 (A10), U510.27 (A10), U511.27 (A10); no longer U502.28 (A9), U503.28 (A9), U504.28 (A9), U505.28 (A9), U506.26 (A9), U507.26 (A9), U508.28 (A9), U509.28 (A9), U510.28 (A9), U511.28 (A9)
- net A12: now also U502.26 (A11), U503.26 (A11), U504.26 (A11), U505.26 (A11), U506.25 (A11), U507.25 (A11), U508.26 (A11), U509.26 (A11), U510.26 (A11), U511.26 (A11); no longer U502.27 (A10), U503.27 (A10), U504.27 (A10), U505.27 (A10), U506.23 (A10), U507.23 (A10), U508.27 (A10), U509.27 (A10), U510.27 (A10), U511.27 (A10)
- net A13: now also U502.25 (A12), U503.25 (A12), U504.25 (A12), U505.25 (A12), U506.4 (A12), U507.4 (A12), U508.25 (A12), U509.25 (A12), U510.25 (A12), U511.25 (A12); no longer U502.26 (A11), U503.26 (A11), U504.26 (A11), U505.26 (A11), U506.25 (A11), U507.25 (A11), U508.26 (A11), U509.26 (A11), U510.26 (A11), U511.26 (A11)
- net A14: now also U502.24 (A13), U503.24 (A13), U504.24 (A13), U505.24 (A13), U506.28 (A13), U507.28 (A13), U508.24 (A13), U509.24 (A13), U510.24 (A13), U511.24 (A13); no longer U502.25 (A12), U503.25 (A12), U504.25 (A12), U505.25 (A12), U506.4 (A12), U507.4 (A12), U508.25 (A12), U509.25 (A12), U510.25 (A12), U511.25 (A12)
- net A15: now also U502.23 (A14), U503.23 (A14), U504.23 (A14), U505.23 (A14), U506.29 (A14), U507.29 (A14), U508.23 (A14), U509.23 (A14), U510.23 (A14), U511.23 (A14); no longer U502.24 (A13), U503.24 (A13), U504.24 (A13), U505.24 (A13), U506.28 (A13), U507.28 (A13), U508.24 (A13), U509.24 (A13), U510.24 (A13), U511.24 (A13)
- net A16: now also U502.22 (A15), U503.22 (A15), U504.22 (A15), U505.22 (A15), U506.3 (A15), U507.3 (A15), U508.22 (A15), U509.22 (A15), U510.22 (A15), U511.22 (A15); no longer U502.23 (A14), U503.23 (A14), U504.23 (A14), U505.23 (A14), U506.29 (A14), U507.29 (A14), U508.23 (A14), U509.23 (A14), U510.23 (A14), U511.23 (A14)
- net A17: now also U502.21 (A16), U503.21 (A16), U504.21 (A16), U505.21 (A16), U506.2 (A16), U507.2 (A16), U508.21 (A16), U509.21 (A16), U510.21 (A16), U511.21 (A16); no longer U502.22 (A15), U503.22 (A15), U504.22 (A15), U505.22 (A15), U506.3 (A15), U507.3 (A15), U508.22 (A15), U509.22 (A15), U510.22 (A15), U511.22 (A15)
- net A18: now also U502.20 (A17), U503.20 (A17), U504.20 (A17), U505.20 (A17), U506.30 (A17), U507.30 (A17), U508.20 (A17), U509.20 (A17), U510.20 (A17), U511.20 (A17); no longer U502.21 (A16), U503.21 (A16), U504.21 (A16), U505.21 (A16), U506.2 (A16), U507.2 (A16), U508.21 (A16), U509.21 (A16), U510.21 (A16), U511.21 (A16)
- net A19: now also U502.19 (A18), U503.19 (A18), U504.19 (A18), U505.19 (A18), U506.1 (A18), U507.1 (A18), U508.19 (A18), U509.19 (A18), U510.19 (A18), U511.19 (A18); no longer U502.20 (A17), U503.20 (A17), U504.20 (A17), U505.20 (A17), U506.30 (A17), U507.30 (A17), U508.20 (A17), U509.20 (A17), U510.20 (A17), U511.20 (A17)
- net A2: now also U502.4 (A1), U503.4 (A1), U504.4 (A1), U505.4 (A1), U506.11 (A1), U507.11 (A1), U508.4 (A1), U509.4 (A1), U510.4 (A1), U511.4 (A1); no longer U502.5 (A0), U503.5 (A0), U504.5 (A0), U505.5 (A0), U506.12 (A0), U507.12 (A0), U508.5 (A0), U509.5 (A0), U510.5 (A0), U511.5 (A0)
- net A20: now also U502.18 (A19), U503.18 (A19), U504.18 (A19), U505.18 (A19), U508.18 (A19), U509.18 (A19), U510.18 (A19), U511.18 (A19); no longer U502.19 (A18), U503.19 (A18), U504.19 (A18), U505.19 (A18), U506.1 (A18), U507.1 (A18), U508.19 (A18), U509.19 (A18), U510.19 (A18), U511.19 (A18)
- net A21: no longer U502.18 (A19), U503.18 (A19), U504.18 (A19), U505.18 (A19), U508.18 (A19), U509.18 (A19), U510.18 (A19), U511.18 (A19)
- net A3: now also U502.3 (A2), U503.3 (A2), U504.3 (A2), U505.3 (A2), U506.10 (A2), U507.10 (A2), U508.3 (A2), U509.3 (A2), U510.3 (A2), U511.3 (A2); no longer U502.4 (A1), U503.4 (A1), U504.4 (A1), U505.4 (A1), U506.11 (A1), U507.11 (A1), U508.4 (A1), U509.4 (A1), U510.4 (A1), U511.4 (A1)
- net A4: now also U502.2 (A3), U503.2 (A3), U504.2 (A3), U505.2 (A3), U506.9 (A3), U507.9 (A3), U508.2 (A3), U509.2 (A3), U510.2 (A3), U511.2 (A3); no longer U502.3 (A2), U503.3 (A2), U504.3 (A2), U505.3 (A2), U506.10 (A2), U507.10 (A2), U508.3 (A2), U509.3 (A2), U510.3 (A2), U511.3 (A2)
- net A5: now also U502.1 (A4), U503.1 (A4), U504.1 (A4), U505.1 (A4), U506.8 (A4), U507.8 (A4), U508.1 (A4), U509.1 (A4), U510.1 (A4), U511.1 (A4); no longer U502.2 (A3), U503.2 (A3), U504.2 (A3), U505.2 (A3), U506.9 (A3), U507.9 (A3), U508.2 (A3), U509.2 (A3), U510.2 (A3), U511.2 (A3)
- net A6: now also U502.44 (A5), U503.44 (A5), U504.44 (A5), U505.44 (A5), U506.7 (A5), U507.7 (A5), U508.44 (A5), U509.44 (A5), U510.44 (A5), U511.44 (A5); no longer U502.1 (A4), U503.1 (A4), U504.1 (A4), U505.1 (A4), U506.8 (A4), U507.8 (A4), U508.1 (A4), U509.1 (A4), U510.1 (A4), U511.1 (A4)
- net A7: now also U502.43 (A6), U503.43 (A6), U504.43 (A6), U505.43 (A6), U506.6 (A6), U507.6 (A6), U508.43 (A6), U509.43 (A6), U510.43 (A6), U511.43 (A6); no longer U502.44 (A5), U503.44 (A5), U504.44 (A5), U505.44 (A5), U506.7 (A5), U507.7 (A5), U508.44 (A5), U509.44 (A5), U510.44 (A5), U511.44 (A5)
- net A8: now also U502.42 (A7), U503.42 (A7), U504.42 (A7), U505.42 (A7), U506.5 (A7), U507.5 (A7), U508.42 (A7), U509.42 (A7), U510.42 (A7), U511.42 (A7); no longer U502.43 (A6), U503.43 (A6), U504.43 (A6), U505.43 (A6), U506.6 (A6), U507.6 (A6), U508.43 (A6), U509.43 (A6), U510.43 (A6), U511.43 (A6)
- net A9: now also U502.39 (A8), U503.39 (A8), U504.39 (A8), U505.39 (A8), U506.27 (A8), U507.27 (A8), U508.39 (A8), U509.39 (A8), U510.39 (A8), U511.39 (A8); no longer U502.42 (A7), U503.42 (A7), U504.42 (A7), U505.42 (A7), U506.5 (A7), U507.5 (A7), U508.42 (A7), U509.42 (A7), U510.42 (A7), U511.42 (A7)
- net GND: now also C520.2, C521.2, C522.2; no longer U502.6 (~{CE1}), U503.6 (~{CE1}), U504.6 (~{CE1}), U505.6 (~{CE1}), U506.22 (CE), U507.22 (CE), U508.6 (~{CE1}), U509.6 (~{CE1}), U510.6 (~{CE1}), U511.6 (~{CE1})
- net ~{OBMEM_RAM0SEL}: now also U502.6 (~{CE1}), U503.6 (~{CE1})
- net ~{OBMEM_RAM1SEL}: now also U504.6 (~{CE1}), U505.6 (~{CE1})
- net ~{OBMEM_RAM2SEL}: now also U508.6 (~{CE1}), U509.6 (~{CE1})
- net ~{OBMEM_RAM3SEL}: now also U510.6 (~{CE1}), U511.6 (~{CE1})
- net ~{OBMEM_ROMSEL}: now also U506.22 (CE), U507.22 (CE)
- net TMS: now reaches U501.13 (I/O/TMS)
- net TCK: now reaches U501.32 (I/O/TCK)
- net BERR_TDI: now reaches U501.38 (I/O/TDO)
- net MEMCTL_TDI: now reaches U501.7 (I/O/TDI)
- new net A1: U502.5 (A0), U503.5 (A0), U504.5 (A0), U505.5 (A0), U506.12 (A0), U507.12 (A0), U508.5 (A0), U509.5 (A0), U510.5 (A0), U511.5 (A0)

Commit message: MMU now has Bus Error Register integrated.
Connections:
- net BERR_TDI renamed TDO

Commit message: A bunch of routing for the RAM.
Parts:
- renumbered U504 to U502, U505 to U503, U502 to U504, U503 to U505, U510 to U508, U511 to U509, U508 to U510, U509 to U511
Connections:
- net ~{OBMEM_RAM0SEL}: now also U502.6 (~{CE1}), U503.6 (~{CE1}); no longer U504.6 (~{CE1}), U505.6 (~{CE1})
- net ~{OBMEM_RAM1SEL}: now also U504.6 (~{CE1}), U505.6 (~{CE1}); no longer U502.6 (~{CE1}), U503.6 (~{CE1})
- net ~{OBMEM_RAM2SEL}: now also U508.6 (~{CE1}), U509.6 (~{CE1}); no longer U510.6 (~{CE1}), U511.6 (~{CE1})
- net ~{OBMEM_RAM3SEL}: now also U510.6 (~{CE1}), U511.6 (~{CE1}); no longer U508.6 (~{CE1}), U509.6 (~{CE1})
Changed lines of the file:
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@@
 		)
 	)
-	(label "~{OBMEM_RAM1SEL}"
+	(label "~{OBMEM_RAM0SEL}"
 		(at 80.01 173.99 180)
 		(effects
@@
 		)
 	)
-	(label "~{OBMEM_RAM1SEL}"
+	(label "~{OBMEM_RAM0SEL}"
 		(at 80.01 86.36 180)
 		(effects
@@
 		)
 	)
-	(label "~{OBMEM_RAM3SEL}"
+	(label "~{OBMEM_RAM2SEL}"
 		(at 171.45 86.36 180)
 		(effects
@@
 		)
 	)
-	(label "~{OBMEM_RAM0SEL}"
+	(label "~{OBMEM_RAM1SEL}"
 		(at 33.02 86.36 180)
 		(effects
@@
 		)
 	)
-	(label "~{OBMEM_RAM2SEL}"
+	(label "~{OBMEM_RAM3SEL}"
 		(at 124.46 86.36 180)
 		(effects
@@
 		)
 	)
-	(label "~{OBMEM_RAM3SEL}"
+	(label "~{OBMEM_RAM2SEL}"
 		(at 171.45 173.99 180)
 		(effects
@@
 		)
 	)
-	(label "~{OBMEM_RAM2SEL}"
+	(label "~{OBMEM_RAM3SEL}"
 		(at 124.46 173.99 180)
 		(effects
@@
 		)
 	)
-	(label "~{OBMEM_RAM0SEL}"
+	(label "~{OBMEM_RAM1SEL}"
 		(at 33.02 173.99 180)
 		(effects
@@
 		(dnp no)
 		(fields_autoplaced yes)
-		(property "Reference" "U503"
+		(property "Reference" "U505"
 			(at 47.8633 109.22 0)
 			(effects
@@
 			(project "cpu010"
 				(path "/65f80d66-eea1-4882-b29a-ae1b65892b55/7792efab-b43b-475d-b2b8-8a6079701be8"
-					(reference "U503")
+					(reference "U505")
 					(unit 1)
 				)
@@
 		(dnp no)
 		(fields_autoplaced yes)
-		(property "Reference" "U511"
+		(property "Reference" "U509"
 			(at 186.2933 109.22 0)
 			(effects
@@
 			(project "cpu010"
 				(path "/65f80d66-eea1-4882-b29a-ae1b65892b55/7792efab-b43b-475d-b2b8-8a6079701be8"
-					(reference "U511")
+					(reference "U509")
 					(unit 1)
 				)
@@
 		(dnp no)
 		(fields_autoplaced yes)
-		(property "Reference" "U502"
+		(property "Reference" "U504"
 			(at 47.8633 21.59 0)
 			(effects
@@
 			(project ""
 				(path "/65f80d66-eea1-4882-b29a-ae1b65892b55/7792efab-b43b-475d-b2b8-8a6079701be8"
-					(reference "U502")
+					(reference "U504")
 					(unit 1)
 				)
@@
 		(dnp no)
 		(fields_autoplaced yes)
-		(property "Reference" "U509"
+		(property "Reference" "U511"
 			(at 139.3033 109.22 0)
 			(effects
@@
 			(project "cpu010"
 				(path "/65f80d66-eea1-4882-b29a-ae1b65892b55/7792efab-b43b-475d-b2b8-8a6079701be8"
-					(reference "U509")
+					(reference "U511")
 					(unit 1)
 				)
@@
 		(dnp no)
 		(fields_autoplaced yes)
-		(property "Reference" "U510"
+		(property "Reference" "U508"
 			(at 186.2933 21.59 0)
 			(effects
@@
 			(project "cpu010"
 				(path "/65f80d66-eea1-4882-b29a-ae1b65892b55/7792efab-b43b-475d-b2b8-8a6079701be8"
-					(reference "U510")
+					(reference "U508")
 					(unit 1)
 				)
@@
 		(dnp no)
 		(fields_autoplaced yes)
-		(property "Reference" "U504"
+		(property "Reference" "U502"
 			(at 94.8533 21.59 0)
 			(effects
@@
 			(project "cpu010"
 				(path "/65f80d66-eea1-4882-b29a-ae1b65892b55/7792efab-b43b-475d-b2b8-8a6079701be8"
-					(reference "U504")
+					(reference "U502")
 					(unit 1)
 				)
@@
 		(dnp no)
 		(fields_autoplaced yes)
-		(property "Reference" "U505"
+		(property "Reference" "U503"
 			(at 94.8533 109.22 0)
 			(effects
@@
 			(project "cpu010"
 				(path "/65f80d66-eea1-4882-b29a-ae1b65892b55/7792efab-b43b-475d-b2b8-8a6079701be8"
-					(reference "U505")
+					(reference "U503")
 					(unit 1)
 				)
@@
 		(dnp no)
 		(fields_autoplaced yes)
-		(property "Reference" "U508"
+		(property "Reference" "U510"
 			(at 139.3033 21.59 0)
 			(effects
@@
 			(project "cpu010"
 				(path "/65f80d66-eea1-4882-b29a-ae1b65892b55/7792efab-b43b-475d-b2b8-8a6079701be8"
-					(reference "U508")
+					(reference "U510")
 					(unit 1)
 				)

Commit message: Beef up the power supply a little.
Parts:
- added C523, C524, C525, C526: 100µF, Capacitor_THT:CP_Radial_D6.3mm_P2.50mm, symbol Device:C_Polarized_Small
Connections:
- net +5V: now also C523.1, C524.1, C525.1, C526.1
- net GND: now also C523.2, C524.2, C525.2, C526.2
