File: cpu010/design-files/cpu010-psu.kicad_sch (KiCad schematic)
At the start: 12 parts, among them J801 ATX-24, SW801 Power, U801 MAX16054

Commit message: Fix Errata A.2 -- Buffer the PWR_OK output to the LED and the DS1813 with a new N-FET / P-FET high-side switch controlled by PWR_OK from the PSU.
Parts:
- added Q801: BSS138, Package_TO_SOT_SMD:SOT-23, symbol Transistor_FET:BSS138
- added Q802: MMFTP3334K, Package_TO_SOT_SMD:SOT-23, symbol Transistor_FET:BSS84
- added R804, R805: 10K, Resistor_SMD:R_0805_2012Metric_Pad1.20x1.40mm_HandSolder, symbol Device:R_Small
Connections:
- net +5V: now also Q802.3 (D), R804.1
- net GND: now also Q801.2 (S), R805.2
- net PWR_OK: now also Q802.2 (S); no longer J801.8 (PWR_OK)
- new net: Q801.3 (D), Q802.1 (G), R804.2
- new net: J801.8 (PWR_OK), Q801.1 (G), R805.1
Other:
- note added: "A BSS84 would probably be OK here, but the low-Rds MMFTP3334K should provide a lot of margin for the DS1813."

Commit message: Add Mouser and LCSC part numbers for Q801 and Q802.
Parts:
- Q801: LCSC (none) -> C52895; Mouser (none) -> 512-BSS138
- Q802: LCSC (none) -> C49256473; Mouser (none) -> 637-MMFTP3334K
Changed lines of the file:
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@@
+			)
+		)
+		(property "Mouser" "637-MMFTP3334K"
+			(at 215.9 55.88 0)
+			(effects
+				(font
+					(size 1.27 1.27)
+				)
+				(hide yes)
+			)
+		)
+		(property "LCSC" "C49256473"
+			(at 215.9 55.88 0)
+			(effects
+				(font
+					(size 1.27 1.27)
+				)
+				(hide yes)
 			)
 		)
@@
 			(at 198.12 63.5 0)
 			(effects
+				(font
+					(size 1.27 1.27)
+				)
+				(hide yes)
+			)
+		)
+		(property "Mouser" "512-BSS138"
+			(at 198.12 63.5 0)
+			(effects
+				(font
+					(size 1.27 1.27)
+				)
+				(hide yes)
+			)
+		)
+		(property "LCSC" "C52895"
+			(at 198.12 63.5 0)
+			(effects

Commit message: Oops, fix swapped source/drain on Q802.
Parts:
- Q802: value MMFTP3334K -> Si2301CDS; LCSC C49256473 -> C10487; Mouser 637-MMFTP3334K -> 781-SI2301CDS-T1-GE3
Connections:
- net +5V: now also Q802.2 (S); no longer Q802.3 (D)
- net PWR_OK: now also Q802.3 (D); no longer Q802.2 (S)
Other:
- note added: "A BSS84 would probably be OK here, but the low-Rds Si2301CDS should provide a lot of margin for the DS1813. Alternatives in case Si2301CDS isn't available: - MMFTP3334K - AO3401A - DMG2305X"
- note removed: "A BSS84 would probably be OK here, but the low-Rds MMFTP3334K should provide a lot of margin for the DS1813."
Changed lines of the file:
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@@
 		)
 	)
-	(text "A BSS84 would probably be OK here, but the\nlow-Rds MMFTP3334K should provide a lot of\nmargin for the DS1813."
+	(text "A BSS84 would probably be OK here, but the\nlow-Rds Si2301CDS should provide a lot of\nmargin for the DS1813.\n\nAlternatives in case Si2301CDS isn't available:\n- MMFTP3334K\n- AO3401A\n- DMG2305X"
 		(exclude_from_sim no)
-		(at 212.598 37.592 0)
+		(at 221.996 41.91 0)
 		(effects
 			(font
@@
 		(lib_id "Transistor_FET:BSS84")
 		(at 215.9 55.88 0)
+		(mirror x)
 		(unit 1)
 		(exclude_from_sim no)
@@
 		(on_board yes)
 		(dnp no)
-		(fields_autoplaced yes)
 		(property "Reference" "Q802"
-			(at 222.25 54.6099 0)
-			(effects
-				(font
-					(size 1.27 1.27)
-				)
-				(justify left)
-			)
-		)
-		(property "Value" "MMFTP3334K"
-			(at 222.25 57.1499 0)
+			(at 222.25 57.1501 0)
+			(effects
+				(font
+					(size 1.27 1.27)
+				)
+				(justify left)
+			)
+		)
+		(property "Value" "Si2301CDS"
+			(at 222.25 54.6101 0)
 			(effects
 				(font
@@
 		)
 		(property "Footprint" "Package_TO_SOT_SMD:SOT-23"
-			(at 220.98 57.785 0)
+			(at 220.98 53.975 0)
 			(effects
 				(font
@@
 			)
 		)
-		(property "Datasheet" "http://assets.nexperia.com/documents/data-sheet/BSS84.pdf"
-			(at 220.98 59.69 0)
-			(effects
-				(font
-					(size 1.27 1.27)
-				)
-				(justify left)
-				(hide yes)
-			)
-		)
-		(property "Description" "-0.13A Id, -50V Vds, P-Channel MOSFET, SOT-23"
+		(property "Datasheet" ""
+			(at 220.98 52.07 0)
+			(effects
+				(font
+					(size 1.27 1.27)
+				)
+				(justify left)
+				(hide yes)
+			)
+		)
+		(property "Description" ""
 			(at 215.9 55.88 0)
 			(effects
@@
 			)
 		)
-		(property "Mouser" "637-MMFTP3334K"
+		(property "Mouser" "781-SI2301CDS-T1-GE3"
 			(at 215.9 55.88 0)
 			(effects
@@
 			)
 		)
-		(property "LCSC" "C49256473"
+		(property "LCSC" "C10487"
 			(at 215.9 55.88 0)
 			(effects
