File: nqvme_template/design-files/nqvme_interface.kicad_sch (KiCad schematic)
At the start: 1 part, among them J201 DIN41612_03x32_ABC

Commit message: Lay out the 22V10.
Parts:
- added C201, C202, C203: 100nF, Capacitor_SMD:C_0603_1608Metric_Pad1.08x0.95mm_HandSolder, symbol Device:C_Small
- added R201: 10K, Resistor_SMD:R_0603_1608Metric_Pad0.98x0.95mm_HandSolder, symbol Device:R_Small
- added SW201: SW_DIP_x03, Button_Switch_THT:SW_DIP_SPSTx03_Slide_9.78x9.8mm_W7.62mm_P2.54mm, symbol Switch:SW_DIP_x03
- added U201: AT24C01, Package_DIP:DIP-8_W7.62mm_Socket, symbol Memory_EEPROM:M24C01-FMN
- added U202: CD74HCT688M96, Package_SO:SOIC-20W_7.5x12.8mm_P1.27mm, symbol 74xx:74HCT688
- added U203: GAL22V10, Package_DIP:DIP-24_W7.62mm_Socket, symbol jrt-ICs:GAL22V10
Connections:
- net +5V: now also C201.1, C202.1, C203.1, R201.2, U201.7 (~{WC}), U201.8 (VCC), U202.20 (VCC), U203.24 (VCC)
- net A21: now also U202.13 (P5)
- net A22: now also U202.15 (P6)
- net A23: now also U202.17 (P7)
- net AM0: now also U203.10 (I10)
- net AM1: now also U203.9 (I9)
- net AM2: now also U203.8 (I8)
- net AM3: now also U203.7 (I7)
- net AM4: now also U203.6 (I6)
- net AM5: now also U203.11 (I11)
- net GND: now also C201.2, C202.2, C203.2, U201.4 (VSS), U202.1 (G), U202.10 (GND), U202.11 (P4), U202.12 (R4), U202.2 (P0), U202.3 (R0), U202.4 (P1), U202.5 (R1), U202.6 (P2), U202.7 (R2), U202.8 (P3), U202.9 (R3), U203.12 (GND)
- net R/~{W}: now also U203.3 (I3)
- net SCL: now also U201.5 (SDA)
- net SDA: now also U201.6 (SCL)
- net ~{AS}: now also U203.13 (I12)
- net ~{LDS}: now also U203.4 (I4)
- net ~{UDS}: now also U203.5 (I5)
- new net: R201.1, SW201.4, SW201.5, SW201.6
- new net A21M: SW201.3, U201.1 (E0), U202.14 (R5)
- new net A22M: SW201.2, U201.2 (E1), U202.16 (R6)
- new net A23M: SW201.1, U201.3 (E2), U202.18 (R7)
- new net ~{RMATCH}: U202.19 (P=R), U203.1 (I1/CLK)
- new net ~{VMEAS}: U203.23 (IO10)
- no-connect marks 23 -> 33
