File: nqvme_template/design-files/nqvme_template.kicad_pcb (KiCad board)
At the start: 2 copper layers, 151.9 x 99.8 mm, 1 part, among them J201 DIN41612_03x32_ABC

Commit message: Lay out the 22V10.
Parts:
- added C201: 100nF, Capacitor_SMD:C_0603_1608Metric_Pad1.08x0.95mm_HandSolder, F.Cu at (85.1, 118.0)
- added C202: 100nF, Capacitor_SMD:C_0603_1608Metric_Pad1.08x0.95mm_HandSolder, F.Cu at (85.6, 96.5)
- added C203: 100nF, Capacitor_SMD:C_0603_1608Metric_Pad1.08x0.95mm_HandSolder, F.Cu at (87.6, 117.1)
- added R201: 10K, Resistor_SMD:R_0603_1608Metric_Pad0.98x0.95mm_HandSolder, F.Cu at (86.4, 46.7)
- added SW201: SW_DIP_x03, Button_Switch_THT:SW_DIP_SPSTx03_Slide_9.78x9.8mm_W7.62mm_P2.54mm, F.Cu at (76.2, 53.3)
- added U201: AT24C01, Package_DIP:DIP-8_W7.62mm_Socket, F.Cu at (74.9, 117.1)
- added U202: CD74HCT688M96, Package_SO:SOIC-20W_7.5x12.8mm_P1.27mm, F.Cu at (78.7, 101.2)
- added U203: GAL22V10, Package_DIP:DIP-24_W7.62mm_Socket, F.Cu at (90.2, 124.7)
Other:
- copper layers 2 -> 4
- board text added: "0"
- board text added: "1"
- board text added: "2"
- board text added: "NQVME ID EEPROM"
- board text added: "NQVME Region Selector"
- board text added: "NQVMEGLU"
